Commit message: Added Inertia, CoM, Mass, Visual and Collision for L/R HipRoll leg

File: bigman_urdf/urdf/bigman_robot.urdf.xacro (robot description, xacro)
@@ -12,4 +12,4 @@
 <!-- YARP PLUGINS for GAZEBO SIMULATION -->
   <xacro:include filename="$(find bigman_urdf)/urdf/gazebo/yarp_control.gazebo.xacro" />
-  <origin xyz="0.0 0.0 0.575" rpy="0 0 0" />
+  <origin xyz="0.0 0.0 0.79" rpy="0 0 0" />
 </robot>

File: bigman_urdf/urdf/parts/legs.urdf.xacro (robot description, xacro)
@@ -1,4 +1,7 @@
 <?xml version="1.0"?>
 <robot xmlns:xacro="http://ros.org/wiki/xacro">
+<xacro:property name="mmTom" value="0.001" />
+<xacro:property name="mm2Tom2" value="${0.001*0.001}" />
+<xacro:property name="tonsToKg" value="1000.0" />
 <xacro:property name="PI" value="3.14159265359" />
 <xacro:property name="PI_2" value="1.57079632679" />
@@ -8,18 +11,18 @@
 <link name ="RHipMot">
     <inertial>
-      <origin xyz="-3.269678E-4 -0.023587321 -2.6496509E-4" rpy="0 0 0"/>
-      <mass value="0.89258227"/>
-      <inertia ixx="4.7672294E-4"  ixy="-3.9936567E-6"  ixz="-2.4802574E-6" iyy="5.458038E-4" iyz="-3.3389575E-6" izz="5.126859E-4" />
-    </inertial>
-    <visual>
-      <origin xyz="0.0 0.023 -0.52" rpy="0 0 ${PI}"/>
+      <origin xyz="${-1.0348188e+02*mmTom} ${-1.0919813e+02*mmTom} ${-6.4924056e+01*mmTom}" rpy="0 0 0"/>
+      <mass value="${3.7958197e-03*tonsToKg}"/>
+      <inertia ixx="${1.5639017e+01*mm2Tom2*tonsToKg}"  ixy="${1.8504661*mm2Tom2*tonsToKg}"  ixz="${2.3907793*mm2Tom2*tonsToKg}" iyy="${2.3519749e+01*mm2Tom2*tonsToKg}" iyz="${-2.3303162*mm2Tom2*tonsToKg}" izz="${2.0953643e+01*mm2Tom2*tonsToKg}" />
+    </inertial>
+    <visual>
+      <origin xyz="0 0 0" rpy="0 0 0"/>
       <geometry name="RHipMot_visual">
-        <mesh filename="package://bigman_urdf/meshes/collada/asm0001_collada_20_prt.dae" scale="${SF} ${SF} ${SF}" />
-      </geometry>
-    </visual>
-    <collision>
-      <origin xyz="0.0 0.023 -0.52" rpy="0 0 ${PI}"/>
+        <mesh filename="package://bigman_urdf/meshes/HipRoll.STL" scale="0.001 0.001 0.001" />
+      </geometry>
+    </visual>
+    <collision>
+      <origin xyz="0 0 0" rpy="0 0 0"/>
       <geometry name="RHipMot_collision">
-        <mesh filename="package://bigman_urdf/meshes/collada/simple/simple_asm0001_collada_20_prt.stl" scale="${SF} ${SF} ${SF}" />
+        <mesh filename="package://bigman_urdf/meshes/simple/HipRoll.STL" scale="0.001 0.001 0.001" />
       </geometry>
     </collision>
@@ -123,18 +126,18 @@
   <link name ="LHipMot">
     <inertial>
-      <origin xyz="-3.269678E-4 0.023587321 -2.6496509E-4" rpy="0 0 0"/>
-      <mass value="0.89258227"/>
-      <inertia ixx="4.7672294E-4"  ixy="3.9936567E-6"  ixz="-2.4802574E-6" iyy="5.458038E-4" iyz="3.3389575E-6" izz="5.126859E-4" />
-    </inertial>
-    <visual>
-      <origin xyz="0.0 -0.023 -0.52" rpy="0 0 ${PI}"/>
+      <origin xyz="${-1.0348188e+02*mmTom} ${1.0919813e+02*mmTom} ${-6.4924056e+01*mmTom}" rpy="0 0 0"/>
+      <mass value="${3.7958197e-03*tonsToKg}"/>
+      <inertia ixx="${1.5639017e+01*mm2Tom2*tonsToKg}"  ixy="${-1.8504661*mm2Tom2*tonsToKg}"  ixz="${2.3907793*mm2Tom2*tonsToKg}" iyy="${2.3519749e+01*mm2Tom2*tonsToKg}" iyz="${2.3303162*mm2Tom2*tonsToKg}" izz="${2.0953643e+01*mm2Tom2*tonsToKg}" />
+    </inertial>
+    <visual>
+      <origin xyz="0 0 0" rpy="0 0 0"/>
       <geometry name="RHipMot_visual">
-        <mesh filename="package://bigman_urdf/meshes/collada/asm0001_collada_06_prt.dae" scale="${SF} ${SF} ${SF}" />
-      </geometry>
-    </visual>
-    <collision>
-      <origin xyz="0.0 -0.023 -0.52" rpy="0 0 ${PI}"/>
+        <mesh filename="package://bigman_urdf/meshes/HipRoll.STL" scale="0.001 -0.001 0.001" />
+      </geometry>
+    </visual>
+    <collision>
+      <origin xyz="0 0 0" rpy="0 0 0"/>
       <geometry name="RHipMot_collision">
-        <mesh filename="package://bigman_urdf/meshes/collada/simple/simple_asm0001_collada_06_prt.stl" scale="${SF} ${SF} ${SF}" />
+        <mesh filename="package://bigman_urdf/meshes/simple/HipRoll.STL" scale="0.001 -0.001 0.001" />
       </geometry>
     </collision>
@@ -240,6 +243,6 @@
     <parent link="Waist"/>
     <child link="RHipMot"/>
-    <origin xyz="0.0 -0.023 0.0" rpy="0 0 0" />
-    <axis xyz="0 1 0" />
+    <origin xyz="0.1059 -0.06 0.0" rpy="0 0 0" />
+    <axis xyz="1 0 0" />
     <limit velocity="4.0" effort="50" lower="-1.9199" upper="0.7854" />
     <dynamics friction="0" damping="3.0"/>
@@ -248,6 +251,6 @@
     <parent link="RHipMot"/>
     <child link="RThighUpLeg"/>
-    <origin xyz="0.0 -0.0496 0.0" rpy="0 0 0" />
-    <axis xyz="1 0 0" />
+    <origin xyz="-0.0889 -0.121032 -0.217872" rpy="0 0 0" />
+    <axis xyz="0 0 1" />
     <limit velocity="4.0" effort="50" lower="-1.0472" upper="0.4363" />
     <dynamics friction="0" damping="3.0"/>
@@ -289,6 +292,6 @@
     <parent link="Waist"/>
     <child link="LHipMot"/>
-    <origin xyz="0.0 0.023 0.0" rpy="0 0 0" />
-    <axis xyz="0 1 0" />
+    <origin xyz="0.1059 0.06 0.0" rpy="0 0 0" />
+    <axis xyz="1 0 0" />
     <limit velocity="4.0" effort="50" lower="-1.9199" upper="0.7854" />
     <dynamics friction="0" damping="3.0"/>
@@ -297,6 +300,6 @@
     <parent link="LHipMot"/>
     <child link="LThighUpLeg"/>
-    <origin xyz="0.0 0.0496 0.0" rpy="0 0 0" />
-    <axis xyz="1 0 0" />
+    <origin xyz="-0.0889 0.121032 -0.217872" rpy="0 0 0" />
+    <axis xyz="0 0 1" />
     <limit velocity="4.0" effort="50" lower="-0.4363" upper="1.0472" />
     <dynamics friction="0" damping="3.0"/>

Commit message: Added R/L HipPitch Mass, Inertia, visualization and collision

File: bigman_urdf/urdf/bigman_robot.urdf.xacro (robot description, xacro)
@@ -12,4 +12,4 @@
 <!-- YARP PLUGINS for GAZEBO SIMULATION -->
   <xacro:include filename="$(find bigman_urdf)/urdf/gazebo/yarp_control.gazebo.xacro" />
-  <origin xyz="0.0 0.0 0.79" rpy="0 0 0" />
+  <origin xyz="0.0 0.0 0.920" rpy="0 0 0" />
 </robot>

File: bigman_urdf/urdf/parts/legs.urdf.xacro (robot description, xacro)
@@ -49,18 +49,18 @@
   <link name ="RThighLowLeg">
     <inertial>
-      <origin xyz="9.8720058E-4 6.7037262E-4 -0.075716843" rpy="0 0 0"/>
-      <mass value="1.7001134"/>
-      <inertia ixx="0.0038979546"  ixy="1.7802399E-6"  ixz="2.6403262E-5" iyy="0.0039360845" iyz="4.522711E-5" izz="9.0218711E-4" />
-    </inertial>
-    <visual>
-      <origin xyz="0.0 0.0726 -0.4176" rpy="0 0 ${PI}"/>
+      <origin xyz="${3.7746286e+01*mmTom} ${-2.8539939e+01*mmTom} ${-1.9310133e+02*mmTom}" rpy="0 0 0"/>
+      <mass value="5.0950736"/>
+      <inertia ixx="${5.1607858e+04*mm2Tom2}"  ixy="${2.2253472e+03*mm2Tom2}"  ixz="${2.4529790e+03*mm2Tom2}" iyy="${4.4349153e+04*mm2Tom2}" iyz="${-4.1006942e+03*mm2Tom2}" izz="${2.3374453e+04*mm2Tom2}" />
+    </inertial>
+    <visual>
+      <origin xyz="0 0 0" rpy="0 0 0"/>
       <geometry name="RThighLowLeg_visual">
-        <mesh filename="package://bigman_urdf/meshes/collada/asm0001_collada_18_prt.dae" scale="${SF} ${SF} ${SF}" />
-      </geometry>
-    </visual>
-    <collision>
-      <origin xyz="0.0 0.0726 -0.4176" rpy="0 0 ${PI}"/>
+        <mesh filename="package://bigman_urdf/meshes/HipPitch.STL" scale="0.001 0.001 0.001" />
+      </geometry>
+    </visual>
+    <collision>
+      <origin xyz="0 0 0" rpy="0 0 0"/>
       <geometry name="RThighLowLeg_collision">
-        <mesh filename="package://bigman_urdf/meshes/collada/simple/simple_asm0001_collada_18_prt.stl" scale="${SF} ${SF} ${SF}" />
+        <mesh filename="package://bigman_urdf/meshes/simple/HipPitch.STL" scale="0.001 0.001 0.001" />
       </geometry>
     </collision>
@@ -164,18 +164,18 @@
   <link name ="LThighLowLeg">
     <inertial>
-      <origin xyz="9.8720058E-4 -6.7037262E-4 -0.075716843" rpy="0 0 0"/>
-      <mass value="1.7001134"/>
-      <inertia ixx="0.0038979546"  ixy="-1.7802399E-6"  ixz="2.6403262E-5" iyy="0.0039360845" iyz="-4.5227110E-5" izz="9.0218711E-4" />
-    </inertial>
-    <visual>
-      <origin xyz="0.0 -0.0726 -0.4176" rpy="0 0 ${PI}"/>
-      <geometry name="LThighLowLeg_visual">
-        <mesh filename="package://bigman_urdf/meshes/collada/asm0001_collada_04_prt.dae" scale="${SF} ${SF} ${SF}" />
-      </geometry>
-    </visual>
-    <collision>
-      <origin xyz="0.0 -0.0726 -0.4176" rpy="0 0 ${PI}"/>
-      <geometry name="LThighLowLeg_collision">
-        <mesh filename="package://bigman_urdf/meshes/collada/simple/simple_asm0001_collada_04_prt.stl" scale="${SF} ${SF} ${SF}" />
+      <origin xyz="${3.7746286e+01*mmTom} ${2.8539939e+01*mmTom} ${-1.9310133e+02*mmTom}" rpy="0 0 0"/>
+      <mass value="5.0950736"/>
+      <inertia ixx="${5.1607858e+04*mm2Tom2}"  ixy="${-2.2253472e+03*mm2Tom2}"  ixz="${2.4529790e+03*mm2Tom2}" iyy="${4.4349153e+04*mm2Tom2}" iyz="${4.1006942e+03*mm2Tom2}" izz="${2.3374453e+04*mm2Tom2}" />
+    </inertial>
+    <visual>
+      <origin xyz="0 0 0" rpy="0 0 0"/>
+      <geometry name="RThighLowLeg_visual">
+        <mesh filename="package://bigman_urdf/meshes/HipPitch.STL" scale="0.001 -0.001 0.001" />
+      </geometry>
+    </visual>
+    <collision>
+      <origin xyz="0 0 0" rpy="0 0 0"/>
+      <geometry name="RThighLowLeg_collision">
+        <mesh filename="package://bigman_urdf/meshes/simple/HipPitch.STL" scale="0.001 -0.001 0.001" />
       </geometry>
     </collision>
@@ -267,5 +267,5 @@
     <parent link="RThighLowLeg"/>
     <child link="RLowLeg"/>
-    <origin xyz="0.0 0.0 -0.1234" rpy="0 0 0" />
+    <origin xyz="0.0 0.0 -0.356" rpy="0 0 0" />
     <axis xyz="0 1 0" />
     <limit velocity="4.0" effort="50" lower="-0.1745" upper="1.9199" />
@@ -316,5 +316,5 @@
     <parent link="LThighLowLeg"/>
     <child link="LLowLeg"/>
-    <origin xyz="0.0 0.0 -0.1234" rpy="0 0 0" />
+    <origin xyz="0.0 0.0 -0.356" rpy="0 0 0" />
     <axis xyz="0 1 0" />
     <limit velocity="4.0" effort="50" lower="-0.1745" upper="1.9199" />

Commit message: Added L/R KneePitch Mass, Inertia, CoM, visualization and collision

File: bigman_urdf/urdf/bigman_robot.urdf.xacro (robot description, xacro)
@@ -12,4 +12,4 @@
 <!-- YARP PLUGINS for GAZEBO SIMULATION -->
   <xacro:include filename="$(find bigman_urdf)/urdf/gazebo/yarp_control.gazebo.xacro" />
-  <origin xyz="0.0 0.0 0.920" rpy="0 0 0" />
+  <origin xyz="0.0 0.0 1.12" rpy="0 0 0" />
 </robot>

File: bigman_urdf/urdf/parts/legs.urdf.xacro (robot description, xacro)
@@ -68,18 +68,18 @@
   <link name ="RLowLeg">
     <inertial>
-      <origin xyz="0.0024612666 -0.0053099614 -0.08598948" rpy="0 0 0"/>
-      <mass value="1.4098179"/>
-      <inertia ixx="0.0040604004"  ixy="1.1227206E-5"  ixz="1.2260973E-5" iyy="0.004005652855" iyz="5.1899176E-4" izz="0.0012414054" />
-    </inertial>
-    <visual>
-      <origin xyz="0.0 0.0726 -0.2942" rpy="0 0 ${PI}"/>
+      <origin xyz="${-5.0828668*mmTom} ${3.7732093*mmTom} ${-7.2605017e+01*mmTom}" rpy="0 0 0"/>
+      <mass value="5.6495309"/>
+      <inertia ixx="${1.0535542e+05*mm2Tom2}"  ixy="${-5.8199221e+02*mm2Tom2}"  ixz="${1.6743598e+03*mm2Tom2}" iyy="${9.7857796e+04*mm2Tom2}" iyz="${-3.3770181e+03*mm2Tom2}" izz="${2.0854086e+04*mm2Tom2}" />
+    </inertial>
+    <visual>
+      <origin xyz="0 0 0" rpy="0 0 0"/>
       <geometry name="RLowLeg_visual">
-        <mesh filename="package://bigman_urdf/meshes/collada/asm0001_collada_17_prt.dae" scale="${SF} ${SF} ${SF}" />
-      </geometry>
-    </visual>
-    <collision>
-      <origin xyz="0.0 0.0726 -0.2942" rpy="0 0 ${PI}"/>
+        <mesh filename="package://bigman_urdf/meshes/KneePitch.STL" scale="0.001 0.001 0.001" />
+      </geometry>
+    </visual>
+    <collision>
+      <origin xyz="0 0 0" rpy="0 0 0"/>
       <geometry name="RLowLeg_collision">
-        <mesh filename="package://bigman_urdf/meshes/collada/simple/simple_asm0001_collada_17_prt.stl" scale="${SF} ${SF} ${SF}" />
+        <mesh filename="package://bigman_urdf/meshes/simple/KneePitch.STL" scale="0.001 0.001 0.001" />
       </geometry>
     </collision>
@@ -183,18 +183,18 @@
   <link name ="LLowLeg">
     <inertial>
-      <origin xyz="0.0024612666 0.0053099614 -0.085989484" rpy="0 0 0"/>
-      <mass value="1.4098179"/>
-      <inertia ixx="0.0040604004"  ixy="-1.1227206E-5"  ixz="1.2260973E-5" iyy="0.004005652855" iyz="-5.1899176E-4" izz="0.0012414054" />
-    </inertial>
-    <visual>
-      <origin xyz="0.0 -0.0726 -0.2942" rpy="0 0 ${PI}"/>
-      <geometry name="LLowLeg_visual">
-        <mesh filename="package://bigman_urdf/meshes/collada/asm0001_collada_03_prt.dae" scale="${SF} ${SF} ${SF}" />
-      </geometry>
-    </visual>
-    <collision>
-      <origin xyz="0.0 -0.0726 -0.2942" rpy="0 0 ${PI}"/>
-      <geometry name="LLowLeg_collision">
-        <mesh filename="package://bigman_urdf/meshes/collada/simple/simple_asm0001_collada_03_prt.stl" scale="${SF} ${SF} ${SF}" />
+      <origin xyz="${-5.0828668*mmTom} ${-3.7732093*mmTom} ${-7.2605017e+01*mmTom}" rpy="0 0 0"/>
+      <mass value="5.6495309"/>
+      <inertia ixx="${1.0535542e+05*mm2Tom2}"  ixy="${5.8199221e+02*mm2Tom2}"  ixz="${1.6743598e+03*mm2Tom2}" iyy="${9.7857796e+04*mm2Tom2}" iyz="${3.3770181e+03*mm2Tom2}" izz="${2.0854086e+04*mm2Tom2}" />
+    </inertial>
+    <visual>
+      <origin xyz="0 0 0" rpy="0 0 0"/>
+      <geometry name="RLowLeg_visual">
+        <mesh filename="package://bigman_urdf/meshes/KneePitch.STL" scale="0.001 0.001 0.001" />
+      </geometry>
+    </visual>
+    <collision>
+      <origin xyz="0 0 0" rpy="0 0 0"/>
+      <geometry name="RLowLeg_collision">
+        <mesh filename="package://bigman_urdf/meshes/simple/KneePitch.STL" scale="0.001 0.001 0.001" />
       </geometry>
     </collision>
@@ -275,6 +275,6 @@
     <parent link="RLowLeg"/>
     <child link="RFootmot"/>
-    <origin xyz="0.0 0.0 -0.201" rpy="0 0 0" />
-    <axis xyz="1 0 0" />
+    <origin xyz="0.0 0.0 -0.4" rpy="0 0 0" />
+    <axis xyz="0 1 0" />
     <limit velocity="4.0" effort="50" lower="-0.6109" upper="0.6109" />
     <dynamics friction="0" damping="3.0"/>
@@ -324,6 +324,6 @@
     <parent link="LLowLeg"/>
     <child link="LFootmot"/>
-    <origin xyz="0.0 0.0 -0.201" rpy="0 0 0" />
-    <axis xyz="1 0 0" />
+    <origin xyz="0.0 0.0 -0.4" rpy="0 0 0" />
+    <axis xyz="0 1 0" />
     <limit velocity="4.0" effort="50" lower="-0.6109" upper="0.6109" />
     <dynamics friction="0" damping="3.0"/>
