Commit message: Updated scripts

File: bigman_urdf/urdf/bigman_config.urdf.xacro (robot description, xacro)
@@ -1,6 +1,6 @@
 <?xml version="1.0"?>
 <robot xmlns:xacro="http://ros.org/wiki/xacro" name="BIGMAN">
-<xacro:property name="model_name" value="IIT Bigman w/ Softhand" />
-<xacro:property name="model_version" value="0.1" />
+<xacro:property name="model_name" value="IIT Bigman" />
+<xacro:property name="model_version" value="1.0" />
 <!--
 ####################################################
@@ -42,13 +42,13 @@
 -->
 <!-- 2) 7DOFS_FOREARMS -->
+<xacro:property name="GAZEBO_BIGMAN_USES_NO_FOREARMS" value="false" />
+<xacro:property name="GAZEBO_BIGMAN_USES_7DOF_FOREARMS_DRC_14" value="true" />
+<xacro:property name="GAZEBO_BIGMAN_USES_SOFTHANDS_DRC_sw1_14" value="false" />
+<!-- 3) 7DOFS_FOREARMS + SOFT_HANDS -->
 <!--
 <xacro:property name="GAZEBO_BIGMAN_USES_NO_FOREARMS" value="false" />
 <xacro:property name="GAZEBO_BIGMAN_USES_7DOF_FOREARMS_DRC_14" value="true" />
-<xacro:property name="GAZEBO_BIGMAN_USES_SOFTHANDS_DRC_sw1_14" value="false" />
+<xacro:property name="GAZEBO_BIGMAN_USES_SOFTHANDS_DRC_sw1_14" value="true" />
 -->
-<!-- 3) 7DOFS_FOREARMS + SOFT_HANDS -->
-<xacro:property name="GAZEBO_BIGMAN_USES_NO_FOREARMS" value="false" />
-<xacro:property name="GAZEBO_BIGMAN_USES_7DOF_FOREARMS_DRC_14" value="true" />
-<xacro:property name="GAZEBO_BIGMAN_USES_SOFTHANDS_DRC_sw1_14" value="true" />
 <!--
 ####################################################

Commit message: Small modification

File: bigman_urdf/urdf/bigman_config.urdf.xacro (robot description, xacro)
@@ -1,6 +1,6 @@
 <?xml version="1.0"?>
 <robot xmlns:xacro="http://ros.org/wiki/xacro" name="BIGMAN">
-<xacro:property name="model_name" value="IIT Bigman" />
-<xacro:property name="model_version" value="1.0" />
+<xacro:property name="model_name" value="IIT Bigman w/ Softhand" />
+<xacro:property name="model_version" value="0.1" />
 <!--
 ####################################################
@@ -42,13 +42,13 @@
 -->
 <!-- 2) 7DOFS_FOREARMS -->
+<!--
 <xacro:property name="GAZEBO_BIGMAN_USES_NO_FOREARMS" value="false" />
 <xacro:property name="GAZEBO_BIGMAN_USES_7DOF_FOREARMS_DRC_14" value="true" />
 <xacro:property name="GAZEBO_BIGMAN_USES_SOFTHANDS_DRC_sw1_14" value="false" />
+-->
 <!-- 3) 7DOFS_FOREARMS + SOFT_HANDS -->
-<!--
 <xacro:property name="GAZEBO_BIGMAN_USES_NO_FOREARMS" value="false" />
 <xacro:property name="GAZEBO_BIGMAN_USES_7DOF_FOREARMS_DRC_14" value="true" />
 <xacro:property name="GAZEBO_BIGMAN_USES_SOFTHANDS_DRC_sw1_14" value="true" />
--->
 <!--
 ####################################################

Commit message: Deleted optrions for feet.

File: bigman_urdf/urdf/bigman_config.urdf.xacro (robot description, xacro)
@@ -1,23 +1,6 @@
 <?xml version="1.0"?>
 <robot xmlns:xacro="http://ros.org/wiki/xacro" name="BIGMAN">
-<xacro:property name="model_name" value="IIT Bigman w/ Softhand" />
+<xacro:property name="model_name" value="IIT Bigman" />
 <xacro:property name="model_version" value="0.1" />
-<!--
-####################################################
-##
-##  FEET SELECTION
-##
-##
-## options:
-## 1) round feet
-## 2) simple feet
-##
-####################################################
-# TODO checks (must be mutually exclusive)
--->
-<!-- 1) round feet -->
-<xacro:property name="GAZEBO_BIGMAN_USES_ROUND_FEET_13" value="false" />
-<!-- 2) simple feet -->
-<xacro:property name="GAZEBO_BIGMAN_USES_SIMPLE_FEET_DRC_sw1_14" value="true" />
 <!--
 ####################################################

File: bigman_urdf/urdf/parts/legs.urdf.xacro (robot description, xacro)
@@ -102,12 +102,7 @@
   </link>
 <xacro:unless value="${GAZEBO_BIGMAN_USES_ACCURATE_FT}">
-    <xacro:if value="${GAZEBO_BIGMAN_USES_ROUND_FEET_13}">
-      <xacro:include filename="$(find bigman_urdf)/urdf/parts/subparts/round_feet_13/round_foot_R_13.urdf.xacro" />
-    </xacro:if>
-    <xacro:if value="${GAZEBO_BIGMAN_USES_SIMPLE_FEET_DRC_sw1_14}">
       <xacro:include filename="$(find bigman_urdf)/urdf/parts/subparts/simple_feet_DRC_sw1_14/simple_foot_R_DRC_sw1_14.urdf.xacro" />
-    </xacro:if>
-  </xacro:unless>
-  <xacro:if value="${GAZEBO_BIGMAN_USES_ACCURATE_FT}">
+</xacro:unless>
+<xacro:if value="${GAZEBO_BIGMAN_USES_ACCURATE_FT}">
     <link name ="RFootFTSensor">
       <inertial>
@@ -117,11 +112,6 @@
       </inertial>
     </link>
-    <xacro:if value="${GAZEBO_BIGMAN_USES_ROUND_FEET_13}">
-      <xacro:include filename="$(find bigman_urdf)/urdf/parts/subparts/round_feet_13/accurate_FT_round_foot_R_13.urdf.xacro" />
-    </xacro:if>
-    <xacro:if value="${GAZEBO_BIGMAN_USES_SIMPLE_FEET_DRC_sw1_14}">
       <xacro:include filename="$(find bigman_urdf)/urdf/parts/subparts/simple_feet_DRC_sw1_14/accurate_FT_simple_foot_R_DRC_sw1_14.urdf.xacro" />
-    </xacro:if>
-  </xacro:if>
+ </xacro:if>
 <!-- ********************LEFT LEG******************** -->
   <link name ="LHipMot">
@@ -221,10 +211,5 @@
   </link>
   <xacro:unless value="${GAZEBO_BIGMAN_USES_ACCURATE_FT}">
-    <xacro:if value="${GAZEBO_BIGMAN_USES_ROUND_FEET_13}">
-      <xacro:include filename="$(find bigman_urdf)/urdf/parts/subparts/round_feet_13/round_foot_L_13.urdf.xacro" />
-    </xacro:if>
-    <xacro:if value="${GAZEBO_BIGMAN_USES_SIMPLE_FEET_DRC_sw1_14}">
       <xacro:include filename="$(find bigman_urdf)/urdf/parts/subparts/simple_feet_DRC_sw1_14/simple_foot_L_DRC_sw1_14.urdf.xacro" />
-    </xacro:if>
   </xacro:unless>
   <xacro:if value="${GAZEBO_BIGMAN_USES_ACCURATE_FT}">
@@ -236,10 +221,5 @@
       </inertial>
     </link>
-    <xacro:if value="${GAZEBO_BIGMAN_USES_ROUND_FEET_13}">
-      <xacro:include filename="$(find bigman_urdf)/urdf/parts/subparts/round_feet_13/accurate_FT_round_foot_L_13.urdf.xacro" />
-    </xacro:if>
-    <xacro:if value="${GAZEBO_BIGMAN_USES_SIMPLE_FEET_DRC_sw1_14}">
       <xacro:include filename="$(find bigman_urdf)/urdf/parts/subparts/simple_feet_DRC_sw1_14/accurate_FT_simple_foot_L_DRC_sw1_14.urdf.xacro" />
-    </xacro:if>
   </xacro:if>
 <!-- JOINTS -->

Commit message: Deleted useless .ini files. Delted variables in config. Problems with bigman.gazebo.wtf

File: bigman_urdf/urdf/bigman_config.urdf.xacro (robot description, xacro)
@@ -12,38 +12,4 @@
 <!-- 7DOFS_FOREARMS + SOFT_HANDS -->
 <xacro:property name="GAZEBO_BIGMAN_USES_SOFTHANDS_DRC_sw1_14" value="true" />
-<!--
-####################################################
-##
-##  MIDDLEWARE SELECTION
-##
-##
-## options:
-#  notice how, regardless of the middleware selected
-#  a bare version of the robot is created (.urdf)
-#  1) yarp
-#	The robot is created using yarp plugins for
-#	the IMU and F/T sensors. The controlboard
-#	plugins used to control joints and get
-#	encoder and torque information are to be
-#	inserted using the .world file, where the
-#	initial configuration for the joints can
-#	be specified (for example, look at the
-#	worlds folder)
-#  2) ros
-#	The sdf is created including ros plugins
-#
-##
-####################################################
-#
-# 1) yarp
-#
--->
-<xacro:property name="GAZEBO_BIGMAN_USES_ROS" value="false" />
-<!--
-#
-# 2) ros
-#
--->
-<xacro:property name="GAZEBO_BIGMAN_USES_YARP" value="true" />
 <!--
 ####################################################

File: bigman_urdf/urdf/gazebo/microstrain_3dmgx2_imu.gazebo.xacro (robot description, xacro)
@@ -6,22 +6,4 @@
   This file groups files to use BIGMAN in GAZEBO
   -->
-  <xacro:if value="$(optenv GAZEBO_BIGMAN_USES_ROS false)">
-    <gazebo>
-        <plugin name="quadrotor_imu_sim" filename="libhector_gazebo_ros_imu.so">
-          <updateRate>100.0</updateRate>
-          <bodyName>imu_link</bodyName>
-          <topicName>BIGMAN/raw_imu</topicName>
-          <rpyOffsets>0 0 0</rpyOffsets> <!-- deprecated -->
-          <gaussianNoise>0</gaussianNoise>  <!-- deprecated -->
-          <accelDrift>0.5 0.5 0.5</accelDrift>
-          <accelGaussianNoise>0.35 0.35 0.3</accelGaussianNoise>
-          <rateDrift>0.1 0.1 0.1</rateDrift>
-          <rateGaussianNoise>0.05 0.05 0.015</rateGaussianNoise>
-          <headingDrift>0.1</headingDrift>
-          <headingGaussianNoise>0.05</headingGaussianNoise>
-        </plugin>
-      </gazebo>
-  </xacro:if>
-  <xacro:if value="$(optenv GAZEBO_BIGMAN_USES_YARP true)">
     <gazebo reference="imu_link">
         <sensor name="imu_sensor" type="imu">
@@ -54,4 +36,3 @@
         </sensor>
        </gazebo>
-  </xacro:if>
 </robot>

Commit message: Added flag to decide between fixed and moving hokuyo link in multisense.

File: bigman_urdf/urdf/bigman_config.urdf.xacro (robot description, xacro)
@@ -6,8 +6,24 @@
 ####################################################
 ##
-##  HAND SELECTION
+##  BIGMAN_FIXED_HANDS
+##  if "true" a fixed joint between wrist and hand
+##  will be used otherwise a rotative joints will
+##  be used.
+##
 ##
 ####################################################
 -->
 <xacro:property name="BIGMAN_FIXED_HANDS" value="true" />
+<!--
+####################################################
+##
+##  BIGMAN_FIXED_MULTISENSE
+##  if "true" a fixed joint between "head" and
+##  "hokuyo_link" will be used otherwise a continuous
+##  joints will be used.
+##
+##
+####################################################
+-->
+<xacro:property name="BIGMAN_FIXED_MULTISENSE" value="true" />
 </robot>

File: bigman_urdf/urdf/config/bigman_gazebo.urdf.xacro (robot description, xacro)
@@ -6,8 +6,24 @@
 ####################################################
 ##
-##  HAND SELECTION
+##  BIGMAN_FIXED_HANDS
+##  if "true" a fixed joint between wrist and hand
+##  will be used otherwise a rotative joints will
+##  be used.
+##
 ##
 ####################################################
 -->
 <xacro:property name="BIGMAN_FIXED_HANDS" value="false" />
+<!--
+####################################################
+##
+##  BIGMAN_FIXED_MULTISENSE
+##  if "true" a fixed joint between "head" and
+##  "hokuyo_link" will be used otherwise a continuous
+##  joints will be used.
+##
+##
+####################################################
+-->
+<xacro:property name="BIGMAN_FIXED_MULTISENSE" value="false" />
 </robot>

File: bigman_urdf/urdf/sensors/multisense_sl.urdf.xacro (robot description, xacro)
@@ -71,5 +71,5 @@
   </gazebo>
 -->
-<!--
+<xacro:if value="${BIGMAN_FIXED_MULTISENSE}">
   <joint name="hokuyo_joint" type="continuous">
     <origin xyz="-0.0446 0 0.0880" rpy="0 0 0" />
@@ -79,5 +79,6 @@
     <dynamics damping="0.01" friction="0"/>
   </joint>
--->
+</xacro:if>
+<xacro:unless value="${BIGMAN_FIXED_MULTISENSE}">
   <joint name="hokuyo_joint" type="fixed">
     <origin xyz="-0.0446 0 0.0880" rpy="0 0 0" />
@@ -85,4 +86,5 @@
     <child link="hokuyo_link" />
   </joint>
+</xacro:unless>
 <!-- Remove frome here!
   <gazebo reference="hokuyo_joint">

Commit message: Added a new variable in config to select between old and new version of the Chest

File: bigman_urdf/urdf/bigman_config.urdf.xacro (robot description, xacro)
@@ -3,4 +3,15 @@
 <xacro:property name="model_name" value="IIT Bigman Ctrl" />
 <xacro:property name="model_version" value="0.1" />
+<!--
+####################################################
+##
+##  BIGMAN_OLD_CHEST
+##  if "true" the old version of the chest will be
+##  used.
+##
+##
+####################################################
+-->
+<xacro:property name="BIGMAN_OLD_CHEST" value="false" />
 <!--
 ####################################################

File: bigman_urdf/urdf/config/bigman_gazebo.urdf.xacro (robot description, xacro)
@@ -3,4 +3,15 @@
 <xacro:property name="model_name" value="IIT Bigman" />
 <xacro:property name="model_version" value="0.1" />
+<!--
+####################################################
+##
+##  BIGMAN_OLD_CHEST
+##  if "true" the old version of the chest will be
+##  used.
+##
+##
+####################################################
+-->
+<xacro:property name="BIGMAN_OLD_CHEST" value="false" />
 <!--
 ####################################################

File: bigman_urdf/urdf/parts/arms.urdf.xacro (robot description, xacro)
@@ -166,6 +166,10 @@
     <parent link="DWYTorso"/>
     <child link="RShp"/>
-    <!--origin xyz="0.0 -0.2 0.0" rpy="0 0 0" /-->
+<xacro:if value="${BIGMAN_OLD_CHEST}">
+    <origin xyz="0.0 -0.2 0.0" rpy="0 0 0" />
+</xacro:if>
+<xacro:unless value="${BIGMAN_OLD_CHEST}">
     <origin xyz="0.045646 -0.219164 0.001531" rpy="0 0 0.3491" />
+</xacro:unless>
     <axis xyz="0 ${cos_42} ${-sin_42}" />
     <limit velocity="6.283" effort="120" lower="-2.844" upper="2.844" />
@@ -200,6 +204,10 @@
     <parent link="DWYTorso"/>
     <child link="LShp"/>
-    <!--origin xyz="0.0 0.2 0.0" rpy="0 0 0" /-->
+<xacro:if value="${BIGMAN_OLD_CHEST}">
+    <origin xyz="0.0 0.2 0.0" rpy="0 0 0" />
+</xacro:if>
+<xacro:unless value="${BIGMAN_OLD_CHEST}">
     <origin xyz="0.045646 0.219164 0.001531" rpy="0 0 -0.3491" />
+</xacro:unless>
     <axis xyz="0.0 ${cos_42} ${sin_42}" />
     <limit velocity="6.283" effort="120" lower="-2.844" upper="2.844" />

File: bigman_urdf/urdf/parts/torso.urdf.xacro (robot description, xacro)
@@ -81,6 +81,10 @@
       <origin xyz="0.0 0.0 0.0" rpy="0 0 0"/>
       <geometry name="DWYTorso_visual">
-        <!--mesh filename="package://bigman_urdf/meshes/Chest.STL" scale="0.001 0.001 0.001" /-->
+<xacro:if value="${BIGMAN_OLD_CHEST}">
+        <mesh filename="package://bigman_urdf/meshes/Chest.STL" scale="0.001 0.001 0.001" />
+</xacro:if>
+<xacro:unless value="${BIGMAN_OLD_CHEST}">
         <mesh filename="package://bigman_urdf/meshes/NewChest.STL" scale="0.001 0.001 0.001" />
+</xacro:unless>
       </geometry>
     </visual>
@@ -88,6 +92,10 @@
       <origin xyz="0.0 0.0 0.0" rpy="0 0 0"/>
       <geometry name="DWYTorso_collision">
-        <!--mesh filename="package://bigman_urdf/meshes/simple/Chest.STL" scale="0.001 0.001 0.001" /-->
+<xacro:if value="${BIGMAN_OLD_CHEST}">
+        <mesh filename="package://bigman_urdf/meshes/simple/Chest.STL" scale="0.001 0.001 0.001" />
+</xacro:if>
+<xacro:unless value="${BIGMAN_OLD_CHEST}">
         <mesh filename="package://bigman_urdf/meshes/simple/NewChest.STL" scale="0.001 0.001 0.001" />
+</xacro:unless>
       </geometry>
     </collision>

Commit message: Added new variable to add/delete protections

File: bigman_urdf/urdf/bigman_config.urdf.xacro (robot description, xacro)
@@ -72,3 +72,13 @@
 -->
 <xacro:property name="BIGMAN_HEAD" value="true" />
+<!--
+####################################################
+##
+##  BIGMAN_ADD_PROTECTIONS
+##  if "true" the protections are added to the model.
+##
+##
+####################################################
+-->
+<xacro:property name="BIGMAN_ADD_PROTECTIONS" value="true" />
 </robot>

File: bigman_urdf/urdf/config/bigman_gazebo.urdf.xacro (robot description, xacro)
@@ -72,3 +72,13 @@
 -->
 <xacro:property name="BIGMAN_HEAD" value="true" />
+<!--
+####################################################
+##
+##  BIGMAN_ADD_PROTECTIONS
+##  if "true" the protections are added to the model.
+##
+##
+####################################################
+-->
+<xacro:property name="BIGMAN_ADD_PROTECTIONS" value="true" />
 </robot>

File: bigman_urdf/urdf/config/bigman_only_legs.urdf.xacro (robot description, xacro)
@@ -72,3 +72,13 @@
 -->
 <xacro:property name="BIGMAN_HEAD" value="true" />
+<!--
+####################################################
+##
+##  BIGMAN_ADD_PROTECTIONS
+##  if "true" the protections are added to the model.
+##
+##
+####################################################
+-->
+<xacro:property name="BIGMAN_ADD_PROTECTIONS" value="false" />
 </robot>

File: bigman_urdf/urdf/config/bigman_only_upper_body.urdf.xacro (robot description, xacro)
@@ -72,3 +72,13 @@
 -->
 <xacro:property name="BIGMAN_HEAD" value="true" />
+<!--
+####################################################
+##
+##  BIGMAN_ADD_PROTECTIONS
+##  if "true" the protections are added to the model.
+##
+##
+####################################################
+-->
+<xacro:property name="BIGMAN_ADD_PROTECTIONS" value="true" />
 </robot>

File: bigman_urdf/urdf/config/bigman_only_upper_body_gazebo.urdf.xacro (robot description, xacro)
@@ -72,3 +72,13 @@
 -->
 <xacro:property name="BIGMAN_HEAD" value="true" />
+<!--
+####################################################
+##
+##  BIGMAN_ADD_PROTECTIONS
+##  if "true" the protections are added to the model.
+##
+##
+####################################################
+-->
+<xacro:property name="BIGMAN_ADD_PROTECTIONS" value="true" />
 </robot>

File: bigman_urdf/urdf/config/bigman_real.urdf.xacro (robot description, xacro)
@@ -72,3 +72,13 @@
 -->
 <xacro:property name="BIGMAN_HEAD" value="false" />
+<!--
+####################################################
+##
+##  BIGMAN_ADD_PROTECTIONS
+##  if "true" the protections are added to the model.
+##
+##
+####################################################
+-->
+<xacro:property name="BIGMAN_ADD_PROTECTIONS" value="true" />
 </robot>

File: bigman_urdf/urdf/parts/torso.urdf.xacro (robot description, xacro)
@@ -84,4 +84,5 @@
     </collision>
   </link>
+<xacro:if value="${BIGMAN_ADD_PROTECTIONS}">
 <link name ="TorsoProtections">
     <inertial>
@@ -104,5 +105,7 @@
     </collision>
   </link>
+</xacro:if>
 <!-- JOINTS -->
+<xacro:if value="${BIGMAN_ADD_PROTECTIONS}">
 <joint name="torso_protection_joint" type="fixed">
     <parent link="DWYTorso"/>
@@ -110,4 +113,5 @@
     <origin xyz="0.0 0 0.0" rpy="${-PI_2} 0 0" />
 </joint>
+</xacro:if>
 <joint name="torso_joint" type="fixed">
     <parent link="DWYTorso"/>

Commit message: Added flag to add/remove backpack

File: bigman_urdf/urdf/bigman_config.urdf.xacro (robot description, xacro)
@@ -82,3 +82,13 @@
 -->
 <xacro:property name="BIGMAN_ADD_PROTECTIONS" value="true" />
+<!--
+####################################################
+##
+##  BIGMAN_ADD_BACKPACK
+##  if "true" the backpack is added to the model.
+##
+##
+####################################################
+-->
+<xacro:property name="BIGMAN_ADD_BACKPACK" value="false" />
 </robot>

File: bigman_urdf/urdf/config/bigman.urdf.xacro (robot description, xacro)
@@ -82,3 +82,13 @@
 -->
 <xacro:property name="BIGMAN_ADD_PROTECTIONS" value="true" />
+<!--
+####################################################
+##
+##  BIGMAN_ADD_BACKPACK
+##  if "true" the backpack is added to the model.
+##
+##
+####################################################
+-->
+<xacro:property name="BIGMAN_ADD_BACKPACK" value="true" />
 </robot>

File: bigman_urdf/urdf/config/bigman_gazebo.urdf.xacro (robot description, xacro)
@@ -82,3 +82,13 @@
 -->
 <xacro:property name="BIGMAN_ADD_PROTECTIONS" value="true" />
+<!--
+####################################################
+##
+##  BIGMAN_ADD_BACKPACK
+##  if "true" the backpack is added to the model.
+##
+##
+####################################################
+-->
+<xacro:property name="BIGMAN_ADD_BACKPACK" value="true" />
 </robot>

File: bigman_urdf/urdf/config/bigman_only_legs.urdf.xacro (robot description, xacro)
@@ -82,3 +82,13 @@
 -->
 <xacro:property name="BIGMAN_ADD_PROTECTIONS" value="false" />
+<!--
+####################################################
+##
+##  BIGMAN_ADD_BACKPACK
+##  if "true" the backpack is added to the model.
+##
+##
+####################################################
+-->
+<xacro:property name="BIGMAN_ADD_BACKPACK" value="false" />
 </robot>

File: bigman_urdf/urdf/config/bigman_only_upper_body.urdf.xacro (robot description, xacro)
@@ -82,3 +82,13 @@
 -->
 <xacro:property name="BIGMAN_ADD_PROTECTIONS" value="true" />
+<!--
+####################################################
+##
+##  BIGMAN_ADD_BACKPACK
+##  if "true" the backpack is added to the model.
+##
+##
+####################################################
+-->
+<xacro:property name="BIGMAN_ADD_BACKPACK" value="true" />
 </robot>

File: bigman_urdf/urdf/config/bigman_only_upper_body_gazebo.urdf.xacro (robot description, xacro)
@@ -82,3 +82,13 @@
 -->
 <xacro:property name="BIGMAN_ADD_PROTECTIONS" value="true" />
+<!--
+####################################################
+##
+##  BIGMAN_ADD_BACKPACK
+##  if "true" the backpack is added to the model.
+##
+##
+####################################################
+-->
+<xacro:property name="BIGMAN_ADD_BACKPACK" value="true" />
 </robot>

File: bigman_urdf/urdf/config/bigman_real.urdf.xacro (robot description, xacro)
@@ -82,3 +82,13 @@
 -->
 <xacro:property name="BIGMAN_ADD_PROTECTIONS" value="true" />
+<!--
+####################################################
+##
+##  BIGMAN_ADD_BACKPACK
+##  if "true" the backpack is added to the model.
+##
+##
+####################################################
+-->
+<xacro:property name="BIGMAN_ADD_BACKPACK" value="true" />
 </robot>

File: bigman_urdf/urdf/parts/torso.urdf.xacro (robot description, xacro)
@@ -108,4 +108,5 @@
 </xacro:if>
 <!-- UPDATE DATA FOR TORSO PROTECTION! -->
+<xacro:if value="${BIGMAN_ADD_BACKPACK}">
 <link name="backpack">
     <inertial>
@@ -128,5 +129,7 @@
     </collision>
 </link>
+</xacro:if>
 <!-- JOINTS -->
+<xacro:if value="${BIGMAN_ADD_BACKPACK}">
 <joint name="backpack_joint" type="fixed">
     <parent link="DWYTorso"/>
@@ -134,4 +137,5 @@
     <origin xyz="-0.185 0 -0.025" rpy="0 0 0" />
 </joint>
+</xacro:if>
 <xacro:if value="${BIGMAN_ADD_PROTECTIONS}">
 <joint name="torso_protection_joint" type="fixed">

Commit message: Changed value

File: bigman_urdf/urdf/bigman_config.urdf.xacro (robot description, xacro)
@@ -91,4 +91,4 @@
 ####################################################
 -->
-<xacro:property name="BIGMAN_ADD_BACKPACK" value="false" />
+<xacro:property name="BIGMAN_ADD_BACKPACK" value="true" />
 </robot>
