Commit message: Fixed bug that was causing the use of the wrong reference frames with the new feet. Set NEW_BIGMAN_FEET to true as default.

File: bigman_urdf/urdf/bigman_config.urdf.xacro (robot description, xacro)
@@ -112,4 +112,4 @@
 ####################################################
 -->
-<xacro:property name="BIGMAN_NEW_FEET" value="false" />
+<xacro:property name="BIGMAN_NEW_FEET" value="true" />
 </robot>

File: bigman_urdf/urdf/config/bigman_gazebo.urdf.xacro (robot description, xacro)
@@ -112,4 +112,4 @@
 ####################################################
 -->
-<xacro:property name="BIGMAN_NEW_FEET" value="false" />
+<xacro:property name="BIGMAN_NEW_FEET" value="true" />
 </robot>

File: bigman_urdf/urdf/config/bigman_real.urdf.xacro (robot description, xacro)
@@ -112,4 +112,4 @@
 ####################################################
 -->
-<xacro:property name="BIGMAN_NEW_FEET" value="false" />
+<xacro:property name="BIGMAN_NEW_FEET" value="true" />
 </robot>

File: bigman_urdf/urdf/parts/foot_reference_frame.urdf.xacro (robot description, xacro)
@@ -10,4 +10,13 @@
 		</joint>
 	</xacro:macro>
+       <xacro:unless value="${BIGMAN_NEW_FEET}">
+	       <xacro:macro name="references_frame_foot" params="parent name mirror_y">
+	       <!-- macro for reference frames in foot -->
+		       <xacro:reference_frame_foot parent="${parent}" name="${name}_upper_right" x="0.195" y="${mirror_y*-0.07}" />
+		       <xacro:reference_frame_foot parent="${parent}" name="${name}_upper_left" x="0.195" y="${mirror_y*0.09}" />
+		       <xacro:reference_frame_foot parent="${parent}" name="${name}_lower_right" x="-0.111" y="${mirror_y*-0.07}" />
+		       <xacro:reference_frame_foot parent="${parent}" name="${name}_lower_left" x="-0.111" y="${mirror_y*0.09}" />
+	       </xacro:macro>
+       </xacro:unless>
        <xacro:if value="${BIGMAN_NEW_FEET}">
               <xacro:macro name="references_frame_foot" params="parent name mirror_y">
@@ -19,13 +28,4 @@
               </xacro:macro>
        </xacro:if>
-       <xacro:unless value="${BIGMAN_NEW_FEET}">
-	       <xacro:macro name="references_frame_foot" params="parent name mirror_y">
-	       <!-- macro for reference frames in foot -->
-		       <xacro:reference_frame_foot parent="${parent}" name="${name}_upper_right" x="0.195" y="${mirror_y*-0.07}" />
-		       <xacro:reference_frame_foot parent="${parent}" name="${name}_upper_left" x="0.195" y="${mirror_y*0.09}" />
-		       <xacro:reference_frame_foot parent="${parent}" name="${name}_lower_right" x="-0.111" y="${mirror_y*-0.07}" />
-		       <xacro:reference_frame_foot parent="${parent}" name="${name}_lower_left" x="-0.111" y="${mirror_y*0.09}" />
-	       </xacro:macro>
-       </xacro:unless>
 	<xacro:references_frame_foot parent="l_sole" name="l_foot" mirror_y="1.0"/>
 	<xacro:references_frame_foot parent="r_sole" name="r_foot" mirror_y="-1.0"/>
