Commit message: better handling of parameters, enabled whole_robot control

File: bigman_urdf/urdf/bigman_config.urdf.xacro (robot description, xacro)
@@ -1,85 +1,7 @@
 <?xml version="1.0"?>
 <robot xmlns:xacro="http://ros.org/wiki/xacro" name="BIGMAN">
+<xacro:include filename="$(find bigman_urdf)/urdf/config/bigman_default_params.xacro"/>
 <xacro:property name="model_name" value="IIT Bigman Ctrl" />
 <xacro:property name="model_version" value="0.1" />
-<!--
-####################################################
-##
-##  BIGMAN_UPPER_BODY
-##  if "true" the kinematic chains of the arms and torso
-##  will be used to generate the model
-##
-####################################################
--->
-<xacro:property name="BIGMAN_UPPER_BODY" value="true" />
-<!--
-####################################################
-##
-##  BIGMAN_LEGS
-##  if "true" the kinematic chains of the legs
-##  will be used to generate the model
-##
-####################################################
--->
-<xacro:property name="BIGMAN_LEGS" value="true" />
-<!--
-####################################################
-##
-##  BIGMAN_OLD_CHEST
-##  if "true" the old version of the chest will be
-##  used.
-##
-##
-####################################################
--->
-<xacro:property name="BIGMAN_OLD_CHEST" value="false" />
-<!--
-####################################################
-##
-##  BIGMAN_FIXED_HANDS
-##  if "true" a fixed joint between wrist and hand
-##  will be used otherwise a rotative joints will
-##  be used.
-##
-##
-####################################################
--->
-<xacro:property name="BIGMAN_FIXED_HANDS" value="true" />
-<!--
-####################################################
-##
-##  BIGMAN_FIXED_MULTISENSE
-##  if "true" a fixed joint between "head" and
-##  "hokuyo_link" will be used otherwise a continuous
-##  joints will be used.
-##
-##
-####################################################
--->
-<xacro:property name="BIGMAN_FIXED_MULTISENSE" value="true" />
-<!--
-####################################################
-##
-##  BIGMAN_HEAD
-##  if "true" a fixed joint between "NeckPitch" and
-##  "head" will be used to connect the head to the rest
-##  of the body. If "false" the head will not be added
-##  to the model (this is the case when the multisense
-##  from the launch file is used).
-##
-##
-####################################################
--->
-<xacro:property name="BIGMAN_HEAD" value="true" />
-<!--
-####################################################
-##
-##  BIGMAN_ADD_PROTECTIONS
-##  if "true" the protections are added to the model.
-##
-##
-####################################################
--->
-<xacro:property name="BIGMAN_ADD_PROTECTIONS" value="true" />
 <!--
 ####################################################

File: bigman_urdf/urdf/config/bigman_gazebo.urdf.xacro (robot description, xacro)
@@ -1,37 +1,7 @@
 <?xml version="1.0"?>
 <robot xmlns:xacro="http://ros.org/wiki/xacro" name="BIGMAN">
+<xacro:include filename="$(find bigman_urdf)/urdf/config/bigman_default_params.xacro"/>
 <xacro:property name="model_name" value="IIT Bigman" />
 <xacro:property name="model_version" value="0.1" />
-<!--
-####################################################
-##
-##  BIGMAN_UPPER_BODY
-##  if "true" the kinematic chains of the arms and torso
-##  will be used to generate the model
-##
-####################################################
--->
-<xacro:property name="BIGMAN_UPPER_BODY" value="true" />
-<!--
-####################################################
-##
-##  BIGMAN_LEGS
-##  if "true" the kinematic chains of the legs
-##  will be used to generate the model
-##
-####################################################
--->
-<xacro:property name="BIGMAN_LEGS" value="true" />
-<!--
-####################################################
-##
-##  BIGMAN_OLD_CHEST
-##  if "true" the old version of the chest will be
-##  used.
-##
-##
-####################################################
--->
-<xacro:property name="BIGMAN_OLD_CHEST" value="false" />
 <!--
 ####################################################
@@ -58,28 +28,4 @@
 -->
 <xacro:property name="BIGMAN_FIXED_MULTISENSE" value="false" />
-<!--
-####################################################
-##
-##  BIGMAN_HEAD
-##  if "true" a fixed joint between "NeckPitch" and
-##  "head" will be used to connect the head to the rest
-##  of the body. If "false" the head will not be added
-##  to the model (this is the case when the multisense
-##  from the launch file is used).
-##
-##
-####################################################
--->
-<xacro:property name="BIGMAN_HEAD" value="true" />
-<!--
-####################################################
-##
-##  BIGMAN_ADD_PROTECTIONS
-##  if "true" the protections are added to the model.
-##
-##
-####################################################
--->
-<xacro:property name="BIGMAN_ADD_PROTECTIONS" value="true" />
 <!--
 ####################################################

File: bigman_urdf/urdf/config/bigman_only_legs.urdf.xacro (robot description, xacro)
@@ -1,4 +1,5 @@
 <?xml version="1.0"?>
 <robot xmlns:xacro="http://ros.org/wiki/xacro" name="BIGMAN">
+<xacro:include filename="$(find bigman_urdf)/urdf/config/bigman_default_params.xacro"/>
 <xacro:property name="model_name" value="IIT Bigman Legs" />
 <xacro:property name="model_version" value="0.1" />
@@ -13,63 +14,4 @@
 -->
 <xacro:property name="BIGMAN_UPPER_BODY" value="false" />
-<!--
-####################################################
-##
-##  BIGMAN_LEGS
-##  if "true" the kinematic chains of the legs
-##  will be used to generate the model
-##
-####################################################
--->
-<xacro:property name="BIGMAN_LEGS" value="true" />
-<!--
-####################################################
-##
-##  BIGMAN_OLD_CHEST
-##  if "true" the old version of the chest will be
-##  used.
-##
-##
-####################################################
--->
-<xacro:property name="BIGMAN_OLD_CHEST" value="false" />
-<!--
-####################################################
-##
-##  BIGMAN_FIXED_HANDS
-##  if "true" a fixed joint between wrist and hand
-##  will be used otherwise a rotative joints will
-##  be used.
-##
-##
-####################################################
--->
-<xacro:property name="BIGMAN_FIXED_HANDS" value="true" />
-<!--
-####################################################
-##
-##  BIGMAN_FIXED_MULTISENSE
-##  if "true" a fixed joint between "head" and
-##  "hokuyo_link" will be used otherwise a continuous
-##  joints will be used.
-##
-##
-####################################################
--->
-<xacro:property name="BIGMAN_FIXED_MULTISENSE" value="true" />
-<!--
-####################################################
-##
-##  BIGMAN_HEAD
-##  if "true" a fixed joint between "NeckPitch" and
-##  "head" will be used to connect the head to the rest
-##  of the body. If "false" the head will not be added
-##  to the model (this is the case when the multisense
-##  from the launch file is used).
-##
-##
-####################################################
--->
-<xacro:property name="BIGMAN_HEAD" value="true" />
 <!--
 ####################################################

File: bigman_urdf/urdf/config/bigman_only_upper_body.urdf.xacro (robot description, xacro)
@@ -1,16 +1,7 @@
 <?xml version="1.0"?>
 <robot xmlns:xacro="http://ros.org/wiki/xacro" name="BIGMAN">
+<xacro:include filename="$(find bigman_urdf)/urdf/config/bigman_default_params.xacro"/>
 <xacro:property name="model_name" value="IIT Bigman Upper Body Ctrl" />
 <xacro:property name="model_version" value="0.1" />
-<!--
-####################################################
-##
-##  BIGMAN_UPPER_BODY
-##  if "true" the kinematic chains of the arms and torso
-##  will be used to generate the model
-##
-####################################################
--->
-<xacro:property name="BIGMAN_UPPER_BODY" value="true" />
 <!--
 ####################################################
@@ -34,52 +25,4 @@
 -->
 <xacro:property name="BIGMAN_OLD_CHEST" value="false" />
-<!--
-####################################################
-##
-##  BIGMAN_FIXED_HANDS
-##  if "true" a fixed joint between wrist and hand
-##  will be used otherwise a rotative joints will
-##  be used.
-##
-##
-####################################################
--->
-<xacro:property name="BIGMAN_FIXED_HANDS" value="true" />
-<!--
-####################################################
-##
-##  BIGMAN_FIXED_MULTISENSE
-##  if "true" a fixed joint between "head" and
-##  "hokuyo_link" will be used otherwise a continuous
-##  joints will be used.
-##
-##
-####################################################
--->
-<xacro:property name="BIGMAN_FIXED_MULTISENSE" value="true" />
-<!--
-####################################################
-##
-##  BIGMAN_HEAD
-##  if "true" a fixed joint between "NeckPitch" and
-##  "head" will be used to connect the head to the rest
-##  of the body. If "false" the head will not be added
-##  to the model (this is the case when the multisense
-##  from the launch file is used).
-##
-##
-####################################################
--->
-<xacro:property name="BIGMAN_HEAD" value="true" />
-<!--
-####################################################
-##
-##  BIGMAN_ADD_PROTECTIONS
-##  if "true" the protections are added to the model.
-##
-##
-####################################################
--->
-<xacro:property name="BIGMAN_ADD_PROTECTIONS" value="true" />
 <!--
 ####################################################

File: bigman_urdf/urdf/config/bigman_only_upper_body_gazebo.urdf.xacro (robot description, xacro)
@@ -1,16 +1,7 @@
 <?xml version="1.0"?>
 <robot xmlns:xacro="http://ros.org/wiki/xacro" name="BIGMAN">
+<xacro:include filename="$(find bigman_urdf)/urdf/config/bigman_default_params.xacro"/>
 <xacro:property name="model_name" value="IIT Bigman Upper Body" />
 <xacro:property name="model_version" value="0.1" />
-<!--
-####################################################
-##
-##  BIGMAN_UPPER_BODY
-##  if "true" the kinematic chains of the arms and torso
-##  will be used to generate the model
-##
-####################################################
--->
-<xacro:property name="BIGMAN_UPPER_BODY" value="true" />
 <!--
 ####################################################
@@ -23,15 +14,4 @@
 -->
 <xacro:property name="BIGMAN_LEGS" value="false" />
-<!--
-####################################################
-##
-##  BIGMAN_OLD_CHEST
-##  if "true" the old version of the chest will be
-##  used.
-##
-##
-####################################################
--->
-<xacro:property name="BIGMAN_OLD_CHEST" value="false" />
 <!--
 ####################################################
@@ -58,28 +38,4 @@
 -->
 <xacro:property name="BIGMAN_FIXED_MULTISENSE" value="false" />
-<!--
-####################################################
-##
-##  BIGMAN_HEAD
-##  if "true" a fixed joint between "NeckPitch" and
-##  "head" will be used to connect the head to the rest
-##  of the body. If "false" the head will not be added
-##  to the model (this is the case when the multisense
-##  from the launch file is used).
-##
-##
-####################################################
--->
-<xacro:property name="BIGMAN_HEAD" value="true" />
-<!--
-####################################################
-##
-##  BIGMAN_ADD_PROTECTIONS
-##  if "true" the protections are added to the model.
-##
-##
-####################################################
--->
-<xacro:property name="BIGMAN_ADD_PROTECTIONS" value="true" />
 <!--
 ####################################################

File: bigman_urdf/urdf/config/bigman_real.urdf.xacro (robot description, xacro)
@@ -1,61 +1,7 @@
 <?xml version="1.0"?>
 <robot xmlns:xacro="http://ros.org/wiki/xacro" name="BIGMAN">
+<xacro:include filename="$(find bigman_urdf)/urdf/config/bigman_default_params.xacro"/>
 <xacro:property name="model_name" value="IIT Bigman Real" />
 <xacro:property name="model_version" value="0.1" />
-<!--
-####################################################
-##
-##  BIGMAN_UPPER_BODY
-##  if "true" the kinematic chains of the arms and torso
-##  will be used to generate the model
-##
-####################################################
--->
-<xacro:property name="BIGMAN_UPPER_BODY" value="true" />
-<!--
-####################################################
-##
-##  BIGMAN_LEGS
-##  if "true" the kinematic chains of the legs
-##  will be used to generate the model
-##
-####################################################
--->
-<xacro:property name="BIGMAN_LEGS" value="true" />
-<!--
-####################################################
-##
-##  BIGMAN_OLD_CHEST
-##  if "true" the old version of the chest will be
-##  used.
-##
-##
-####################################################
--->
-<xacro:property name="BIGMAN_OLD_CHEST" value="false" />
-<!--
-####################################################
-##
-##  BIGMAN_FIXED_HANDS
-##  if "true" a fixed joint between wrist and hand
-##  will be used otherwise a rotative joints will
-##  be used.
-##
-##
-####################################################
--->
-<xacro:property name="BIGMAN_FIXED_HANDS" value="true" />
-<!--
-####################################################
-##
-##  BIGMAN_FIXED_MULTISENSE
-##  if "true" a fixed joint between "head" and
-##  "hokuyo_link" will be used otherwise a continuous
-##  joints will be used.
-##
-##
-####################################################
--->
-<xacro:property name="BIGMAN_FIXED_MULTISENSE" value="true" />
 <!--
 ####################################################
@@ -72,14 +18,4 @@
 -->
 <xacro:property name="BIGMAN_HEAD" value="false" />
-<!--
-####################################################
-##
-##  BIGMAN_ADD_PROTECTIONS
-##  if "true" the protections are added to the model.
-##
-##
-####################################################
--->
-<xacro:property name="BIGMAN_ADD_PROTECTIONS" value="true" />
 <!--
 ####################################################

File: bigman_urdf/urdf/gazebo/yarp_control.gazebo.xacro (robot description, xacro)
@@ -2,4 +2,11 @@
 <robot xmlns:xacro="http://ros.org/wiki/xacro">
 <gazebo>
+<xacro:if value="${BIGMAN_WHOLE_BODY}">
+      <plugin name='bigman_yarp_gazebo_plugin_whole_body' filename='libgazebo_yarp_controlboard.so'>
+      <yarpConfigurationFile>model://bigman_urdf/conf/bigman/bigman_gazebo.ini</yarpConfigurationFile>
+      <initialConfiguration>0.0 0.0 0.0 0.0 0.0 0.0 0.0 0.0 0.0 0.0 0.0 0.0 0.0 0.0 0.0 0.0 0.0 0.0 0.0 -0.17 0.0 0.0 0.0 0.0 0.0 0.0 0.17 0.0 0.0 0.0 0.0 0.0 0.0 0.0</initialConfiguration>
+    </plugin>
+</xacro:if>
+<xacro:unless value="${BIGMAN_WHOLE_BODY}">
 <xacro:if value="${BIGMAN_UPPER_BODY}">
 <!-- TORSO -->
@@ -84,4 +91,5 @@
 <!-- plugin name="bigman_yarp_gazebo_plugin_external_wrench" filename="libgazebo_yarp_externalwrench.so"/ -->
 <plugin name="bigman_show_model_com" filename="libgazebo_yarp_showmodelcom.so"/>
+</xacro:unless>
 </gazebo>
 </robot>

File: bigman_urdf/urdf/parts/soft_hand.urdf.xacro (robot description, xacro)
@@ -72,67 +72,132 @@
 </xacro:if>
 <xacro:unless value="${BIGMAN_FIXED_HANDS}">
+<xacro:property name="a" value="0.08" />
+<xacro:property name="b" value="0.08" />
+<xacro:property name="c" value="0.1" />
+<!-- For the hand we use the inertia of a parallelepiped -->
 <!-- LINKS -->
-<!-- ## WRONG NUMBERS FOR... ok lasciamo perde... FIX THEM!! ## -->
-  <link name="RSoftHand">
-    <inertial>
-      <origin xyz="0 0 -0.17" rpy="0 0 0"/>
-      <mass value="1.2"/>
-      <inertia ixx="${1.2*(b*b+c*c)/12.0}"  ixy="0"  ixz="0" iyy="${1.2*(a*a+c*c)/12.0}" iyz="0" izz="${1.2*(a*a+b*b)/12.0}" />
-    </inertial>
-    <visual>
-     <origin xyz="0 0 0" rpy="0 0 0" />
-     <geometry>
-        <box size="0.07 0.07 0.07" />
-     </geometry>
-     <material name="Cyan">
-       <color rgba="0 1.0 1.0 1.0"/>
-     </material>
-   </visual>
-   <collision>
-     <origin xyz="0 0 0" rpy="0 0 0"/>
-     <geometry>
-       <box size="0.07 0.07 0.07" />
-     </geometry>
-   </collision>
-  </link>
-  <link name="LSoftHand">
-    <inertial>
-      <origin xyz="0 0 -0.17" rpy="0 0 0"/>
-      <mass value="1.2"/>
-      <inertia ixx="${1.2*(b*b+c*c)/12.0}"  ixy="0"  ixz="0" iyy="${1.2*(a*a+c*c)/12.0}" iyz="0" izz="${1.2*(a*a+b*b)/12.0}" />
-    </inertial>
-    <visual>
-     <origin xyz="0 0 0" rpy="0 0 0" />
-     <geometry>
-        <box size="0.07 0.07 0.07" />
-     </geometry>
-     <material name="Cyan">
-       <color rgba="0 1.0 1.0 1.0"/>
-     </material>
-   </visual>
-   <collision>
-     <origin xyz="0 0 0" rpy="0 0 0"/>
-     <geometry>
-       <box size="0.07 0.07 0.07" />
-     </geometry>
+<link name="RSoftHand"/>
+<link name="r_palm"/>
+<link name="R_visual_cube">
+    <inertial>
+        <origin xyz="0 0 0" rpy="0 0 0"/>
+        <mass value="1.0e-5"/>
+        <inertia ixx="0"  ixy="0"  ixz="0" iyy="0" iyz="0" izz="0" />
+    </inertial>
+    <visual>
+        <origin xyz="0 0 0" rpy="0 0 0" />
+        <geometry>
+            <box size="0.08 0.08 0.08" />
+        </geometry>
+    </visual>
+</link>
+<gazebo reference="R_visual_cube">
+    <material>Gazebo/RedBright</material>
+</gazebo>
+<link name="RSoftHandLink">
+    <inertial>
+      <origin xyz="${1.1908576e+01*mmTom} ${2.1833446*mmTom} ${-1.5361558e+02*mmTom}" rpy="0 0 0"/>
+      <mass value="5.0e-01"/>
+      <inertia ixx="${5.0e-01*(a*a+c*c)/12.0}"  ixy="0"  ixz="0" iyy="${5.0e-01*(b*b+c*c)/12.0}" iyz="0" izz="${5.0e-01*(a*a+b*b)/12.0}" />
+    </inertial>
+    <visual>
+      <origin xyz="0.0 0.0 0.0" rpy="0.0 0.0 0.0"/>
+      <geometry name="RSoftHandLink_visual">
+        <mesh filename="package://bigman_urdf/meshes/SoftHandOpen.STL" scale="0.001 0.001 0.001" />
+      </geometry>
+      <material name="black"/>
+   </visual>
+   <collision>
+      <origin xyz="0.0 0.0 0.0" rpy="0.0 0.0 0.0"/>
+      <geometry name="RSoftHandLink_collision">
+        <mesh filename="package://bigman_urdf/meshes/simple/SoftHandOpen.STL" scale="0.001 0.001 0.001" />
+      </geometry>
+   </collision>
+  </link>
+  <link name="LSoftHand"/>
+  <link name="l_palm"/>
+  <link name="L_visual_cube">
+      <inertial>
+          <origin xyz="0 0 0" rpy="0 0 0"/>
+          <mass value="1.0e-5"/>
+          <inertia ixx="0"  ixy="0"  ixz="0" iyy="0" iyz="0" izz="0" />
+      </inertial>
+      <visual>
+          <origin xyz="0 0 0" rpy="0 0 0" />
+          <geometry>
+              <box size="0.08 0.08 0.08" />
+          </geometry>
+      </visual>
+  </link>
+  <gazebo reference="L_visual_cube">
+      <material>Gazebo/RedBright</material>
+  </gazebo>
+  <link name="LSoftHandLink">
+    <inertial>
+      <origin xyz="${1.1908576e+01*mmTom} ${-2.1833446*mmTom} ${-1.5361558e+02*mmTom}" rpy="0 0 0"/>
+      <mass value="5.0e-01"/>
+      <inertia ixx="${5.0e-01*(a*a+c*c)/12.0}"  ixy="0"  ixz="0" iyy="${5.0e-01*(b*b+c*c)/12.0}" iyz="0" izz="${5.0e-01*(a*a+b*b)/12.0}" />
+    </inertial>
+    <visual>
+      <origin xyz="0.0 0.0 0.0" rpy="0.0 0.0 0.0"/>
+      <geometry name="LSoftHandLink_visual">
+        <mesh filename="package://bigman_urdf/meshes/SoftHandOpen.STL" scale="0.001 -0.001 0.001" />
+      </geometry>
+      <material name="black"/>
+   </visual>
+   <collision>
+     <origin xyz="0.0 0.0 0.0" rpy="0.0 0.0 0.0"/>
+      <geometry name="LSoftHandLink_collision">
+        <mesh filename="package://bigman_urdf/meshes/simple/SoftHandOpen.STL" scale="0.001 -0.001 0.001" />
+      </geometry>
    </collision>
   </link>
 <!-- JOINTS -->
-<joint name="r_handj" type="revolute">
+  <joint name="r_handj" type="revolute">
+      <parent link="RWrMot3"/>
+      <child link="R_visual_cube"/>
+      <origin xyz="0 0 -0.04" rpy="0 0 0"/>
+      <axis xyz="1 0 0" />
+      <limit velocity="4.0" effort="5" lower="0.0" upper="1.7" />
+      <dynamics friction="0" damping="3.0"/>
+  </joint>
+  <joint name="r_handj1" type="fixed">
         <parent link="RWrMot3"/>
+        <child link="RSoftHandLink"/>
+        <origin xyz="0 0 0" rpy="0 0 0"/>
+  </joint>
+  <joint name="r_handj2" type="fixed">
+        <parent link="RSoftHandLink"/>
         <child link="RSoftHand"/>
-        <origin xyz="0 0 -0.04" rpy="0 0 0"/>
-        <axis xyz="1 0 0" />
-        <limit velocity="4.0" effort="5" lower="0.0" upper="5.0" />
-        <dynamics friction="0" damping="3.0"/>
-</joint>
-<joint name="l_handj" type="revolute">
+        <origin xyz="${1.1908576e+01*mmTom} ${2.1833446*mmTom} ${-1.5361558e+02*mmTom}" rpy="0 0 0"/>
+  </joint>
+  <joint name="r_handj3" type="fixed">
+        <parent link="RSoftHand"/>
+        <child link="r_palm"/>
+        <origin xyz="0 ${2.0696923e+01*mmTom+5.0*mmTom} 0.0" rpy="0 0 0"/>
+  </joint>
+  <joint name="l_handj" type="revolute">
+      <parent link="LWrMot3"/>
+      <child link="L_visual_cube"/>
+      <origin xyz="0 0 -0.04" rpy="0 0 0"/>
+      <axis xyz="-1 0 0" />
+      <limit velocity="4.0" effort="5" lower="0" upper="1.7" />
+      <dynamics friction="0" damping="3.0"/>
+  </joint>
+  <joint name="l_handj1" type="fixed">
         <parent link="LWrMot3"/>
+        <child link="LSoftHandLink"/>
+        <origin xyz="0 0 0" rpy="0 0 0"/>
+  </joint>
+  <joint name="l_handj2" type="fixed">
+        <parent link="LSoftHandLink"/>
         <child link="LSoftHand"/>
-        <origin xyz="0 0 -0.04" rpy="0 0 0"/>
-        <axis xyz="-1 0 0" />
-        <limit velocity="4.0" effort="5" lower="0" upper="5.0" />
-        <dynamics friction="0" damping="3.0"/>
-</joint>
+        <origin xyz="${1.1908576e+01*mmTom} ${-2.1833446*mmTom} ${-1.5361558e+02*mmTom}" rpy="0 0 0"/>
+  </joint>
+  <joint name="l_handj3" type="fixed">
+        <parent link="LSoftHand"/>
+        <child link="l_palm"/>
+        <origin xyz="0 ${-2.0696923e+01*mmTom-5.0*mmTom} 0.0" rpy="0 0 0"/>
+  </joint>
 </xacro:unless>
 </robot>
