Commit message: Added flag to select between safe joint limits or normal joint limits.

File: bigman_urdf/urdf/bigman_config.urdf.xacro (robot description, xacro)
@@ -113,3 +113,15 @@
 -->
 <xacro:property name="BIGMAN_NEW_FEET" value="true" />
+<!--
+####################################################
+##
+##  BIGMAN_SAFETY_JOINT_LIMITS_X
+##  if "true" the more strict joint limits are used
+##  for the X part
+##
+##
+####################################################
+-->
+<xacro:property name="BIGMAN_SAFETY_JOINT_LIMITS_ARMS" value="true" />
+<xacro:property name="BIGMAN_SAFETY_JOINT_LIMITS_TORSO" value="false" />
 </robot>

File: bigman_urdf/urdf/bigman_robot.urdf.xacro (robot description, xacro)
@@ -28,5 +28,5 @@
 <xacro:if value="${BIGMAN_LEGS}">
   <origin xyz="0.0 0.0 1.12" rpy="0 0 0" />
-  <xacro:include filename="$(find bigman_urdf)/urdf/gazebo/microstrain_3dmgx2_imu.gazebo.xacro" />
+  <!--xacro:include filename="$(find bigman_urdf)/urdf/gazebo/microstrain_3dmgx2_imu.gazebo.xacro" /-->
 </xacro:if>
   <xacro:include filename="$(find bigman_urdf)/urdf/gazebo/force_torque.gazebo.xacro" />

File: bigman_urdf/urdf/config/bigman_gazebo.urdf.xacro (robot description, xacro)
@@ -113,3 +113,15 @@
 -->
 <xacro:property name="BIGMAN_NEW_FEET" value="true" />
+<!--
+####################################################
+##
+##  BIGMAN_SAFETY_JOINT_LIMITS_X
+##  if "true" the more strict joint limits are used
+##  for the X part
+##
+##
+####################################################
+-->
+<xacro:property name="BIGMAN_SAFETY_JOINT_LIMITS_ARMS" value="true" />
+<xacro:property name="BIGMAN_SAFETY_JOINT_LIMITS_TORSO" value="false" />
 </robot>

File: bigman_urdf/urdf/config/bigman_only_legs.urdf.xacro (robot description, xacro)
@@ -113,3 +113,15 @@
 -->
 <xacro:property name="BIGMAN_NEW_FEET" value="true" />
+<!--
+####################################################
+##
+##  BIGMAN_SAFETY_JOINT_LIMITS_X
+##  if "true" the more strict joint limits are used
+##  for the X part
+##
+##
+####################################################
+-->
+<xacro:property name="BIGMAN_SAFETY_JOINT_LIMITS_ARMS" value="true" />
+<xacro:property name="BIGMAN_SAFETY_JOINT_LIMITS_TORSO" value="false" />
 </robot>

File: bigman_urdf/urdf/config/bigman_only_upper_body.urdf.xacro (robot description, xacro)
@@ -113,3 +113,15 @@
 -->
 <xacro:property name="BIGMAN_NEW_FEET" value="false" />
+<!--
+####################################################
+##
+##  BIGMAN_SAFETY_JOINT_LIMITS_X
+##  if "true" the more strict joint limits are used
+##  for the X part
+##
+##
+####################################################
+-->
+<xacro:property name="BIGMAN_SAFETY_JOINT_LIMITS_ARMS" value="true" />
+<xacro:property name="BIGMAN_SAFETY_JOINT_LIMITS_TORSO" value="false" />
 </robot>

File: bigman_urdf/urdf/config/bigman_only_upper_body_gazebo.urdf.xacro (robot description, xacro)
@@ -113,3 +113,15 @@
 -->
 <xacro:property name="BIGMAN_NEW_FEET" value="false" />
+<!--
+####################################################
+##
+##  BIGMAN_SAFETY_JOINT_LIMITS_X
+##  if "true" the more strict joint limits are used
+##  for the X part
+##
+##
+####################################################
+-->
+<xacro:property name="BIGMAN_SAFETY_JOINT_LIMITS_ARMS" value="true" />
+<xacro:property name="BIGMAN_SAFETY_JOINT_LIMITS_TORSO" value="false" />
 </robot>

File: bigman_urdf/urdf/config/bigman_real.urdf.xacro (robot description, xacro)
@@ -113,3 +113,15 @@
 -->
 <xacro:property name="BIGMAN_NEW_FEET" value="true" />
+<!--
+####################################################
+##
+##  BIGMAN_SAFETY_JOINT_LIMITS_X
+##  if "true" the more strict joint limits are used
+##  for the X part
+##
+##
+####################################################
+-->
+<xacro:property name="BIGMAN_SAFETY_JOINT_LIMITS_ARMS" value="true" />
+<xacro:property name="BIGMAN_SAFETY_JOINT_LIMITS_TORSO" value="false" />
 </robot>

File: bigman_urdf/urdf/parts/torso.urdf.xacro (robot description, xacro)
@@ -155,5 +155,10 @@
     <origin xyz="0.1115 0 0.195982" rpy="0 0 0" />
     <axis xyz="${cos_26} 0 ${sin_26}" />
-    <limit velocity="6.283" effort="120" lower="${-15.0*toRad}" upper="${15.0*toRad}" />
+    <xacro:if value="${BIGMAN_SAFETY_JOINT_LIMITS_TORSO}">
+    	<limit velocity="6.283" effort="120" lower="${-15.0*toRad}" upper="${15.0*toRad}" />
+    </xacro:if>
+    <xacro:unless value="${BIGMAN_SAFETY_JOINT_LIMITS_TORSO}">
+    	<limit velocity="6.283" effort="120" lower="${-35.0*toRad}" upper="${35.0*toRad}" />
+    </xacro:unless>
     <dynamics friction="0" damping="3.0"/>
 </joint>
@@ -163,5 +168,10 @@
     <origin xyz="0 0 0" rpy="0 0 0" />
     <axis xyz="0 1 0" />
-    <limit velocity="6.283" effort="220" lower="${-10.0*toRad}" upper="${40.0*toRad}" />
+    <xacro:if value="${BIGMAN_SAFETY_JOINT_LIMITS_TORSO}">
+    	<limit velocity="6.283" effort="220" lower="${-10.0*toRad}" upper="${40.0*toRad}" />
+    </xacro:if>
+    <xacro:unless value="${BIGMAN_SAFETY_JOINT_LIMITS_TORSO}">
+    	<limit velocity="6.283" effort="220" lower="${-20.0*toRad}" upper="${80.0*toRad}" />
+    </xacro:unless>
     <dynamics friction="0" damping="3.0"/>
   </joint>
@@ -171,5 +181,10 @@
     <origin xyz="0 0 0.22275" rpy="0 0 0" />
     <axis xyz="0 0 1" />
-    <limit velocity="6.283" effort="120" lower="${-100.0*toRad}" upper="${100.0*toRad}" />
+    <xacro:if value="${BIGMAN_SAFETY_JOINT_LIMITS_TORSO}">
+    	<limit velocity="6.283" effort="120" lower="${-100.0*toRad}" upper="${100.0*toRad}" />
+    </xacro:if>
+    <xacro:unless value="${BIGMAN_SAFETY_JOINT_LIMITS_TORSO}">
+    	<limit velocity="6.283" effort="120" lower="${-163.0*toRad}" upper="${163.0*toRad}" />
+    </xacro:unless>
     <dynamics friction="0" damping="3.0"/>
   </joint>

Commit message: Added flag to use safety joint limits in arms

File: bigman_urdf/urdf/bigman_config.urdf.xacro (robot description, xacro)
@@ -123,5 +123,5 @@
 ####################################################
 -->
-<xacro:property name="BIGMAN_SAFETY_JOINT_LIMITS_ARMS" value="true" />
+<xacro:property name="BIGMAN_SAFETY_JOINT_LIMITS_ARMS" value="false" />
 <xacro:property name="BIGMAN_SAFETY_JOINT_LIMITS_TORSO" value="false" />
 </robot>

File: bigman_urdf/urdf/config/bigman_gazebo.urdf.xacro (robot description, xacro)
@@ -123,5 +123,5 @@
 ####################################################
 -->
-<xacro:property name="BIGMAN_SAFETY_JOINT_LIMITS_ARMS" value="true" />
+<xacro:property name="BIGMAN_SAFETY_JOINT_LIMITS_ARMS" value="false" />
 <xacro:property name="BIGMAN_SAFETY_JOINT_LIMITS_TORSO" value="false" />
 </robot>

File: bigman_urdf/urdf/config/bigman_only_legs.urdf.xacro (robot description, xacro)
@@ -123,5 +123,5 @@
 ####################################################
 -->
-<xacro:property name="BIGMAN_SAFETY_JOINT_LIMITS_ARMS" value="true" />
+<xacro:property name="BIGMAN_SAFETY_JOINT_LIMITS_ARMS" value="false" />
 <xacro:property name="BIGMAN_SAFETY_JOINT_LIMITS_TORSO" value="false" />
 </robot>

File: bigman_urdf/urdf/config/bigman_only_upper_body.urdf.xacro (robot description, xacro)
@@ -123,5 +123,5 @@
 ####################################################
 -->
-<xacro:property name="BIGMAN_SAFETY_JOINT_LIMITS_ARMS" value="true" />
+<xacro:property name="BIGMAN_SAFETY_JOINT_LIMITS_ARMS" value="false" />
 <xacro:property name="BIGMAN_SAFETY_JOINT_LIMITS_TORSO" value="false" />
 </robot>

File: bigman_urdf/urdf/config/bigman_only_upper_body_gazebo.urdf.xacro (robot description, xacro)
@@ -123,5 +123,5 @@
 ####################################################
 -->
-<xacro:property name="BIGMAN_SAFETY_JOINT_LIMITS_ARMS" value="true" />
+<xacro:property name="BIGMAN_SAFETY_JOINT_LIMITS_ARMS" value="false" />
 <xacro:property name="BIGMAN_SAFETY_JOINT_LIMITS_TORSO" value="false" />
 </robot>

File: bigman_urdf/urdf/config/bigman_real.urdf.xacro (robot description, xacro)
@@ -123,5 +123,5 @@
 ####################################################
 -->
-<xacro:property name="BIGMAN_SAFETY_JOINT_LIMITS_ARMS" value="true" />
+<xacro:property name="BIGMAN_SAFETY_JOINT_LIMITS_ARMS" value="false" />
 <xacro:property name="BIGMAN_SAFETY_JOINT_LIMITS_TORSO" value="false" />
 </robot>

File: bigman_urdf/urdf/parts/arms.urdf.xacro (robot description, xacro)
@@ -183,6 +183,10 @@
 </xacro:unless>
     <axis xyz="0 ${cos_42} ${-sin_42}" />
-    <!--limit velocity="6.283" effort="120" lower="${-163*toRad}" upper="${161.0*toRad}" /-->
-    <limit velocity="6.283" effort="120" lower="${-55*toRad}" upper="${85.0*toRad}" /> <!-- <limit velocity="6.283" effort="120" lower="${-57*toRad}" upper="${89.0*toRad}" /> -->
+    <xacro:if value="${BIGMAN_SAFETY_JOINT_LIMITS_ARMS}">
+    	<limit velocity="6.283" effort="120" lower="${-55*toRad}" upper="${85.0*toRad}" />
+    </xacro:if>
+    <xacro:unless value="${BIGMAN_SAFETY_JOINT_LIMITS_ARMS}">
+    	<limit velocity="6.283" effort="120" lower="${-163*toRad}" upper="${161.0*toRad}" />
+    </xacro:unless>
     <dynamics friction="0" damping="3.0"/>
 </joint>
@@ -192,6 +196,10 @@
     <origin xyz="0.0 -0.116568264 0.03364" rpy="0 0 0" />
     <axis xyz="1 0 0" />
-    <!--limit velocity="6.283" effort="120" lower="${-221.0*toRad}" upper="${-7.0*toRad}" /-->
-    <limit velocity="6.283" effort="120" lower="${-120.0*toRad}" upper="${-7.0*toRad}" />
+    <xacro:if value="${BIGMAN_SAFETY_JOINT_LIMITS_ARMS}">
+    	<limit velocity="6.283" effort="120" lower="${-120.0*toRad}" upper="${-7.0*toRad}" />
+    </xacro:if>
+    <xacro:unless value="${BIGMAN_SAFETY_JOINT_LIMITS_ARMS}">
+    	<limit velocity="6.283" effort="120" lower="${-221.0*toRad}" upper="${-7.0*toRad}" />
+    </xacro:unless>
     <dynamics friction="0" damping="3.0"/>
 </joint>
@@ -223,6 +231,10 @@
 </xacro:unless>
     <axis xyz="0.0 ${cos_42} ${sin_42}" />
-    <!--limit velocity="6.283" effort="120" lower="${-165.0*toRad}" upper="${160.0*toRad}" /-->
-    <limit velocity="6.283" effort="120" lower="${-55.0*toRad}" upper="${85.0*toRad}" /><!-- <limit velocity="6.283" effort="120" lower="${-57*toRad}" upper="${89.0*toRad}" /> -->
+    <xacro:if value="${BIGMAN_SAFETY_JOINT_LIMITS_ARMS}">
+    	<limit velocity="6.283" effort="120" lower="${-55.0*toRad}" upper="${85.0*toRad}" />
+    </xacro:if>
+    <xacro:unless value="${BIGMAN_SAFETY_JOINT_LIMITS_ARMS}">
+    	<limit velocity="6.283" effort="120" lower="${-165.0*toRad}" upper="${160.0*toRad}" />
+    </xacro:unless>
     <dynamics friction="0" damping="3.0"/>
 </joint>
@@ -232,6 +244,10 @@
     <origin xyz="0.0 0.116568264 0.03364" rpy="0 0 0" />
     <axis xyz="1 0 0" />
-    <!--limit velocity="6.283" effort="120" lower="${5.0*toRad}" upper="${221.0*toRad}" /-->
-    <limit velocity="6.283" effort="120" lower="${5.0*toRad}" upper="${120.0*toRad}" />
+    <xacro:if value="${BIGMAN_SAFETY_JOINT_LIMITS_ARMS}">
+    	<limit velocity="6.283" effort="120" lower="${5.0*toRad}" upper="${120.0*toRad}" />
+    </xacro:if>
+    <xacro:unless value="${BIGMAN_SAFETY_JOINT_LIMITS_ARMS}">
+    	<limit velocity="6.283" effort="120" lower="${5.0*toRad}" upper="${221.0*toRad}" />
+    </xacro:unless>
     <dynamics friction="0" damping="3.0"/>
 </joint>

Commit message: Added xacro properties to control the robot using YARP or XBOT. XBOT enabled, YARP disabled.

File: bigman_urdf/urdf/bigman_config.urdf.xacro (robot description, xacro)
@@ -3,4 +3,23 @@
 <xacro:property name="model_name" value="IIT Bigman Ctrl" />
 <xacro:property name="model_version" value="0.1" />
+<!--
+####################################################
+##
+##  BIGMAN_YARP
+##  if "true" the bigman robot is controlled via YARP
+##
+####################################################
+-->
+<xacro:property name="BIGMAN_YARP" value="false" />
+<!--
+####################################################
+##
+##  BIGMAN_XBOT
+##  if "true" the bigman robot is controlled via
+##  XBotCore Suite
+##
+####################################################
+-->
+<xacro:property name="BIGMAN_XBOT" value="true" />
 <!--
 ####################################################

File: bigman_urdf/urdf/bigman_robot.urdf.xacro (robot description, xacro)
@@ -8,6 +8,5 @@
   -->
   <!-- Uncomment this to have the robot rigidly connected to the world -->
-<!--
-  <link name="world"/>
+<!--  <link name="world"/>
    <joint name="fixed" type="fixed">
     <parent link="world"/>
@@ -33,6 +32,12 @@
   <xacro:include filename="$(find bigman_urdf)/urdf/gazebo/force_torque.gazebo.xacro" />
   <xacro:include filename="$(find bigman_urdf)/urdf/gazebo/bigman.gazebo.xacro" />
+  <!-- XBOTCORE PLUGINS for GAZEBO SIMULATION -->
+  <xacro:if value="${BIGMAN_XBOT}">
+    <xacro:include filename="$(find bigman_urdf)/urdf/gazebo/xbot_control.gazebo.xacro" />
+  </xacro:if>
 <!-- YARP PLUGINS for GAZEBO SIMULATION -->
-  <xacro:include filename="$(find bigman_urdf)/urdf/gazebo/yarp_control.gazebo.xacro" />
+  <xacro:if value="${BIGMAN_YARP}">
+    <xacro:include filename="$(find bigman_urdf)/urdf/gazebo/yarp_control.gazebo.xacro" />
+  </xacro:if>
   <xacro:include filename="$(find bigman_urdf)/urdf/gazebo/bigman_materials.gazebo.xacro" />
 </robot>

File: bigman_urdf/urdf/config/bigman_gazebo.urdf.xacro (robot description, xacro)
@@ -3,4 +3,23 @@
 <xacro:property name="model_name" value="IIT Bigman" />
 <xacro:property name="model_version" value="0.1" />
+<!--
+####################################################
+##
+##  BIGMAN_YARP
+##  if "true" the bigman robot is controlled via YARP
+##
+####################################################
+-->
+<xacro:property name="BIGMAN_YARP" value="false" />
+<!--
+####################################################
+##
+##  BIGMAN_XBOT
+##  if "true" the bigman robot is controlled via
+##  XBotCore Suite
+##
+####################################################
+-->
+<xacro:property name="BIGMAN_XBOT" value="true" />
 <!--
 ####################################################

File: bigman_urdf/urdf/config/bigman_only_legs.urdf.xacro (robot description, xacro)
@@ -3,4 +3,23 @@
 <xacro:property name="model_name" value="IIT Bigman Legs" />
 <xacro:property name="model_version" value="0.1" />
+<!--
+####################################################
+##
+##  BIGMAN_YARP
+##  if "true" the bigman robot is controlled via YARP
+##
+####################################################
+-->
+<xacro:property name="BIGMAN_YARP" value="false" />
+<!--
+####################################################
+##
+##  BIGMAN_XBOT
+##  if "true" the bigman robot is controlled via
+##  XBotCore Suite
+##
+####################################################
+-->
+<xacro:property name="BIGMAN_XBOT" value="true" />
 <!--
 ####################################################

File: bigman_urdf/urdf/config/bigman_only_upper_body.urdf.xacro (robot description, xacro)
@@ -3,4 +3,23 @@
 <xacro:property name="model_name" value="IIT Bigman Upper Body Ctrl" />
 <xacro:property name="model_version" value="0.1" />
+<!--
+####################################################
+##
+##  BIGMAN_YARP
+##  if "true" the bigman robot is controlled via YARP
+##
+####################################################
+-->
+<xacro:property name="BIGMAN_YARP" value="false" />
+<!--
+####################################################
+##
+##  BIGMAN_XBOT
+##  if "true" the bigman robot is controlled via
+##  XBotCore Suite
+##
+####################################################
+-->
+<xacro:property name="BIGMAN_XBOT" value="true" />
 <!--
 ####################################################
@@ -45,5 +64,5 @@
 ####################################################
 -->
-<xacro:property name="BIGMAN_FIXED_HANDS" value="true" />
+<xacro:property name="BIGMAN_FIXED_HANDS" value="false" />
 <!--
 ####################################################

File: bigman_urdf/urdf/config/bigman_only_upper_body_gazebo.urdf.xacro (robot description, xacro)
@@ -3,4 +3,23 @@
 <xacro:property name="model_name" value="IIT Bigman Upper Body" />
 <xacro:property name="model_version" value="0.1" />
+<!--
+####################################################
+##
+##  BIGMAN_YARP
+##  if "true" the bigman robot is controlled via YARP
+##
+####################################################
+-->
+<xacro:property name="BIGMAN_YARP" value="false" />
+<!--
+####################################################
+##
+##  BIGMAN_XBOT
+##  if "true" the bigman robot is controlled via
+##  XBotCore Suite
+##
+####################################################
+-->
+<xacro:property name="BIGMAN_XBOT" value="true" />
 <!--
 ####################################################

File: bigman_urdf/urdf/config/bigman_real.urdf.xacro (robot description, xacro)
@@ -3,4 +3,23 @@
 <xacro:property name="model_name" value="IIT Bigman Real" />
 <xacro:property name="model_version" value="0.1" />
+<!--
+####################################################
+##
+##  BIGMAN_YARP
+##  if "true" the bigman robot is controlled via YARP
+##
+####################################################
+-->
+<xacro:property name="BIGMAN_YARP" value="false" />
+<!--
+####################################################
+##
+##  BIGMAN_XBOT
+##  if "true" the bigman robot is controlled via
+##  XBotCore Suite
+##
+####################################################
+-->
+<xacro:property name="BIGMAN_XBOT" value="true" />
 <!--
 ####################################################

File: bigman_urdf/urdf/gazebo/force_torque.gazebo.xacro (robot description, xacro)
@@ -18,7 +18,9 @@
 			<update_rate>1000</update_rate>
                      <pose>0 0 -0.0565 0 0 0</pose>
-			<plugin name="RForearmPlate_FT_plugin" filename="libgazebo_yarp_forcetorque.so">
-				<yarpConfigurationFile>model://bigman_urdf/conf/bigman/bigman_gazebo_right_arm_ft.ini</yarpConfigurationFile>
-			</plugin>
+                        <xacro:if value="${BIGMAN_YARP}">
+			  <plugin name="RForearmPlate_FT_plugin" filename="libgazebo_yarp_forcetorque.so">
+			  	<yarpConfigurationFile>model://bigman_urdf/conf/bigman/bigman_gazebo_right_arm_ft.ini</yarpConfigurationFile>
+			  </plugin>
+                        </xacro:if>
 		</sensor>
 	</gazebo>
@@ -33,7 +35,9 @@
 			<update_rate>1000</update_rate>
                      <pose>0 0 -0.0565 0 0 0</pose>
+                     <xacro:if value="${BIGMAN_YARP}">
 			<plugin name="LForearmPlate_FT_plugin" filename="libgazebo_yarp_forcetorque.so">
 				<yarpConfigurationFile>model://bigman_urdf/conf/bigman/bigman_gazebo_left_arm_ft.ini</yarpConfigurationFile>
 			</plugin>
+                     </xacro:if>
 		</sensor>
 	</gazebo>
@@ -50,7 +54,9 @@
 			<update_rate>1000</update_rate>
 			<pose>0.005 0 -0.107 0 0 0</pose>
-			<plugin name="LAnkSag_FT_plugin" filename="libgazebo_yarp_forcetorque.so">
+                        <xacro:if value="${BIGMAN_YARP}">
+			  <plugin name="LAnkSag_FT_plugin" filename="libgazebo_yarp_forcetorque.so">
 				<yarpConfigurationFile>model://bigman_urdf/conf/bigman/bigman_gazebo_left_leg_ft.ini</yarpConfigurationFile>
-			</plugin>
+			  </plugin>
+                        </xacro:if>
 		</sensor>
 	</gazebo>
@@ -65,7 +71,9 @@
 			<update_rate>1000</update_rate>
 			<pose>0.005 0 -0.107 0 0 0</pose>
-			<plugin name="RAnkSag_FT_plugin" filename="libgazebo_yarp_forcetorque.so">
+                        <xacro:if value="${BIGMAN_YARP}">
+			  <plugin name="RAnkSag_FT_plugin" filename="libgazebo_yarp_forcetorque.so">
 				<yarpConfigurationFile>model://bigman_urdf/conf/bigman/bigman_gazebo_right_leg_ft.ini</yarpConfigurationFile>
-	        	</plugin>
+	        	  </plugin>
+                        </xacro:if>
 		</sensor>
 	</gazebo>

File: bigman_urdf/urdf/gazebo/microstrain_3dmgx2_imu.gazebo.xacro (robot description, xacro)
@@ -31,7 +31,9 @@
           -->
          </imu>
-         <plugin name="bigman_yarp_gazebo_plugin_IMU" filename="libgazebo_yarp_imu.so">
-           <yarpConfigurationFile>model://bigman_urdf/conf/bigman/bigman_gazebo_inertial.ini</yarpConfigurationFile>
-         </plugin>
+         <xacro:if value="${BIGMAN_YARP}">
+           <plugin name="bigman_yarp_gazebo_plugin_IMU" filename="libgazebo_yarp_imu.so">
+             <yarpConfigurationFile>model://bigman_urdf/conf/bigman/bigman_gazebo_inertial.ini</yarpConfigurationFile>
+           </plugin>
+         </xacro:if>
         </sensor>
        </gazebo>
@@ -61,7 +63,9 @@
           -->
          </imu>
-         <plugin name="bigman_yarp_gazebo_plugin_IMU2" filename="libgazebo_yarp_imu.so">
-           <yarpConfigurationFile>model://bigman_urdf/conf/bigman/bigman_gazebo_inertial2.ini</yarpConfigurationFile>
-         </plugin>
+         <xacro:if value="${BIGMAN_YARP}">
+           <plugin name="bigman_yarp_gazebo_plugin_IMU2" filename="libgazebo_yarp_imu.so">
+             <yarpConfigurationFile>model://bigman_urdf/conf/bigman/bigman_gazebo_inertial2.ini</yarpConfigurationFile>
+           </plugin>
+         </xacro:if>
         </sensor>
        </gazebo>
