Commit message: Added the magnetic_attach plugin to the robot

File: bigman_urdf/urdf/bigman_config.urdf.xacro (robot description, xacro)
@@ -144,3 +144,14 @@
 <xacro:property name="BIGMAN_SAFETY_JOINT_LIMITS_ARMS" value="false" />
 <xacro:property name="BIGMAN_SAFETY_JOINT_LIMITS_TORSO" value="false" />
+<!--
+####################################################
+##
+##  BIGMAN_MAGNETIC_ATTACH_ROS
+##  if "true" the magnetic_attach_ros plugin is used
+##  for the hands
+##
+##
+####################################################
+-->
+<xacro:property name="BIGMAN_MAGNETIC_ATTACH_ROS" value="true" />
 </robot>

File: bigman_urdf/urdf/bigman_robot.urdf.xacro (robot description, xacro)
@@ -40,4 +40,7 @@
     <xacro:include filename="$(find bigman_urdf)/urdf/gazebo/yarp_control.gazebo.xacro" />
   </xacro:if>
+  <xacro:if value="${BIGMAN_MAGNETIC_ATTACH_ROS}">
+    <xacro:include filename="$(find bigman_urdf)/urdf/gazebo/magnetic_attach_ros.gazebo.xacro" />
+  </xacro:if>
   <xacro:include filename="$(find bigman_urdf)/urdf/gazebo/bigman_materials.gazebo.xacro" />
 </robot>

File: bigman_urdf/urdf/config/bigman_gazebo.urdf.xacro (robot description, xacro)
@@ -144,3 +144,14 @@
 <xacro:property name="BIGMAN_SAFETY_JOINT_LIMITS_ARMS" value="false" />
 <xacro:property name="BIGMAN_SAFETY_JOINT_LIMITS_TORSO" value="false" />
+<!--
+####################################################
+##
+##  BIGMAN_MAGNETIC_ATTACH_ROS
+##  if "true" the magnetic_attach_ros plugin is used
+##  for the hands
+##
+##
+####################################################
+-->
+<xacro:property name="BIGMAN_MAGNETIC_ATTACH_ROS" value="true" />
 </robot>

File: bigman_urdf/urdf/config/bigman_only_legs.urdf.xacro (robot description, xacro)
@@ -144,3 +144,14 @@
 <xacro:property name="BIGMAN_SAFETY_JOINT_LIMITS_ARMS" value="false" />
 <xacro:property name="BIGMAN_SAFETY_JOINT_LIMITS_TORSO" value="false" />
+<!--
+####################################################
+##
+##  BIGMAN_MAGNETIC_ATTACH_ROS
+##  if "true" the magnetic_attach_ros plugin is used
+##  for the hands
+##
+##
+####################################################
+-->
+<xacro:property name="BIGMAN_MAGNETIC_ATTACH_ROS" value="false" />
 </robot>

File: bigman_urdf/urdf/config/bigman_only_upper_body.urdf.xacro (robot description, xacro)
@@ -144,3 +144,14 @@
 <xacro:property name="BIGMAN_SAFETY_JOINT_LIMITS_ARMS" value="false" />
 <xacro:property name="BIGMAN_SAFETY_JOINT_LIMITS_TORSO" value="false" />
+<!--
+####################################################
+##
+##  BIGMAN_MAGNETIC_ATTACH_ROS
+##  if "true" the magnetic_attach_ros plugin is used
+##  for the hands
+##
+##
+####################################################
+-->
+<xacro:property name="BIGMAN_MAGNETIC_ATTACH_ROS" value="true" />
 </robot>

File: bigman_urdf/urdf/config/bigman_only_upper_body_gazebo.urdf.xacro (robot description, xacro)
@@ -144,3 +144,14 @@
 <xacro:property name="BIGMAN_SAFETY_JOINT_LIMITS_ARMS" value="false" />
 <xacro:property name="BIGMAN_SAFETY_JOINT_LIMITS_TORSO" value="false" />
+<!--
+####################################################
+##
+##  BIGMAN_MAGNETIC_ATTACH_ROS
+##  if "true" the magnetic_attach_ros plugin is used
+##  for the hands
+##
+##
+####################################################
+-->
+<xacro:property name="BIGMAN_MAGNETIC_ATTACH_ROS" value="true" />
 </robot>

File: bigman_urdf/urdf/config/bigman_real.urdf.xacro (robot description, xacro)
@@ -144,3 +144,14 @@
 <xacro:property name="BIGMAN_SAFETY_JOINT_LIMITS_ARMS" value="false" />
 <xacro:property name="BIGMAN_SAFETY_JOINT_LIMITS_TORSO" value="false" />
+<!--
+####################################################
+##
+##  BIGMAN_MAGNETIC_ATTACH_ROS
+##  if "true" the magnetic_attach_ros plugin is used
+##  for the hands
+##
+##
+####################################################
+-->
+<xacro:property name="BIGMAN_MAGNETIC_ATTACH_ROS" value="true" />
 </robot>

File: bigman_urdf/urdf/gazebo/bigman.gazebo.xacro (robot description, xacro)
@@ -171,4 +171,15 @@
     <provideFeedback>true</provideFeedback>
    </gazebo>
+   <!-- The reference tag has to be the link that will be present in gazebo while the
+   collision tag will be the collision under the link present in the sdf -->
+   <xacro:if value="${BIGMAN_MAGNETIC_ATTACH_ROS}">
+    <gazebo reference="RWrMot3">
+     <sensor name='RWrMot3_contact_sensor' type='contact'>
+      <contact>
+       <collision>RWrMot3_fixed_joint_lump__RSoftHandLink_collision_1</collision>
+      </contact>
+     </sensor>
+    </gazebo>
+   </xacro:if>
     <xacro:unless value="${BIGMAN_FIXED_HANDS}">
       <gazebo reference="r_handj">
@@ -205,4 +216,15 @@
     <provideFeedback>true</provideFeedback>
    </gazebo>
+   <!-- The reference tag has to be the link that will be present in gazebo while the
+   collision tag will be the collision under the link present in the sdf -->
+   <xacro:if value="${BIGMAN_MAGNETIC_ATTACH_ROS}">
+    <gazebo reference="LWrMot3">
+     <sensor name='LWrMot3_contact_sensor' type='contact'>
+      <contact>
+       <collision>LWrMot3_fixed_joint_lump__LSoftHandLink_collision_1</collision>
+      </contact>
+     </sensor>
+    </gazebo>
+   </xacro:if>
     <xacro:unless value="${BIGMAN_FIXED_HANDS}">
       <gazebo reference="l_handj">
