Commit message: Deleted xtion from bigman

File: bigman_urdf/urdf/bigman.urdf.xacro (robot description, xacro)
@@ -15,14 +15,9 @@
 The coordinate frame called gaze defines the head position and orientation. The orientation indicates in which direction the head appears to be looking regardless of any sensors (camera for instance). -->
 <link name="gaze"/>
-<xacro:if value="${GAZEBO_BIGMAN_USES_XTION}">
-	<xacro:include filename="$(find bigman_urdf)/urdf/sensors/xtion.urdf.xacro" />
-</xacro:if>
-<xacro:unless value="${GAZEBO_BIGMAN_USES_XTION}">
-	<joint name="gaze_joint" type="fixed">
-		<parent link="torso"/>
-		<child link="gaze"/>
-		<origin xyz="0 0 0.1" rpy="0 0 0" />
-	</joint>
-</xacro:unless>
+<joint name="gaze_joint" type="fixed">
+	<parent link="torso"/>
+	<child link="gaze"/>
+	<origin xyz="0 0 0.1" rpy="0 0 0" />
+</joint>
 <!-- ************ COMAN BASE ************** -->
 <xacro:include filename="$(find bigman_urdf)/urdf/bigman_base.urdf.xacro"/>

File: bigman_urdf/urdf/bigman_config.urdf.xacro (robot description, xacro)
@@ -106,21 +106,3 @@
 -->
 <xacro:property name="GAZEBO_BIGMAN_USES_ACCURATE_FT" value="false" />
-<!--
-####################################################
-##
-##  Xtion SELECTION
-##
-##
-## options:
-## 1) BIGMAN classic without the staff to carry the sensor.
-##      Torso frame is connected to gaze link through a gaze_joint "fixed"
-## 2) BIGMAN with staff and xtion sensor. Torso frame is connected to a xtion_staff_link through
-##      a xtion_staff_joint "fixed". Xtion_staff_link is then connected to gaze_link through gaze_joint "fixed".
-##
-####################################################
-#
-# 1/2 (true/false)
-#
--->
-<xacro:property name="GAZEBO_BIGMAN_USES_XTION" value="true" />
 </robot>

File: bigman_urdf/urdf/bigman_robot.urdf.xacro (robot description, xacro)
@@ -9,7 +9,4 @@
   <xacro:include filename="$(find bigman_urdf)/urdf/gazebo/microstrain_3dmgx2_imu.gazebo.xacro" />
   <xacro:include filename="$(find bigman_urdf)/urdf/gazebo/bigman.gazebo.xacro" />
-  <xacro:if value="${GAZEBO_BIGMAN_USES_XTION}">
-	<xacro:include filename="$(find bigman_urdf)/urdf/gazebo/openni_kinect.gazebo.xacro" />
-  </xacro:if>
 <!-- YARP PLUGINS for GAZEBO SIMULATION -->
   <xacro:include filename="$(find bigman_urdf)/urdf/gazebo/yarp_control.gazebo.xacro" />

Commit message: Deleted files regarding coman without forearms

File: bigman_urdf/urdf/bigman.urdf.xacro (robot description, xacro)
@@ -28,7 +28,4 @@
 <link name="l_wrist"/>
 <link name="r_wrist"/>
-<xacro:if value="${GAZEBO_BIGMAN_USES_NO_FOREARMS}">
-    <xacro:include filename="$(find bigman_urdf)/urdf/parts/no_forearms.urdf.xacro" />
-</xacro:if>
 <xacro:if value="${GAZEBO_BIGMAN_USES_7DOF_FOREARMS_DRC_14}">
     <xacro:include filename="$(find bigman_urdf)/urdf/parts/7DOF_forearms_DRC_14.urdf.xacro" />

File: bigman_urdf/urdf/bigman_config.urdf.xacro (robot description, xacro)
@@ -48,5 +48,4 @@
 -->
 <!-- 3) 7DOFS_FOREARMS + SOFT_HANDS -->
-<xacro:property name="GAZEBO_BIGMAN_USES_NO_FOREARMS" value="false" />
 <xacro:property name="GAZEBO_BIGMAN_USES_7DOF_FOREARMS_DRC_14" value="true" />
 <xacro:property name="GAZEBO_BIGMAN_USES_SOFTHANDS_DRC_sw1_14" value="true" />

File: bigman_urdf/urdf/gazebo/yarp_control.gazebo.xacro (robot description, xacro)
@@ -68,26 +68,4 @@
 	</xacro:unless>
 </xacro:if>
-<xacro:if value="${GAZEBO_BIGMAN_USES_NO_FOREARMS}">
-	<plugin name="bigman_yarp_gazebo_plugin_left_arm" filename="libgazebo_yarp_controlboard.so">
-		<yarpConfigurationFile>model://bigman_urdf/conf/bigman_no_forearms/bigman_gazebo_left_arm.ini</yarpConfigurationFile>
-		<initialConfiguration>0.0 0.17 0.0 0.0</initialConfiguration>
-	</plugin>
-    <plugin name="bigman_yarp_gazebo_plugin_left_arm_speed" filename="libgazebo_yarp_jointsensors.so">
-        <yarpConfigurationFile>model://bigman_urdf/conf/bigman_no_forearms/bigman_gazebo_left_arm_speed.ini</yarpConfigurationFile>
-    </plugin>
-    <plugin name="bigman_yarp_gazebo_plugin_left_arm_torque" filename="libgazebo_yarp_jointsensors.so">
-        <yarpConfigurationFile>model://bigman_urdf/conf/bigman_no_forearms/bigman_gazebo_left_arm_torque.ini</yarpConfigurationFile>
-    </plugin>
-	<plugin name="bigman_yarp_gazebo_plugin_right_arm" filename="libgazebo_yarp_controlboard.so">
-		<yarpConfigurationFile>model://bigman_urdf/conf/bigman_no_forearms/bigman_gazebo_right_arm.ini</yarpConfigurationFile>
-		<initialConfiguration>0.0 -0.17 0.0 0.0</initialConfiguration>
-	</plugin>
-    <plugin name="bigman_yarp_gazebo_plugin_right_arm_speed" filename="libgazebo_yarp_jointsensors.so">
-        <yarpConfigurationFile>model://bigman_urdf/conf/bigman_no_forearms/bigman_gazebo_right_arm_speed.ini</yarpConfigurationFile>
-    </plugin>
-    <plugin name="bigman_yarp_gazebo_plugin_right_arm_torque" filename="libgazebo_yarp_jointsensors.so">
-        <yarpConfigurationFile>model://bigman_urdf/conf/bigman_no_forearms/bigman_gazebo_right_arm_torque.ini</yarpConfigurationFile>
-    </plugin>
-</xacro:if>
 <!-- Plugin to apply external wrenches to the robot -->
 <plugin name="bigman_yarp_gazebo_plugin_external_wrench" filename="libgazebo_yarp_externalwrench.so"/>

Commit message: Deleted variable for coman with 7DOF forearm

File: bigman_urdf/urdf/bigman.urdf.xacro (robot description, xacro)
@@ -28,11 +28,7 @@
 <link name="l_wrist"/>
 <link name="r_wrist"/>
-<xacro:if value="${GAZEBO_BIGMAN_USES_7DOF_FOREARMS_DRC_14}">
-    <xacro:include filename="$(find bigman_urdf)/urdf/parts/7DOF_forearms_DRC_14.urdf.xacro" />
-</xacro:if>
+<xacro:include filename="$(find bigman_urdf)/urdf/parts/7DOF_forearms_DRC_14.urdf.xacro" />
 <!-- ************ HANDS ************ -->
-<xacro:if value="${GAZEBO_BIGMAN_USES_7DOF_FOREARMS_DRC_14}">
-    <xacro:include filename="$(find bigman_urdf)/urdf/parts/soft_hand.urdf.xacro" />
-</xacro:if>
+<xacro:include filename="$(find bigman_urdf)/urdf/parts/soft_hand.urdf.xacro" />
 <!-- IMU -->
 <xacro:include filename="$(find bigman_urdf)/urdf/sensors/imu.urdf.xacro"/>

File: bigman_urdf/urdf/bigman_config.urdf.xacro (robot description, xacro)
@@ -25,28 +25,7 @@
 ##  FOREARMS & HANDS SELECTION
 ##
-##
-## options:
-## 1) no forearms
-## 2) 7dof forearms
-## 3) 7dof forearms + soft hands
-##
 ####################################################
-# TODO: checks (must be mutually exclusive).. eventually, a menu!... documentation!
-#       at the moment just the only combinations that work are:
 -->
-<!-- 1) NO_FOREARMS -->
-<!--
-<xacro:property name="GAZEBO_BIGMAN_USES_NO_FOREARMS" value="true" />
-<xacro:property name="GAZEBO_BIGMAN_USES_7DOF_FOREARMS_DRC_14" value="false" />
-<xacro:property name="GAZEBO_BIGMAN_USES_SOFTHANDS_DRC_sw1_14" value="false" />
--->
-<!-- 2) 7DOFS_FOREARMS -->
-<!--
-<xacro:property name="GAZEBO_BIGMAN_USES_NO_FOREARMS" value="false" />
-<xacro:property name="GAZEBO_BIGMAN_USES_7DOF_FOREARMS_DRC_14" value="true" />
-<xacro:property name="GAZEBO_BIGMAN_USES_SOFTHANDS_DRC_sw1_14" value="false" />
--->
-<!-- 3) 7DOFS_FOREARMS + SOFT_HANDS -->
-<xacro:property name="GAZEBO_BIGMAN_USES_7DOF_FOREARMS_DRC_14" value="true" />
+<!-- 7DOFS_FOREARMS + SOFT_HANDS -->
 <xacro:property name="GAZEBO_BIGMAN_USES_SOFTHANDS_DRC_sw1_14" value="true" />
 <!--

File: bigman_urdf/urdf/gazebo/bigman.gazebo.xacro (robot description, xacro)
@@ -126,5 +126,4 @@
     <provideFeedback>true</provideFeedback>
    </gazebo>
-<xacro:if value="${GAZEBO_BIGMAN_USES_7DOF_FOREARMS_DRC_14}">
    <gazebo reference="RForearmPlate">
     <cfmDamping>1</cfmDamping>
@@ -139,6 +138,4 @@
     <provideFeedback>true</provideFeedback>
    </gazebo>
-</xacro:if>
-<xacro:if value="${GAZEBO_BIGMAN_USES_7DOF_FOREARMS_DRC_14}">
     <xacro:unless value="${GAZEBO_BIGMAN_USES_SOFTHANDS_DRC_sw1_14}">
       <gazebo reference="r_handj">
@@ -147,5 +144,4 @@
       </gazebo>
     </xacro:unless>
-</xacro:if>
    <gazebo reference="LShSag">
     <cfmDamping>1</cfmDamping>
@@ -164,5 +160,4 @@
     <provideFeedback>true</provideFeedback>
    </gazebo>
-<xacro:if value="${GAZEBO_BIGMAN_USES_7DOF_FOREARMS_DRC_14}">
    <gazebo reference="LForearmPlate">
     <cfmDamping>1</cfmDamping>
@@ -177,6 +172,4 @@
     <provideFeedback>true</provideFeedback>
    </gazebo>
-</xacro:if>
-<xacro:if value="${GAZEBO_BIGMAN_USES_7DOF_FOREARMS_DRC_14}">
     <xacro:unless value="${GAZEBO_BIGMAN_USES_SOFTHANDS_DRC_sw1_14}">
       <gazebo reference="l_handj">
@@ -185,4 +178,3 @@
       </gazebo>
     </xacro:unless>
-</xacro:if>
 </robot>

File: bigman_urdf/urdf/gazebo/yarp_control.gazebo.xacro (robot description, xacro)
@@ -35,5 +35,4 @@
 </plugin>
 <!-- ARMS -->
-<xacro:if value="${GAZEBO_BIGMAN_USES_7DOF_FOREARMS_DRC_14}">
 	<plugin name="bigman_yarp_gazebo_plugin_left_arm" filename="libgazebo_yarp_controlboard.so">
 		<yarpConfigurationFile>model://bigman_urdf/conf/bigman/bigman_gazebo_left_arm.ini</yarpConfigurationFile>
@@ -67,5 +66,4 @@
 		</plugin>
 	</xacro:unless>
-</xacro:if>
 <!-- Plugin to apply external wrenches to the robot -->
 <plugin name="bigman_yarp_gazebo_plugin_external_wrench" filename="libgazebo_yarp_externalwrench.so"/>

Commit message: Added multisense head in simulation. Only kinematics and dynamics, not yet camera and laser simulation

File: bigman_urdf/urdf/bigman.urdf.xacro (robot description, xacro)
@@ -35,3 +35,10 @@
 <!-- IMU -->
 <xacro:include filename="$(find bigman_urdf)/urdf/sensors/imu.urdf.xacro"/>
+<!-- multisense_sl_v4 -->
+<xacro:include filename="$(find bigman_urdf)/urdf/sensors/multisense_sl.urdf.xacro"/>
+<joint name="neck_joint" type="fixed">
+    <parent link="DWYTorso"/>
+    <child link="head"/>
+    <origin xyz="0.05 0 0.3" rpy="0 0 0" />
+</joint>
 </robot>

Commit message: Added chest link, moved DWYtorso joint ant torso. Still missing Inertia, Mass and CoM.

File: bigman_urdf/urdf/bigman.urdf.xacro (robot description, xacro)
@@ -40,5 +40,5 @@
     <parent link="DWYTorso"/>
     <child link="head"/>
-    <origin xyz="0.05 0 0.3" rpy="0 0 0" />
+    <origin xyz="0.05 0 0.05" rpy="0 0 0" />
 </joint>
 </robot>

File: bigman_urdf/urdf/parts/arms.urdf.xacro (robot description, xacro)
@@ -163,5 +163,5 @@
     <parent link="DWYTorso"/>
     <child link="RShp"/>
-    <origin xyz="-0.014976503999999998 -0.0825 0.15770847" rpy="0 0 0" />
+    <origin xyz="0.0 -0.2 0.0" rpy="0 0 0" />
     <axis xyz="0 1 0" />
     <limit velocity="4.0" effort="50" lower="-3.4034" upper="1.6581" />
@@ -196,5 +196,5 @@
     <parent link="DWYTorso"/>
     <child link="LShp"/>
-    <origin xyz="-0.014976503999999998 0.0825 0.15770847" rpy="0 0 0" />
+    <origin xyz="0.0 0.2 0.0" rpy="0 0 0" />
     <axis xyz="0 1 0" />
     <limit velocity="4.0" effort="50" lower="-3.4034" upper="1.6581" />

File: bigman_urdf/urdf/parts/torso.urdf.xacro (robot description, xacro)
@@ -78,13 +78,13 @@
     </inertial>
     <visual>
-      <origin xyz="-0.020281504 0.0 -0.68662053" rpy="0 0 ${PI}"/>
+      <origin xyz="0.0 0.0 0.0" rpy="0 0 0"/>
       <geometry name="DWYTorso_visual">
-        <mesh filename="package://bigman_urdf/meshes/collada/asm0001_collada_10_prt.dae" scale="${SF} ${SF} ${SF}" />
+        <mesh filename="package://bigman_urdf/meshes/Chest.STL" scale="0.001 0.001 0.001" />
       </geometry>
     </visual>
     <collision>
-      <origin xyz="-0.020281504 0.0 -0.68662053" rpy="0 0 ${PI}"/>
+      <origin xyz="0.0 0.0 0.0" rpy="0 0 0"/>
       <geometry name="DWYTorso_collision">
-        <mesh filename="package://bigman_urdf/meshes/collada/simple/simple_asm0001_collada_10_prt.stl" scale="${SF} ${SF} ${SF}" />
+        <mesh filename="package://bigman_urdf/meshes/simple/Chest.STL" scale="0.001 0.001 0.001" />
       </geometry>
     </collision>
@@ -99,5 +99,5 @@
     <parent link="DWYTorso"/>
     <child link="torso"/>
-    <origin xyz="-0.014976503999999998 0 0.15770847" rpy="0 0 0" />
+    <origin xyz="0.0 0 0.0" rpy="0 0 0" />
 </joint>
 <joint name="WaistLat" type="revolute">
@@ -121,5 +121,5 @@
     <parent link="DWS"/>
     <child link="DWYTorso"/>
-    <origin xyz="0 0 0.04749999" rpy="0 0 0" />
+    <origin xyz="0 0 0.22222" rpy="0 0 0" />
     <axis xyz="0 0 1" />
     <limit velocity="4.0" effort="50" lower="-1.3963" upper="1.3962" />

Commit message: Added new model bigman_gazebo

File: bigman_urdf/urdf/bigman.urdf.xacro (robot description, xacro)
@@ -20,5 +20,5 @@
 	<origin xyz="0 0 0.1" rpy="0 0 0" />
 </joint>
-<!-- ************ COMAN BASE ************** -->
+<!-- ************ BIGMAN BASE ************** -->
 <xacro:include filename="$(find bigman_urdf)/urdf/bigman_base.urdf.xacro"/>
 <!-- ************ FOREARMS ************ -->
@@ -35,5 +35,5 @@
 <!-- IMU -->
 <xacro:include filename="$(find bigman_urdf)/urdf/sensors/imu.urdf.xacro"/>
-<!-- multisense_sl_v4 -->
+<!-- multisense_sl_v4 with fixed joints (NOT FOR SIMULATION) -->
 <xacro:include filename="$(find bigman_urdf)/urdf/sensors/multisense_sl.urdf.xacro"/>
 <joint name="neck_joint" type="fixed">

File: bigman_urdf/urdf/config/bigman.urdf.xacro (robot description, xacro)
@@ -1,35 +1,13 @@
 <?xml version="1.0"?>
 <robot xmlns:xacro="http://ros.org/wiki/xacro" name="BIGMAN">
-<xacro:property name="model_name" value="IIT Bigman" />
+<xacro:property name="model_name" value="IIT Bigman Ctrl" />
 <xacro:property name="model_version" value="0.1" />
 <!--
 ####################################################
 ##
-##  FOREARMS & HANDS SELECTION
+##  HAND SELECTION
 ##
 ####################################################
 -->
-<!-- 7DOFS_FOREARMS + SOFT_HANDS -->
-<xacro:property name="GAZEBO_BIGMAN_USES_SOFTHANDS_DRC_sw1_14" value="true" />
-<!--
-####################################################
-##
-##  F/T SELECTION
-##
-##
-## options:
-## 1) accurate (ft sensors located at exact spot)
-#	FT sensors are defined as children of
-#	underactuated joints, added specifically
-#	to create a frame for accurate reading,
-#	and to take into account the bias given
-#	by the sensor's inertia.
-## 2) non-accurate (ft sensors at the nearest joint)
-##
-####################################################
-#
-# 1/2 (true/false)
-#
--->
-<xacro:property name="GAZEBO_BIGMAN_USES_ACCURATE_FT" value="false" />
+<xacro:property name="BIGMAN_FIXED_HANDS" value="true" />
 </robot>

File: bigman_urdf/urdf/config/bigman_gazebo.urdf.xacro (robot description, xacro)
@@ -1,5 +1,5 @@
 <?xml version="1.0"?>
 <robot xmlns:xacro="http://ros.org/wiki/xacro" name="BIGMAN">
-<xacro:property name="model_name" value="IIT Bigman Ctrl" />
+<xacro:property name="model_name" value="IIT Bigman" />
 <xacro:property name="model_version" value="0.1" />
 <!--
@@ -10,4 +10,4 @@
 ####################################################
 -->
-<xacro:property name="BIGMAN_FIXED_HANDS" value="true" />
+<xacro:property name="BIGMAN_FIXED_HANDS" value="false" />
 </robot>

File: bigman_urdf/urdf/gazebo/bigman.gazebo.xacro (robot description, xacro)
@@ -138,5 +138,5 @@
     <provideFeedback>true</provideFeedback>
    </gazebo>
-    <xacro:unless value="${GAZEBO_BIGMAN_USES_SOFTHANDS_DRC_sw1_14}">
+    <xacro:unless value="${BIGMAN_FIXED_HANDS}">
       <gazebo reference="r_handj">
         <cfmDamping>1</cfmDamping>
@@ -172,5 +172,5 @@
     <provideFeedback>true</provideFeedback>
    </gazebo>
-    <xacro:unless value="${GAZEBO_BIGMAN_USES_SOFTHANDS_DRC_sw1_14}">
+    <xacro:unless value="${BIGMAN_FIXED_HANDS}">
       <gazebo reference="l_handj">
         <cfmDamping>1</cfmDamping>

File: bigman_urdf/urdf/gazebo/yarp_control.gazebo.xacro (robot description, xacro)
@@ -56,5 +56,5 @@
     </plugin>
 	<!-- HANDS -->
-	<xacro:unless value="${GAZEBO_BIGMAN_USES_SOFTHANDS_DRC_sw1_14}">
+	<xacro:unless value="${BIGMAN_FIXED_HANDS}">
 		<plugin name="bigman_yarp_gazebo_plugin_left_hand" filename="libgazebo_yarp_controlboard.so">
 			<yarpConfigurationFile>model://bigman_urdf/conf/bigman/bigman_gazebo_left_hand.ini</yarpConfigurationFile>

File: bigman_urdf/urdf/parts/soft_hand.urdf.xacro (robot description, xacro)
@@ -1,5 +1,5 @@
 <?xml version="1.0"?>
 <robot xmlns:xacro="http://ros.org/wiki/xacro" name="SoftHand">
-<xacro:if value="${GAZEBO_BIGMAN_USES_SOFTHANDS_DRC_sw1_14}">
+<xacro:if value="${BIGMAN_FIXED_HANDS}">
 <!-- LINKS -->
 <link name="RSoftHand">
@@ -53,5 +53,5 @@
   </joint>
 </xacro:if>
-<xacro:unless value="${GAZEBO_BIGMAN_USES_SOFTHANDS_DRC_sw1_14}">
+<xacro:unless value="${BIGMAN_FIXED_HANDS}">
 <!-- LINKS -->
 <!-- ## WRONG NUMBERS FOR... ok lasciamo perde... FIX THEM!! ## -->

File: bigman_urdf/urdf/sensors/multisense_sl.urdf.xacro (robot description, xacro)
@@ -71,4 +71,5 @@
   </gazebo>
 -->
+<!--
   <joint name="hokuyo_joint" type="continuous">
     <origin xyz="-0.0446 0 0.0880" rpy="0 0 0" />
@@ -77,4 +78,10 @@
     <axis xyz="1 0 0" />
     <dynamics damping="0.01" friction="0"/>
+  </joint>
+-->
+  <joint name="hokuyo_joint" type="fixed">
+    <origin xyz="-0.0446 0 0.0880" rpy="0 0 0" />
+    <parent link="head" />
+    <child link="hokuyo_link" />
   </joint>
 <!-- Remove frome here!

Commit message: Corrected bug in position of the ft sensors in the legs. Corrected bug in generation of the robot. Added ref frames in legs for ft sensors.

File: bigman_urdf/urdf/bigman.urdf.xacro (robot description, xacro)
@@ -22,4 +22,17 @@
 <!-- ************ BIGMAN BASE ************** -->
 <xacro:include filename="$(find bigman_urdf)/urdf/bigman_base.urdf.xacro"/>
+<!-- ***** LEGS F/T SENSOR REF FRAMES *******-->
+<link name="l_leg_ft"/>
+<link name="r_leg_ft"/>
+<joint name="l_leg_ft_joint" type="fixed">
+    <parent link="LFootmot"/>
+    <child link="l_leg_ft"/>
+    <origin xyz="0.005 0 -0.107" rpy="0 0 0" />
+</joint>
+<joint name="r_leg_ft_joint" type="fixed">
+    <parent link="RFootmot"/>
+    <child link="r_leg_ft"/>
+    <origin xyz="0.005 0 -0.107" rpy="0 0 0" />
+</joint>
 <!-- ************ FOREARMS ************ -->
 <!-- This links are defined in order to be compliant with http://www.ros.org/reps/rep-0120.html#coordinate-frames

File: bigman_urdf/urdf/gazebo/force_torque.gazebo.xacro (robot description, xacro)
@@ -29,5 +29,5 @@
 			<visualize>true</visualize>
 			<update_rate>1000</update_rate>
-			<pose>0.05 0 -0.107 0 0 0</pose>
+			<pose>0.005 0 -0.107 0 0 0</pose>
 			<plugin name="LAnkSag_FT_plugin" filename="libgazebo_yarp_forcetorque.so">
 				<yarpConfigurationFile>model://bigman_urdf/conf/bigman/bigman_gazebo_left_leg_ft.ini</yarpConfigurationFile>
@@ -41,5 +41,5 @@
 			<visualize>true</visualize>
 			<update_rate>1000</update_rate>
-			<pose>0.05 0 -0.107 0 0 0</pose>
+			<pose>0.005 0 -0.107 0 0 0</pose>
 			<plugin name="RAnkSag_FT_plugin" filename="libgazebo_yarp_forcetorque.so">
 				<yarpConfigurationFile>model://bigman_urdf/conf/bigman/bigman_gazebo_right_leg_ft.ini</yarpConfigurationFile>

File: bigman_urdf/urdf/sensors/multisense_sl.urdf.xacro (robot description, xacro)
@@ -71,5 +71,5 @@
   </gazebo>
 -->
-<xacro:if value="${BIGMAN_FIXED_MULTISENSE}">
+<xacro:unless value="${BIGMAN_FIXED_MULTISENSE}">
   <joint name="hokuyo_joint" type="continuous">
     <origin xyz="-0.0446 0 0.0880" rpy="0 0 0" />
@@ -79,6 +79,6 @@
     <dynamics damping="0.01" friction="0"/>
   </joint>
-</xacro:if>
-<xacro:unless value="${BIGMAN_FIXED_MULTISENSE}">
+</xacro:unless>
+<xacro:if value="${BIGMAN_FIXED_MULTISENSE}">
   <joint name="hokuyo_joint" type="fixed">
     <origin xyz="-0.0446 0 0.0880" rpy="0 0 0" />
@@ -86,5 +86,5 @@
     <child link="hokuyo_link" />
   </joint>
-</xacro:unless>
+</xacro:if>
 <!-- Remove frome here!
   <gazebo reference="hokuyo_joint">

Commit message: Added simplified contact for feet using a box, not a mesh convex hull.

File: bigman_urdf/urdf/bigman.urdf.xacro (robot description, xacro)
@@ -28,10 +28,10 @@
     <parent link="LFootmot"/>
     <child link="l_leg_ft"/>
-    <origin xyz="0.005 0 -0.107" rpy="0 0 0" />
+    <origin xyz="0.005 0 -0.107" rpy="0 0 0"/>
 </joint>
 <joint name="r_leg_ft_joint" type="fixed">
     <parent link="RFootmot"/>
     <child link="r_leg_ft"/>
-    <origin xyz="0.005 0 -0.107" rpy="0 0 0" />
+    <origin xyz="0.005 0 -0.107" rpy="0 0 0"/>
 </joint>
 <link name="l_arm_ft"/>

Commit message: Fixed bug in sensor ref frame

File: bigman_urdf/urdf/bigman.urdf.xacro (robot description, xacro)
@@ -26,10 +26,10 @@
 <link name="r_leg_ft"/>
 <joint name="l_leg_ft_joint" type="fixed">
-    <parent link="LFootmot"/>
+    <parent link="LFoot"/>
     <child link="l_leg_ft"/>
     <origin xyz="0.005 0 -0.107" rpy="0 0 0"/>
 </joint>
 <joint name="r_leg_ft_joint" type="fixed">
-    <parent link="RFootmot"/>
+    <parent link="RFoot"/>
     <child link="r_leg_ft"/>
     <origin xyz="0.005 0 -0.107" rpy="0 0 0"/>
