Commit message: CHanged BIGMAN_ONLY_LEGS variable in BIGMAN_LEGS. Added BIGMAN_UPPER_BODY variable. Added files to generate and use only upper body. Need to be finished!

File: bigman_urdf/urdf/bigman.urdf.xacro (robot description, xacro)
@@ -10,5 +10,5 @@
 <!-- ************ MODEL CONFIGURATION ************ -->
 <xacro:include filename="$(find bigman_urdf)/urdf/bigman_config.urdf.xacro" />
-<xacro:unless value="${BIGMAN_ONLY_LEGS}">
+<xacro:if value="${BIGMAN_UPPER_BODY}">
 <!-- Head -->
 <!-- This links are defined in order to be compliant with http://www.ros.org/reps/rep-0120.html#coordinate-frames
@@ -21,51 +21,53 @@
 	<origin xyz="0 0 0.1" rpy="0 0 0" />
 </joint>
-</xacro:unless>
+</xacro:if>
 <!-- ************ BIGMAN BASE ************** -->
 <xacro:include filename="$(find bigman_urdf)/urdf/bigman_base.urdf.xacro"/>
-<!-- ***** LEGS F/T SENSOR REF FRAMES *******-->
-<link name="l_leg_ft"/>
-<link name="r_leg_ft"/>
-<joint name="l_leg_ft_joint" type="fixed">
-    <parent link="LFoot"/>
-    <child link="l_leg_ft"/>
-    <origin xyz="0.005 0 -0.107" rpy="0 0 0"/>
-</joint>
-<joint name="r_leg_ft_joint" type="fixed">
-    <parent link="RFoot"/>
-    <child link="r_leg_ft"/>
-    <origin xyz="0.005 0 -0.107" rpy="0 0 0"/>
-</joint>
-<xacro:unless value="${BIGMAN_ONLY_LEGS}">
-<link name="l_arm_ft"/>
-<link name="r_arm_ft"/>
-<joint name="l_arm_ft_joint" type="fixed">
-    <parent link="LWrMot3"/>
-    <child link="l_arm_ft"/>
-    <origin xyz="0 0 -0.0565" rpy="0 0 0" />
-</joint>
-<joint name="r_arm_ft_joint" type="fixed">
-    <parent link="RWrMot3"/>
-    <child link="r_arm_ft"/>
-    <origin xyz="0 0 -0.0565" rpy="0 0 0" />
-</joint>
-<!-- ************ FOREARMS ************ -->
-<!-- This links are defined in order to be compliant with http://www.ros.org/reps/rep-0120.html#coordinate-frames
-and to define the end effectors of the robot -->
-<!-- position and orientation of the arm regardless of the tool (grasping device for instance) attached to it -->
-<link name="l_wrist"/>
-<link name="r_wrist"/>
-<xacro:include filename="$(find bigman_urdf)/urdf/parts/forearms.urdf.xacro" />
-<xacro:include filename="$(find bigman_urdf)/urdf/parts/forearm_reference_frame.urdf.xacro" />
-<!-- ************ HANDS ************ -->
-<xacro:include filename="$(find bigman_urdf)/urdf/parts/soft_hand.urdf.xacro" />
-<!-- multisense_sl_v4 with fixed joints (NOT FOR SIMULATION) -->
-<xacro:include filename="$(find bigman_urdf)/urdf/sensors/multisense_sl.urdf.xacro"/>
-<joint name="neck_joint" type="fixed">
-    <parent link="DWYTorso"/>
-    <child link="head"/>
-    <origin xyz="0.05 0 0.05" rpy="0 0 0" />
-</joint>
-</xacro:unless>
+<xacro:if value="${BIGMAN_LEGS}">
+	<!-- ***** LEGS F/T SENSOR REF FRAMES *******-->
+	<link name="l_leg_ft"/>
+	<link name="r_leg_ft"/>
+	<joint name="l_leg_ft_joint" type="fixed">
+	    <parent link="LFoot"/>
+	    <child link="l_leg_ft"/>
+	    <origin xyz="0.005 0 -0.107" rpy="0 0 0"/>
+	</joint>
+	<joint name="r_leg_ft_joint" type="fixed">
+	    <parent link="RFoot"/>
+	    <child link="r_leg_ft"/>
+	    <origin xyz="0.005 0 -0.107" rpy="0 0 0"/>
+	</joint>
+</xacro:if>
+<xacro:if value="${BIGMAN_UPPER_BODY}">
+	<link name="l_arm_ft"/>
+	<link name="r_arm_ft"/>
+	<joint name="l_arm_ft_joint" type="fixed">
+	    <parent link="LWrMot3"/>
+	    <child link="l_arm_ft"/>
+	    <origin xyz="0 0 -0.0565" rpy="0 0 0" />
+	</joint>
+	<joint name="r_arm_ft_joint" type="fixed">
+	    <parent link="RWrMot3"/>
+	    <child link="r_arm_ft"/>
+	    <origin xyz="0 0 -0.0565" rpy="0 0 0" />
+	</joint>
+	<!-- ************ FOREARMS ************ -->
+	<!-- This links are defined in order to be compliant with http://www.ros.org/reps/rep-0120.html#coordinate-frames
+	and to define the end effectors of the robot -->
+	<!-- position and orientation of the arm regardless of the tool (grasping device for instance) attached to it -->
+	<link name="l_wrist"/>
+	<link name="r_wrist"/>
+	<xacro:include filename="$(find bigman_urdf)/urdf/parts/forearms.urdf.xacro" />
+	<xacro:include filename="$(find bigman_urdf)/urdf/parts/forearm_reference_frame.urdf.xacro" />
+	<!-- ************ HANDS ************ -->
+	<xacro:include filename="$(find bigman_urdf)/urdf/parts/soft_hand.urdf.xacro" />
+	<!-- multisense_sl_v4 with fixed joints (NOT FOR SIMULATION) -->
+	<xacro:include filename="$(find bigman_urdf)/urdf/sensors/multisense_sl.urdf.xacro"/>
+	<joint name="neck_joint" type="fixed">
+	    <parent link="DWYTorso"/>
+	    <child link="head"/>
+	    <origin xyz="0.05 0 0.05" rpy="0 0 0" />
+	</joint>
+</xacro:if>
 <!-- IMU -->
 <xacro:include filename="$(find bigman_urdf)/urdf/sensors/imu.urdf.xacro"/>

File: bigman_urdf/urdf/bigman_base.urdf.xacro (robot description, xacro)
@@ -35,61 +35,65 @@
     <origin xyz="0 0 0" rpy="0 0 0" />
 </joint>
-<xacro:if value="${BIGMAN_ONLY_LEGS}">
-       <!-- ********************FAKE TORSO******************** -->
-       <xacro:include filename="$(find bigman_urdf)/urdf/parts/pelvis_weight_bench.urdf.xacro" />
+<xacro:if value="${BIGMAN_LEGS}">
+       <xacro:unless value="${BIGMAN_UPPER_BODY}">
+		<!-- ********************FAKE TORSO******************** -->
+		<xacro:include filename="$(find bigman_urdf)/urdf/parts/pelvis_weight_bench.urdf.xacro" />
+       </xacro:unless>
 </xacro:if>
-<xacro:unless value="${BIGMAN_ONLY_LEGS}">
+<xacro:if value="${BIGMAN_UPPER_BODY}">
        <!-- ********************TORSO******************** -->
        <!-- first real link of the robot, inertial reference frame -->
        <xacro:include filename="$(find bigman_urdf)/urdf/parts/torso.urdf.xacro" />
-</xacro:unless>
-<!-- ********************LEGS******************** -->
-<!-- This links are defined in order to be compliant with http://www.ros.org/reps/rep-0120.html#coordinate-frames
-and to define the end effectors of the robot -->
-<!--  position and orientation of the leg regardless of the support body geometry -->
-  <link name="l_ankle"/>
-  <link name="r_ankle"/>
-<!-- position and orientation of the left leg support body. The (X,Y) plane of this frame must be coplanar with the support body contact surface. It is recommended to choose the origin as the projection of the support body origin on the contact surface. The Z coordinate of this frame should be on the ground level when standing. -->
-  <link name="l_sole"/>
-  <link name="r_sole"/>
-<!--  position and orientation of the leg toe body. The (X,Y) plan of this frame must be coplanar with the toe body contact surface. It is recommended to choose the origin as the projection of the body center on the contact surface. -->
-  <link name="l_toe"/>
-  <link name="r_toe"/>
-<xacro:include filename="$(find bigman_urdf)/urdf/parts/legs.urdf.xacro" />
-  <joint name="l_ankle_joint" type="fixed">
-     <parent link="LFoot"/>
-     <child link="l_ankle"/>
-     <origin xyz="0 0 0" rpy="0 0 0" />
-  </joint>
-  <joint name="r_ankle_joint" type="fixed">
-    <parent link="RFoot"/>
-    <child link="r_ankle"/>
-    <origin xyz="0 0 0" rpy="0 0 0" />
-  </joint>
-  <joint name="l_sole_joint" type="fixed">
-    <parent link="LFoot"/>
-    <child link="l_sole"/>
-    <origin xyz="0 0 -0.1435" rpy="0 0 0" />
-  </joint>
-  <joint name="r_sole_joint" type="fixed">
-    <parent link="RFoot"/>
-    <child link="r_sole"/>
-    <origin xyz="0 0 -0.1435" rpy="0 0 0" />
-  </joint>
-  <joint name="l_toe_joint" type="fixed">
-    <parent link="l_sole"/>
-    <child link="l_toe"/>
-    <origin xyz="0.195 0 0" rpy="0 0 0" />
-  </joint>
-  <joint name="r_toe_joint" type="fixed">
-    <parent link="r_sole"/>
-    <child link="r_toe"/>
-    <origin xyz="0.195 0 0" rpy="0 0 0" />
-  </joint>
-<!-- Reference frames in feet -->
-<xacro:include filename="$(find bigman_urdf)/urdf/parts/foot_reference_frame.urdf.xacro" />
-<xacro:unless value="${BIGMAN_ONLY_LEGS}">
+</xacro:if>
+<xacro:if value="${BIGMAN_LEGS}">
+	<!-- ********************LEGS******************** -->
+	<!-- This links are defined in order to be compliant with http://www.ros.org/reps/rep-0120.html#coordinate-frames
+	and to define the end effectors of the robot -->
+	<!--  position and orientation of the leg regardless of the support body geometry -->
+	  <link name="l_ankle"/>
+	  <link name="r_ankle"/>
+	<!-- position and orientation of the left leg support body. The (X,Y) plane of this frame must be coplanar with the support body contact surface. It is recommended to choose the origin as the projection of the support body origin on the contact surface. The Z coordinate of this frame should be on the ground level when standing. -->
+	  <link name="l_sole"/>
+	  <link name="r_sole"/>
+	<!--  position and orientation of the leg toe body. The (X,Y) plan of this frame must be coplanar with the toe body contact surface. It is recommended to choose the origin as the projection of the body center on the contact surface. -->
+	  <link name="l_toe"/>
+	  <link name="r_toe"/>
+	<xacro:include filename="$(find bigman_urdf)/urdf/parts/legs.urdf.xacro" />
+  	<joint name="l_ankle_joint" type="fixed">
+	     <parent link="LFoot"/>
+	     <child link="l_ankle"/>
+	     <origin xyz="0 0 0" rpy="0 0 0" />
+        </joint>
+	  <joint name="r_ankle_joint" type="fixed">
+	    <parent link="RFoot"/>
+	    <child link="r_ankle"/>
+	    <origin xyz="0 0 0" rpy="0 0 0" />
+	  </joint>
+	  <joint name="l_sole_joint" type="fixed">
+	    <parent link="LFoot"/>
+	    <child link="l_sole"/>
+	    <origin xyz="0 0 -0.1435" rpy="0 0 0" />
+	  </joint>
+	  <joint name="r_sole_joint" type="fixed">
+	    <parent link="RFoot"/>
+	    <child link="r_sole"/>
+	    <origin xyz="0 0 -0.1435" rpy="0 0 0" />
+	  </joint>
+	  <joint name="l_toe_joint" type="fixed">
+	    <parent link="l_sole"/>
+	    <child link="l_toe"/>
+	    <origin xyz="0.195 0 0" rpy="0 0 0" />
+	  </joint>
+	  <joint name="r_toe_joint" type="fixed">
+	    <parent link="r_sole"/>
+	    <child link="r_toe"/>
+	    <origin xyz="0.195 0 0" rpy="0 0 0" />
+	  </joint>
+	<!-- Reference frames in feet -->
+	<xacro:include filename="$(find bigman_urdf)/urdf/parts/foot_reference_frame.urdf.xacro" />
+</xacro:if>
+<xacro:if value="${BIGMAN_UPPER_BODY}">
        <!-- ********************ARMS******************** -->
        <xacro:include filename="$(find bigman_urdf)/urdf/parts/arms.urdf.xacro" />
-</xacro:unless>
+</xacro:if>
 </robot>

File: bigman_urdf/urdf/config/bigman.urdf.xacro (robot description, xacro)
@@ -6,14 +6,21 @@
 ####################################################
 ##
-##  BIGMAN_ONLY_LEGS
-##  if "true" only the kinematic chains of the legs
-##  will be used to generate the model, the flags
-##  regarding the upper body will not be taken in
-##  consideration.
-##
+##  BIGMAN_UPPER_BODY
+##  if "true" the kinematic chains of the arms and torso
+##  will be used to generate the model
 ##
 ####################################################
 -->
-<xacro:property name="BIGMAN_ONLY_LEGS" value="false" />
+<xacro:property name="BIGMAN_UPPER_BODY" value="true" />
+<!--
+####################################################
+##
+##  BIGMAN_LEGS
+##  if "true" the kinematic chains of the legs
+##  will be used to generate the model
+##
+####################################################
+-->
+<xacro:property name="BIGMAN_LEGS" value="true" />
 <!--
 ####################################################

File: bigman_urdf/urdf/config/bigman_gazebo.urdf.xacro (robot description, xacro)
@@ -6,14 +6,21 @@
 ####################################################
 ##
-##  BIGMAN_ONLY_LEGS
-##  if "true" only the kinematic chains of the legs
-##  will be used to generate the model, the flags
-##  regarding the upper body will not be taken in
-##  consideration.
-##
+##  BIGMAN_UPPER_BODY
+##  if "true" the kinematic chains of the arms and torso
+##  will be used to generate the model
 ##
 ####################################################
 -->
-<xacro:property name="BIGMAN_ONLY_LEGS" value="false" />
+<xacro:property name="BIGMAN_UPPER_BODY" value="true" />
+<!--
+####################################################
+##
+##  BIGMAN_LEGS
+##  if "true" the kinematic chains of the legs
+##  will be used to generate the model
+##
+####################################################
+-->
+<xacro:property name="BIGMAN_LEGS" value="true" />
 <!--
 ####################################################

File: bigman_urdf/urdf/config/bigman_only_legs.urdf.xacro (robot description, xacro)
@@ -6,14 +6,32 @@
 ####################################################
 ##
-##  BIGMAN_ONLY_LEGS
-##  if "true" only the kinematic chains of the legs
-##  will be used to generate the model, the flags
-##  regarding the upper body will not be taken in
-##  consideration.
+##  BIGMAN_UPPER_BODY
+##  if "true" the kinematic chains of the arms and torso
+##  will be used to generate the model
+##
+####################################################
+-->
+<xacro:property name="BIGMAN_UPPER_BODY" value="false" />
+<!--
+####################################################
+##
+##  BIGMAN_LEGS
+##  if "true" the kinematic chains of the legs
+##  will be used to generate the model
+##
+####################################################
+-->
+<xacro:property name="BIGMAN_LEGS" value="true" />
+<!--
+####################################################
+##
+##  BIGMAN_OLD_CHEST
+##  if "true" the old version of the chest will be
+##  used.
 ##
 ##
 ####################################################
 -->
-<xacro:property name="BIGMAN_ONLY_LEGS" value="true" />
+<xacro:property name="BIGMAN_OLD_CHEST" value="false" />
 <!--
 ####################################################

File: bigman_urdf/urdf/config/bigman_only_upper_body.urdf.xacro (robot description, xacro)
@@ -1,5 +1,5 @@
 <?xml version="1.0"?>
 <robot xmlns:xacro="http://ros.org/wiki/xacro" name="BIGMAN">
-<xacro:property name="model_name" value="IIT Bigman Ctrl" />
+<xacro:property name="model_name" value="IIT Bigman Upper Body" />
 <xacro:property name="model_version" value="0.1" />
 <!--
@@ -22,5 +22,5 @@
 ####################################################
 -->
-<xacro:property name="BIGMAN_LEGS" value="true" />
+<xacro:property name="BIGMAN_LEGS" value="false" />
 <!--
 ####################################################

File: bigman_urdf/urdf/gazebo/bigman.gazebo.xacro (robot description, xacro)
@@ -1,4 +1,5 @@
 <?xml version="1.0"?>
 <robot xmlns:xacro="http://ros.org/wiki/xacro">
+<xacro:if value="${BIGMAN_LEGS}">
 <!-- contact model for foot surface -->
    <gazebo reference="LFoot">
@@ -20,4 +21,6 @@
      <minDepth>0.0</minDepth>
    </gazebo>
+</xacro:if>
+<xacro:if value="${BIGMAN_UPPER_BODY}">
 <!-- contact model for hand surface -->
    <gazebo reference="LSoftHand">
@@ -39,4 +42,6 @@
      <minDepth>0.0</minDepth>
    </gazebo>
+</xacro:if>
+<xacro:if value="${BIGMAN_LEGS}">
 <!-- Other parameters... -->
    <gazebo reference="RHipSag">
@@ -88,5 +93,6 @@
     <provideFeedback>true</provideFeedback>
    </gazebo>
-<xacro:unless value="${BIGMAN_ONLY_LEGS}">
+</xacro:if>
+<xacro:if value="${BIGMAN_UPPER_BODY}">
    <gazebo reference="WaistSag">
     <implicitSpringDamper>1</implicitSpringDamper>
@@ -169,4 +175,4 @@
       </gazebo>
     </xacro:unless>
-</xacro:unless>
+</xacro:if>
 </robot>

File: bigman_urdf/urdf/gazebo/force_torque.gazebo.xacro (robot description, xacro)
@@ -7,5 +7,5 @@
 -->
 <robot xmlns:xacro="http:/ros.org/wiki/xacro">
-<xacro:unless value="${BIGMAN_ONLY_LEGS}">
+<xacro:if value="${BIGMAN_UPPER_BODY}">
 	<gazebo reference="RWrj2">
 		<sensor type="force_torque" name="right_arm">
@@ -38,5 +38,6 @@
 		</sensor>
 	</gazebo>
-</xacro:unless>
+</xacro:if>
+<xacro:if value="${BIGMAN_LEGS}">
 	<gazebo reference="LAnkLat">
 		<sensor type="force_torque" name="left_leg">
@@ -69,3 +70,4 @@
 		</sensor>
 	</gazebo>
+</xacro:if>
 </robot>

File: bigman_urdf/urdf/gazebo/yarp_control.gazebo.xacro (robot description, xacro)
@@ -2,5 +2,5 @@
 <robot xmlns:xacro="http://ros.org/wiki/xacro">
 <gazebo>
-<xacro:unless value="${BIGMAN_ONLY_LEGS}">
+<xacro:if value="${BIGMAN_UPPER_BODY}">
 <!-- TORSO -->
 <plugin name="bigman_yarp_gazebo_plugin_torso" filename="libgazebo_yarp_controlboard.so">
@@ -46,5 +46,6 @@
 		</plugin>
 	</xacro:unless>
-</xacro:unless>
+</xacro:if>
+<xacro:if value="${BIGMAN_LEGS}">
 <!-- LEGS -->
 <plugin name="bigman_yarp_gazebo_plugin_left_leg" filename="libgazebo_yarp_controlboard.so">
@@ -70,4 +71,5 @@
 <!-- Plugin to apply external wrenches to the robot -->
 <plugin name="bigman_yarp_gazebo_plugin_external_wrench" filename="libgazebo_yarp_externalwrench.so"/>
+</xacro:if>
 </gazebo>
 </robot>

Commit message: Started implementation of neck

File: bigman_urdf/urdf/bigman.urdf.xacro (robot description, xacro)
@@ -65,5 +65,5 @@
 	<xacro:include filename="$(find bigman_urdf)/urdf/sensors/multisense_sl.urdf.xacro"/>
 	<joint name="neck_joint" type="fixed">
-	    <parent link="DWYTorso"/>
+	    <parent link="NeckPitch"/>
 	    <child link="head"/>
 	    <origin xyz="0.05 0 0.05" rpy="0 0 0" />

File: bigman_urdf/urdf/bigman_base.urdf.xacro (robot description, xacro)
@@ -45,4 +45,6 @@
        <!-- first real link of the robot, inertial reference frame -->
        <xacro:include filename="$(find bigman_urdf)/urdf/parts/torso.urdf.xacro" />
+       <!-- ********************NECK********************* -->
+       <xacro:include filename="$(find bigman_urdf)/urdf/parts/neck.urdf.xacro" />
 </xacro:if>
 <xacro:if value="${BIGMAN_LEGS}">

Commit message: Moved gaze link/joint to bigman_base. Attached gaze to Neck Pitch

File: bigman_urdf/urdf/bigman.urdf.xacro (robot description, xacro)
@@ -10,16 +10,4 @@
 <!-- ************ MODEL CONFIGURATION ************ -->
 <xacro:include filename="$(find bigman_urdf)/urdf/bigman_config.urdf.xacro" />
-<xacro:if value="${BIGMAN_UPPER_BODY}">
-<!-- Head -->
-<!-- This links are defined in order to be compliant with http://www.ros.org/reps/rep-0120.html#coordinate-frames
-and to define the end effectors of the robot.
-The coordinate frame called gaze defines the head position and orientation. The orientation indicates in which direction the head appears to be looking regardless of any sensors (camera for instance). -->
-<link name="gaze"/>
-<joint name="gaze_joint" type="fixed">
-	<parent link="torso"/>
-	<child link="gaze"/>
-	<origin xyz="0 0 0.1" rpy="0 0 0" />
-</joint>
-</xacro:if>
 <!-- ************ BIGMAN BASE ************** -->
 <xacro:include filename="$(find bigman_urdf)/urdf/bigman_base.urdf.xacro"/>

File: bigman_urdf/urdf/bigman_base.urdf.xacro (robot description, xacro)
@@ -47,4 +47,10 @@
        <!-- ********************NECK********************* -->
        <xacro:include filename="$(find bigman_urdf)/urdf/parts/neck.urdf.xacro" />
+       <link name="gaze"/>
+       <joint name="gaze_joint" type="fixed">
+              <parent link="NeckPitch"/>
+              <child link="gaze"/>
+              <origin xyz="0 0 0" rpy="0 0 0" />
+       </joint>
 </xacro:if>
 <xacro:if value="${BIGMAN_LEGS}">

Commit message: Added proper transformation of neck joint.

File: bigman_urdf/urdf/bigman.urdf.xacro (robot description, xacro)
@@ -55,5 +55,5 @@
 	    <parent link="NeckPitch"/>
 	    <child link="head"/>
-	    <origin xyz="0.05 0 0.05" rpy="0 0 0" />
+	    <origin xyz="0.08765 0 0.06475" rpy="0 0 0" />
 	</joint>
 </xacro:if>

File: bigman_urdf/urdf/sensors/multisense_sl.urdf.xacro (robot description, xacro)
@@ -93,12 +93,5 @@
     <child link="head_hokuyo_frame"/>
   </joint>
-  <link name="head_hokuyo_frame">
-    <inertial>
-      <mass value="1e-5" />
-      <!-- collocate with parent link and remove mass from it -->
-      <origin xyz="0.042428 0.0004084 0.0108165" rpy="0 0 0"/>
-      <inertia ixx="1e-6" ixy="0" ixz="0" iyy="1e-6" iyz="0" izz="1e-6" />
-    </inertial>
-  </link>
+  <link name="head_hokuyo_frame"/>
 <!-- Remove frome here!
   <gazebo reference="head_hokuyo_frame">
@@ -251,5 +244,5 @@
   <link name="center_bottom_led_frame"/>
   <joint name="left_led_frame_joint" type="fixed">
-    <origin xyz="-0.01443 0.07452 0.050346" rpy="0 -0.15 0.53"/>
+    <origin xyz="-0.01443 0.07452 0.050346" rpy="0 0 0.6"/>
     <parent link="head"/>
     <child link="left_led_frame"/>
@@ -257,5 +250,6 @@
   <link name="left_led_frame"/>
   <joint name="right_led_frame_joint" type="fixed">
-    <origin xyz="-0.01443 -0.07452 0.050346" rpy="0 -0.15 -0.53"/>
+    <!--origin xyz="-0.01443 -0.07452 0.050346" rpy="0 -0.15 -0.53"/-->
+    <origin xyz="-0.01443 -0.07452 0.050346" rpy="0 0 -0.6"/>
     <parent link="head"/>
     <child link="right_led_frame"/>

Commit message: Added  colors to neck. Moved gaze frame inside head.

File: bigman_urdf/urdf/bigman.urdf.xacro (robot description, xacro)
@@ -59,4 +59,10 @@
 	    <origin xyz="0.08765 0 0.06475" rpy="0 0 0" />
 	</joint>
+       <link name="gaze"/>
+       <joint name="gaze_joint" type="fixed">
+              <parent link="head"/>
+              <child link="gaze"/>
+              <origin xyz="0 0 0" rpy="0 0 0" />
+       </joint>
 </xacro:if>
 <xacro:if value="${BIGMAN_LEGS}">

File: bigman_urdf/urdf/bigman_base.urdf.xacro (robot description, xacro)
@@ -48,10 +48,4 @@
        <!-- ********************NECK********************* -->
        <xacro:include filename="$(find bigman_urdf)/urdf/parts/neck.urdf.xacro" />
-       <link name="gaze"/>
-       <joint name="gaze_joint" type="fixed">
-              <parent link="NeckPitch"/>
-              <child link="gaze"/>
-              <origin xyz="0 0 0" rpy="0 0 0" />
-       </joint>
 </xacro:if>
 <xacro:if value="${BIGMAN_LEGS}">

File: bigman_urdf/urdf/parts/neck.urdf.xacro (robot description, xacro)
@@ -21,4 +21,5 @@
         <mesh filename="package://bigman_urdf/meshes/NeckYaw.STL" scale="0.001 0.001 0.001" />
       </geometry>
+      <material name="grey"/>
     </visual>
     <collision>
@@ -40,4 +41,5 @@
         <mesh filename="package://bigman_urdf/meshes/NeckPitch.STL" scale="0.001 0.001 0.001" />
       </geometry>
+      <material name="grey"/>
     </visual>
     <collision>
