Commit message: Added multisense_namespace parameter to add multisense/ to all the frame related to multisense

File: bigman_urdf/urdf/bigman.urdf.xacro (robot description, xacro)
@@ -56,10 +56,10 @@
 	<joint name="neck_joint" type="fixed">
 	    <parent link="NeckPitch"/>
-	    <child link="head"/>
+	    <child link="${multisense_namespace}/head"/>
 	    <origin xyz="0.08765 0 0.06475" rpy="0 0 0" />
 	</joint>
        <link name="gaze"/>
        <joint name="gaze_joint" type="fixed">
-              <parent link="head"/>
+              <parent link="${multisense_namespace}/head"/>
               <child link="gaze"/>
               <origin xyz="0 0 0" rpy="0 0 0" />

File: bigman_urdf/urdf/sensors/multisense_sl.urdf.xacro (robot description, xacro)
@@ -1,9 +1,10 @@
 <?xml version="1.0"?>
 <robot xmlns:xacro="http://ros.org/wiki/xacro" name="multisense_sl">
+<xacro:property name="multisense_namespace" value="multisense" />
 <!--
        Based on multisense_sl_v4.urdf in multisense_sl_description (DRCSIM)
 -->
   <!-- Head Link Simple Collision Meshes -->
-  <link name="head">
+  <link name="${multisense_namespace}/head">
     <inertial>
       <origin xyz="-0.075493 3.3383E-05 0.02774" rpy="0 0 0" />
@@ -25,5 +26,5 @@
   </collision>
   </link>
-  <link name="hokuyo_link">
+  <link name="${multisense_namespace}/hokuyo_link">
     <inertial>
       <origin xyz="0.032428 0.0004084 -0.0041835" rpy="0 0 0" />
@@ -64,6 +65,6 @@
   <joint name="hokuyo_joint" type="continuous">
     <origin xyz="-0.0446 0 0.0880" rpy="0 0 0" />
-    <parent link="head" />
-    <child link="hokuyo_link" />
+    <parent link="${multisense_namespace}/head" />
+    <child link="${multisense_namespace}/hokuyo_link" />
     <axis xyz="1 0 0" />
     <dynamics damping="0.01" friction="0"/>
@@ -73,6 +74,6 @@
   <joint name="hokuyo_joint" type="fixed">
     <origin xyz="-0.0446 0 0.0880" rpy="0 0 0" />
-    <parent link="head" />
-    <child link="hokuyo_link" />
+    <parent link="${multisense_namespace}/head" />
+    <child link="${multisense_namespace}/hokuyo_link" />
   </joint>
 </xacro:if>
@@ -86,8 +87,8 @@
     <axis xyz="0 1 0" />
     <origin xyz="0.03 0 0.015" rpy="0 0 0"/>
-    <parent link="hokuyo_link"/>
-    <child link="head_hokuyo_frame"/>
-  </joint>
-  <link name="head_hokuyo_frame"/>
+    <parent link="${multisense_namespace}/hokuyo_link"/>
+    <child link="${multisense_namespace}/head_hokuyo_frame"/>
+  </joint>
+  <link name="${multisense_namespace}/head_hokuyo_frame"/>
 <!-- Remove frome here!
   <gazebo reference="head_hokuyo_frame">
@@ -131,14 +132,14 @@
     <!-- optical frame collocated with tilting DOF -->
     <origin xyz="0.0 0.035 -0.002"/>
-    <parent link="head"/>
-    <child link="left_camera_frame"/>
-  </joint>
-  <link name="left_camera_frame"/>
+    <parent link="${multisense_namespace}/head"/>
+    <child link="${multisense_namespace}/left_camera_frame"/>
+  </joint>
+  <link name="${multisense_namespace}/left_camera_frame"/>
   <joint name="left_camera_optical_frame_joint" type="fixed">
     <origin xyz="0 0 0" rpy="-1.5708 0.0 -1.5708" />
-    <parent link="left_camera_frame" />
-    <child link="left_camera_optical_frame"/>
-  </joint>
-  <link name="left_camera_optical_frame"/>
+    <parent link="${multisense_namespace}/left_camera_frame" />
+    <child link="${multisense_namespace}/left_camera_optical_frame"/>
+  </joint>
+  <link name="${multisense_namespace}/left_camera_optical_frame"/>
 <!--
   <gazebo reference="left_camera_frame">
@@ -217,38 +218,38 @@
   <joint name="right_camera_frame_joint" type="fixed">
     <origin xyz="0.0 -0.035 -0.002"/>
-    <parent link="head"/>
-    <child link="right_camera_frame"/>
-  </joint>
-  <link name="right_camera_frame"/>
+    <parent link="${multisense_namespace}/head"/>
+    <child link="${multisense_namespace}/right_camera_frame"/>
+  </joint>
+  <link name="${multisense_namespace}/right_camera_frame"/>
   <joint name="right_camera_optical_frame_joint" type="fixed">
     <origin xyz="0 0 0" rpy="-1.5708 0.0 -1.5708" />
-    <parent link="right_camera_frame" />
-    <child link="right_camera_optical_frame"/>
-  </joint>
-  <link name="right_camera_optical_frame"/>
+    <parent link="${multisense_namespace}/right_camera_frame" />
+    <child link="${multisense_namespace}/right_camera_optical_frame"/>
+  </joint>
+  <link name="${multisense_namespace}/right_camera_optical_frame"/>
   <joint name="center_top_led_frame_joint" type="fixed">
     <origin xyz="0.01125 0.0 0.0105"/>
-    <parent link="head"/>
-    <child link="center_top_led_frame"/>
-  </joint>
-  <link name="center_top_led_frame"/>
+    <parent link="${multisense_namespace}/head"/>
+    <child link="${multisense_namespace}/center_top_led_frame"/>
+  </joint>
+  <link name="${multisense_namespace}/center_top_led_frame"/>
   <joint name="center_bottom_led_frame_joint" type="fixed">
     <origin xyz="0.01125 0.0 -0.0155"/>
-    <parent link="head"/>
-    <child link="center_bottom_led_frame"/>
-  </joint>
-  <link name="center_bottom_led_frame"/>
+    <parent link="${multisense_namespace}/head"/>
+    <child link="${multisense_namespace}/center_bottom_led_frame"/>
+  </joint>
+  <link name="${multisense_namespace}/center_bottom_led_frame"/>
   <joint name="left_led_frame_joint" type="fixed">
     <origin xyz="-0.01443 0.07452 0.050346" rpy="0 0 0.6"/>
-    <parent link="head"/>
-    <child link="left_led_frame"/>
-  </joint>
-  <link name="left_led_frame"/>
+    <parent link="${multisense_namespace}/head"/>
+    <child link="${multisense_namespace}/left_led_frame"/>
+  </joint>
+  <link name="${multisense_namespace}/left_led_frame"/>
   <joint name="right_led_frame_joint" type="fixed">
     <origin xyz="-0.01443 -0.07452 0.050346" rpy="0 0 -0.6"/>
-    <parent link="head"/>
-    <child link="right_led_frame"/>
-  </joint>
-  <link name="right_led_frame"/>
+    <parent link="${multisense_namespace}/head"/>
+    <child link="${multisense_namespace}/right_led_frame"/>
+  </joint>
+  <link name="${multisense_namespace}/right_led_frame"/>
 <!--
   <gazebo>
@@ -257,5 +258,5 @@
 -->
   <!-- imu link -->
-  <link name="head_imu_link">
+  <link name="${multisense_namespace}/head_imu_link">
     <inertial>
       <mass value="1e-5" />
@@ -272,6 +273,6 @@
   </link>
   <joint name="head_imu_joint" type="fixed">
-    <parent link="head"/>
-    <child link="head_imu_link"/>
+    <parent link="${multisense_namespace}/head"/>
+    <child link="${multisense_namespace}/head_imu_link"/>
     <!-- putting it at the same z-level as the stereo -->
     <origin xyz="-0.0475 0.035 0.0" rpy="0 0 0"/>

Commit message: Added new model for real robot

File: bigman_urdf/urdf/bigman.urdf.xacro (robot description, xacro)
@@ -53,16 +53,7 @@
 	<xacro:include filename="$(find bigman_urdf)/urdf/parts/soft_hand.urdf.xacro" />
 	<!-- multisense_sl_v4 with fixed joints (NOT FOR SIMULATION) -->
-	<xacro:include filename="$(find bigman_urdf)/urdf/sensors/multisense_sl.urdf.xacro"/>
-	<joint name="neck_joint" type="fixed">
-	    <parent link="NeckPitch"/>
-	    <child link="${multisense_namespace}/head"/>
-	    <origin xyz="0.08765 0 0.06475" rpy="0 0 0" />
-	</joint>
-       <link name="gaze"/>
-       <joint name="gaze_joint" type="fixed">
-              <parent link="${multisense_namespace}/head"/>
-              <child link="gaze"/>
-              <origin xyz="0 0 0" rpy="0 0 0" />
-       </joint>
+       <xacro:if value="${BIGMAN_HEAD}">
+	       <xacro:include filename="$(find bigman_urdf)/urdf/sensors/multisense_sl.urdf.xacro"/>
+       </xacro:if>
 </xacro:if>
 <xacro:if value="${BIGMAN_LEGS}">

File: bigman_urdf/urdf/bigman_config.urdf.xacro (robot description, xacro)
@@ -58,3 +58,17 @@
 -->
 <xacro:property name="BIGMAN_FIXED_MULTISENSE" value="true" />
+<!--
+####################################################
+##
+##  BIGMAN_HEAD
+##  if "true" a fixed joint between "NeckPitch" and
+##  "head" will be used to connect the head to the rest
+##  of the body. If "false" the head will not be added
+##  to the model (this is the case when the multisense
+##  from the launch file is used).
+##
+##
+####################################################
+-->
+<xacro:property name="BIGMAN_HEAD" value="true" />
 </robot>

File: bigman_urdf/urdf/config/bigman_gazebo.urdf.xacro (robot description, xacro)
@@ -58,3 +58,17 @@
 -->
 <xacro:property name="BIGMAN_FIXED_MULTISENSE" value="false" />
+<!--
+####################################################
+##
+##  BIGMAN_HEAD
+##  if "true" a fixed joint between "NeckPitch" and
+##  "head" will be used to connect the head to the rest
+##  of the body. If "false" the head will not be added
+##  to the model (this is the case when the multisense
+##  from the launch file is used).
+##
+##
+####################################################
+-->
+<xacro:property name="BIGMAN_HEAD" value="true" />
 </robot>

File: bigman_urdf/urdf/config/bigman_only_legs.urdf.xacro (robot description, xacro)
@@ -58,3 +58,17 @@
 -->
 <xacro:property name="BIGMAN_FIXED_MULTISENSE" value="true" />
+<!--
+####################################################
+##
+##  BIGMAN_HEAD
+##  if "true" a fixed joint between "NeckPitch" and
+##  "head" will be used to connect the head to the rest
+##  of the body. If "false" the head will not be added
+##  to the model (this is the case when the multisense
+##  from the launch file is used).
+##
+##
+####################################################
+-->
+<xacro:property name="BIGMAN_HEAD" value="true" />
 </robot>

File: bigman_urdf/urdf/config/bigman_only_upper_body.urdf.xacro (robot description, xacro)
@@ -58,3 +58,17 @@
 -->
 <xacro:property name="BIGMAN_FIXED_MULTISENSE" value="true" />
+<!--
+####################################################
+##
+##  BIGMAN_HEAD
+##  if "true" a fixed joint between "NeckPitch" and
+##  "head" will be used to connect the head to the rest
+##  of the body. If "false" the head will not be added
+##  to the model (this is the case when the multisense
+##  from the launch file is used).
+##
+##
+####################################################
+-->
+<xacro:property name="BIGMAN_HEAD" value="true" />
 </robot>

File: bigman_urdf/urdf/config/bigman_only_upper_body_gazebo.urdf.xacro (robot description, xacro)
@@ -58,3 +58,17 @@
 -->
 <xacro:property name="BIGMAN_FIXED_MULTISENSE" value="false" />
+<!--
+####################################################
+##
+##  BIGMAN_HEAD
+##  if "true" a fixed joint between "NeckPitch" and
+##  "head" will be used to connect the head to the rest
+##  of the body. If "false" the head will not be added
+##  to the model (this is the case when the multisense
+##  from the launch file is used).
+##
+##
+####################################################
+-->
+<xacro:property name="BIGMAN_HEAD" value="true" />
 </robot>

File: bigman_urdf/urdf/sensors/multisense_sl.urdf.xacro (robot description, xacro)
@@ -322,3 +322,14 @@
   </gazebo>
 -->
+  <joint name="neck_joint" type="fixed">
+    <parent link="NeckPitch"/>
+    <child link="${multisense_namespace}/head"/>
+    <origin xyz="0.08765 0 0.06475" rpy="0 0 0" />
+  </joint>
+  <link name="gaze"/>
+  <joint name="gaze_joint" type="fixed">
+    <parent link="${multisense_namespace}/head"/>
+    <child link="gaze"/>
+    <origin xyz="0 0 0" rpy="0 0 0" />
+  </joint>
 </robot>

Commit message: Added flag to add/remove forearms rising support (now are remnoved by default)

File: bigman_urdf/urdf/bigman.urdf.xacro (robot description, xacro)
@@ -49,5 +49,7 @@
 	<link name="r_wrist"/>
 	<xacro:include filename="$(find bigman_urdf)/urdf/parts/forearms.urdf.xacro" />
-	<xacro:include filename="$(find bigman_urdf)/urdf/parts/forearm_reference_frame.urdf.xacro" />
+       <xacro:if value="${BIGMAN_ADD_RAISING_SUPPORT}">
+	       <xacro:include filename="$(find bigman_urdf)/urdf/parts/forearm_reference_frame.urdf.xacro" />
+       </xacro:if>
 	<!-- ************ HANDS ************ -->
 	<xacro:include filename="$(find bigman_urdf)/urdf/parts/soft_hand.urdf.xacro" />

File: bigman_urdf/urdf/bigman_config.urdf.xacro (robot description, xacro)
@@ -92,3 +92,13 @@
 -->
 <xacro:property name="BIGMAN_ADD_BACKPACK" value="true" />
+<!--
+####################################################
+##
+##  BIGMAN_ADD_RAISING_SUPPORT
+##  if "true" the raising support are added to the model.
+##
+##
+####################################################
+-->
+<xacro:property name="BIGMAN_ADD_RAISING_SUPPORT" value="false" />
 </robot>

File: bigman_urdf/urdf/config/bigman_gazebo.urdf.xacro (robot description, xacro)
@@ -92,3 +92,13 @@
 -->
 <xacro:property name="BIGMAN_ADD_BACKPACK" value="true" />
+<!--
+####################################################
+##
+##  BIGMAN_ADD_RAISING_SUPPORT
+##  if "true" the raising support are added to the model.
+##
+##
+####################################################
+-->
+<xacro:property name="BIGMAN_ADD_RAISING_SUPPORT" value="false" />
 </robot>

File: bigman_urdf/urdf/config/bigman_only_legs.urdf.xacro (robot description, xacro)
@@ -92,3 +92,13 @@
 -->
 <xacro:property name="BIGMAN_ADD_BACKPACK" value="false" />
+<!--
+####################################################
+##
+##  BIGMAN_ADD_RAISING_SUPPORT
+##  if "true" the raising support are added to the model.
+##
+##
+####################################################
+-->
+<xacro:property name="BIGMAN_ADD_RAISING_SUPPORT" value="false" />
 </robot>

File: bigman_urdf/urdf/config/bigman_only_upper_body.urdf.xacro (robot description, xacro)
@@ -92,3 +92,13 @@
 -->
 <xacro:property name="BIGMAN_ADD_BACKPACK" value="true" />
+<!--
+####################################################
+##
+##  BIGMAN_ADD_RAISING_SUPPORT
+##  if "true" the raising support are added to the model.
+##
+##
+####################################################
+-->
+<xacro:property name="BIGMAN_ADD_RAISING_SUPPORT" value="false" />
 </robot>

File: bigman_urdf/urdf/config/bigman_only_upper_body_gazebo.urdf.xacro (robot description, xacro)
@@ -92,3 +92,13 @@
 -->
 <xacro:property name="BIGMAN_ADD_BACKPACK" value="true" />
+<!--
+####################################################
+##
+##  BIGMAN_ADD_RAISING_SUPPORT
+##  if "true" the raising support are added to the model.
+##
+##
+####################################################
+-->
+<xacro:property name="BIGMAN_ADD_RAISING_SUPPORT" value="false" />
 </robot>

File: bigman_urdf/urdf/config/bigman_real.urdf.xacro (robot description, xacro)
@@ -92,3 +92,13 @@
 -->
 <xacro:property name="BIGMAN_ADD_BACKPACK" value="true" />
+<!--
+####################################################
+##
+##  BIGMAN_ADD_RAISING_SUPPORT
+##  if "true" the raising support are added to the model.
+##
+##
+####################################################
+-->
+<xacro:property name="BIGMAN_ADD_RAISING_SUPPORT" value="false" />
 </robot>

File: bigman_urdf/urdf/parts/forearms.urdf.xacro (robot description, xacro)
@@ -46,4 +46,5 @@
         </collision>
       </link>
+<xacro:if value="${BIGMAN_ADD_RAISING_SUPPORT}">
       <link name="LRaisingSupport">
         <inertial>
@@ -68,4 +69,5 @@
         </collision>
       </link>
+</xacro:if>
       <link name="LWrMot3">
         <inertial>
@@ -129,4 +131,5 @@
         </collision>
       </link>
+<xacro:if value="${BIGMAN_ADD_RAISING_SUPPORT}">
       <link name="RRaisingSupport">
         <inertial>
@@ -151,4 +154,5 @@
         </collision>
       </link>
+</xacro:if>
       <link name="RWrMot3">
         <inertial>
@@ -189,9 +193,11 @@
     <dynamics friction="0" damping="0.03"/>
   </joint>
-    <joint name="LRaisingSupport_joint" type="fixed">
+<xacro:if value="${BIGMAN_ADD_RAISING_SUPPORT}">
+  <joint name="LRaisingSupport_joint" type="fixed">
     <parent link="LWrMot2"/>
     <child link="LRaisingSupport"/>
     <origin xyz="0.0 0.0 -0.0505" rpy="0 0 0"/>
   </joint>
+</xacro:if>
   <joint name="LWrj2" type="revolute">
     <parent link="LWrMot2"/>
@@ -224,9 +230,11 @@
     <dynamics friction="0" damping="0.03"/>
   </joint>
-    <joint name="RRaisingSupport_joint" type="fixed">
+<xacro:if value="${BIGMAN_ADD_RAISING_SUPPORT}">
+  <joint name="RRaisingSupport_joint" type="fixed">
     <parent link="RWrMot2"/>
     <child link="RRaisingSupport"/>
     <origin xyz="0.0 0.0 -0.0505" rpy="0 0 0"/>
   </joint>
+</xacro:if>
   <joint name="RWrj2" type="revolute">
     <parent link="RWrMot2"/>

Commit message: Added back bigman_urdf/urdf/sensors/multisense_sl_simulation.urdf.xacro since is needed in the launch file. Deleted protections in model since they interefere with the laser scans.

File: bigman_urdf/urdf/bigman.urdf.xacro (robot description, xacro)
@@ -54,5 +54,5 @@
 	<!-- ************ HANDS ************ -->
 	<xacro:include filename="$(find bigman_urdf)/urdf/parts/soft_hand.urdf.xacro" />
-	<!-- multisense_sl_v4 with fixed joints (NOT FOR SIMULATION) -->
+	<!-- multisense_sl_v4 with fixed joints -->
        <xacro:if value="${BIGMAN_HEAD}">
 	       <xacro:include filename="$(find bigman_urdf)/urdf/sensors/multisense_sl.urdf.xacro"/>

File: bigman_urdf/urdf/config/bigman_gazebo.urdf.xacro (robot description, xacro)
@@ -81,5 +81,5 @@
 ####################################################
 -->
-<xacro:property name="BIGMAN_ADD_PROTECTIONS" value="true" />
+<xacro:property name="BIGMAN_ADD_PROTECTIONS" value="false" />
 <!--
 ####################################################

File: bigman_urdf/urdf/sensors/multisense_sl_simulation.urdf.xacro (robot description, xacro)
@@ -61,5 +61,4 @@
     <mu2>0.9</mu2>
   </gazebo>
-<xacro:unless value="${BIGMAN_FIXED_MULTISENSE}">
   <joint name="hokuyo_joint" type="continuous">
     <origin xyz="-0.0446 0 0.0880" rpy="0 0 0" />
@@ -73,12 +72,4 @@
     <implicitSpringDamper>1</implicitSpringDamper>
   </gazebo>
-</xacro:unless>
-<xacro:if value="${BIGMAN_FIXED_MULTISENSE}">
-  <joint name="hokuyo_joint" type="fixed">
-    <origin xyz="-0.0446 0 0.0880" rpy="0 0 0" />
-    <parent link="${multisense_namespace}head_multisense" />
-    <child link="${multisense_namespace}hokuyo_link" />
-  </joint>
-</xacro:if>
   <!-- Hokuyo Laser -->
   <joint name="head_hokuyo_joint" type="fixed">
@@ -315,9 +306,4 @@
     </sensor>
   </gazebo>
-  <joint name="neck_joint" type="fixed">
-    <parent link="head"/>
-    <child link="${multisense_namespace}head_multisense"/>
-    <origin xyz="0.08765 0 0.06475" rpy="0 0 0" />
-  </joint>
   <link name="gaze"/>
   <joint name="gaze_joint" type="fixed">
