Commit message: refactor

File: bigman_urdf/urdf/bigman.urdf.xacro (robot description, xacro)
@@ -56,5 +56,15 @@
 	<!-- multisense_sl_v4 with fixed joints -->
        <xacro:if value="${BIGMAN_HEAD}">
-	       <xacro:include filename="$(find bigman_urdf)/urdf/sensors/multisense_sl.urdf.xacro"/>
+                <joint name="neck_joint" type="fixed">
+                     <parent link="head"/>
+                     <child link="${multisense_namespace}head_multisense"/>
+                     <origin xyz="0.08765 0 0.06475" rpy="0 0 0" />
+                 </joint>
+              <xacro:unless value="${BIGMAN_FIXED_MULTISENSE}">
+                     <xacro:include filename="$(find bigman_urdf)/urdf/sensors/multisense_sl_simulation.urdf.xacro"/>
+              </xacro:unless>
+              <xacro:if value="${BIGMAN_FIXED_MULTISENSE}">
+                     <xacro:include filename="$(find bigman_urdf)/urdf/sensors/multisense_sl.urdf.xacro"/>
+              </xacro:if>
        </xacro:if>
 </xacro:if>

File: bigman_urdf/urdf/sensors/multisense_sl.urdf.xacro (robot description, xacro)
@@ -52,27 +52,4 @@
   </collision>
   </link>
-<!-- Remove frome here! -->
-<gazebo reference="head_multisense">
-    <mu1>0.9</mu1>
-    <mu2>0.9</mu2>
-  </gazebo>
-  <gazebo reference="hokuyo_link">
-    <mu1>0.9</mu1>
-    <mu2>0.9</mu2>
-  </gazebo>
-<xacro:unless value="${BIGMAN_FIXED_MULTISENSE}">
-  <joint name="hokuyo_joint" type="continuous">
-    <origin xyz="-0.0446 0 0.0880" rpy="0 0 0" />
-    <parent link="${multisense_namespace}head_multisense" />
-    <child link="${multisense_namespace}hokuyo_link" />
-    <axis xyz="1 0 0" />
-    <dynamics damping="0.01" friction="0"/>
-  </joint>
-  <!-- Remove frome here! -->
-  <gazebo reference="hokuyo_joint">
-    <implicitSpringDamper>1</implicitSpringDamper>
-  </gazebo>
-</xacro:unless>
-<xacro:if value="${BIGMAN_FIXED_MULTISENSE}">
   <joint name="hokuyo_joint" type="fixed">
     <origin xyz="-0.0446 0 0.0880" rpy="0 0 0" />
@@ -80,5 +57,4 @@
     <child link="${multisense_namespace}hokuyo_link" />
   </joint>
-</xacro:if>
   <!-- Hokuyo Laser -->
   <joint name="head_hokuyo_joint" type="fixed">
@@ -89,42 +65,4 @@
   </joint>
   <link name="${multisense_namespace}head_hokuyo_frame"/>
-<!-- Remove frome here! -->
-  <gazebo reference="head_hokuyo_frame">
-    <!-- sensor type="gpu_ray" name="head_hokuyo_sensor"-->
-    <sensor type="ray" name="head_hokuyo_sensor">
-      <pose>0 0 0 0 0 0</pose>
-      <visualize>true</visualize>
-      <update_rate>40</update_rate>
-      <ray>
-        <scan>
-          <horizontal>
-            <samples>720</samples>
-            <resolution>1</resolution>
-            <min_angle>-1.570796</min_angle>
-            <max_angle>1.570796</max_angle>
-          </horizontal>
-        </scan>
-        <range>
-          <min>0.10</min>
-          <max>30.0</max>
-          <resolution>0.01</resolution>
-        </range>
-        <noise>
-          <type>gaussian</type>
-          <!-- Noise parameters based on published spec for Hokuyo laser
-               achieving "+-30mm" accuracy at range < 10m.  A mean of 0.0m and
-               stddev of 0.01m will put 99.7% of samples within 0.03m of the true
-               reading. -->
-          <mean>0.0</mean>
-          <stddev>0.01</stddev>
-        </noise>
-      </ray>
-      <!--plugin name="gazebo_ros_head_hokuyo_controller" filename="libgazebo_ros_gpu_laser.so"-->
-      <plugin name="gazebo_ros_head_hokuyo_controller" filename="libgazebo_ros_laser.so">
-        <topicName>/multisense/lidar_scan</topicName>
-        <frameName>head_hokuyo_frame</frameName>
-      </plugin>
-    </sensor>
-  </gazebo>
   <!-- Stereo Camera -->
   <joint name="left_camera_frame_joint" type="fixed">
@@ -141,76 +79,4 @@
   </joint>
   <link name="${multisense_namespace}left_camera_optical_frame"/>
-  <gazebo reference="left_camera_frame">
-    <sensor type="multicamera" name="stereo_camera">
-      <!-- see MultiSenseSLPlugin.h for available modes -->
-      <update_rate>30.0</update_rate>
-      <camera name="left">
-        <!-- Spec sheet says 80deg X 45deg @ 1024x544pix.  Based on feedback
-             from teams, we're instead doing 80deg X 80deg @ 800x800pix. -->
-        <horizontal_fov>1.3962634</horizontal_fov>
-        <image>
-          <width>800</width>
-          <height>800</height>
-          <format>R8G8B8</format>
-        </image>
-        <clip>
-          <near>0.02</near>
-          <far>300</far>
-        </clip>
-        <noise>
-          <type>gaussian</type>
-          <!-- Noise is sampled independently per pixel on each frame.
-               That pixel's noise value is added to each of its color
-               channels, which at that point lie in the range [0,1].
-               The stddev value of 0.007 is based on experimental data
-               from a camera in a Sandia hand pointed at a static scene
-               in a couple of different lighting conditions.  -->
-          <mean>0.0</mean>
-          <stddev>0.007</stddev>
-        </noise>
-      </camera>
-      <camera name="right">
-        <pose>0 -0.07 0 0 0 0</pose>
-        <!-- Spec sheet says 80deg X 45deg @ 1024x544pix.  Based on feedback
-             from teams, we're instead doing 80deg X 80deg @ 800x800pix. -->
-        <horizontal_fov>1.3962634</horizontal_fov>
-        <image>
-          <width>800</width>
-          <height>800</height>
-          <format>R8G8B8</format>
-        </image>
-        <clip>
-          <near>0.02</near>
-          <far>300</far>
-        </clip>
-        <noise>
-          <type>gaussian</type>
-          <!-- Noise is sampled independently per pixel on each frame.
-               That pixel's noise value is added to each of its color
-               channels, which at that point lie in the range [0,1].
-               The stddev value of 0.007 is based on experimental data
-               from a camera in a Sandia hand pointed at a static scene
-               in a couple of different lighting conditions.  -->
-          <mean>0.0</mean>
-          <stddev>0.007</stddev>
-        </noise>
-      </camera>
-      <plugin name="stereo_camera_controller" filename="libgazebo_ros_multicamera.so">
-        <alwaysOn>true</alwaysOn>
-        <updateRate>0.0</updateRate>
-        <cameraName>multisense/camera</cameraName>
-        <imageTopicName>image_raw</imageTopicName>
-        <cameraInfoTopicName>camera_info</cameraInfoTopicName>
-        <frameName>left_camera_optical_frame</frameName>
-        <rightFrameName>right_camera_optical_frame</rightFrameName>
-        <hackBaseline>0.07</hackBaseline>
-        <distortionK1>0.0</distortionK1>
-        <distortionK2>0.0</distortionK2>
-        <distortionK3>0.0</distortionK3>
-        <distortionT1>0.0</distortionT1>
-        <distortionT2>0.0</distortionT2>
-      </plugin>
-    </sensor>
-  </gazebo>
   <joint name="right_camera_frame_joint" type="fixed">
     <origin xyz="0.0 -0.035 -0.002"/>
@@ -249,7 +115,4 @@
   </joint>
   <link name="${multisense_namespace}right_led_frame"/>
-  <gazebo>
-    <plugin filename="libMultiSenseSLPlugin.so" name="multisense_plugin"/>
-  </gazebo>
   <!-- imu link -->
   <link name="${multisense_namespace}head_imu_link">
@@ -273,51 +136,4 @@
     <origin xyz="-0.0475 0.035 0.0" rpy="0 0 0"/>
   </joint>
-  <gazebo reference="head_imu_link">
-    <!-- this is expected to be reparented to head with appropriate offset
-         when head_imu_link is reduced by fixed joint reduction -->
-    <!-- todo: this is working with gazebo 1.4, need to write a unit test -->
-     <sensor name="head_imu_sensor" type="imu">
-      <always_on>1</always_on>
-      <update_rate>1000.0</update_rate>
-      <imu>
-        <noise>
-          <type>gaussian</type>
-          <!-- Noise parameters from Boston Dynamics
-               (http://gazebosim.org/wiki/Sensor_noise):
-                 rates (rad/s): mean=0, stddev=2e-4
-                 accels (m/s/s): mean=0, stddev=1.7e-2
-                 rate bias (rad/s): 5e-6 - 1e-5
-                 accel bias (m/s/s): 1e-1
-               Experimentally, simulation provide rates with noise of
-               about 1e-3 rad/s and accels with noise of about 1e-1 m/s/s.
-               So we don't expect to see the noise unless number of inner iterations
-               are increased.
-               We will add bias.  In this model, bias is sampled once for rates
-               and once for accels at startup; the sign (negative or positive)
-               of each bias is then switched with equal probability.  Thereafter,
-               the biases are fixed additive offsets.  We choose
-               bias means and stddevs to produce biases close to the provided
-               data. -->
-          <rate>
-            <mean>0.0</mean>
-            <stddev>2e-4</stddev>
-            <bias_mean>0.0000075</bias_mean>
-            <bias_stddev>0.0000008</bias_stddev>
-          </rate>
-          <accel>
-            <mean>0.0</mean>
-            <stddev>1.7e-2</stddev>
-            <bias_mean>0.1</bias_mean>
-            <bias_stddev>0.001</bias_stddev>
-          </accel>
-        </noise>
-      </imu>
-    </sensor>
-  </gazebo>
-  <joint name="neck_joint" type="fixed">
-    <parent link="head"/>
-    <child link="${multisense_namespace}head_multisense"/>
-    <origin xyz="0.08765 0 0.06475" rpy="0 0 0" />
-  </joint>
   <link name="gaze"/>
   <joint name="gaze_joint" type="fixed">
