Commit message: added multisense/ namespace in front of the frames related to multisense

File: bigman_urdf/urdf/bigman.urdf.xacro (robot description, xacro)
@@ -58,5 +58,5 @@
                 <joint name="neck_joint" type="fixed">
                      <parent link="NeckPitch"/>
-                     <child link="${multisense_namespace}head_multisense"/>
+                     <child link="multisense/head"/>
                      <origin xyz="0.08765 0 0.06475" rpy="0 0 0" />
                  </joint>

File: bigman_urdf/urdf/sensors/multisense_sl.urdf.xacro (robot description, xacro)
@@ -1,10 +1,9 @@
 <?xml version="1.0"?>
 <robot xmlns:xacro="http://ros.org/wiki/xacro" name="multisense_sl">
-<xacro:property name="multisense_namespace" value="" />
 <!--
        Based on multisense_sl_v4.urdf in multisense_sl_description (DRCSIM)
 -->
   <!-- Head Link Simple Collision Meshes -->
-  <link name="${multisense_namespace}head_multisense">
+  <link name="multisense/head">
     <inertial>
       <origin xyz="-0.075493 3.3383E-05 0.02774" rpy="0 0 0" />
@@ -26,5 +25,5 @@
   </collision>
   </link>
-  <link name="${multisense_namespace}hokuyo_link">
+  <link name="multisense/hokuyo_link">
     <inertial>
       <origin xyz="0.032428 0.0004084 -0.0041835" rpy="0 0 0" />
@@ -54,6 +53,6 @@
   <joint name="hokuyo_joint" type="fixed">
     <origin xyz="-0.0446 0 0.0880" rpy="0 0 0" />
-    <parent link="${multisense_namespace}head_multisense" />
-    <child link="${multisense_namespace}hokuyo_link" />
+    <parent link="multisense/head" />
+    <child link="multisense/hokuyo_link" />
   </joint>
   <!-- Hokuyo Laser -->
@@ -61,60 +60,60 @@
     <axis xyz="0 1 0" />
     <origin xyz="0.03 0 0.015" rpy="0 0 0"/>
-    <parent link="${multisense_namespace}hokuyo_link"/>
-    <child link="${multisense_namespace}head_hokuyo_frame"/>
+    <parent link="multisense/hokuyo_link"/>
+    <child link="multisense/head_hokuyo_frame"/>
   </joint>
-  <link name="${multisense_namespace}head_hokuyo_frame"/>
+  <link name="multisense/head_hokuyo_frame"/>
   <!-- Stereo Camera -->
   <joint name="left_camera_frame_joint" type="fixed">
     <!-- optical frame collocated with tilting DOF -->
     <origin xyz="0.0 0.035 -0.002"/>
-    <parent link="${multisense_namespace}head_multisense"/>
-    <child link="${multisense_namespace}left_camera_frame"/>
+    <parent link="multisense/head"/>
+    <child link="multisense/left_camera_frame"/>
   </joint>
-  <link name="${multisense_namespace}left_camera_frame"/>
+  <link name="multisense/left_camera_frame"/>
   <joint name="left_camera_optical_frame_joint" type="fixed">
     <origin xyz="0 0 0" rpy="-1.5708 0.0 -1.5708" />
-    <parent link="${multisense_namespace}left_camera_frame" />
-    <child link="${multisense_namespace}left_camera_optical_frame"/>
+    <parent link="multisense/left_camera_frame" />
+    <child link="multisense/left_camera_optical_frame"/>
   </joint>
-  <link name="${multisense_namespace}left_camera_optical_frame"/>
+  <link name="multisense/left_camera_optical_frame"/>
   <joint name="right_camera_frame_joint" type="fixed">
     <origin xyz="0.0 -0.035 -0.002"/>
-    <parent link="${multisense_namespace}head_multisense"/>
-    <child link="${multisense_namespace}right_camera_frame"/>
+    <parent link="multisense/head"/>
+    <child link="multisense/right_camera_frame"/>
   </joint>
-  <link name="${multisense_namespace}right_camera_frame"/>
+  <link name="multisense/right_camera_frame"/>
   <joint name="right_camera_optical_frame_joint" type="fixed">
     <origin xyz="0 0 0" rpy="-1.5708 0.0 -1.5708" />
-    <parent link="${multisense_namespace}right_camera_frame" />
-    <child link="${multisense_namespace}right_camera_optical_frame"/>
+    <parent link="multisense/right_camera_frame" />
+    <child link="multisense/right_camera_optical_frame"/>
   </joint>
-  <link name="${multisense_namespace}right_camera_optical_frame"/>
+  <link name="multisense/right_camera_optical_frame"/>
   <joint name="center_top_led_frame_joint" type="fixed">
     <origin xyz="0.01125 0.0 0.0105"/>
-    <parent link="${multisense_namespace}head_multisense"/>
-    <child link="${multisense_namespace}center_top_led_frame"/>
+    <parent link="multisense/head"/>
+    <child link="multisense/center_top_led_frame"/>
   </joint>
-  <link name="${multisense_namespace}center_top_led_frame"/>
+  <link name="multisense/center_top_led_frame"/>
   <joint name="center_bottom_led_frame_joint" type="fixed">
     <origin xyz="0.01125 0.0 -0.0155"/>
-    <parent link="${multisense_namespace}head_multisense"/>
-    <child link="${multisense_namespace}center_bottom_led_frame"/>
+    <parent link="multisense/head"/>
+    <child link="multisense/center_bottom_led_frame"/>
   </joint>
-  <link name="${multisense_namespace}center_bottom_led_frame"/>
+  <link name="multisense/center_bottom_led_frame"/>
   <joint name="left_led_frame_joint" type="fixed">
     <origin xyz="-0.01443 0.07452 0.050346" rpy="0 0 0.6"/>
-    <parent link="${multisense_namespace}head_multisense"/>
-    <child link="${multisense_namespace}left_led_frame"/>
+    <parent link="multisense/head"/>
+    <child link="multisense/left_led_frame"/>
   </joint>
-  <link name="${multisense_namespace}left_led_frame"/>
+  <link name="multisense/left_led_frame"/>
   <joint name="right_led_frame_joint" type="fixed">
     <origin xyz="-0.01443 -0.07452 0.050346" rpy="0 0 -0.6"/>
-    <parent link="${multisense_namespace}head_multisense"/>
-    <child link="${multisense_namespace}right_led_frame"/>
+    <parent link="multisense/head"/>
+    <child link="multisense/right_led_frame"/>
   </joint>
-  <link name="${multisense_namespace}right_led_frame"/>
+  <link name="multisense/right_led_frame"/>
   <!-- imu link -->
-  <link name="${multisense_namespace}head_imu_link">
+  <link name="multisense/head_imu_link">
     <inertial>
       <mass value="1e-5" />
@@ -131,6 +130,6 @@
   </link>
   <joint name="head_imu_joint" type="fixed">
-    <parent link="${multisense_namespace}head_multisense"/>
-    <child link="${multisense_namespace}head_imu_link"/>
+    <parent link="multisense/head"/>
+    <child link="multisense/head_imu_link"/>
     <!-- putting it at the same z-level as the stereo -->
     <origin xyz="-0.0475 0.035 0.0" rpy="0 0 0"/>
@@ -138,5 +137,5 @@
   <link name="gaze"/>
   <joint name="gaze_joint" type="fixed">
-    <parent link="${multisense_namespace}head_multisense"/>
+    <parent link="multisense/head"/>
     <child link="gaze"/>
     <origin xyz="0 0 0" rpy="0 0 0" />

File: bigman_urdf/urdf/sensors/multisense_sl_simulation.urdf.xacro (robot description, xacro)
@@ -1,10 +1,9 @@
 <?xml version="1.0"?>
 <robot xmlns:xacro="http://ros.org/wiki/xacro" name="multisense_sl">
-<xacro:property name="multisense_namespace" value="" />
 <!--
        Based on multisense_sl_v4.urdf in multisense_sl_description (DRCSIM)
 -->
   <!-- Head Link Simple Collision Meshes -->
-  <link name="${multisense_namespace}head_multisense">
+  <link name="multisense/head">
     <inertial>
       <origin xyz="-0.075493 3.3383E-05 0.02774" rpy="0 0 0" />
@@ -26,5 +25,5 @@
   </collision>
   </link>
-  <link name="${multisense_namespace}hokuyo_link">
+  <link name="multisense/hokuyo_link">
     <inertial>
       <origin xyz="0.032428 0.0004084 -0.0041835" rpy="0 0 0" />
@@ -53,9 +52,9 @@
   </link>
 <!-- Remove frome here! -->
-<gazebo reference="head_multisense">
+<gazebo reference="multisense/head">
     <mu1>0.9</mu1>
     <mu2>0.9</mu2>
   </gazebo>
-  <gazebo reference="hokuyo_link">
+  <gazebo reference="multisense/hokuyo_link">
     <mu1>0.9</mu1>
     <mu2>0.9</mu2>
@@ -63,6 +62,6 @@
   <joint name="hokuyo_joint" type="continuous">
     <origin xyz="-0.0446 0 0.0880" rpy="0 0 0" />
-    <parent link="${multisense_namespace}head_multisense" />
-    <child link="${multisense_namespace}hokuyo_link" />
+    <parent link="multisense/head" />
+    <child link="multisense/hokuyo_link" />
     <axis xyz="1 0 0" />
     <dynamics damping="0.01" friction="0"/>
@@ -76,10 +75,10 @@
     <axis xyz="0 1 0" />
     <origin xyz="0.03 0 0.015" rpy="0 0 0"/>
-    <parent link="${multisense_namespace}hokuyo_link"/>
-    <child link="${multisense_namespace}head_hokuyo_frame"/>
-  </joint>
-  <link name="${multisense_namespace}head_hokuyo_frame"/>
+    <parent link="multisense/hokuyo_link"/>
+    <child link="multisense/head_hokuyo_frame"/>
+  </joint>
+  <link name="multisense/head_hokuyo_frame"/>
 <!-- Remove frome here! -->
-  <gazebo reference="head_hokuyo_frame">
+  <gazebo reference="multisense/head_hokuyo_frame">
     <!-- sensor type="gpu_ray" name="head_hokuyo_sensor"-->
     <sensor type="ray" name="head_hokuyo_sensor">
@@ -114,5 +113,5 @@
       <plugin name="gazebo_ros_head_hokuyo_controller" filename="libgazebo_ros_laser.so">
         <topicName>/multisense/lidar_scan</topicName>
-        <frameName>head_hokuyo_frame</frameName>
+        <frameName>multisense/head_hokuyo_frame</frameName>
       </plugin>
     </sensor>
@@ -122,15 +121,15 @@
     <!-- optical frame collocated with tilting DOF -->
     <origin xyz="0.0 0.035 -0.002"/>
-    <parent link="${multisense_namespace}head_multisense"/>
-    <child link="${multisense_namespace}left_camera_frame"/>
-  </joint>
-  <link name="${multisense_namespace}left_camera_frame"/>
+    <parent link="multisense/head"/>
+    <child link="multisense/left_camera_frame"/>
+  </joint>
+  <link name="multisense/left_camera_frame"/>
   <joint name="left_camera_optical_frame_joint" type="fixed">
     <origin xyz="0 0 0" rpy="-1.5708 0.0 -1.5708" />
-    <parent link="${multisense_namespace}left_camera_frame" />
-    <child link="${multisense_namespace}left_camera_optical_frame"/>
-  </joint>
-  <link name="${multisense_namespace}left_camera_optical_frame"/>
-  <gazebo reference="left_camera_frame">
+    <parent link="multisense/left_camera_frame" />
+    <child link="multisense/left_camera_optical_frame"/>
+  </joint>
+  <link name="multisense/left_camera_optical_frame"/>
+  <gazebo reference="multisense/left_camera_frame">
     <sensor type="multicamera" name="stereo_camera">
       <!-- see MultiSenseSLPlugin.h for available modes -->
@@ -193,6 +192,6 @@
         <imageTopicName>image_raw</imageTopicName>
         <cameraInfoTopicName>camera_info</cameraInfoTopicName>
-        <frameName>left_camera_optical_frame</frameName>
-        <rightFrameName>right_camera_optical_frame</rightFrameName>
+        <frameName>multisense/left_camera_optical_frame</frameName>
+        <rightFrameName>multisense/right_camera_optical_frame</rightFrameName>
         <hackBaseline>0.07</hackBaseline>
         <distortionK1>0.0</distortionK1>
@@ -206,43 +205,43 @@
   <joint name="right_camera_frame_joint" type="fixed">
     <origin xyz="0.0 -0.035 -0.002"/>
-    <parent link="${multisense_namespace}head_multisense"/>
-    <child link="${multisense_namespace}right_camera_frame"/>
-  </joint>
-  <link name="${multisense_namespace}right_camera_frame"/>
+    <parent link="multisense/head"/>
+    <child link="multisense/right_camera_frame"/>
+  </joint>
+  <link name="multisense/right_camera_frame"/>
   <joint name="right_camera_optical_frame_joint" type="fixed">
     <origin xyz="0 0 0" rpy="-1.5708 0.0 -1.5708" />
-    <parent link="${multisense_namespace}right_camera_frame" />
-    <child link="${multisense_namespace}right_camera_optical_frame"/>
-  </joint>
-  <link name="${multisense_namespace}right_camera_optical_frame"/>
+    <parent link="multisense/right_camera_frame" />
+    <child link="multisense/right_camera_optical_frame"/>
+  </joint>
+  <link name="multisense/right_camera_optical_frame"/>
   <joint name="center_top_led_frame_joint" type="fixed">
     <origin xyz="0.01125 0.0 0.0105"/>
-    <parent link="${multisense_namespace}head_multisense"/>
-    <child link="${multisense_namespace}center_top_led_frame"/>
-  </joint>
-  <link name="${multisense_namespace}center_top_led_frame"/>
+    <parent link="multisense/head"/>
+    <child link="multisense/center_top_led_frame"/>
+  </joint>
+  <link name="multisense/center_top_led_frame"/>
   <joint name="center_bottom_led_frame_joint" type="fixed">
     <origin xyz="0.01125 0.0 -0.0155"/>
-    <parent link="${multisense_namespace}head_multisense"/>
-    <child link="${multisense_namespace}center_bottom_led_frame"/>
-  </joint>
-  <link name="${multisense_namespace}center_bottom_led_frame"/>
+    <parent link="multisense/head"/>
+    <child link="multisense/center_bottom_led_frame"/>
+  </joint>
+  <link name="multisense/center_bottom_led_frame"/>
   <joint name="left_led_frame_joint" type="fixed">
     <origin xyz="-0.01443 0.07452 0.050346" rpy="0 0 0.6"/>
-    <parent link="${multisense_namespace}head_multisense"/>
-    <child link="${multisense_namespace}left_led_frame"/>
-  </joint>
-  <link name="${multisense_namespace}left_led_frame"/>
+    <parent link="multisense/head"/>
+    <child link="multisense/left_led_frame"/>
+  </joint>
+  <link name="multisense/left_led_frame"/>
   <joint name="right_led_frame_joint" type="fixed">
     <origin xyz="-0.01443 -0.07452 0.050346" rpy="0 0 -0.6"/>
-    <parent link="${multisense_namespace}head_multisense"/>
-    <child link="${multisense_namespace}right_led_frame"/>
-  </joint>
-  <link name="${multisense_namespace}right_led_frame"/>
+    <parent link="multisense/head"/>
+    <child link="multisense/right_led_frame"/>
+  </joint>
+  <link name="multisense/right_led_frame"/>
   <gazebo>
     <plugin filename="libMultiSenseSLPlugin2.so" name="multisense_plugin"/>
   </gazebo>
   <!-- imu link -->
-  <link name="${multisense_namespace}head_imu_link">
+  <link name="multisense/head_imu_link">
     <inertial>
       <mass value="1e-5" />
@@ -259,10 +258,10 @@
   </link>
   <joint name="head_imu_joint" type="fixed">
-    <parent link="${multisense_namespace}head_multisense"/>
-    <child link="${multisense_namespace}head_imu_link"/>
+    <parent link="multisense/head"/>
+    <child link="multisense/head_imu_link"/>
     <!-- putting it at the same z-level as the stereo -->
     <origin xyz="-0.0475 0.035 0.0" rpy="0 0 0"/>
   </joint>
-  <gazebo reference="head_imu_link">
+  <gazebo reference="multisense/head_imu_link">
     <!-- this is expected to be reparented to head with appropriate offset
          when head_imu_link is reduced by fixed joint reduction -->
@@ -308,5 +307,5 @@
   <link name="gaze"/>
   <joint name="gaze_joint" type="fixed">
-    <parent link="${multisense_namespace}head_multisense"/>
+    <parent link="multisense/head"/>
     <child link="gaze"/>
     <origin xyz="0 0 0" rpy="0 0 0" />

Commit message: added possibliity to add floating_base kinematic chain

File: bigman_urdf/urdf/bigman.urdf.xacro (robot description, xacro)
@@ -14,4 +14,13 @@
 <!-- ************ BIGMAN BASE ************** -->
 <xacro:include filename="$(find bigman_urdf)/urdf/bigman_base.urdf.xacro"/>
+<xacro:if value="${BIGMAN_FLOATING_BASE}">
+<!-- ************ BIGMAN FLOATING BASE ************** -->
+<link name="world"/>
+  <joint name="reference" type="floating">
+    <origin xyz="0.0 0.0 0.0"/>
+    <parent link="world"/>
+    <child link="base_link"/>
+  </joint>
+</xacro:if>
 <xacro:if value="${BIGMAN_LEGS}">
 	<!-- ***** LEGS F/T SENSOR REF FRAMES *******-->

File: bigman_urdf/urdf/bigman_config.urdf.xacro (robot description, xacro)
@@ -147,4 +147,15 @@
 ####################################################
 ##
+##  BIGMAN_FLOATING_BASE
+##  if "true" virtual kinematic chains is attached between
+##  "world" and "base_link"
+##
+##
+####################################################
+-->
+<xacro:property name="BIGMAN_FLOATING_BASE" value="true" />
+<!--
+####################################################
+##
 ##  BIGMAN_MAGNETIC_ATTACH_ROS
 ##  if "true" the magnetic_attach_ros plugin is used

File: bigman_urdf/urdf/config/bigman_gazebo.urdf.xacro (robot description, xacro)
@@ -147,4 +147,15 @@
 ####################################################
 ##
+##  BIGMAN_FLOATING_BASE
+##  if "true" virtual kinematic chains is attached between
+##  "world" and "base_link"
+##
+##
+####################################################
+-->
+<xacro:property name="BIGMAN_FLOATING_BASE" value="true" />
+<!--
+####################################################
+##
 ##  BIGMAN_MAGNETIC_ATTACH_ROS
 ##  if "true" the magnetic_attach_ros plugin is used

File: bigman_urdf/urdf/config/bigman_only_legs.urdf.xacro (robot description, xacro)
@@ -147,4 +147,15 @@
 ####################################################
 ##
+##  BIGMAN_FLOATING_BASE
+##  if "true" virtual kinematic chains is attached between
+##  "world" and "base_link"
+##
+##
+####################################################
+-->
+<xacro:property name="BIGMAN_FLOATING_BASE" value="true" />
+<!--
+####################################################
+##
 ##  BIGMAN_MAGNETIC_ATTACH_ROS
 ##  if "true" the magnetic_attach_ros plugin is used

File: bigman_urdf/urdf/config/bigman_only_upper_body.urdf.xacro (robot description, xacro)
@@ -147,4 +147,15 @@
 ####################################################
 ##
+##  BIGMAN_FLOATING_BASE
+##  if "true" virtual kinematic chains is attached between
+##  "world" and "base_link"
+##
+##
+####################################################
+-->
+<xacro:property name="BIGMAN_FLOATING_BASE" value="false" />
+<!--
+####################################################
+##
 ##  BIGMAN_MAGNETIC_ATTACH_ROS
 ##  if "true" the magnetic_attach_ros plugin is used

File: bigman_urdf/urdf/config/bigman_only_upper_body_gazebo.urdf.xacro (robot description, xacro)
@@ -147,4 +147,15 @@
 ####################################################
 ##
+##  BIGMAN_FLOATING_BASE
+##  if "true" virtual kinematic chains is attached between
+##  "world" and "base_link"
+##
+##
+####################################################
+-->
+<xacro:property name="BIGMAN_FLOATING_BASE" value="false" />
+<!--
+####################################################
+##
 ##  BIGMAN_MAGNETIC_ATTACH_ROS
 ##  if "true" the magnetic_attach_ros plugin is used

File: bigman_urdf/urdf/config/bigman_real.urdf.xacro (robot description, xacro)
@@ -147,4 +147,15 @@
 ####################################################
 ##
+##  BIGMAN_FLOATING_BASE
+##  if "true" virtual kinematic chains is attached between
+##  "world" and "base_link"
+##
+##
+####################################################
+-->
+<xacro:property name="BIGMAN_FLOATING_BASE" value="false" />
+<!--
+####################################################
+##
 ##  BIGMAN_MAGNETIC_ATTACH_ROS
 ##  if "true" the magnetic_attach_ros plugin is used
