Commit message: Added foot of new bigman/walkman

File: bigman_urdf/urdf/bigman_base.urdf.xacro (robot description, xacro)
@@ -37,20 +37,20 @@
     <parent link="LFoot"/>
     <child link="l_sole"/>
-    <origin xyz="0 0 -0.09" rpy="0 0 0" />
+    <origin xyz="0 0 -0.1435" rpy="0 0 0" />
   </joint>
   <joint name="r_sole_joint" type="fixed">
     <parent link="RFoot"/>
     <child link="r_sole"/>
-    <origin xyz="0 0 -0.09" rpy="0 0 0" />
+    <origin xyz="0 0 -0.1435" rpy="0 0 0" />
   </joint>
   <joint name="l_toe_joint" type="fixed">
     <parent link="l_sole"/>
     <child link="l_toe"/>
-    <origin xyz="0.13 0 0" rpy="0 0 0" />
+    <origin xyz="0.195 0 0" rpy="0 0 0" />
   </joint>
   <joint name="r_toe_joint" type="fixed">
     <parent link="r_sole"/>
     <child link="r_toe"/>
-    <origin xyz="0.13 0 0" rpy="0 0 0" />
+    <origin xyz="0.195 0 0" rpy="0 0 0" />
   </joint>
 <!-- Reference frames in feet -->

File: bigman_urdf/urdf/bigman_robot.urdf.xacro (robot description, xacro)
@@ -12,4 +12,4 @@
 <!-- YARP PLUGINS for GAZEBO SIMULATION -->
   <xacro:include filename="$(find bigman_urdf)/urdf/gazebo/yarp_control.gazebo.xacro" />
-  <origin xyz="0.0 0.0 0.521" rpy="0 0 0" />
+  <origin xyz="0.0 0.0 0.575" rpy="0 0 0" />
 </robot>

File: bigman_urdf/urdf/gazebo/force_torque.gazebo.xacro (robot description, xacro)
@@ -29,5 +29,5 @@
 			<visualize>true</visualize>
 			<update_rate>1000</update_rate>
-			<pose>0 0 -0.065 0 0 0</pose>
+			<pose>0.05 0 -0.107 0 0 0</pose>
 			<plugin name="LAnkSag_FT_plugin" filename="libgazebo_yarp_forcetorque.so">
 				<yarpConfigurationFile>model://bigman_urdf/conf/bigman/bigman_gazebo_left_leg_ft.ini</yarpConfigurationFile>
@@ -41,5 +41,5 @@
 			<visualize>true</visualize>
 			<update_rate>1000</update_rate>
-			<pose>0 0 -0.065 0 0 0</pose>
+			<pose>0.05 0 -0.107 0 0 0</pose>
 			<plugin name="RAnkSag_FT_plugin" filename="libgazebo_yarp_forcetorque.so">
 				<yarpConfigurationFile>model://bigman_urdf/conf/bigman/bigman_gazebo_right_leg_ft.ini</yarpConfigurationFile>

File: bigman_urdf/urdf/parts/foot_reference_frame.urdf.xacro (robot description, xacro)
@@ -1,8 +1,4 @@
 <?xml version="1.0"?>
 <robot xmlns:xacro="http://ros.org/wiki/xacro">
-	<xacro:property name="x_positive" value="0.13" />
-	<xacro:property name="x_negative" value="-0.07" />
-	<xacro:property name="y_positive" value="0.05" />
-	<xacro:property name="y_negative" value="-0.05" />
         <xacro:macro name="reference_frame_foot" params="parent name x y">
 	<!-- macro for one reference frame in foot -->
@@ -14,12 +10,12 @@
 		</joint>
 	</xacro:macro>
-	<xacro:macro name="references_frame_foot" params="parent name">
+	<xacro:macro name="references_frame_foot" params="parent name mirror_y">
 	<!-- macro for reference frames in foot -->
-		<xacro:reference_frame_foot parent="${parent}" name="${name}_upper_right" x="${x_positive}" y="${y_negative}" />
-		<xacro:reference_frame_foot parent="${parent}" name="${name}_upper_left" x="${x_positive}" y="${y_positive}" />
-		<xacro:reference_frame_foot parent="${parent}" name="${name}_lower_right" x="${x_negative}" y="${y_negative}" />
-		<xacro:reference_frame_foot parent="${parent}" name="${name}_lower_left" x="${x_negative}" y="${y_positive}" />
+		<xacro:reference_frame_foot parent="${parent}" name="${name}_upper_right" x="0.195" y="${mirror_y*-0.09}" />
+		<xacro:reference_frame_foot parent="${parent}" name="${name}_upper_left" x="0.195" y="${mirror_y*0.07}" />
+		<xacro:reference_frame_foot parent="${parent}" name="${name}_lower_right" x="-0.111" y="${mirror_y*-0.09}" />
+		<xacro:reference_frame_foot parent="${parent}" name="${name}_lower_left" x="-0.111" y="${mirror_y*0.07}" />
 	</xacro:macro>
-	<xacro:references_frame_foot parent="l_sole" name="l_foot"/>
-	<xacro:references_frame_foot parent="r_sole" name="r_foot"/>
+	<xacro:references_frame_foot parent="l_sole" name="l_foot" mirror_y="1.0"/>
+	<xacro:references_frame_foot parent="r_sole" name="r_foot" mirror_y="-1.0"/>
 </robot>

File: bigman_urdf/urdf/parts/legs.urdf.xacro (robot description, xacro)
@@ -101,17 +101,23 @@
     </collision>
   </link>
-<xacro:unless value="${GAZEBO_BIGMAN_USES_ACCURATE_FT}">
-      <xacro:include filename="$(find bigman_urdf)/urdf/parts/subparts/simple_feet_DRC_sw1_14/simple_foot_R_DRC_sw1_14.urdf.xacro" />
-</xacro:unless>
-<xacro:if value="${GAZEBO_BIGMAN_USES_ACCURATE_FT}">
-    <link name ="RFootFTSensor">
-      <inertial>
-        <origin xyz="0.0 -0.0 -0.0325" rpy="0 0 0"/>
-        <mass value="0.280"/>
-        <inertia ixx="0.0012944808"  ixy="0.0"  ixz="2.0080105E-4" iyy="0.0015851846" iyz="2.7599327E-4" izz="0.0013326766" />
+  <link name ="RFoot">
+     <inertial>
+        <origin xyz="0.00969210464 -0.0090460227 -0.043062308" rpy="0 0 0"/>
+        <mass value="0.66646684"/>
+        <inertia ixx="0.0012944808"  ixy="-9.2387693E-5"  ixz="2.0080105E-4" iyy="0.0015851846" iyz="2.7599327E-4" izz="0.0013326766" />
       </inertial>
-    </link>
-      <xacro:include filename="$(find bigman_urdf)/urdf/parts/subparts/simple_feet_DRC_sw1_14/accurate_FT_simple_foot_R_DRC_sw1_14.urdf.xacro" />
- </xacro:if>
+    <visual>
+      <origin xyz="0 0 0" rpy="0 0 0"/>
+      <geometry name="RFoot_visual">
+        <mesh filename="package://bigman_urdf/meshes/Foot.STL" scale="0.001 -0.001 0.001"/>
+      </geometry>
+    </visual>
+    <collision>
+      <origin xyz="0 0 0" rpy="0 0 0"/>
+      <geometry name="RFoot_collision">
+        <mesh filename="package://bigman_urdf/meshes/simple/Foot.STL" scale="0.001 -0.001 0.001"/>
+      </geometry>
+    </collision>
+  </link>
 <!-- ********************LEFT LEG******************** -->
   <link name ="LHipMot">
@@ -210,17 +216,23 @@
     </collision>
   </link>
-  <xacro:unless value="${GAZEBO_BIGMAN_USES_ACCURATE_FT}">
-      <xacro:include filename="$(find bigman_urdf)/urdf/parts/subparts/simple_feet_DRC_sw1_14/simple_foot_L_DRC_sw1_14.urdf.xacro" />
-  </xacro:unless>
-  <xacro:if value="${GAZEBO_BIGMAN_USES_ACCURATE_FT}">
-    <link name ="LFootFTSensor">
+  <link name ="LFoot">
       <inertial>
-        <origin xyz="0.0 -0.0 -0.0325" rpy="0 0 0"/>
-        <mass value="0.280"/>
-        <inertia ixx="0.0012944808"  ixy="-9.2387693E-5"  ixz="2.0080105E-4" iyy="0.0015851846" iyz="2.7599327E-4" izz="0.0013326766" />
+        <origin xyz="0.0096921046 0.0090460227 -0.043062308" rpy="0 0 0"/>
+        <mass value="0.66646684"/>
+        <inertia ixx="0.0012944808"  ixy="9.2387693E-5"  ixz="2.0080105E-4" iyy="0.0015851846" iyz="-2.7599327E-4" izz="0.0013326766" />
       </inertial>
-    </link>
-      <xacro:include filename="$(find bigman_urdf)/urdf/parts/subparts/simple_feet_DRC_sw1_14/accurate_FT_simple_foot_L_DRC_sw1_14.urdf.xacro" />
-  </xacro:if>
+      <visual>
+      <origin xyz="0 0 0" rpy="0 0 0"/>
+      <geometry name="LFoot_visual">
+        <mesh filename="package://bigman_urdf/meshes/Foot.STL" scale="0.001 0.001 0.001"/>
+      </geometry>
+    </visual>
+    <collision>
+      <origin xyz="0 0 0" rpy="0 0 0"/>
+      <geometry name="LFoot_collision">
+        <mesh filename="package://bigman_urdf/meshes/simple/Foot.STL" scale="0.001 0.001 0.001"/>
+      </geometry>
+    </collision>
+   </link>
 <!-- JOINTS -->
 <!-- ********************RIGHT LEG******************** -->
@@ -265,5 +277,4 @@
     <dynamics friction="0" damping="3.0"/>
   </joint>
- <xacro:unless value="${GAZEBO_BIGMAN_USES_ACCURATE_FT}">
     <joint name="RAnkSag" type="revolute">
       <parent link="RFootmot"/>
@@ -274,23 +285,4 @@
       <dynamics friction="0" damping="3.0"/>
     </joint>
-  </xacro:unless>
-  <xacro:if value="${GAZEBO_BIGMAN_USES_ACCURATE_FT}">
-    <joint name="RAnkSag" type="revolute">
-      <parent link="RFootmot"/>
-      <child link="RFootFTSensor"/>
-      <origin xyz="0.0 0.0 0.0" rpy="0 0 0" />
-      <axis xyz="0 1 0" />
-      <limit velocity="4.0" effort="50" lower="-1.2217" upper="1.2217" />
-      <dynamics friction="0" damping="3.0"/>
-    </joint>
-    <joint name="RAnkSagFT" type="revolute">
-      <parent link="RFootFTSensor"/>
-      <child link="RFoot"/>
-      <origin xyz="0.0 0.0 -0.065" rpy="0 0 0" />
-      <axis xyz="0 1 0" />
-      <limit velocity="0.0" effort="0" lower="-0.0" upper="0.0" />
-      <dynamics friction="0" damping="3.0"/>
-    </joint>
-  </xacro:if>
 <!-- ********************LEFT LEG******************** -->
   <joint name="LHipSag" type="revolute">
@@ -334,31 +326,11 @@
     <dynamics friction="0" damping="3.0"/>
   </joint>
-<xacro:unless value="${GAZEBO_BIGMAN_USES_ACCURATE_FT}">
-    <joint name="LAnkSag" type="revolute">
-      <parent link="LFootmot"/>
-      <child link="LFoot"/>
-      <origin xyz="0.0 0.0 0.0" rpy="0 0 0" />
-      <axis xyz="0 1 0" />
-      <limit velocity="4.0" effort="50" lower="-1.2217" upper="1.2217" />
-      <dynamics friction="0" damping="3.0"/>
-    </joint>
-  </xacro:unless>
-  <xacro:if value="${GAZEBO_BIGMAN_USES_ACCURATE_FT}">
-    <joint name="LAnkSag" type="revolute">
-      <parent link="LFootmot"/>
-      <child link="LFootFTSensor"/>
-      <origin xyz="0.0 0.0 0.0" rpy="0 0 0" />
-      <axis xyz="0 1 0" />
-      <limit velocity="4.0" effort="50" lower="-1.2217" upper="1.2217" />
-      <dynamics friction="0" damping="3.0"/>
-    </joint>
-    <joint name="LAnkSagFT" type="revolute">
-      <parent link="LFootFTSensor"/>
-      <child link="LFoot"/>
-      <origin xyz="0.0 0.0 -0.065" rpy="0 0 0" />
-      <axis xyz="0 1 0" />
-      <limit velocity="0.0" effort="0" lower="-0.0" upper="0.0" />
-      <dynamics friction="0" damping="3.0"/>
-    </joint>
-  </xacro:if>
+  <joint name="LAnkSag" type="revolute">
+    <parent link="LFootmot"/>
+    <child link="LFoot"/>
+    <origin xyz="0.0 0.0 0.0" rpy="0 0 0" />
+    <axis xyz="0 1 0" />
+    <limit velocity="4.0" effort="50" lower="-1.2217" upper="1.2217" />
+    <dynamics friction="0" damping="3.0"/>
+  </joint>
 </robot>

Commit message: Moved pelvis weight bench in parts, added variable mass.

File: bigman_urdf/urdf/bigman_base.urdf.xacro (robot description, xacro)
@@ -35,4 +35,8 @@
     <origin xyz="0 0 0" rpy="0 0 0" />
 </joint>
+<xacro:if value="${BIGMAN_ONLY_LEGS}">
+       <!-- ********************FAKE TORSO******************** -->
+       <xacro:include filename="$(find bigman_urdf)/urdf/parts/pelvis_weight_bench.urdf.xacro" />
+</xacro:if>
 <xacro:unless value="${BIGMAN_ONLY_LEGS}">
        <!-- ********************TORSO******************** -->

File: bigman_urdf/urdf/parts/legs.urdf.xacro (robot description, xacro)
@@ -7,25 +7,4 @@
 <xacro:property name="PI_2" value="1.57079632679" />
 <!-- LINKS -->
-<xacro:if value="${BIGMAN_ONLY_LEGS}">
-<link name ="PelvisWeightBench">
-    <inertial>
-      <origin xyz="0.0 0.0 ${1.8846109e+02*mmTom}" rpy="0 0 0"/>
-      <mass value="5.5278386"/>
-      <inertia ixx="${1.5195067e+05*mm2Tom2}"  ixy="0.0"  ixz="${-2.4191890e-01*mm2Tom2}" iyy="${1.5213465e+05*mm2Tom2}" iyz="0.0" izz="${5.1389419e+03*mm2Tom2}" />
-    </inertial>
-    <visual>
-      <origin xyz="0 0 0" rpy="0 0 0"/>
-      <geometry name="PelvisWeightBench_visual">
-        <mesh filename="package://bigman_urdf/meshes/PelvisWeightBench.STL" scale="0.001 0.001 0.001" />
-      </geometry>
-    </visual>
-    <collision>
-      <origin xyz="0 0 0" rpy="0 0 0"/>
-      <geometry name="PelvisWeightBench_collision">
-        <mesh filename="package://bigman_urdf/meshes/simple/PelvisWeightBench.STL" scale="0.001 0.001 0.001" />
-      </geometry>
-    </collision>
-</link>
-</xacro:if>
 <!-- ********************RIGHT LEG******************** -->
 <link name ="RHipMot">
@@ -269,11 +248,4 @@
    </link>
 <!-- JOINTS -->
-<xacro:if value="${BIGMAN_ONLY_LEGS}">
-       <joint name="PelvisWeightBench_joint" type="fixed">
-           <parent link="Waist"/>
-           <child link="PelvisWeightBench"/>
-           <origin xyz="-0.035 0 0.075" rpy="0 0 ${PI_2}" />
-       </joint>
-</xacro:if>
 <!-- ********************RIGHT LEG******************** -->
   <joint name="RHipLat" type="revolute">

Commit message: more realistic colors in the urdfs

File: bigman_urdf/urdf/bigman_base.urdf.xacro (robot description, xacro)
@@ -22,4 +22,5 @@
         <mesh filename="package://bigman_urdf/meshes/Waist.STL" scale="0.001 0.001 0.001"/>
       </geometry>
+      <material name="grey"/>
     </visual>
     <collision>

File: bigman_urdf/urdf/parts/arms.urdf.xacro (robot description, xacro)
@@ -19,4 +19,5 @@
         <mesh filename="package://bigman_urdf/meshes/ShoulderPitch.STL" scale="0.001 0.001 0.001" />
       </geometry>
+      <material name="dark_grey"/>
     </visual>
     <collision>
@@ -38,4 +39,5 @@
         <mesh filename="package://bigman_urdf/meshes/TopUpperArm.STL" scale="0.001 0.001 0.001" />
       </geometry>
+      <material name="dark_grey"/>
     </visual>
     <collision>
@@ -57,4 +59,5 @@
         <mesh filename="package://bigman_urdf/meshes/BottomUpperArm.STL" scale="0.001 0.001 0.001" />
       </geometry>
+      <material name="dark_grey"/>
     </visual>
     <collision>
@@ -76,4 +79,5 @@
             <mesh filename="package://bigman_urdf/meshes/Elbow.STL" scale="0.001 0.001 0.001" />
           </geometry>
+	  <material name="dark_grey"/>
         </visual>
         <collision>
@@ -96,4 +100,5 @@
         <mesh filename="package://bigman_urdf/meshes/ShoulderPitch.STL" scale="0.001 -0.001 0.001" />
       </geometry>
+      <material name="dark_grey"/>
     </visual>
     <collision>
@@ -115,4 +120,5 @@
         <mesh filename="package://bigman_urdf/meshes/TopUpperArm.STL" scale="0.001 -0.001 0.001" />
       </geometry>
+      <material name="dark_grey"/>
     </visual>
     <collision>
@@ -134,4 +140,5 @@
         <mesh filename="package://bigman_urdf/meshes/BottomUpperArm.STL" scale="0.001 -0.001 0.001" />
       </geometry>
+      <material name="dark_grey"/>
     </visual>
     <collision>
@@ -153,4 +160,5 @@
             <mesh filename="package://bigman_urdf/meshes/Elbow.STL" scale="0.001 -0.001 0.001" />
           </geometry>
+	  <material name="dark_grey"/>
         </visual>
         <collision>

File: bigman_urdf/urdf/parts/forearms.urdf.xacro (robot description, xacro)
@@ -17,4 +17,5 @@
             <mesh filename="package://bigman_urdf/meshes/Forearm.STL" scale="0.001 -0.001 0.001" />
           </geometry>
+	  <material name="dark_grey"/>
         </visual>
         <collision>
@@ -36,4 +37,5 @@
             <mesh filename="package://bigman_urdf/meshes/ForearmPitch.STL" scale="0.001 -0.001 0.001" />
           </geometry>
+	  <material name="dark_grey"/>
         </visual>
         <collision>
@@ -55,4 +57,5 @@
             <mesh filename="package://bigman_urdf/meshes/RaisingSupport.STL" scale="0.001 -0.001 0.001" />
           </geometry>
+	  <material name="dark_grey"/>
         </visual>
         <collision>
@@ -76,4 +79,5 @@
             <mesh filename="package://bigman_urdf/meshes/ForearmRoll.STL" scale="0.001 -0.001 0.001" />
           </geometry>
+	  <material name="blue"/>
         </visual>
         <collision>
@@ -96,4 +100,5 @@
             <mesh filename="package://bigman_urdf/meshes/Forearm.STL" scale="0.001 0.001 0.001" />
           </geometry>
+	  <material name="dark_grey"/>
         </visual>
         <collision>
@@ -115,4 +120,5 @@
             <mesh filename="package://bigman_urdf/meshes/ForearmPitch.STL" scale="0.001 0.001 0.001" />
           </geometry>
+	  <material name="dark_grey"/>
         </visual>
         <collision>
@@ -134,4 +140,5 @@
             <mesh filename="package://bigman_urdf/meshes/RaisingSupport.STL" scale="0.001 0.001 0.001" />
           </geometry>
+	  <material name="dark_grey"/>
         </visual>
         <collision>
@@ -155,4 +162,5 @@
             <mesh filename="package://bigman_urdf/meshes/ForearmRoll.STL" scale="0.001 0.001 0.001" />
           </geometry>
+	  <material name="blue"/>
         </visual>
         <collision>

File: bigman_urdf/urdf/parts/legs.urdf.xacro (robot description, xacro)
@@ -19,4 +19,5 @@
         <mesh filename="package://bigman_urdf/meshes/HipRoll.STL" scale="0.001 0.001 0.001" />
       </geometry>
+      <material name="dark_grey"/>
     </visual>
     <collision>
@@ -38,4 +39,5 @@
         <mesh filename="package://bigman_urdf/meshes/HipYaw.STL" scale="0.001 0.001 0.001" />
       </geometry>
+      <material name="dark_grey"/>
     </visual>
     <collision>
@@ -57,4 +59,5 @@
         <mesh filename="package://bigman_urdf/meshes/HipPitch.STL" scale="0.001 0.001 0.001" />
       </geometry>
+      <material name="grey"/>
     </visual>
     <collision>
@@ -76,4 +79,5 @@
         <mesh filename="package://bigman_urdf/meshes/KneePitchCalf.STL" scale="0.001 0.001 0.001" />
       </geometry>
+      <material name="dark_grey"/>
     </visual>
     <collision>
@@ -95,4 +99,5 @@
         <mesh filename="package://bigman_urdf/meshes/AnklePitch.STL" scale="0.001 0.001 0.001" />
       </geometry>
+      <material name="dark_grey"/>
     </visual>
     <collision>
@@ -114,4 +119,5 @@
         <mesh filename="package://bigman_urdf/meshes/Foot.STL" scale="0.001 -0.001 0.001"/>
       </geometry>
+      <material name="dark_grey"/>
     </visual>
     <collision>
@@ -138,4 +144,5 @@
         <mesh filename="package://bigman_urdf/meshes/HipRoll.STL" scale="0.001 -0.001 0.001" />
       </geometry>
+      <material name="dark_grey"/>
     </visual>
     <collision>
@@ -157,4 +164,5 @@
         <mesh filename="package://bigman_urdf/meshes/HipYaw.STL" scale="0.001 -0.001 0.001" />
       </geometry>
+      <material name="dark_grey"/>
     </visual>
     <collision>
@@ -176,4 +184,5 @@
         <mesh filename="package://bigman_urdf/meshes/HipPitch.STL" scale="0.001 -0.001 0.001" />
       </geometry>
+      <material name="grey"/>
     </visual>
     <collision>
@@ -195,4 +204,5 @@
         <mesh filename="package://bigman_urdf/meshes/KneePitchCalf.STL" scale="0.001 0.001 0.001" />
       </geometry>
+      <material name="dark_grey"/>
     </visual>
     <collision>
@@ -214,4 +224,5 @@
         <mesh filename="package://bigman_urdf/meshes/AnklePitch.STL" scale="0.001 -0.001 0.001" />
       </geometry>
+      <material name="dark_grey"/>
     </visual>
     <collision>
@@ -233,4 +244,5 @@
         <mesh filename="package://bigman_urdf/meshes/Foot.STL" scale="0.001 0.001 0.001"/>
       </geometry>
+      <material name="dark_grey"/>
     </visual>
     <collision>

File: bigman_urdf/urdf/parts/pelvis_weight_bench.urdf.xacro (robot description, xacro)
@@ -24,4 +24,5 @@
         <mesh filename="package://bigman_urdf/meshes/PelvisWeightBench.STL" scale="0.001 0.001 0.001" />
       </geometry>
+      <material name="grey"/>
     </visual>
     <collision>
@@ -43,4 +44,5 @@
         <cylinder length="${CYLINDER_HEIGHT}" radius="${CYLINDER_RADIUS}"/>
       </geometry>
+      <material name="grey"/>
     </visual>
     <collision>

File: bigman_urdf/urdf/parts/soft_hand.urdf.xacro (robot description, xacro)
@@ -20,4 +20,5 @@
         <mesh filename="package://bigman_urdf/meshes/SoftHandOpen.STL" scale="0.001 0.001 0.001" />
       </geometry>
+      <material name="black"/>
    </visual>
    <collision>
@@ -41,4 +42,5 @@
         <mesh filename="package://bigman_urdf/meshes/SoftHandOpen.STL" scale="0.001 -0.001 0.001" />
       </geometry>
+      <material name="black"/>
    </visual>
    <collision>

File: bigman_urdf/urdf/parts/torso.urdf.xacro (robot description, xacro)
@@ -24,4 +24,5 @@
         <mesh filename="package://bigman_urdf/meshes/TorsoRoll.STL" scale="0.001 0.001 0.001" />
       </geometry>
+      <material name="dark_grey"/>
     </visual>
     <collision>
@@ -43,4 +44,5 @@
         <mesh filename="package://bigman_urdf/meshes/TorsoYawPitch.STL" scale="0.001 0.001 0.001" />
       </geometry>
+      <material name="dark_grey"/>
     </visual>
     <collision>
@@ -67,4 +69,5 @@
 </xacro:unless>
       </geometry>
+      <material name="blue"/>
     </visual>
     <collision>

File: bigman_urdf/urdf/sensors/multisense_sl.urdf.xacro (robot description, xacro)
@@ -16,7 +16,5 @@
                 <mesh filename="package://bigman_urdf/meshes/multisense.STL"/>
             </geometry>
-            <material name="">
-                <color rgba="0.9098 0.44314 0.031373 1" />
-            </material>
+            <material name="dark_grey"/>
         </visual>
   <collision>
@@ -44,7 +42,5 @@
         <mesh filename="package://bigman_urdf/meshes/hokuyo_link.STL"/>
       </geometry>
-      <material name="">
-        <color rgba="0.72941 0.35686 0.023529 1" />
-      </material>
+      <material name="black"/>
     </visual>
   <collision>

Commit message: Added new version of Waist. Updated documentation

File: bigman_urdf/urdf/bigman_base.urdf.xacro (robot description, xacro)
@@ -13,7 +13,7 @@
 <link name="Waist">
     <inertial>
-      <origin xyz="${-3.2862932e+01*mmTom} ${-5.0930727e-01*mmTom} ${-1.2899617*mmTom}" rpy="0.0 0.0 0.0"/>
-      <mass value="6.4080904"/>
-      <inertia ixx="${3.8826078e+04*mm2Tom2}"  ixy="${2.9047605e+02*mm2Tom2}"  ixz="${6.8975598e+02*mm2Tom2}" iyy="${2.5050374e+04*mm2Tom2}" iyz="${-1.3370623e+01*mm2Tom2}" izz="${4.8055286e+04*mm2Tom2}" />
+      <origin xyz="${-2.2813402e+01*mmTom} ${-7.3935443e-01*mmTom} ${3.0422909e+01*mmTom}" rpy="0.0 0.0 0.0"/>
+      <mass value="1.1046081e+01"/>
+      <inertia ixx="${9.6207978e+04*mm2Tom2}"  ixy="${1.4081043e+02*mm2Tom2}"  ixz="${3.1258127e+03*mm2Tom2}" iyy="${9.8511158e+04*mm2Tom2}" iyz="${1.3938149e+02*mm2Tom2}" izz="${8.6541531e+04*mm2Tom2}" />
     </inertial>
     <visual>

File: bigman_urdf/urdf/parts/torso.urdf.xacro (robot description, xacro)
@@ -93,5 +93,5 @@
     <parent link="Waist"/>
     <child link="DWL"/>
-    <origin xyz="0.0715192 0 0.195982" rpy="0 0 0" />
+    <origin xyz="0.1115 0 0.195982" rpy="0 0 0" />
     <axis xyz="${cos_26} 0 ${sin_26}" />
     <limit velocity="6.283" effort="120" lower="${-35.0*toRad}" upper="${35.0*toRad}" />
