Commit message: Added new feet to model. Added new variable in config to set new/old feet (actual default is false). Fixed small error in cog position in old foot.

File: bigman_urdf/urdf/bigman_base.urdf.xacro (robot description, xacro)
@@ -86,10 +86,20 @@
 	    <parent link="l_sole"/>
 	    <child link="l_toe"/>
-	    <origin xyz="0.195 0 0" rpy="0 0 0" />
+           <xacro:unless value="${BIGMAN_NEW_FEET}">
+	      <origin xyz="0.195 0 0" rpy="0 0 0" />
+           </xacro:unless>
+           <xacro:if value="${BIGMAN_NEW_FEET}">
+	      <origin xyz="0.16 0 0" rpy="0 0 0" />
+           </xacro:if>
 	  </joint>
 	  <joint name="r_toe_joint" type="fixed">
 	    <parent link="r_sole"/>
 	    <child link="r_toe"/>
-	    <origin xyz="0.195 0 0" rpy="0 0 0" />
+	    <xacro:unless value="${BIGMAN_NEW_FEET}">
+	      <origin xyz="0.195 0 0" rpy="0 0 0" />
+           </xacro:unless>
+           <xacro:if value="${BIGMAN_NEW_FEET}">
+	      <origin xyz="0.16 0 0" rpy="0 0 0" />
+           </xacro:if>
 	  </joint>
 	<!-- Reference frames in feet -->

File: bigman_urdf/urdf/bigman_config.urdf.xacro (robot description, xacro)
@@ -102,3 +102,14 @@
 -->
 <xacro:property name="BIGMAN_ADD_RAISING_SUPPORT" value="false" />
+<!--
+####################################################
+##
+##  BIGMAN_NEW_FEET
+##  if "true" the new feet with the joint in the middle
+##  are used to the model.
+##
+##
+####################################################
+-->
+<xacro:property name="BIGMAN_NEW_FEET" value="false" />
 </robot>

File: bigman_urdf/urdf/config/bigman_gazebo.urdf.xacro (robot description, xacro)
@@ -102,3 +102,14 @@
 -->
 <xacro:property name="BIGMAN_ADD_RAISING_SUPPORT" value="false" />
+<!--
+####################################################
+##
+##  BIGMAN_NEW_FEET
+##  if "true" the new feet with the joint in the middle
+##  are used to the model.
+##
+##
+####################################################
+-->
+<xacro:property name="BIGMAN_NEW_FEET" value="false" />
 </robot>

File: bigman_urdf/urdf/config/bigman_only_legs.urdf.xacro (robot description, xacro)
@@ -102,3 +102,14 @@
 -->
 <xacro:property name="BIGMAN_ADD_RAISING_SUPPORT" value="false" />
+<!--
+####################################################
+##
+##  BIGMAN_NEW_FEET
+##  if "true" the new feet with the joint in the middle
+##  are used to the model.
+##
+##
+####################################################
+-->
+<xacro:property name="BIGMAN_NEW_FEET" value="true" />
 </robot>

File: bigman_urdf/urdf/config/bigman_only_upper_body.urdf.xacro (robot description, xacro)
@@ -102,3 +102,14 @@
 -->
 <xacro:property name="BIGMAN_ADD_RAISING_SUPPORT" value="false" />
+<!--
+####################################################
+##
+##  BIGMAN_NEW_FEET
+##  if "true" the new feet with the joint in the middle
+##  are used to the model.
+##
+##
+####################################################
+-->
+<xacro:property name="BIGMAN_NEW_FEET" value="false" />
 </robot>

File: bigman_urdf/urdf/config/bigman_only_upper_body_gazebo.urdf.xacro (robot description, xacro)
@@ -102,3 +102,14 @@
 -->
 <xacro:property name="BIGMAN_ADD_RAISING_SUPPORT" value="false" />
+<!--
+####################################################
+##
+##  BIGMAN_NEW_FEET
+##  if "true" the new feet with the joint in the middle
+##  are used to the model.
+##
+##
+####################################################
+-->
+<xacro:property name="BIGMAN_NEW_FEET" value="false" />
 </robot>

File: bigman_urdf/urdf/config/bigman_real.urdf.xacro (robot description, xacro)
@@ -102,3 +102,14 @@
 -->
 <xacro:property name="BIGMAN_ADD_RAISING_SUPPORT" value="false" />
+<!--
+####################################################
+##
+##  BIGMAN_NEW_FEET
+##  if "true" the new feet with the joint in the middle
+##  are used to the model.
+##
+##
+####################################################
+-->
+<xacro:property name="BIGMAN_NEW_FEET" value="false" />
 </robot>

File: bigman_urdf/urdf/parts/foot_reference_frame.urdf.xacro (robot description, xacro)
@@ -10,11 +10,22 @@
 		</joint>
 	</xacro:macro>
-	<xacro:macro name="references_frame_foot" params="parent name mirror_y">
-	<!-- macro for reference frames in foot -->
-		<xacro:reference_frame_foot parent="${parent}" name="${name}_upper_right" x="0.195" y="${mirror_y*-0.07}" />
-		<xacro:reference_frame_foot parent="${parent}" name="${name}_upper_left" x="0.195" y="${mirror_y*0.09}" />
-		<xacro:reference_frame_foot parent="${parent}" name="${name}_lower_right" x="-0.111" y="${mirror_y*-0.07}" />
-		<xacro:reference_frame_foot parent="${parent}" name="${name}_lower_left" x="-0.111" y="${mirror_y*0.09}" />
-	</xacro:macro>
+       <xacro:if value="${BIGMAN_NEW_FEET}">
+              <xacro:macro name="references_frame_foot" params="parent name mirror_y">
+              <!-- macro for reference frames in foot -->
+                     <xacro:reference_frame_foot parent="${parent}" name="${name}_upper_right" x="0.16" y="${mirror_y*-0.07}" />
+                     <xacro:reference_frame_foot parent="${parent}" name="${name}_upper_left" x="0.16" y="${mirror_y*0.09}" />
+                     <xacro:reference_frame_foot parent="${parent}" name="${name}_lower_right" x="-0.16" y="${mirror_y*-0.07}" />
+                     <xacro:reference_frame_foot parent="${parent}" name="${name}_lower_left" x="-0.16" y="${mirror_y*0.09}" />
+              </xacro:macro>
+       </xacro:if>
+       <xacro:unless value="${BIGMAN_NEW_FEET}">
+	       <xacro:macro name="references_frame_foot" params="parent name mirror_y">
+	       <!-- macro for reference frames in foot -->
+		       <xacro:reference_frame_foot parent="${parent}" name="${name}_upper_right" x="0.195" y="${mirror_y*-0.07}" />
+		       <xacro:reference_frame_foot parent="${parent}" name="${name}_upper_left" x="0.195" y="${mirror_y*0.09}" />
+		       <xacro:reference_frame_foot parent="${parent}" name="${name}_lower_right" x="-0.111" y="${mirror_y*-0.07}" />
+		       <xacro:reference_frame_foot parent="${parent}" name="${name}_lower_left" x="-0.111" y="${mirror_y*0.09}" />
+	       </xacro:macro>
+       </xacro:unless>
 	<xacro:references_frame_foot parent="l_sole" name="l_foot" mirror_y="1.0"/>
 	<xacro:references_frame_foot parent="r_sole" name="r_foot" mirror_y="-1.0"/>

File: bigman_urdf/urdf/parts/legs.urdf.xacro (robot description, xacro)
@@ -110,12 +110,24 @@
   <link name ="RFoot">
      <inertial>
-        <origin xyz="0.01282904 -0.00463694 -0.10109499" rpy="0 0 0"/>
-        <mass value="3.33109981"/>
-        <inertia ixx="0.01006627"  ixy="-0.00051955"  ixz="-0.00374069" iyy="0.02882577" iyz="0.00044505" izz="0.02819025" />
+        <xacro:if value="${BIGMAN_NEW_FEET}">
+          <origin xyz="-0.00653584 -0.00479384 -0.10180375" rpy="0 0 0"/>
+          <mass value="3.42638110"/>
+          <inertia ixx="0.01032886"  ixy="-0.00016407"  ixz="-0.00201294" iyy="0.02854025" iyz="0.00046315" izz="0.02799499" />
+        </xacro:if>
+        <xacro:unless value="${BIGMAN_NEW_FEET}">
+          <origin xyz="0.01282904 -0.00463694 -0.10109499" rpy="0 0 0"/>
+          <mass value="3.33109981"/>
+          <inertia ixx="0.01006627"  ixy="-0.00051955"  ixz="-0.00374069" iyy="0.02882577" iyz="0.00044505" izz="0.02819025" />
+        </xacro:unless>
       </inertial>
     <visual>
       <origin xyz="0 0 0" rpy="0 0 0"/>
       <geometry name="RFoot_visual">
-        <mesh filename="package://bigman_urdf/meshes/Foot.STL" scale="0.001 -0.001 0.001"/>
+        <xacro:if value="${BIGMAN_NEW_FEET}">
+              <mesh filename="package://bigman_urdf/meshes/NewFoot.STL" scale="0.001 0.001 0.001"/>
+        </xacro:if>
+        <xacro:unless value="${BIGMAN_NEW_FEET}">
+              <mesh filename="package://bigman_urdf/meshes/Foot.STL" scale="0.001 -0.001 0.001"/>
+        </xacro:unless>
       </geometry>
       <material name="dark_grey"/>
@@ -126,8 +138,16 @@
         <mesh filename="package://bigman_urdf/meshes/simple/Foot.STL" scale="0.001 -0.001 0.001"/>
       </geometry>-->
-     <origin xyz="0.047 -0.01 -0.1359" rpy="0 0 0"/>
-     <geometry>
-       <box size="0.306 0.16 0.015" />
-     </geometry>
+     <xacro:if value="${BIGMAN_NEW_FEET}">
+       <origin xyz="0.005 -0.01 -0.1359" rpy="0 0 0"/>
+       <geometry>
+         <box size="0.32 0.16 0.015" />
+       </geometry>
+     </xacro:if>
+     <xacro:unless value="${BIGMAN_NEW_FEET}">
+       <origin xyz="0.047 -0.01 -0.1359" rpy="0 0 0"/>
+       <geometry>
+         <box size="0.306 0.16 0.015" />
+       </geometry>
+     </xacro:unless>
     </collision>
   </link>
@@ -235,12 +255,24 @@
   <link name ="LFoot">
       <inertial>
-        <origin xyz="0.01282904 -0.00463694 -0.10109499" rpy="0 0 0"/>
-        <mass value="3.33109981"/>
-        <inertia ixx="0.01006627"  ixy="0.00051955"  ixz="-0.00374069" iyy="0.02882577" iyz="-0.00044505" izz="0.02819025" />
+        <xacro:if value="${BIGMAN_NEW_FEET}">
+          <origin xyz="-0.00653584 0.00479384 -0.10180375" rpy="0 0 0"/>
+          <mass value="3.42638110"/>
+          <inertia ixx="0.01032886"  ixy="-0.00016407"  ixz="-0.00201294" iyy="0.02854025" iyz="0.00046315" izz="0.02799499" />
+        </xacro:if>
+        <xacro:unless value="${BIGMAN_NEW_FEET}">
+          <origin xyz="0.01282904 0.00463694 -0.10109499" rpy="0 0 0"/>
+          <mass value="3.33109981"/>
+          <inertia ixx="0.01006627"  ixy="0.00051955"  ixz="-0.00374069" iyy="0.02882577" iyz="-0.00044505" izz="0.02819025" />
+        </xacro:unless>
       </inertial>
       <visual>
       <origin xyz="0 0 0" rpy="0 0 0"/>
       <geometry name="LFoot_visual">
-        <mesh filename="package://bigman_urdf/meshes/Foot.STL" scale="0.001 0.001 0.001"/>
+        <xacro:if value="${BIGMAN_NEW_FEET}">
+              <mesh filename="package://bigman_urdf/meshes/NewFoot.STL" scale="0.001 -0.001 0.001"/>
+        </xacro:if>
+        <xacro:unless value="${BIGMAN_NEW_FEET}">
+              <mesh filename="package://bigman_urdf/meshes/Foot.STL" scale="0.001 0.001 0.001"/>
+        </xacro:unless>
       </geometry>
       <material name="dark_grey"/>
@@ -253,8 +285,16 @@
       </geometry>
       -->
-     <origin xyz="0.047 0.01 -0.1359" rpy="0 0 0"/>
-     <geometry>
-       <box size="0.306 0.16 0.015" />
-     </geometry>
+     <xacro:if value="${BIGMAN_NEW_FEET}">
+       <origin xyz="0.005 0.01 -0.1359" rpy="0 0 0"/>
+       <geometry>
+        <box size="0.32 0.16 0.015" />
+       </geometry>
+     </xacro:if>
+     <xacro:unless value="${BIGMAN_NEW_FEET}">
+       <origin xyz="0.047 0.01 -0.1359" rpy="0 0 0"/>
+       <geometry>
+        <box size="0.306 0.16 0.015" />
+       </geometry>
+     </xacro:unless>
     </collision>
    </link>

Commit message: Added ref frames for optitrack and updated doc

File: bigman_urdf/urdf/bigman_base.urdf.xacro (robot description, xacro)
@@ -109,5 +109,5 @@
        <!-- ********************ARMS******************** -->
        <xacro:include filename="$(find bigman_urdf)/urdf/parts/arms.urdf.xacro" />
-       <xacro:include filename="$(find bigman_urdf)/urdf/parts/wrist_calibration_frames.urdf.xacro" />
+       <xacro:include filename="$(find bigman_urdf)/urdf/parts/calibration_frames.urdf.xacro" />
 </xacro:if>
 </robot>

File: bigman_urdf/urdf/parts/calibration_frames.urdf.xacro (robot description, xacro)
@@ -29,4 +29,28 @@
 </joint>
 <!-- L_WRIST CALIBRATION FRAMES -->
+<joint name="l_wrist_calib_joint_base" type="fixed">
+    <parent link="LWrMot3"/>
+    <child link="l_wrist_calibration_link_base"/>
+    <origin xyz="${0.0*mmTom} ${-55.0*mmTom} ${-49.5*mmTom}" rpy="0 0 ${-M_PI_2}" />
+</joint>
+<link name="l_wrist_calibration_link_base"/>
+<link name="l_wrist_calibration_link_A"/>
+<link name="l_wrist_calibration_link_B"/>
+<link name="l_wrist_calibration_link_C"/>
+<joint name="l_wrist_calib_joint_A" type="fixed">
+    <parent link="l_wrist_calibration_link_base"/>
+    <child link="l_wrist_calibration_link_A"/>
+    <origin xyz="${11.3*mmTom} ${21.2132*mmTom} ${21.2132*mmTom}" rpy="0 0 0" />
+</joint>
+<joint name="l_wrist_calib_joint_B" type="fixed">
+    <parent link="l_wrist_calibration_link_base"/>
+    <child link="l_wrist_calibration_link_B"/>
+    <origin xyz="${11.3*mmTom} ${11.5702*mmTom} ${-13.7888*mmTom}" rpy="0 0 0" />
+</joint>
+<joint name="l_wrist_calib_joint_C" type="fixed">
+    <parent link="l_wrist_calibration_link_base"/>
+    <child link="l_wrist_calibration_link_C"/>
+    <origin xyz="${11.3*mmTom} ${-39.5075*mmTom} ${-6.25738*mmTom}" rpy="0 0 0" />
+</joint>
 <!-- WAIST CALIBRATION FRAMES -->
 <joint name="pelvis_calib_joint_base" type="fixed">
