Commit message: Added missing STLs. Added L/R forearm Inertia, CoM, Mass, Visualization and COllision

File: bigman_urdf/urdf/parts/7DOF_forearms_DRC_14.urdf.xacro (robot description, xacro)
@@ -1,4 +1,6 @@
 <?xml version="1.0"?>
 <robot xmlns:xacro="http://ros.org/wiki/xacro">
+<xacro:property name="mmTom" value="0.001" />
+<xacro:property name="mm2Tom2" value="${0.001*0.001}" />
 <!-- distance from last motor to FT sensor
 		The value needs to be subtracted to the *FOrearmPlate joint z origin,
@@ -9,22 +11,20 @@
 <!-- ****************LINKS**************** -->
 <!-- ****************LEFT FOREARM**************** -->
-      <!-- ## WRONG NUMBERS FOR INERTIAL!!! FIX THEM!! ## -->
-      <!-- In ROBOTRAN this link is named LFARM -->
       <link name ="LForearm">
         <inertial>
-          <origin xyz="0 0 ${-0.085 + Wrj1_to_FT}" rpy="0 0 0"/>
-          <mass value="0.93351655"/>
-          <inertia ixx="0.001"  ixy="0.0"  ixz="0.0" iyy="0.001" iyz="0.0" izz="0.001" />
+          <origin xyz="${1.2625599e-02*mmTom} ${-4.2975381*mmTom} ${4.4717986e+01*mmTom}" rpy="0 0 0"/>
+          <mass value="2.2127686"/>
+          <inertia ixx="${6.5428368e+03*mm2Tom2}"  ixy="${4.1196967e+01*mm2Tom2}"  ixz="${3.2727270*mm2Tom2}" iyy="${5.5878290e+03*mm2Tom2}" iyz="${-4.2088668e+02*mm2Tom2}" izz="${2.4783023e+03*mm2Tom2}" />
         </inertial>
         <visual>
-          <origin xyz="0 0 ${0.015 + Wrj1_to_FT}" rpy="3.14159265359 0 1.570796326795"/>
+          <origin xyz="0 0 0" rpy="0 0 0"/>
           <geometry name="LForearm_visual">
-            <mesh filename="package://bigman_urdf/meshes/collada/forearms/forearm_lowpoly.dae" scale="0.1 0.1 0.1" />
+            <mesh filename="package://bigman_urdf/meshes/Forearm.STL" scale="0.001 0.001 0.001" />
           </geometry>
         </visual>
         <collision>
-          <origin xyz="0 0 ${0.015 + Wrj1_to_FT}" rpy="0 3.14159265359 1.570796326795"/>
+          <origin xyz="0 0 0" rpy="0 0 0"/>
           <geometry name="LForearm_collision">
-            <mesh filename="package://bigman_urdf/meshes/collada/simple/forearms/forearm.stl" scale="1.0 1.0 1.0" />
+            <mesh filename="package://bigman_urdf/meshes/simple/Forearm.STL" scale="0.001 0.001 0.001" />
           </geometry>
         </collision>
@@ -73,22 +73,20 @@
       </link>
 <!-- ****************RIGHT FOREARM**************** -->
-      <!-- ## WRONG NUMBERS FOR INERTIAL!!! FIX THEM!! ## -->
-      <!-- In ROBOTRAN this link is named RFArm -->
       <link name ="RForearm">
         <inertial>
-          <origin xyz="0 0 ${-0.085 + Wrj1_to_FT}" rpy="0 0 0"/>
-          <mass value="0.93351655"/>
-          <inertia ixx="0.001"  ixy="0.0"  ixz="0.0" iyy="0.001" iyz="0.0" izz="0.001" />
+          <origin xyz="${1.2625599e-02*mmTom} ${4.2975381*mmTom} ${4.4717986e+01*mmTom}" rpy="0 0 0"/>
+          <mass value="2.2127686"/>
+          <inertia ixx="${6.5428368e+03*mm2Tom2}"  ixy="${-4.1196967e+01*mm2Tom2}"  ixz="${3.2727270*mm2Tom2}" iyy="${5.5878290e+03*mm2Tom2}" iyz="${4.2088668e+02*mm2Tom2}" izz="${2.4783023e+03*mm2Tom2}" />
         </inertial>
         <visual>
-          <origin xyz="0 0 ${0.015 + Wrj1_to_FT}" rpy="3.14159265359 0 1.570796326795"/>
+          <origin xyz="0 0 0" rpy="0 0 0"/>
           <geometry name="RForearm_visual">
-            <mesh filename="package://bigman_urdf/meshes/collada/forearms/forearm_lowpoly.dae" scale="0.1 0.1 0.1" />
+            <mesh filename="package://bigman_urdf/meshes/Forearm.STL" scale="0.001 -0.001 0.001" />
           </geometry>
         </visual>
         <collision>
-          <origin xyz="0 0 ${0.015 + Wrj1_to_FT}" rpy="0 3.14159265359 1.570796326795"/>
+          <origin xyz="0 0 0" rpy="0 0 0"/>
           <geometry name="RForearm_collision">
-            <mesh filename="package://bigman_urdf/meshes/collada/simple/forearms/forearm.stl" scale="1.0 1.0 1.0" />
+            <mesh filename="package://bigman_urdf/meshes/simple/Forearm.STL" scale="0.001 -0.001 0.001" />
           </geometry>
         </collision>
@@ -141,7 +139,7 @@
     <parent link="LElb"/>
     <child link="LForearm"/>
-    <origin xyz="-0.015 0.0 ${-0.051 - Wrj1_to_FT}" rpy="0 0 0"/>
+    <origin xyz="-0.075 0.0 -0.1955" rpy="0 0 0"/>
     <axis xyz="0 0 1" />
-    <limit velocity="4.0" effort="5" lower="-1.5708" upper="1.5708" />
+    <limit velocity="6.283" effort="60" lower="-2.529" upper="2.529" />
     <dynamics friction="0" damping="0.03"/>
   </joint>
@@ -171,7 +169,7 @@
     <parent link="RElb"/>
     <child link="RForearm"/>
-    <origin xyz="-0.015 0.0 ${-0.051 - Wrj1_to_FT}" rpy="0 0 0"/>
+    <origin xyz="-0.075 0.0 -0.1955" rpy="0 0 0"/>
     <axis xyz="0 0 1" />
-    <limit velocity="4.0" effort="5" lower="-1.5708" upper="1.5708" />
+    <limit velocity="6.283" effort="60" lower="-2.529" upper="2.529" />
     <dynamics friction="0" damping="0.03"/>
   </joint>

Commit message: Added Missing STLs, Added L/R forearm pitch Visual, COllision, Mass, inertia and com. Fixed wrong dynamic parameter in previous links.

File: bigman_urdf/urdf/parts/7DOF_forearms_DRC_14.urdf.xacro (robot description, xacro)
@@ -13,12 +13,12 @@
       <link name ="LForearm">
         <inertial>
-          <origin xyz="${1.2625599e-02*mmTom} ${-4.2975381*mmTom} ${4.4717986e+01*mmTom}" rpy="0 0 0"/>
+          <origin xyz="${1.2625599e-02*mmTom} ${4.2975381*mmTom} ${4.4717986e+01*mmTom}" rpy="0 0 0"/>
           <mass value="2.2127686"/>
-          <inertia ixx="${6.5428368e+03*mm2Tom2}"  ixy="${4.1196967e+01*mm2Tom2}"  ixz="${3.2727270*mm2Tom2}" iyy="${5.5878290e+03*mm2Tom2}" iyz="${-4.2088668e+02*mm2Tom2}" izz="${2.4783023e+03*mm2Tom2}" />
+          <inertia ixx="${6.5428368e+03*mm2Tom2}"  ixy="${-4.1196967e+01*mm2Tom2}"  ixz="${3.2727270*mm2Tom2}" iyy="${5.5878290e+03*mm2Tom2}" iyz="${4.2088668e+02*mm2Tom2}" izz="${2.4783023e+03*mm2Tom2}" />
         </inertial>
         <visual>
           <origin xyz="0 0 0" rpy="0 0 0"/>
           <geometry name="LForearm_visual">
-            <mesh filename="package://bigman_urdf/meshes/Forearm.STL" scale="0.001 0.001 0.001" />
+            <mesh filename="package://bigman_urdf/meshes/Forearm.STL" scale="0.001 -0.001 0.001" />
           </geometry>
         </visual>
@@ -26,26 +26,24 @@
           <origin xyz="0 0 0" rpy="0 0 0"/>
           <geometry name="LForearm_collision">
-            <mesh filename="package://bigman_urdf/meshes/simple/Forearm.STL" scale="0.001 0.001 0.001" />
+            <mesh filename="package://bigman_urdf/meshes/simple/Forearm.STL" scale="0.001 -0.001 0.001" />
           </geometry>
         </collision>
       </link>
-      <!-- ## WRONG NUMBERS FOR INERTIAL!!! FIX THEM!! ## -->
-      <!-- Here I have used the inertia of a full cylinder with r = 0.02 [m] and h = 0.07 [m] -->
       <link name="LWrMot2">
         <inertial>
-          <origin xyz="0 0 0" rpy="0 0 0"/>
-          <mass value="0.26070556"/>
-          <inertia ixx="0.000132"  ixy="0"  ixz="0" iyy="0.000132" iyz="0" izz="5.213E-5" />
+          <origin xyz="${9.8193770*mmTom} ${1.3797184*mmTom} ${-8.0380065e+01*mmTom}" rpy="0 0 0"/>
+          <mass value="1.2838072"/>
+          <inertia ixx="${1.9941240e+03*mm2Tom2}"  ixy="${2.5697060e+01*mm2Tom2}"  ixz="${1.7443538e+02*mm2Tom2}" iyy="${2.1755329e+03*mm2Tom2}" iyz="${-1.2100987e+02*mm2Tom2}" izz="${1.8303760e+03*mm2Tom2}" />
         </inertial>
         <visual>
-          <origin xyz="0.025 0 0" rpy="0 1.570796326795 3.14159265359"/>
+          <origin xyz="0 0 0" rpy="0 0 0"/>
           <geometry name="LWrMot2_visual">
-            <mesh filename="package://bigman_urdf/meshes/collada/forearms/fa_asm_3_right_sw0001.dae" scale="0.001 0.001 0.001" />
+            <mesh filename="package://bigman_urdf/meshes/ForearmPitch.STL" scale="0.001 -0.001 0.001" />
           </geometry>
         </visual>
         <collision>
-          <origin xyz="0.025 0 0" rpy="0 1.570796326795 3.14159265359"/>
+          <origin xyz="0 0 0" rpy="0 0 0"/>
           <geometry name="LWrMot2_collision">
-            <mesh filename="package://bigman_urdf/meshes/collada/simple/forearms/simple_fa_asm_3_right_sw0001.stl" scale="0.001 0.001 0.001" />
+            <mesh filename="package://bigman_urdf/meshes/simple/ForearmPitch.STL" scale="0.001 -0.001 0.001" />
           </geometry>
         </collision>
@@ -75,12 +73,12 @@
       <link name ="RForearm">
         <inertial>
-          <origin xyz="${1.2625599e-02*mmTom} ${4.2975381*mmTom} ${4.4717986e+01*mmTom}" rpy="0 0 0"/>
+          <origin xyz="${1.2625599e-02*mmTom} ${-4.2975381*mmTom} ${4.4717986e+01*mmTom}" rpy="0 0 0"/>
           <mass value="2.2127686"/>
-          <inertia ixx="${6.5428368e+03*mm2Tom2}"  ixy="${-4.1196967e+01*mm2Tom2}"  ixz="${3.2727270*mm2Tom2}" iyy="${5.5878290e+03*mm2Tom2}" iyz="${4.2088668e+02*mm2Tom2}" izz="${2.4783023e+03*mm2Tom2}" />
+          <inertia ixx="${6.5428368e+03*mm2Tom2}"  ixy="${4.1196967e+01*mm2Tom2}"  ixz="${3.2727270*mm2Tom2}" iyy="${5.5878290e+03*mm2Tom2}" iyz="${-4.2088668e+02*mm2Tom2}" izz="${2.4783023e+03*mm2Tom2}" />
         </inertial>
         <visual>
           <origin xyz="0 0 0" rpy="0 0 0"/>
           <geometry name="RForearm_visual">
-            <mesh filename="package://bigman_urdf/meshes/Forearm.STL" scale="0.001 -0.001 0.001" />
+            <mesh filename="package://bigman_urdf/meshes/Forearm.STL" scale="0.001 0.001 0.001" />
           </geometry>
         </visual>
@@ -88,26 +86,24 @@
           <origin xyz="0 0 0" rpy="0 0 0"/>
           <geometry name="RForearm_collision">
-            <mesh filename="package://bigman_urdf/meshes/simple/Forearm.STL" scale="0.001 -0.001 0.001" />
+            <mesh filename="package://bigman_urdf/meshes/simple/Forearm.STL" scale="0.001 0.001 0.001" />
           </geometry>
         </collision>
       </link>
-      <!-- ## WRONG NUMBERS FOR INERTIAL!!! FIX THEM!! ## -->
-      <!-- Here I have used the inertia of a full cylinder with r = 0.02 [m] and h = 0.07 [m] -->
       <link name="RWrMot2">
         <inertial>
-          <origin xyz="0 0 0" rpy="0 0 0"/>
-          <mass value="0.26070556"/>
-          <inertia ixx="0.000132"  ixy="0"  ixz="0" iyy="0.000132" iyz="0" izz="5.213E-5" />
+          <origin xyz="${9.8193770*mmTom} ${-1.3797184*mmTom} ${-8.0380065e+01*mmTom}" rpy="0 0 0"/>
+          <mass value="1.2838072"/>
+          <inertia ixx="${1.9941240e+03*mm2Tom2}"  ixy="${-2.5697060e+01*mm2Tom2}"  ixz="${1.7443538e+02*mm2Tom2}" iyy="${2.1755329e+03*mm2Tom2}" iyz="${1.2100987e+02*mm2Tom2}" izz="${1.8303760e+03*mm2Tom2}" />
         </inertial>
         <visual>
-          <origin xyz="0.025 0 0" rpy="0 1.570796326795 3.14159265359"/>
+          <origin xyz="0 0 0" rpy="0 0 0"/>
           <geometry name="RWrMot2_visual">
-            <mesh filename="package://bigman_urdf/meshes/collada/forearms/fa_asm_3_right_sw0001.dae" scale="0.001 0.001 0.001" />
+            <mesh filename="package://bigman_urdf/meshes/ForearmPitch.STL" scale="0.001 0.001 0.001" />
           </geometry>
         </visual>
         <collision>
-          <origin xyz="0.025 0 0" rpy="0 1.570796326795 3.14159265359"/>
+          <origin xyz="0 0 0" rpy="0 0 0"/>
           <geometry name="RWrMot2_collision">
-            <mesh filename="package://bigman_urdf/meshes/collada/simple/forearms/simple_fa_asm_3_right_sw0001.stl" scale="0.001 0.001 0.001" />
+            <mesh filename="package://bigman_urdf/meshes/simple/ForearmPitch.STL" scale="0.001 0.001 0.001" />
           </geometry>
         </collision>
@@ -147,7 +143,7 @@
     <parent link="LForearm"/>
     <child link="LWrMot2"/>
-    <origin xyz="0 0 ${-0.14368 + Wrj1_to_FT}" rpy="0 0 0"/>
+    <origin xyz="0 0 0" rpy="0 0 0"/>
     <axis xyz="0 1 0"/>
-    <limit velocity="4.0" effort="5" lower="-0.524" upper="0.524" />
+    <limit velocity="6.283" effort="60" lower="-1.48" upper="1.48" />
     <dynamics friction="0" damping="0.03"/>
   </joint>
@@ -155,7 +151,7 @@
     <parent link="LWrMot2"/>
     <child link="LWrMot3"/>
-    <origin xyz="0 0 0.0" rpy="0 0 0"/>
+    <origin xyz="0 0 -0.092" rpy="0 0 0"/>
     <axis xyz="1 0 0"/>
-    <limit velocity="4.0" effort="5" lower="-0.785375" upper="1.395" />
+    <limit velocity="6.283" effort="60" lower="-0.785375" upper="1.395" />
     <dynamics friction="0" damping="0.03"/>
   </joint>
@@ -177,7 +173,7 @@
     <parent link="RForearm"/>
     <child link="RWrMot2"/>
-    <origin xyz="0 0 ${-0.14368 + Wrj1_to_FT}" rpy="0 0 0"/>
+    <origin xyz="0 0 0" rpy="0 0 0"/>
     <axis xyz="0 1 0"/>
-    <limit velocity="4.0" effort="5" lower="-0.524" upper="0.524" />
+    <limit velocity="6.283" effort="60" lower="-1.48" upper="1.48" />
     <dynamics friction="0" damping="0.03"/>
   </joint>
@@ -185,7 +181,7 @@
     <parent link="RWrMot2"/>
     <child link="RWrMot3"/>
-    <origin xyz="0 0 0.0" rpy="0 0 0"/>
+    <origin xyz="0 0 -0.092" rpy="0 0 0"/>
     <axis xyz="1 0 0"/>
-    <limit velocity="4.0" effort="5" lower="-1.395" upper="0.785375" />
+    <limit velocity="6.283" effort="60" lower="-1.395" upper="0.785375" />
     <dynamics friction="0" damping="0.03"/>
   </joint>

Commit message: Added L/R forearm pitch collision, visualization, CoM, Mass and Inertia

File: bigman_urdf/urdf/parts/7DOF_forearms_DRC_14.urdf.xacro (robot description, xacro)
@@ -49,22 +49,20 @@
         </collision>
       </link>
-      <!-- ## WRONG NUMBERS FOR INERTIAL!!! FIX THEM!! ## -->
-      <!-- Here I have used the inertia of a concave cylinder with r = 0.02 [m] -->
       <link name="LWrMot3">
         <inertial>
-          <origin xyz="0 0 0" rpy="0 0 0"/>
-          <mass value="0.054007518"/>
-          <inertia ixx="2.16E-5"  ixy="0"  ixz="0" iyy="2.16E-5" iyz="0" izz="2.16E-5" />
+          <origin xyz="${7.0380706*mmTom} ${-1.0811188e-02*mmTom} ${-3.9669274e+01*mmTom}" rpy="0 0 0"/>
+          <mass value="4.2801447e-01"/>
+          <inertia ixx="${2.8620156e+02*mm2Tom2}"  ixy="${5.2570457e-02*mm2Tom2}"  ixz="${-3.9174213e+01*mm2Tom2}" iyy="${7.1261855e+02*mm2Tom2}" iyz="${-9.5020266e-02*mm2Tom2}" izz="${6.1444258e+02*mm2Tom2}" />
         </inertial>
         <visual>
-          <origin xyz="0.025 -0.012 -0.02" rpy="0 3.14159265359 1.570796326795"/>
+          <origin xyz="0 0 0" rpy="0 0 0"/>
           <geometry name="LWrMot3_visual">
-            <mesh filename="package://bigman_urdf/meshes/collada/forearms/fa_hand_interface_rig_sw0001.dae" scale="0.001 0.001 0.001" />
+            <mesh filename="package://bigman_urdf/meshes/ForearmRoll.STL" scale="0.001 -0.001 0.001" />
           </geometry>
         </visual>
         <collision>
-          <origin xyz="0.025 -0.012 -0.02" rpy="0 3.14159265359 1.570796326795"/>
+          <origin xyz="0 0 0" rpy="0 0 0"/>
           <geometry name="LWrMot3_collision">
-            <mesh filename="package://bigman_urdf/meshes/collada/simple/forearms/simple_fa_hand_interface_rig_sw0001.stl" scale="0.001 0.001 0.001" />
+            <mesh filename="package://bigman_urdf/meshes/simple/ForearmRoll.STL" scale="0.001 -0.001 0.001" />
           </geometry>
         </collision>
@@ -109,22 +107,20 @@
         </collision>
       </link>
-      <!-- ## WRONG NUMBERS FOR INERTIAL!!! FIX THEM!! ## -->
-      <!-- Here I have used the inertia of a concave cylinder with r = 0.02 [m] -->
       <link name="RWrMot3">
         <inertial>
-          <origin xyz="0 0 0" rpy="0 0 0"/>
-          <mass value="0.054007518"/>
-          <inertia ixx="2.16E-5"  ixy="0"  ixz="0" iyy="2.16E-5" iyz="0" izz="2.16E-5" />
+          <origin xyz="${7.0380706*mmTom} ${1.0811188e-02*mmTom} ${-3.9669274e+01*mmTom}" rpy="0 0 0"/>
+          <mass value="4.2801447e-01"/>
+          <inertia ixx="${2.8620156e+02*mm2Tom2}"  ixy="${-5.2570457e-02*mm2Tom2}"  ixz="${-3.9174213e+01*mm2Tom2}" iyy="${7.1261855e+02*mm2Tom2}" iyz="${9.5020266e-02*mm2Tom2}" izz="${6.1444258e+02*mm2Tom2}" />
         </inertial>
         <visual>
-          <origin xyz="0.025 -0.012 -0.02" rpy="0 3.14159265359 1.570796326795"/>
+          <origin xyz="0 0 0" rpy="0 0 0"/>
           <geometry name="RWrMot3_visual">
-            <mesh filename="package://bigman_urdf/meshes/collada/forearms/fa_hand_interface_rig_sw0001.dae" scale="0.001 0.001 0.001" />
+            <mesh filename="package://bigman_urdf/meshes/ForearmRoll.STL" scale="0.001 0.001 0.001" />
           </geometry>
         </visual>
         <collision>
-          <origin xyz="0.025 -0.012 -0.02" rpy="0 3.14159265359 1.570796326795"/>
+          <origin xyz="0 0 0" rpy="0 0 0"/>
           <geometry name="RWrMot3_collision">
-            <mesh filename="package://bigman_urdf/meshes/collada/simple/forearms/simple_fa_hand_interface_rig_sw0001.stl" scale="0.001 0.001 0.001" />
+            <mesh filename="package://bigman_urdf/meshes/simple/ForearmRoll.STL" scale="0.001 0.001 0.001" />
           </geometry>
         </collision>
@@ -153,5 +149,5 @@
     <origin xyz="0 0 -0.092" rpy="0 0 0"/>
     <axis xyz="1 0 0"/>
-    <limit velocity="6.283" effort="60" lower="-0.785375" upper="1.395" />
+    <limit velocity="6.283" effort="60" lower="-1.48" upper="1.48" />
     <dynamics friction="0" damping="0.03"/>
   </joint>
@@ -183,5 +179,5 @@
     <origin xyz="0 0 -0.092" rpy="0 0 0"/>
     <axis xyz="1 0 0"/>
-    <limit velocity="6.283" effort="60" lower="-1.395" upper="0.785375" />
+    <limit velocity="6.283" effort="60" lower="-1.48" upper="1.48" />
     <dynamics friction="0" damping="0.03"/>
   </joint>
