Commit message: Added new documentation. Added proper Inertia, Mass and CoM for sticks. Added reference frames.

File: bigman_urdf/urdf/parts/forearm_reference_frame.urdf.xacro (robot description, xacro)
@@ -1,10 +1,12 @@
 <?xml version="1.0"?>
 <robot xmlns:xacro="http://ros.org/wiki/xacro">
-       <xacro:property name="x_positive" value="0.08" />
-	<xacro:property name="x_negative" value="-0.08" />
-       <xacro:macro name="reference_frame_forearm" params="parent name x">
+       <xacro:property name="x_positive" value="0.097" />
+	<xacro:property name="x_negative" value="-0.081" />
+       <xacro:property name="z_offset" value="-0.132" />
+       <xacro:property name="ball_radius" value="0.02" />
+       <xacro:macro name="reference_frame_forearm" params="parent name x z">
 		<link name="${name}_link"/>
 		<joint name="${name}_joint" type="fixed">
-			<origin xyz="${x} 0 -0.07" rpy="0 0 0" />
+			<origin xyz="${x} 0 ${z}" rpy="0 0 0" />
 			<parent link="${parent}"/>
 			<child link="${name}_link"/>
@@ -12,7 +14,7 @@
 	</xacro:macro>
        <xacro:macro name="references_frame_forearm" params="parent name">
-		<xacro:reference_frame_forearm parent="${parent}" name="${name}_forward_contact" x="${x_positive}" />
-		<xacro:reference_frame_forearm parent="${parent}" name="${name}_backward_contact" x="${x_negative}" />
-              <xacro:reference_frame_forearm parent="${parent}" name="${name}_central_contact" x="0.0" />
+		<xacro:reference_frame_forearm parent="${parent}" name="${name}_forward_contact" x="${x_positive}" z="${z_offset}" />
+		<xacro:reference_frame_forearm parent="${parent}" name="${name}_backward_contact" x="${x_negative}" z="${z_offset}"/>
+              <xacro:reference_frame_forearm parent="${parent}" name="${name}_central_contact" x="0.0" z="${z_offset-ball_radius}"/>
 	</xacro:macro>
        <xacro:references_frame_forearm parent="LRaisingSupport" name="l_forearm"/>

File: bigman_urdf/urdf/parts/forearms.urdf.xacro (robot description, xacro)
@@ -3,4 +3,5 @@
 <xacro:property name="mmTom" value="0.001" />
 <xacro:property name="mm2Tom2" value="${0.001*0.001}" />
+<xacro:property name="tonsToKg" value="1000.0" />
 <!-- ****************LINKS**************** -->
 <!-- ****************LEFT FOREARM**************** -->
@@ -25,4 +26,9 @@
       </link>
       <link name="LRaisingSupport">
+        <inertial>
+          <origin xyz="${7.2667838*mmTom} ${1.2370624*mmTom} ${-6.9076044e+01*mmTom}" rpy="0 0 0"/>
+          <mass value="${1.3789343e-03*tonsToKg}"/>
+          <inertia ixx="${5.9368721*mm2Tom2*tonsToKg}"  ixy="${1.6171173e-02*mm2Tom2*tonsToKg}"  ixz="${4.7369581e-02*mm2Tom2*tonsToKg}" iyy="${1.3268985e+01*mm2Tom2*tonsToKg}" iyz="${-1.3188343e-01*mm2Tom2*tonsToKg}" izz="${9.5878298*mm2Tom2*tonsToKg}" />
+        </inertial>
         <visual>
           <origin xyz="0 0 0" rpy="0 0 0"/>
@@ -97,4 +103,9 @@
       </link>
       <link name="RRaisingSupport">
+        <inertial>
+          <origin xyz="${7.2667838*mmTom} ${-1.2370624*mmTom} ${-6.9076044e+01*mmTom}" rpy="0 0 0"/>
+          <mass value="${1.3789343e-03*tonsToKg}"/>
+          <inertia ixx="${5.9368721*mm2Tom2*tonsToKg}"  ixy="${-1.6171173e-02*mm2Tom2*tonsToKg}"  ixz="${4.7369581e-02*mm2Tom2*tonsToKg}" iyy="${1.3268985e+01*mm2Tom2*tonsToKg}" iyz="${1.3188343e-01*mm2Tom2*tonsToKg}" izz="${9.5878298*mm2Tom2*tonsToKg}" />
+        </inertial>
         <visual>
           <origin xyz="0 0 0" rpy="0 0 0"/>
