Commit message: Starting adding RaisingSupports

File: bigman_urdf/urdf/parts/forearms.urdf.xacro (robot description, xacro)
@@ -24,4 +24,18 @@
         </collision>
       </link>
+      <link name="LRaisingSupport">
+        <visual>
+          <origin xyz="0 0 0" rpy="0 0 0"/>
+          <geometry name="LRaisingSupport_visual">
+            <mesh filename="package://bigman_urdf/meshes/RaisingSupport.STL" scale="0.001 -0.001 0.001" />
+          </geometry>
+        </visual>
+        <collision>
+          <origin xyz="0 0 0" rpy="0 0 0"/>
+          <geometry name="LRaisingSupport_collision">
+            <mesh filename="package://bigman_urdf/meshes/simple/RaisingSupport.STL" scale="0.001 -0.001 0.001" />
+          </geometry>
+        </collision>
+      </link>
       <link name="LWrMot2">
         <inertial>
@@ -79,4 +93,18 @@
           <geometry name="RForearm_collision">
             <mesh filename="package://bigman_urdf/meshes/simple/Forearm.STL" scale="0.001 0.001 0.001" />
+          </geometry>
+        </collision>
+      </link>
+      <link name="RRaisingSupport">
+        <visual>
+          <origin xyz="0 0 0" rpy="0 0 0"/>
+          <geometry name="RRaisingSupport_visual">
+            <mesh filename="package://bigman_urdf/meshes/RaisingSupport.STL" scale="0.001 0.001 0.001" />
+          </geometry>
+        </visual>
+        <collision>
+          <origin xyz="0 0 0" rpy="0 0 0"/>
+          <geometry name="RRaisingSupport_collision">
+            <mesh filename="package://bigman_urdf/meshes/simple/RaisingSupport.STL" scale="0.001 0.001 0.001" />
           </geometry>
         </collision>
@@ -129,4 +157,9 @@
     <limit velocity="6.283" effort="60" lower="-2.529" upper="2.529" />
     <dynamics friction="0" damping="0.03"/>
+  </joint>
+  <joint name="LRaisingSupport_joint" type="fixed">
+    <parent link="LForearm"/>
+    <child link="LRaisingSupport"/>
+    <origin xyz="0.0 0.0 -0.0505" rpy="0 0 0"/>
   </joint>
   <joint name="LWrj1" type="revolute">
@@ -160,4 +193,9 @@
     <dynamics friction="0" damping="0.03"/>
   </joint>
+  <joint name="RRaisingSupport_joint" type="fixed">
+    <parent link="RForearm"/>
+    <child link="RRaisingSupport"/>
+    <origin xyz="0.0 0.0 -0.0505" rpy="0 0 0"/>
+  </joint>
   <joint name="RWrj1" type="revolute">
     <parent link="RForearm"/>

Commit message: Added SoftHands, fixed bug in sticks

File: bigman_urdf/urdf/parts/forearms.urdf.xacro (robot description, xacro)
@@ -25,4 +25,23 @@
         </collision>
       </link>
+      <link name="LWrMot2">
+        <inertial>
+          <origin xyz="${9.8193770*mmTom} ${1.3797184*mmTom} ${-8.0380065e+01*mmTom}" rpy="0 0 0"/>
+          <mass value="1.2838072"/>
+          <inertia ixx="${1.9941240e+03*mm2Tom2}"  ixy="${2.5697060e+01*mm2Tom2}"  ixz="${1.7443538e+02*mm2Tom2}" iyy="${2.1755329e+03*mm2Tom2}" iyz="${-1.2100987e+02*mm2Tom2}" izz="${1.8303760e+03*mm2Tom2}" />
+        </inertial>
+        <visual>
+          <origin xyz="0 0 0" rpy="0 0 0"/>
+          <geometry name="LWrMot2_visual">
+            <mesh filename="package://bigman_urdf/meshes/ForearmPitch.STL" scale="0.001 -0.001 0.001" />
+          </geometry>
+        </visual>
+        <collision>
+          <origin xyz="0 0 0" rpy="0 0 0"/>
+          <geometry name="LWrMot2_collision">
+            <mesh filename="package://bigman_urdf/meshes/simple/ForearmPitch.STL" scale="0.001 -0.001 0.001" />
+          </geometry>
+        </collision>
+      </link>
       <link name="LRaisingSupport">
         <inertial>
@@ -44,23 +63,4 @@
         </collision>
       </link>
-      <link name="LWrMot2">
-        <inertial>
-          <origin xyz="${9.8193770*mmTom} ${1.3797184*mmTom} ${-8.0380065e+01*mmTom}" rpy="0 0 0"/>
-          <mass value="1.2838072"/>
-          <inertia ixx="${1.9941240e+03*mm2Tom2}"  ixy="${2.5697060e+01*mm2Tom2}"  ixz="${1.7443538e+02*mm2Tom2}" iyy="${2.1755329e+03*mm2Tom2}" iyz="${-1.2100987e+02*mm2Tom2}" izz="${1.8303760e+03*mm2Tom2}" />
-        </inertial>
-        <visual>
-          <origin xyz="0 0 0" rpy="0 0 0"/>
-          <geometry name="LWrMot2_visual">
-            <mesh filename="package://bigman_urdf/meshes/ForearmPitch.STL" scale="0.001 -0.001 0.001" />
-          </geometry>
-        </visual>
-        <collision>
-          <origin xyz="0 0 0" rpy="0 0 0"/>
-          <geometry name="LWrMot2_collision">
-            <mesh filename="package://bigman_urdf/meshes/simple/ForearmPitch.STL" scale="0.001 -0.001 0.001" />
-          </geometry>
-        </collision>
-      </link>
       <link name="LWrMot3">
         <inertial>
@@ -102,4 +102,23 @@
         </collision>
       </link>
+      <link name="RWrMot2">
+        <inertial>
+          <origin xyz="${9.8193770*mmTom} ${-1.3797184*mmTom} ${-8.0380065e+01*mmTom}" rpy="0 0 0"/>
+          <mass value="1.2838072"/>
+          <inertia ixx="${1.9941240e+03*mm2Tom2}"  ixy="${-2.5697060e+01*mm2Tom2}"  ixz="${1.7443538e+02*mm2Tom2}" iyy="${2.1755329e+03*mm2Tom2}" iyz="${1.2100987e+02*mm2Tom2}" izz="${1.8303760e+03*mm2Tom2}" />
+        </inertial>
+        <visual>
+          <origin xyz="0 0 0" rpy="0 0 0"/>
+          <geometry name="RWrMot2_visual">
+            <mesh filename="package://bigman_urdf/meshes/ForearmPitch.STL" scale="0.001 0.001 0.001" />
+          </geometry>
+        </visual>
+        <collision>
+          <origin xyz="0 0 0" rpy="0 0 0"/>
+          <geometry name="RWrMot2_collision">
+            <mesh filename="package://bigman_urdf/meshes/simple/ForearmPitch.STL" scale="0.001 0.001 0.001" />
+          </geometry>
+        </collision>
+      </link>
       <link name="RRaisingSupport">
         <inertial>
@@ -118,23 +137,4 @@
           <geometry name="RRaisingSupport_collision">
             <mesh filename="package://bigman_urdf/meshes/simple/RaisingSupport.STL" scale="0.001 0.001 0.001" />
-          </geometry>
-        </collision>
-      </link>
-      <link name="RWrMot2">
-        <inertial>
-          <origin xyz="${9.8193770*mmTom} ${-1.3797184*mmTom} ${-8.0380065e+01*mmTom}" rpy="0 0 0"/>
-          <mass value="1.2838072"/>
-          <inertia ixx="${1.9941240e+03*mm2Tom2}"  ixy="${-2.5697060e+01*mm2Tom2}"  ixz="${1.7443538e+02*mm2Tom2}" iyy="${2.1755329e+03*mm2Tom2}" iyz="${1.2100987e+02*mm2Tom2}" izz="${1.8303760e+03*mm2Tom2}" />
-        </inertial>
-        <visual>
-          <origin xyz="0 0 0" rpy="0 0 0"/>
-          <geometry name="RWrMot2_visual">
-            <mesh filename="package://bigman_urdf/meshes/ForearmPitch.STL" scale="0.001 0.001 0.001" />
-          </geometry>
-        </visual>
-        <collision>
-          <origin xyz="0 0 0" rpy="0 0 0"/>
-          <geometry name="RWrMot2_collision">
-            <mesh filename="package://bigman_urdf/meshes/simple/ForearmPitch.STL" scale="0.001 0.001 0.001" />
           </geometry>
         </collision>
@@ -169,9 +169,4 @@
     <dynamics friction="0" damping="0.03"/>
   </joint>
-  <joint name="LRaisingSupport_joint" type="fixed">
-    <parent link="LForearm"/>
-    <child link="LRaisingSupport"/>
-    <origin xyz="0.0 0.0 -0.0505" rpy="0 0 0"/>
-  </joint>
   <joint name="LWrj1" type="revolute">
     <parent link="LForearm"/>
@@ -181,4 +176,9 @@
     <limit velocity="6.283" effort="60" lower="-1.48" upper="1.48" />
     <dynamics friction="0" damping="0.03"/>
+  </joint>
+    <joint name="LRaisingSupport_joint" type="fixed">
+    <parent link="LWrMot2"/>
+    <child link="LRaisingSupport"/>
+    <origin xyz="0.0 0.0 -0.0505" rpy="0 0 0"/>
   </joint>
   <joint name="LWrj2" type="revolute">
@@ -204,9 +204,4 @@
     <dynamics friction="0" damping="0.03"/>
   </joint>
-  <joint name="RRaisingSupport_joint" type="fixed">
-    <parent link="RForearm"/>
-    <child link="RRaisingSupport"/>
-    <origin xyz="0.0 0.0 -0.0505" rpy="0 0 0"/>
-  </joint>
   <joint name="RWrj1" type="revolute">
     <parent link="RForearm"/>
@@ -217,4 +212,9 @@
     <dynamics friction="0" damping="0.03"/>
   </joint>
+    <joint name="RRaisingSupport_joint" type="fixed">
+    <parent link="RWrMot2"/>
+    <child link="RRaisingSupport"/>
+    <origin xyz="0.0 0.0 -0.0505" rpy="0 0 0"/>
+  </joint>
   <joint name="RWrj2" type="revolute">
     <parent link="RWrMot2"/>

File: bigman_urdf/urdf/parts/soft_hand.urdf.xacro (robot description, xacro)
@@ -3,5 +3,7 @@
 <xacro:if value="${BIGMAN_FIXED_HANDS}">
 <!-- LINKS -->
-<link name="RSoftHand">
+<link name="RSoftHand"/>
+<link name="r_palm"/>
+<link name="RSoftHandLink">
     <inertial>
       <origin xyz="0 0 0" rpy="0 0 0"/>
@@ -10,17 +12,19 @@
     </inertial>
     <visual>
-      <origin xyz="0.007 0.01 -0.04" rpy="${-3.14159265359/2} 0 ${3.14159265359}"/>
-      <geometry name="RSoftHand_visual">
-        <mesh filename="package://bigman_urdf/meshes/collada/forearms/R_soft_hand_open_lowpoly.dae" scale="0.1 0.1 0.1" />
+      <origin xyz="0.0 0.0 0.0" rpy="0.0 0.0 0.0"/>
+      <geometry name="RSoftHandLink_visual">
+        <mesh filename="package://bigman_urdf/meshes/SoftHandOpen.STL" scale="0.001 0.001 0.001" />
       </geometry>
    </visual>
    <collision>
-      <origin xyz="0 0.01 -0.04" rpy="0 0 3.14159265359"/>
-      <geometry name="RSoftHand_collision">
-        <mesh filename="package://bigman_urdf/meshes/collada/simple/forearms/R_soft_hand_open.stl" scale="1E-3 1E-3 1E-3" />
+      <origin xyz="0.0 0.0 0.0" rpy="0.0 0.0 0.0"/>
+      <geometry name="RSoftHandLink_collision">
+        <mesh filename="package://bigman_urdf/meshes/simple/SoftHandOpen.STL" scale="0.001 0.001 0.001" />
       </geometry>
    </collision>
   </link>
-  <link name="LSoftHand">
+  <link name="LSoftHand"/>
+  <link name="l_palm"/>
+  <link name="LSoftHandLink">
     <inertial>
       <origin xyz="0 0 0" rpy="0 0 0"/>
@@ -29,13 +33,13 @@
     </inertial>
     <visual>
-      <origin xyz="0.007 -0.012 -0.04" rpy="${-3.14159265359/2} 0 ${3.14159265359/2}"/>
-      <geometry name="LSoftHand_visual">
-        <mesh filename="package://bigman_urdf/meshes/collada/forearms/L_soft_hand_open_lowpoly.dae" scale="0.1 0.1 0.1" />
+      <origin xyz="0.0 0.0 0.0" rpy="0.0 0.0 0.0"/>
+      <geometry name="LSoftHandLink_visual">
+        <mesh filename="package://bigman_urdf/meshes/SoftHandOpen.STL" scale="0.001 -0.001 0.001" />
       </geometry>
    </visual>
    <collision>
-     <origin xyz="0.007 -0.012 -0.04" rpy="0 0 ${3.14159265359/2}"/>
-      <geometry name="LSoftHand_collision">
-        <mesh filename="package://bigman_urdf/meshes/collada/simple/forearms/L_soft_hand_open.stl" scale="1E-3 1E-3 1E-3" />
+     <origin xyz="0.0 0.0 0.0" rpy="0.0 0.0 0.0"/>
+      <geometry name="LSoftHandLink_collision">
+        <mesh filename="package://bigman_urdf/meshes/simple/SoftHandOpen.STL" scale="0.001 -0.001 0.001" />
       </geometry>
    </collision>
@@ -44,11 +48,31 @@
   <joint name="r_handj" type="fixed">
         <parent link="RWrMot3"/>
+        <child link="RSoftHandLink"/>
+        <origin xyz="0 0 0" rpy="0 0 0"/>
+  </joint>
+  <joint name="r_handj2" type="fixed">
+        <parent link="RSoftHandLink"/>
         <child link="RSoftHand"/>
-        <origin xyz="0 0 -0.11" rpy="0 0 0"/>
+        <origin xyz="${1.1908576e+01*mmTom} ${2.1833446*mmTom} ${-1.5361558e+02*mmTom}" rpy="0 0 0"/>
+  </joint>
+  <joint name="r_handj3" type="fixed">
+        <parent link="RSoftHand"/>
+        <child link="r_palm"/>
+        <origin xyz="0 0.05 0.0" rpy="0 0 0"/>
   </joint>
   <joint name="l_handj" type="fixed">
         <parent link="LWrMot3"/>
+        <child link="LSoftHandLink"/>
+        <origin xyz="0 0 0" rpy="0 0 0"/>
+  </joint>
+  <joint name="l_handj2" type="fixed">
+        <parent link="LSoftHandLink"/>
         <child link="LSoftHand"/>
-        <origin xyz="0 0 -0.11" rpy="0 0 0"/>
+        <origin xyz="${1.1908576e+01*mmTom} ${-2.1833446*mmTom} ${-1.5361558e+02*mmTom}" rpy="0 0 0"/>
+  </joint>
+  <joint name="l_handj3" type="fixed">
+        <parent link="LSoftHand"/>
+        <child link="l_palm"/>
+        <origin xyz="0 -0.05 0.0" rpy="0 0 0"/>
   </joint>
 </xacro:if>

Commit message: Simplified contact model for raising support

File: bigman_urdf/urdf/parts/forearms.urdf.xacro (robot description, xacro)
@@ -57,7 +57,9 @@
         </visual>
         <collision>
-          <origin xyz="0 0 0" rpy="0 0 0"/>
+          <origin xyz="0.008 0 -0.076" rpy="0 0 0"/>
+          <!--origin xyz="0 0 0" rpy="0 0 0"/-->
           <geometry name="LRaisingSupport_collision">
-            <mesh filename="package://bigman_urdf/meshes/simple/RaisingSupport.STL" scale="0.001 -0.001 0.001" />
+            <box size="0.218 0.04 0.152" />
+            <!--mesh filename="package://bigman_urdf/meshes/simple/RaisingSupport.STL" scale="0.001 -0.001 0.001" /-->
           </geometry>
         </collision>
@@ -134,7 +136,9 @@
         </visual>
         <collision>
-          <origin xyz="0 0 0" rpy="0 0 0"/>
+          <origin xyz="0.008 0 -0.076" rpy="0 0 0"/>
+          <!--origin xyz="0 0 0" rpy="0 0 0"/-->
           <geometry name="RRaisingSupport_collision">
-            <mesh filename="package://bigman_urdf/meshes/simple/RaisingSupport.STL" scale="0.001 0.001 0.001" />
+            <box size="0.218 0.04 0.152" />
+            <!--mesh filename="package://bigman_urdf/meshes/simple/RaisingSupport.STL" scale="0.001 0.001 0.001" /-->
           </geometry>
         </collision>

Commit message: arms longer 15 cm

File: bigman_urdf/urdf/parts/forearms.urdf.xacro (robot description, xacro)
@@ -176,5 +176,5 @@
     <parent link="LElb"/>
     <child link="LForearm"/>
-    <origin xyz="-0.075 0.0 -0.1955" rpy="0 0 0"/>
+    <origin xyz="-0.075 0.0 -0.3455" rpy="0 0 0"/>
     <axis xyz="0 0 1" />
     <limit velocity="6.283" effort="60" lower="-2.529" upper="2.529" />
@@ -211,5 +211,5 @@
     <parent link="RElb"/>
     <child link="RForearm"/>
-    <origin xyz="-0.075 0.0 -0.1955" rpy="0 0 0"/>
+    <origin xyz="-0.075 0.0 -0.3455" rpy="0 0 0"/>
     <axis xyz="0 0 1" />
     <limit velocity="6.283" effort="60" lower="-2.529" upper="2.529" />
