Commit message: Added Inertia, CoM and Mass to Chest Link

File: bigman_urdf/urdf/parts/torso.urdf.xacro (robot description, xacro)
@@ -73,7 +73,7 @@
   <link name ="DWYTorso">
     <inertial>
-      <origin xyz="-0.0358501 1.8286043E-5 0.117557148" rpy="0 0 0"/>
-      <mass value="6.3617175"/>
-      <inertia ixx="0.034089342"  ixy="-9.8308572E-6"  ixz="-7.5649290E-4" iyy="0.030117357" iyz="6.2443771E-6" izz="0.025296582" />
+      <origin xyz="-0.10981228 -0.00551229 -0.06272896" rpy="0 0 0"/>
+      <mass value="22.38913469"/>
+      <inertia ixx="0.15989993"  ixy="0.00087514"  ixz="0.01598045" iyy="0.11274359" iyz="0.00019540" izz="0.21318148" />
     </inertial>
     <visual>

Commit message: Added visual, collision, CoM, Mass and Inertia of Torso Yaw

File: bigman_urdf/urdf/parts/torso.urdf.xacro (robot description, xacro)
@@ -54,18 +54,18 @@
   <link name ="DWS">
     <inertial>
-      <origin xyz="-0.0021273416 0.0033575235 -0.0010076896" rpy="0 0 0"/>
-      <mass value="0.75398402"/>
-      <inertia ixx="3.4093348E-4"  ixy="-6.2120042E-6"  ixz="-1.3863473E-6" iyy="3.9581916E-4" iyz="1.443019E-6" izz="3.7449753E-4" />
+      <origin xyz="0.00010203 0.00928164 0.08113610" rpy="0 0 0"/>
+      <mass value="5.28825567"/>
+      <inertia ixx="0.01628069"  ixy="-0.00000323"  ixz="0.00001424" iyy="0.01424286" iyz="0.00075458" izz="0.00994169" />
     </inertial>
     <visual>
-      <origin xyz="-0.020281504 0 -0.63912053" rpy="0 0 ${PI}"/>
+      <origin xyz="0.0 0.0 0.0" rpy="0 0 0"/>
       <geometry name="DWS_visual">
-        <mesh filename="package://bigman_urdf/meshes/collada/asm0001_collada_08_prt.dae" scale="${SF} ${SF} ${SF}" />
+        <mesh filename="package://bigman_urdf/meshes/TorsoYawPitch.STL" scale="0.001 0.001 0.001" />
       </geometry>
     </visual>
     <collision>
-      <origin xyz="-0.020281504 0 -0.63912053" rpy="0 0 ${PI}"/>
+      <origin xyz="0.0 0.0 0.0" rpy="0 0 0"/>
       <geometry name="DWS_collision">
-        <mesh filename="package://bigman_urdf/meshes/collada/simple/simple_asm0001_collada_08_prt.stl" scale="${SF} ${SF} ${SF}" />
+        <mesh filename="package://bigman_urdf/meshes/simple/TorsoYawPitch.STL" scale="0.001 0.001 0.001" />
       </geometry>
     </collision>
@@ -121,5 +121,5 @@
     <parent link="DWS"/>
     <child link="DWYTorso"/>
-    <origin xyz="0 0 0.22222" rpy="0 0 0" />
+    <origin xyz="0 0 0.22275" rpy="0 0 0" />
     <axis xyz="0 0 1" />
     <limit velocity="4.0" effort="50" lower="-1.3963" upper="1.3962" />

Commit message: Added visual, collision, CoM, Mass and Inertia of Torso Roll/pitch link

File: bigman_urdf/urdf/parts/torso.urdf.xacro (robot description, xacro)
@@ -35,18 +35,18 @@
   <link name ="DWL">
     <inertial>
-      <origin xyz="4.2999707E-4 -0.0097650317 0.033011157" rpy="0 0 0"/>
-      <mass value="0.54588774"/>
-      <inertia ixx="9.7126578E-4"  ixy="-7.2101244E-7"  ixz="1.1440119E-6" iyy="7.4686706E-4" iyz="-1.7450917E-4" izz="6.2196235E-4" />
+      <origin xyz="-0.04610869 0.02232230 -0.02249514" rpy="0 0 0"/>
+      <mass value="1.44965471"/>
+      <inertia ixx="0.01096760"  ixy="0.00111556"  ixz="0.00030030" iyy="0.00409572" iyz="0.00054456" izz="0.01143795" />
     </inertial>
     <visual>
-      <origin xyz="-0.020281504 0 -0.63912053" rpy="0 0 ${PI}"/>
+      <origin xyz="0.0 0.0 0.0" rpy="0 0 0"/>
       <geometry name="DWL_visual">
-        <mesh filename="package://bigman_urdf/meshes/collada/asm0001_collada_09_prt.dae" scale="${SF} ${SF} ${SF}" />
+        <mesh filename="package://bigman_urdf/meshes/TorsoRoll.STL" scale="0.001 0.001 0.001" />
       </geometry>
     </visual>
     <collision>
-      <origin xyz="-0.020281504 0 -0.63912053" rpy="0 0 ${PI}"/>
+      <origin xyz="0.0 0.0 0.0" rpy="0 0 0"/>
       <geometry name="DWL_collision">
-        <mesh filename="package://bigman_urdf/meshes/collada/simple/simple_asm0001_collada_09_prt.stl" scale="${SF} ${SF} ${SF}" />
+        <mesh filename="package://bigman_urdf/meshes/simple/TorsoRoll.STL" scale="0.001 0.001 0.001" />
       </geometry>
     </collision>

Commit message: Added Waist Inertia, CoM, Mass viasual and collision

File: bigman_urdf/urdf/parts/torso.urdf.xacro (robot description, xacro)
@@ -1,8 +1,9 @@
 <?xml version="1.0"?>
 <robot xmlns:xacro="http://ros.org/wiki/xacro">
+<xacro:property name="mmTom" value="0.001" />
+<xacro:property name="mm2Tom2" value="${0.001*0.001}" />
 <xacro:property name="PI" value="3.14159265359" />
 <xacro:property name="PI_2" value="1.57079632679" />
 <xacro:property name="SF" value="0.03937" /> <!-- Scale factor for meshes -->
-<xacro:property name="base_link_z_translation" value="-0.52" />
 <xacro:property name="cos_20" value="0.93969262078" />
 <xacro:property name="sin_20" value="0.34202014332" />
@@ -16,18 +17,18 @@
 <link name="Waist">
     <inertial>
-      <origin xyz="-0.026391145 -5.8216364E-4 0.052632312" rpy="0.0 0.0 0.0"/>
-      <mass value="1.8008695"/>
-      <inertia ixx="0.0051032982"  ixy="-5.7170981E-5"  ixz="0.0016920543" iyy="0.006241636" iyz="1.7225949E-5" izz="0.0024517762" />
+      <origin xyz="${-3.2862932e+01*mmTom} ${-5.0930727e-01*mmTom} ${-1.2899617*mmTom}" rpy="0.0 0.0 0.0"/>
+      <mass value="6.4080904"/>
+      <inertia ixx="${3.8826078e+04*mm2Tom2}"  ixy="${2.9047605e+02*mm2Tom2}"  ixz="${6.8975598e+02*mm2Tom2}" iyy="${2.5050374e+04*mm2Tom2}" iyz="${-1.3370623e+01*mm2Tom2}" izz="${4.8055286e+04*mm2Tom2}" />
     </inertial>
     <visual>
-      <origin xyz="0 0 ${base_link_z_translation}" rpy="0 0 ${PI}"/>
+      <origin xyz="0 0 0" rpy="0 0 0"/>
       <geometry name="Waist_visual">
-        <mesh filename="package://bigman_urdf/meshes/collada/asm0001_collada_07_prt.dae" scale="${SF} ${SF} ${SF}"/>
+        <mesh filename="package://bigman_urdf/meshes/Waist.STL" scale="0.001 0.001 0.001"/>
       </geometry>
     </visual>
     <collision>
-      <origin xyz="0 0 ${base_link_z_translation}" rpy="0 0 ${PI}"/>
+      <origin xyz="0 0 0" rpy="0 0 0"/>
       <geometry name="Waist_collision">
-        <mesh filename="package://bigman_urdf/meshes/collada/simple/simple_asm0001_collada_07_prt.stl" scale="${SF} ${SF} ${SF}"/>
+        <mesh filename="package://bigman_urdf/meshes/simple/Waist.STL" scale="0.001 0.001 0.001"/>
       </geometry>
     </collision>

Commit message: Added right angle in torso lat

File: bigman_urdf/urdf/parts/torso.urdf.xacro (robot description, xacro)
@@ -6,6 +6,6 @@
 <xacro:property name="PI_2" value="1.57079632679" />
 <xacro:property name="SF" value="0.03937" /> <!-- Scale factor for meshes -->
-<xacro:property name="cos_20" value="0.93969262078" />
-<xacro:property name="sin_20" value="0.34202014332" />
+<xacro:property name="cos_26" value="0.89879991307" />
+<xacro:property name="sin_26" value="0.43835911792" />
 <!-- LINKS -->
 <!-- This links are defined in order to be compliant with http://www.ros.org/reps/rep-0120.html#coordinate-frames
@@ -106,5 +106,5 @@
     <child link="DWL"/>
     <origin xyz="0.020281504 0 0.11912053" rpy="0 0 0" />
-    <axis xyz="${cos_20} 0 ${sin_20}" />
+    <axis xyz="${cos_26} 0 ${sin_26}" />
     <limit velocity="6.283" effort="120" lower="-0.610" upper="0.610" />
     <!-- dynamics friction="0" damping="0.3"/ -->

Commit message: Moved torso in right position

File: bigman_urdf/urdf/parts/torso.urdf.xacro (robot description, xacro)
@@ -105,5 +105,5 @@
     <parent link="Waist"/>
     <child link="DWL"/>
-    <origin xyz="0.020281504 0 0.11912053" rpy="0 0 0" />
+    <origin xyz="0.0715192 0 0.195982" rpy="0 0 0" />
     <axis xyz="${cos_26} 0 ${sin_26}" />
     <limit velocity="6.283" effort="120" lower="-0.610" upper="0.610" />

Commit message: Changed max torque torso pitch joint

File: bigman_urdf/urdf/parts/torso.urdf.xacro (robot description, xacro)
@@ -116,5 +116,5 @@
     <origin xyz="0 0 0" rpy="0 0 0" />
     <axis xyz="0 1 0" />
-    <limit velocity="6.283" effort="120" lower="-0.349" upper="1.396" />
+    <limit velocity="6.283" effort="220" lower="-0.349" upper="1.396" />
     <dynamics friction="0" damping="3.0"/>
   </joint>

Commit message: Added protection system mesh and collisions

File: bigman_urdf/urdf/parts/torso.urdf.xacro (robot description, xacro)
@@ -84,5 +84,30 @@
     </collision>
   </link>
+<link name ="TorsoProtections">
+    <inertial>
+      <origin xyz="0.00010203 0.00928164 0.08113610" rpy="0 0 0"/>
+      <mass value="3.0"/>
+      <inertia ixx="0.01628069"  ixy="-0.00000323"  ixz="0.00001424" iyy="0.01424286" iyz="0.00075458" izz="0.00994169" />
+    </inertial>
+    <visual>
+      <origin xyz="0.0 0.0 0.0" rpy="0 0 0"/>
+      <geometry name="TorsoProtections_visual">
+        <mesh filename="package://bigman_urdf/meshes/ProtectionSystem.STL" scale="0.001 0.001 0.001" />
+      </geometry>
+      <material name="dark_grey"/>
+    </visual>
+    <collision>
+      <origin xyz="0.0 0.0 0.0" rpy="0 0 0"/>
+      <geometry name="TorsoProtections_collision">
+        <mesh filename="package://bigman_urdf/meshes/simple/ProtectionSystem.STL" scale="0.001 0.001 0.001" />
+      </geometry>
+    </collision>
+  </link>
 <!-- JOINTS -->
+<joint name="torso_protection_joint" type="fixed">
+    <parent link="DWYTorso"/>
+    <child link="TorsoProtections"/>
+    <origin xyz="0.0 0 0.0" rpy="${-PI_2} 0 0" />
+</joint>
 <joint name="torso_joint" type="fixed">
     <parent link="DWYTorso"/>

Commit message: Added new version of torso protections. Added mass and inertia parametrs for torso protection.

File: bigman_urdf/urdf/parts/torso.urdf.xacro (robot description, xacro)
@@ -87,7 +87,7 @@
 <link name ="TorsoProtections">
     <inertial>
-      <origin xyz="0.00010203 0.00928164 0.08113610" rpy="0 0 0"/>
-      <mass value="3.0"/>
-      <inertia ixx="0.01628069"  ixy="-0.00000323"  ixz="0.00001424" iyy="0.01424286" iyz="0.00075458" izz="0.00994169" />
+      <origin xyz="${-8.2963193e+01*mmTom} ${7.0747291e-04*mmTom} ${7.5409106e+01*mmTom}" rpy="0 0 0"/>
+      <mass value="2.9346303"/>
+      <inertia ixx="${1.4773769e+05*mm2Tom2}"  ixy="${0.0*mm2Tom2}"  ixz="${-2.9780072e+04*mm2Tom2}" iyy="${1.6085511e+05*mm2Tom2}" iyz="${0.0*mm2Tom2}" izz="${1.5409381e+05*mm2Tom2}" />
     </inertial>
     <visual>
@@ -111,5 +111,5 @@
     <parent link="DWYTorso"/>
     <child link="TorsoProtections"/>
-    <origin xyz="0.0 0 0.0" rpy="${-PI_2} 0 0" />
+    <origin xyz="0.0 0 0.0" rpy="0 0 0" />
 </joint>
 </xacro:if>

Commit message: Added approximated backpack

File: bigman_urdf/urdf/parts/torso.urdf.xacro (robot description, xacro)
@@ -84,9 +84,10 @@
     </collision>
   </link>
+<!-- UPDATE DATA FOR TORSO PROTECTION! -->
 <xacro:if value="${BIGMAN_ADD_PROTECTIONS}">
 <link name ="TorsoProtections">
     <inertial>
       <origin xyz="${-8.2963193e+01*mmTom} ${7.0747291e-04*mmTom} ${7.5409106e+01*mmTom}" rpy="0 0 0"/>
-      <mass value="2.9346303"/>
+      <mass value="4.7"/>
       <inertia ixx="${1.4773769e+05*mm2Tom2}"  ixy="${0.0*mm2Tom2}"  ixz="${-2.9780072e+04*mm2Tom2}" iyy="${1.6085511e+05*mm2Tom2}" iyz="${0.0*mm2Tom2}" izz="${1.5409381e+05*mm2Tom2}" />
     </inertial>
@@ -106,5 +107,31 @@
   </link>
 </xacro:if>
+<!-- UPDATE DATA FOR TORSO PROTECTION! -->
+<link name="backpack">
+    <inertial>
+      <origin xyz="0 0 -0.065" rpy="0 0 0"/>
+      <mass value="10.0"/>
+      <inertia ixx="${(10.0/12.0)*(0.3*0.3+0.13*0.13)}"  ixy="0.0"  ixz="0.0" iyy="${(10.0/12.0)*(0.16*0.16+0.13*0.13)}" iyz="0.0" izz="${(10.0/12.0)*(0.16*0.16+0.3*0.3)}" />
+    </inertial>
+    <visual>
+      <origin xyz="0.0 0.0 0.0" rpy="0 0 0"/>
+      <geometry name="backpack_visual">
+        <box size="0.16 0.3 0.22" />
+      </geometry>
+      <material name="dark_grey"/>
+    </visual>
+    <collision>
+      <origin xyz="0.0 0.0 0.0" rpy="0 0 0"/>
+      <geometry name="backpack_collision">
+        <box size="0.16 0.3 0.22" />
+      </geometry>
+    </collision>
+</link>
 <!-- JOINTS -->
+<joint name="backpack_joint" type="fixed">
+    <parent link="DWYTorso"/>
+    <child link="backpack"/>
+    <origin xyz="-0.185 0 -0.025" rpy="0 0 0" />
+</joint>
 <xacro:if value="${BIGMAN_ADD_PROTECTIONS}">
 <joint name="torso_protection_joint" type="fixed">

Commit message: Changed torso values

File: bigman_urdf/urdf/parts/torso.urdf.xacro (robot description, xacro)
@@ -155,5 +155,5 @@
     <origin xyz="0.1115 0 0.195982" rpy="0 0 0" />
     <axis xyz="${cos_26} 0 ${sin_26}" />
-    <limit velocity="6.283" effort="120" lower="${-35.0*toRad}" upper="${35.0*toRad}" />
+    <limit velocity="6.283" effort="120" lower="${-15.0*toRad}" upper="${15.0*toRad}" />
     <dynamics friction="0" damping="3.0"/>
 </joint>
@@ -163,5 +163,5 @@
     <origin xyz="0 0 0" rpy="0 0 0" />
     <axis xyz="0 1 0" />
-    <limit velocity="6.283" effort="220" lower="${-20.0*toRad}" upper="${80.0*toRad}" />
+    <limit velocity="6.283" effort="220" lower="${-10.0*toRad}" upper="${80.0*toRad}" />
     <dynamics friction="0" damping="3.0"/>
   </joint>
@@ -171,5 +171,5 @@
     <origin xyz="0 0 0.22275" rpy="0 0 0" />
     <axis xyz="0 0 1" />
-    <limit velocity="6.283" effort="120" lower="${-120.0*toRad}" upper="${120.0*toRad}" />
+    <limit velocity="6.283" effort="120" lower="${-100.0*toRad}" upper="${100.0*toRad}" />
     <dynamics friction="0" damping="3.0"/>
   </joint>

Commit message: - com pos tuned

File: bigman_urdf/urdf/parts/torso.urdf.xacro (robot description, xacro)
@@ -56,5 +56,5 @@
   <link name ="DWYTorso">
     <inertial>
-        <origin xyz="0.0 0.00 0.3" rpy="0 0 0"/>
+        <origin xyz="0.09 -0.03 0.5" rpy="0 0 0"/>
         <mass value="26"/>
       <inertia ixx="0.18629757"  ixy="0.00008160"  ixz="0.00030250" iyy="0.02013829" iyz="-0.00001790" izz="0.18850541" />

Commit message: - torso com position modified for walking

File: bigman_urdf/urdf/parts/torso.urdf.xacro (robot description, xacro)
@@ -56,5 +56,5 @@
   <link name ="DWYTorso">
     <inertial>
-        <origin xyz="0.09 -0.03 0.5" rpy="0 0 0"/>
+        <origin xyz="0.09 -0.06 0.5" rpy="0 0 0"/>
         <mass value="26"/>
       <inertia ixx="0.18629757"  ixy="0.00008160"  ixz="0.00030250" iyy="0.02013829" iyz="-0.00001790" izz="0.18850541" />

Commit message: - x direction tuned for walking

File: bigman_urdf/urdf/parts/torso.urdf.xacro (robot description, xacro)
@@ -56,5 +56,5 @@
   <link name ="DWYTorso">
     <inertial>
-        <origin xyz="0.09 -0.06 0.5" rpy="0 0 0"/>
+        <origin xyz="0.05 -0.06 0.5" rpy="0 0 0"/>
         <mass value="26"/>
       <inertia ixx="0.18629757"  ixy="0.00008160"  ixz="0.00030250" iyy="0.02013829" iyz="-0.00001790" izz="0.18850541" />

Commit message: changed torso roll limits

File: bigman_urdf/urdf/parts/torso.urdf.xacro (robot description, xacro)
@@ -155,5 +155,5 @@
     <origin xyz="0.1115 0 0.195982" rpy="0 0 0" />
     <axis xyz="${cos_26} 0 ${sin_26}" />
-    <limit velocity="6.283" effort="120" lower="${-15.0*toRad}" upper="${15.0*toRad}" />
+    <limit velocity="6.283" effort="120" lower="${-0.11*toRad}" upper="${0.11*toRad}" />
     <dynamics friction="0" damping="3.0"/>
 </joint>

Commit message: changed torso roll (WaistLat) limits

File: bigman_urdf/urdf/parts/torso.urdf.xacro (robot description, xacro)
@@ -155,5 +155,5 @@
     <origin xyz="0.1115 0 0.195982" rpy="0 0 0" />
     <axis xyz="${cos_26} 0 ${sin_26}" />
-    <limit velocity="6.283" effort="120" lower="${-0.11*toRad}" upper="${0.11*toRad}" />
+    <limit velocity="6.283" effort="120" lower="${-0.6*toRad}" upper="${0*toRad}" />
     <dynamics friction="0" damping="3.0"/>
 </joint>
