Commit message: changed neckpitch link into head

File: bigman_urdf/urdf/parts/neck.urdf.xacro (robot description, xacro)
@@ -30,5 +30,5 @@
     </collision>
   </link>
-  <link name ="NeckPitch">
+  <link name ="head">
     <inertial>
       <origin xyz="0.0 0.0 0.0" rpy="0 0 0"/>
@@ -61,5 +61,5 @@
 <joint name="NeckPitchj" type="revolute">
     <parent link="NeckYaw"/>
-    <child link="NeckPitch"/>
+    <child link="head"/>
     <origin xyz="0 0 0.1155" rpy="0 0 0" />
     <axis xyz="0 1 0" />

Commit message: Added new inertia and mass values for the chest that does not take into account the Backpack. Changed inertia to the neck (still not the right values). Updated documentation

File: bigman_urdf/urdf/parts/neck.urdf.xacro (robot description, xacro)
@@ -14,5 +14,5 @@
       <origin xyz="0.0 0.0 0.0" rpy="0 0 0"/>
       <mass value="1.0"/>
-      <inertia ixx="0.01"  ixy="0.0"  ixz="0.0" iyy="0.01" iyz="0.0" izz="0.01" />
+      <inertia ixx="0.001"  ixy="0.0"  ixz="0.0" iyy="0.001" iyz="0.0" izz="0.001" />
     </inertial>
     <visual>
@@ -34,5 +34,5 @@
       <origin xyz="0.0 0.0 0.0" rpy="0 0 0"/>
       <mass value="1.0"/>
-      <inertia ixx="0.01"  ixy="0.0"  ixz="0.0" iyy="0.01" iyz="0.0" izz="0.01" />
+      <inertia ixx="0.001"  ixy="0.0"  ixz="0.0" iyy="0.001" iyz="0.0" izz="0.001" />
     </inertial>
     <visual>

File: bigman_urdf/urdf/parts/torso.urdf.xacro (robot description, xacro)
@@ -56,7 +56,7 @@
   <link name ="DWYTorso">
     <inertial>
-      <origin xyz="-0.10981228 -0.00551229 -0.06272896" rpy="0 0 0"/>
-      <mass value="22.38913469"/>
-      <inertia ixx="0.15989993"  ixy="0.00087514"  ixz="0.01598045" iyy="0.11274359" iyz="0.00019540" izz="0.21318148" />
+      <origin xyz="0.02049278 -0.00000767 -0.03249378" rpy="0 0 0"/>
+      <mass value="7.31313212"/>
+      <inertia ixx="0.18629757"  ixy="0.00008160"  ixz="0.00030250" iyy="0.02013829" iyz="-0.00001790" izz="0.18850541" />
     </inertial>
     <visual>

Commit message: Added approximated inertias for the neck yaw and neck pitch + pc104

File: bigman_urdf/urdf/parts/neck.urdf.xacro (robot description, xacro)
@@ -12,7 +12,7 @@
   <link name ="NeckYaw">
     <inertial>
-      <origin xyz="0.0 0.0 0.0" rpy="0 0 0"/>
-      <mass value="1.0"/>
-      <inertia ixx="0.001"  ixy="0.0"  ixz="0.0" iyy="0.001" iyz="0.0" izz="0.001" />
+      <origin xyz="0.0 0.0 ${1.1550000e+02*mmTom}" rpy="0 0 0"/>
+      <mass value="0.35"/>
+      <inertia ixx="${3.2840119e+02*mm2Tom2}"  ixy="0.0"  ixz="0.0" iyy="${7.0371675e+01*mm2Tom2}" iyz="0.0" izz="${3.2840111e+02*mm2Tom2}" />
     </inertial>
     <visual>
@@ -32,7 +32,7 @@
   <link name ="NeckPitch">
     <inertial>
-      <origin xyz="0.0 0.0 0.0" rpy="0 0 0"/>
-      <mass value="1.0"/>
-      <inertia ixx="0.001"  ixy="0.0"  ixz="0.0" iyy="0.001" iyz="0.0" izz="0.001" />
+      <origin xyz="${-1.020e+02*mmTom} 0.0 ${2.6575000e+02*mmTom}" rpy="0 0 0"/>
+      <mass value="0.623"/>
+      <inertia ixx="${1.0388333e+03*mm2Tom2}"  ixy="0.0"  ixz="0.0" iyy="${5.4689381e+02*mm2Tom2}" iyz="0.0" izz="${5.4689381e+02*mm2Tom2}" />
     </inertial>
     <visual>

Commit message: Added new joint limits for the head

File: bigman_urdf/urdf/parts/neck.urdf.xacro (robot description, xacro)
@@ -8,5 +8,4 @@
 <xacro:property name="sin_26" value="0.43835911792" />
 <xacro:property name="toRad" value="${PI/180.0}" />
-<xacro:property name="safety" value="5.0" />
 <!-- LINKS -->
   <link name ="NeckYaw">
@@ -56,5 +55,6 @@
     <origin xyz="0 0 0" rpy="0 0 0" />
     <axis xyz="0 0 1" />
-    <limit velocity="6.283" effort="120" lower="${(-175.0+safety)*toRad}" upper="${(175.0-safety)*toRad}" />
+    <!--limit velocity="6.283" effort="120" lower="${(-175.0)*toRad}" upper="${(175.0)*toRad}" /-->
+    <limit velocity="6.283" effort="120" lower="${(-35.0)*toRad}" upper="${(35.0)*toRad}" />
     <dynamics friction="0" damping="3.0"/>
 </joint>
@@ -64,5 +64,6 @@
     <origin xyz="0 0 0.1155" rpy="0 0 0" />
     <axis xyz="0 1 0" />
-    <limit velocity="6.283" effort="120" lower="${(-30.0+safety)*toRad}" upper="${(70.0-safety)*toRad}" />
+    <!--limit velocity="6.283" effort="120" lower="${(-30.0)*toRad}" upper="${(70.0)*toRad}" /-->
+    <limit velocity="6.283" effort="120" lower="${(-25.0)*toRad}" upper="${(60.0)*toRad}" />
     <dynamics friction="0" damping="3.0"/>
 </joint>

Commit message: put old values for NeckYawj limits

File: bigman_urdf/urdf/parts/neck.urdf.xacro (robot description, xacro)
@@ -55,6 +55,6 @@
     <origin xyz="0 0 0" rpy="0 0 0" />
     <axis xyz="0 0 1" />
-    <!--limit velocity="6.283" effort="120" lower="${(-175.0)*toRad}" upper="${(175.0)*toRad}" /-->
-    <limit velocity="6.283" effort="120" lower="${(-35.0)*toRad}" upper="${(35.0)*toRad}" />
+    <limit velocity="6.283" effort="120" lower="${(-175.0)*toRad}" upper="${(175.0)*toRad}" />
+    <!--limit velocity="6.283" effort="120" lower="${(-35.0)*toRad}" upper="${(35.0)*toRad}" /-->
     <dynamics friction="0" damping="3.0"/>
 </joint>

Commit message: fixed small error in neck (missing 1.5 mm)

File: bigman_urdf/urdf/parts/neck.urdf.xacro (robot description, xacro)
@@ -62,5 +62,5 @@
     <parent link="NeckYaw"/>
     <child link="NeckPitch"/>
-    <origin xyz="0 0 0.1155" rpy="0 0 0" />
+    <origin xyz="0 0 0.117" rpy="0 0 0" />
     <axis xyz="0 1 0" />
     <!--limit velocity="6.283" effort="120" lower="${(-30.0)*toRad}" upper="${(70.0)*toRad}" /-->
