Commit message: Added Shoulders, missing Inertia, CoM and Mass

File: bigman_urdf/urdf/parts/arms.urdf.xacro (robot description, xacro)
@@ -2,4 +2,6 @@
 <robot xmlns:xacro="http://ros.org/wiki/xacro">
 <xacro:property name="PI" value="3.14159265359" />
+<xacro:property name="cos_42" value="0.743144825" />
+<xacro:property name="sin_42" value="0.669130606" />
 <xacro:property name="SF" value="0.03937" /> <!-- Scale factor for meshes -->
 <!-- LINKS -->
@@ -12,13 +14,13 @@
     </inertial>
     <visual>
-      <origin xyz="-0.005305 0.0825 -0.844329" rpy="0 0 ${PI}"/>
+      <origin xyz="0 0 0" rpy="0 0 0"/>
       <geometry name="RShp_visual">
-        <mesh filename="package://bigman_urdf/meshes/collada/asm0001_collada_24_prt.dae" scale="${SF} ${SF} ${SF}" />
-      </geometry>
-    </visual>
-    <collision>
-      <origin xyz="-0.005305 0.0825 -0.844329" rpy="0 0 ${PI}"/>
+        <mesh filename="package://bigman_urdf/meshes/ShoulderPitch.STL" scale="0.001 0.001 0.001" />
+      </geometry>
+    </visual>
+    <collision>
+      <origin xyz="0 0 0" rpy="0 0 0"/>
       <geometry name="RShp_collision">
-        <mesh filename="package://bigman_urdf/meshes/collada/simple/simple_asm0001_collada_24_prt.stl" scale="${SF} ${SF} ${SF}" />
+        <mesh filename="package://bigman_urdf/meshes/simple/ShoulderPitch.STL" scale="0.001 0.001 0.001" />
       </geometry>
     </collision>
@@ -89,13 +91,13 @@
     </inertial>
     <visual>
-      <origin xyz="-0.005305 -0.0825 -0.844329" rpy="0 0 ${PI}"/>
-      <geometry name="LShp_visual">
-        <mesh filename="package://bigman_urdf/meshes/collada/asm0001_collada_14_prt.dae" scale="${SF} ${SF} ${SF}" />
-      </geometry>
-    </visual>
-    <collision>
-      <origin xyz="-0.005305 -0.0825 -0.844329" rpy="0 0 ${PI}"/>
-      <geometry name="LShp_collision">
-        <mesh filename="package://bigman_urdf/meshes/collada/simple/simple_asm0001_collada_14_prt.stl" scale="${SF} ${SF} ${SF}" />
+      <origin xyz="0 0 0" rpy="0 0 0"/>
+      <geometry name="RShp_visual">
+        <mesh filename="package://bigman_urdf/meshes/ShoulderPitch.STL" scale="0.001 -0.001 0.001" />
+      </geometry>
+    </visual>
+    <collision>
+      <origin xyz="0 0 0" rpy="0 0 0"/>
+      <geometry name="RShp_collision">
+        <mesh filename="package://bigman_urdf/meshes/simple/ShoulderPitch.STL" scale="0.001 -0.001 0.001" />
       </geometry>
     </collision>
@@ -164,5 +166,5 @@
     <child link="RShp"/>
     <origin xyz="0.0 -0.2 0.0" rpy="0 0 0" />
-    <axis xyz="0 1 0" />
+    <axis xyz="0 ${cos_42} ${-sin_42}" />
     <limit velocity="4.0" effort="50" lower="-3.4034" upper="1.6581" />
     <dynamics friction="0" damping="3.0"/>
@@ -171,5 +173,5 @@
     <parent link="RShp"/>
     <child link="RShr"/>
-    <origin xyz="0.0 -0.07329999999999999 0.0" rpy="0 0 0" />
+    <origin xyz="0.0 -0.116568264 0.03364" rpy="0 0 0" />
     <axis xyz="1 0 0" />
     <limit velocity="4.0" effort="50" lower="-2.094" upper="0.31415" />
@@ -197,5 +199,5 @@
     <child link="LShp"/>
     <origin xyz="0.0 0.2 0.0" rpy="0 0 0" />
-    <axis xyz="0 1 0" />
+    <axis xyz="0 ${cos_42} ${sin_42}" />
     <limit velocity="4.0" effort="50" lower="-3.4034" upper="1.6581" />
     <dynamics friction="0" damping="3.0"/>
@@ -204,5 +206,5 @@
     <parent link="LShp"/>
     <child link="LShr"/>
-    <origin xyz="0.0 0.07329999999999999 0.0" rpy="0 0 0" />
+    <origin xyz="0.0 0.116568264 0.03364" rpy="0 0 0" />
     <axis xyz="1 0 0" />
     <limit velocity="4.0" effort="50" lower="-0.31415" upper="2.094" />

Commit message: Added CoM, Inertia and Mass for L/R Shoulder Pitch

File: bigman_urdf/urdf/parts/arms.urdf.xacro (robot description, xacro)
@@ -9,7 +9,7 @@
 <link name ="RShp">
     <inertial>
-      <origin xyz="0.0099500565 -0.038682024 1.6446924E-4" rpy="0 0 0"/>
-      <mass value="0.56782202"/>
-      <inertia ixx="7.8337456E-4"  ixy="1.9035768E-4"  ixz="-3.0037676E-6" iyy="6.3399921E-4" iyz="4.3840774E-6" izz="0.001008054" />
+      <origin xyz="-0.00543349 -0.04480023 0.01581062" rpy="0 0 0"/>
+      <mass value="1.81745527"/>
+      <inertia ixx="0.00571053"  ixy="0.00041083"  ixz="-0.00005130" iyy="0.01126908" iyz="-0.00003461" izz="0.01371197" />
     </inertial>
     <visual>
@@ -86,7 +86,7 @@
 <link name ="LShp">
     <inertial>
-      <origin xyz="0.0099500565 0.038682024 1.6446924E-4" rpy="0 0 0"/>
-      <mass value="0.56782202"/>
-      <inertia ixx="7.8337456E-4"  ixy="-1.9035768E-4"  ixz="-3.0037676E-6" iyy="6.3399921E-4" iyz="-4.3840774E-6" izz="0.001008054" />
+      <origin xyz="-0.00543349 0.04480023 0.01581062" rpy="0 0 0"/>
+      <mass value="1.81745527"/>
+      <inertia ixx="0.00571053"  ixy="-0.00041083"  ixz="-0.00005130" iyy="0.01126908" iyz="0.00003461" izz="0.01371197" />
     </inertial>
     <visual>

Commit message: Added Viasual, collision, CoM, Mass and Inertia for L/R Shoulder Roll

File: bigman_urdf/urdf/parts/arms.urdf.xacro (robot description, xacro)
@@ -28,18 +28,18 @@
 <link name ="RShr">
     <inertial>
-      <origin xyz="-0.0038936743 2.2022151E-6 -0.0048616005" rpy="0 0 0"/>
-      <mass value="0.77683752"/>
-      <inertia ixx="4.5812904E-4"  ixy="-2.4111086E-7"  ixz="9.2521185E-6" iyy="4.3089204E-4" iyz="-4.7216950E-7" izz="3.4174855E-4" />
-    </inertial>
-    <visual>
-      <origin xyz="-0.005305 0.1558 -0.844329" rpy="0 0 ${PI}"/>
+      <origin xyz="0.00729315 0.00002698 -0.07529696" rpy="0 0 0"/>
+      <mass value="5.00486460"/>
+      <inertia ixx="0.01644345"  ixy="-0.00001187"  ixz="-0.00010546" iyy="0.01804804" iyz="-0.00000565" izz="0.00802420" />
+    </inertial>
+    <visual>
+      <origin xyz="0 0 0" rpy="0 0 0"/>
       <geometry name="RShr_visual">
-        <mesh filename="package://bigman_urdf/meshes/collada/asm0001_collada_23_prt.dae" scale="${SF} ${SF} ${SF}" />
-      </geometry>
-    </visual>
-    <collision>
-      <origin xyz="-0.005305 0.1558 -0.844329" rpy="0 0 ${PI}"/>
+        <mesh filename="package://bigman_urdf/meshes/TopUpperArm.STL" scale="0.001 0.001 0.001" />
+      </geometry>
+    </visual>
+    <collision>
+      <origin xyz="0 0 0" rpy="0 0 0"/>
       <geometry name="RShr_collision">
-        <mesh filename="package://bigman_urdf/meshes/collada/simple/simple_asm0001_collada_23_prt.stl" scale="${SF} ${SF} ${SF}" />
+        <mesh filename="package://bigman_urdf/meshes/simple/TopUpperArm.STL" scale="0.001 0.001 0.001" />
       </geometry>
     </collision>
@@ -105,18 +105,18 @@
 <link name ="LShr">
     <inertial>
-      <origin xyz="-0.0038936743 -2.2022151E-6 -0.0048616005" rpy="0 0 0"/>
-      <mass value="0.77683752"/>
-      <inertia ixx="4.5812904E-4"  ixy="2.4111086E-7"  ixz="9.2521185E-6" iyy="4.3089204E-4" iyz="4.721695E-7" izz="3.4174855E-4" />
-    </inertial>
-    <visual>
-      <origin xyz="-0.005305 -0.1558 -0.844329" rpy="0 0 ${PI}"/>
-      <geometry name="LShr_visual">
-        <mesh filename="package://bigman_urdf/meshes/collada/asm0001_collada_13_prt.dae" scale="${SF} ${SF} ${SF}" />
-      </geometry>
-    </visual>
-    <collision>
-      <origin xyz="-0.005305 -0.1558 -0.844329" rpy="0 0 ${PI}"/>
-      <geometry name="LShr_collision">
-        <mesh filename="package://bigman_urdf/meshes/collada/simple/simple_asm0001_collada_13_prt.stl" scale="${SF} ${SF} ${SF}" />
+      <origin xyz="0.00729315 -0.00002698 -0.07529696" rpy="0 0 0"/>
+      <mass value="5.00486460"/>
+      <inertia ixx="0.01644345"  ixy="0.00001187"  ixz="-0.00010546" iyy="0.01804804" iyz="0.00000565" izz="0.00802420" />
+    </inertial>
+    <visual>
+      <origin xyz="0 0 0" rpy="0 0 0"/>
+      <geometry name="RShr_visual">
+        <mesh filename="package://bigman_urdf/meshes/TopUpperArm.STL" scale="0.001 -0.001 0.001" />
+      </geometry>
+    </visual>
+    <collision>
+      <origin xyz="0 0 0" rpy="0 0 0"/>
+      <geometry name="RShr_collision">
+        <mesh filename="package://bigman_urdf/meshes/simple/TopUpperArm.STL" scale="0.001 -0.001 0.001" />
       </geometry>
     </collision>

Commit message: Added Visualization, collision, CoM, Mass and Inertia of elbow

File: bigman_urdf/urdf/parts/arms.urdf.xacro (robot description, xacro)
@@ -47,18 +47,18 @@
 <link name ="RShy">
     <inertial>
-      <origin xyz="0.0022714213 -0.0071091517 -0.057455221" rpy="0 0 0"/>
-      <mass value="1.0462304"/>
-      <inertia ixx="0.0030934574"  ixy="6.6702837E-5"  ixz="3.0222291E-4" iyy="0.0029181573" iyz="-5.2663661E-4" izz="8.0830389E-4" />
-    </inertial>
-    <visual>
-      <origin xyz="-0.005305 0.1558 -0.79952053" rpy="0 0 ${PI}"/>
+      <origin xyz="0.02765373 -0.03258647 -0.12698781" rpy="0 0 0"/>
+      <mass value="3.20289133"/>
+      <inertia ixx="0.01129046"  ixy="0.00013518"  ixz="-0.00134760" iyy="0.00984951" iyz="-0.00026836" izz="0.00728549" />
+    </inertial>
+    <visual>
+      <origin xyz="0 0 0" rpy="0 0 0"/>
       <geometry name="RShy_visual">
-        <mesh filename="package://bigman_urdf/meshes/collada/asm0001_collada_22_prt.dae" scale="${SF} ${SF} ${SF}" />
-      </geometry>
-    </visual>
-    <collision>
-      <origin xyz="-0.005305 0.1558 -0.79952053" rpy="0 0 ${PI}"/>
+        <mesh filename="package://bigman_urdf/meshes/BottomUpperArm.STL" scale="0.001 0.001 0.001" />
+      </geometry>
+    </visual>
+    <collision>
+      <origin xyz="0 0 0" rpy="0 0 0"/>
       <geometry name="RShy_collision">
-        <mesh filename="package://bigman_urdf/meshes/collada/simple/simple_asm0001_collada_22_prt.stl" scale="${SF} ${SF} ${SF}" />
+        <mesh filename="package://bigman_urdf/meshes/simple/BottomUpperArm.STL" scale="0.001 0.001 0.001" />
       </geometry>
     </collision>
@@ -124,18 +124,18 @@
   <link name ="LShy">
     <inertial>
-      <origin xyz="0.0022714213 0.0071091517 -0.057455221" rpy="0 0 0"/>
-      <mass value="1.0462304"/>
-      <inertia ixx="0.0030934574"  ixy="-6.6702837E-5"  ixz="3.0222291E-4" iyy="0.0029181573" iyz="5.2663661E-4" izz="8.0830389E-4" />
-    </inertial>
-    <visual>
-      <origin xyz="-0.005305 -0.1558 -0.79952053" rpy="0 0 ${PI}"/>
-      <geometry name="LShy_visual">
-        <mesh filename="package://bigman_urdf/meshes/collada/asm0001_collada_12_prt.dae" scale="${SF} ${SF} ${SF}" />
-      </geometry>
-    </visual>
-    <collision>
-      <origin xyz="-0.005305 -0.1558 -0.79952053" rpy="0 0 ${PI}"/>
-      <geometry name="LShy_collision">
-        <mesh filename="package://bigman_urdf/meshes/collada/simple/simple_asm0001_collada_12_prt.stl" scale="${SF} ${SF} ${SF}" />
+      <origin xyz="0.02765373 0.03258647 -0.12698781" rpy="0 0 0"/>
+      <mass value="3.20289133"/>
+      <inertia ixx="0.01129046"  ixy="-0.00013518"  ixz="-0.00134760" iyy="0.00984951" iyz="0.00026836" izz="0.00728549" />
+    </inertial>
+    <visual>
+      <origin xyz="0 0 0" rpy="0 0 0"/>
+      <geometry name="RShy_visual">
+        <mesh filename="package://bigman_urdf/meshes/BottomUpperArm.STL" scale="0.001 -0.001 0.001" />
+      </geometry>
+    </visual>
+    <collision>
+      <origin xyz="0 0 0" rpy="0 0 0"/>
+      <geometry name="RShy_collision">
+        <mesh filename="package://bigman_urdf/meshes/simple/BottomUpperArm.STL" scale="0.001 -0.001 0.001" />
       </geometry>
     </collision>
@@ -181,5 +181,5 @@
     <parent link="RShr"/>
     <child link="RShy"/>
-    <origin xyz="0.0 0.0 -0.04480846999999999" rpy="0 0 0" />
+    <origin xyz="0.0 0.0 -0.222" rpy="0 0 0" />
     <axis xyz="0 0 1" />
     <limit velocity="4.0" effort="50" lower="-1.5708" upper="1.5708" />
@@ -214,5 +214,5 @@
     <parent link="LShr"/>
     <child link="LShy"/>
-    <origin xyz="0.0 0.0 -0.04480846999999999" rpy="0 0 0" />
+    <origin xyz="0.0 0.0 -0.222" rpy="0 0 0" />
     <axis xyz="0 0 1" />
     <limit velocity="4.0" effort="50" lower="-1.5708" upper="1.5708" />

Commit message: Moved elbow joint in proper position

File: bigman_urdf/urdf/parts/arms.urdf.xacro (robot description, xacro)
@@ -189,5 +189,5 @@
     <parent link="RShy"/>
     <child link="RElb"/>
-    <origin xyz="0.015 0.0 -0.13519152999999998" rpy="0 0 0" />
+    <origin xyz="0.036 0.0 -0.15" rpy="0 0 0" />
     <axis xyz="0 1 0" />
     <limit velocity="4.0" effort="50" lower="-2.3562" upper="0.0" />
@@ -222,5 +222,5 @@
     <parent link="LShy"/>
     <child link="LElb"/>
-    <origin xyz="0.015 0.0 -0.13519152999999998" rpy="0 0 0" />
+    <origin xyz="0.036 0.0 -0.15" rpy="0 0 0" />
     <axis xyz="0 1 0" />
     <limit velocity="4.0" effort="50" lower="-2.3562" upper="0.0" />

Commit message: Added joint limits for shoulders and torso (still missing elbows and forearms)

File: bigman_urdf/urdf/parts/arms.urdf.xacro (robot description, xacro)
@@ -167,5 +167,5 @@
     <origin xyz="0.0 -0.2 0.0" rpy="0 0 0" />
     <axis xyz="0 ${cos_42} ${-sin_42}" />
-    <limit velocity="4.0" effort="50" lower="-3.4034" upper="1.6581" />
+    <limit velocity="6.283" effort="120" lower="-2.844" upper="2.844" />
     <dynamics friction="0" damping="3.0"/>
 </joint>
@@ -175,5 +175,5 @@
     <origin xyz="0.0 -0.116568264 0.03364" rpy="0 0 0" />
     <axis xyz="1 0 0" />
-    <limit velocity="4.0" effort="50" lower="-2.094" upper="0.31415" />
+    <limit velocity="6.283" effort="120" lower="-3.699" upper="-0.052" />
     <dynamics friction="0" damping="3.0"/>
 </joint>
@@ -183,5 +183,5 @@
     <origin xyz="0.0 0.0 -0.222" rpy="0 0 0" />
     <axis xyz="0 0 1" />
-    <limit velocity="4.0" effort="50" lower="-1.5708" upper="1.5708" />
+    <limit velocity="6.283" effort="120" lower="-2.844" upper="2.844" />
     <dynamics friction="0" damping="3.0"/>
 </joint>
@@ -200,5 +200,5 @@
     <origin xyz="0.0 0.2 0.0" rpy="0 0 0" />
     <axis xyz="0 ${cos_42} ${sin_42}" />
-    <limit velocity="4.0" effort="50" lower="-3.4034" upper="1.6581" />
+    <limit velocity="6.283" effort="120" lower="-2.844" upper="2.844" />
     <dynamics friction="0" damping="3.0"/>
 </joint>
@@ -208,5 +208,5 @@
     <origin xyz="0.0 0.116568264 0.03364" rpy="0 0 0" />
     <axis xyz="1 0 0" />
-    <limit velocity="4.0" effort="50" lower="-0.31415" upper="2.094" />
+    <limit velocity="6.283" effort="120" lower="0.052" upper="3.699" />
     <dynamics friction="0" damping="3.0"/>
 </joint>
@@ -216,5 +216,5 @@
     <origin xyz="0.0 0.0 -0.222" rpy="0 0 0" />
     <axis xyz="0 0 1" />
-    <limit velocity="4.0" effort="50" lower="-1.5708" upper="1.5708" />
+    <limit velocity="6.283" effort="120" lower="-2.844" upper="2.844" />
     <dynamics friction="0" damping="3.0"/>
 </joint>

File: bigman_urdf/urdf/parts/torso.urdf.xacro (robot description, xacro)
@@ -107,5 +107,5 @@
     <origin xyz="0.020281504 0 0.11912053" rpy="0 0 0" />
     <axis xyz="${cos_20} 0 ${sin_20}" />
-    <limit velocity="4.0" effort="50" lower="-0.5236" upper="0.5235" />
+    <limit velocity="6.283" effort="120" lower="-0.610" upper="0.610" />
     <!-- dynamics friction="0" damping="0.3"/ -->
     <dynamics friction="0" damping="3.0"/>
@@ -116,5 +116,5 @@
     <origin xyz="0 0 0" rpy="0 0 0" />
     <axis xyz="0 1 0" />
-    <limit velocity="4.0" effort="50" lower="-0.3491" upper="0.8727" />
+    <limit velocity="6.283" effort="120" lower="-0.349" upper="1.396" />
     <dynamics friction="0" damping="3.0"/>
   </joint>
@@ -124,5 +124,5 @@
     <origin xyz="0 0 0.22275" rpy="0 0 0" />
     <axis xyz="0 0 1" />
-    <limit velocity="4.0" effort="50" lower="-1.3963" upper="1.3962" />
+    <limit velocity="6.283" effort="120" lower="-2.844" upper="2.844" />
     <dynamics friction="0" damping="3.0"/>
   </joint>
