Commit message: Added L/R elbow CoM, Mass, Inertia, Visualization and Collision

File: bigman_urdf/urdf/parts/arms.urdf.xacro (robot description, xacro)
@@ -4,5 +4,6 @@
 <xacro:property name="cos_42" value="0.743144825" />
 <xacro:property name="sin_42" value="0.669130606" />
-<xacro:property name="SF" value="0.03937" /> <!-- Scale factor for meshes -->
+<xacro:property name="mmTom" value="0.001" />
+<xacro:property name="mm2Tom2" value="${0.001*0.001}" />
 <!-- LINKS -->
 <!-- RIGHT ARM -->
@@ -66,18 +67,18 @@
 <link name ="RElb">
         <inertial>
-          <origin xyz="-6.5553403E-4 -9.3464748E-4 -9.3101289E-4" rpy="0 0 0"/>
-          <mass value="0.63306933"/>
-          <inertia ixx="2.2599075E-4"  ixy="-2.6376470E-7"  ixz="-9.8007285E-6" iyy="2.7781302E-4" iyz="-2.0435288E-6" izz="2.1878992E-4" />
+          <origin xyz="${-5.5754915e+01*mmTom} ${-7.5826040*mmTom} ${-4.3820396e+01*mmTom}" rpy="0 0 0"/>
+          <mass value="8.6765385e-01"/>
+          <inertia ixx="${4.0395238e+03*mm2Tom2}"  ixy="${3.4973136e+02*mm2Tom2}"  ixz="${-6.8400465e+02*mm2Tom2}" iyy="${2.2460561e+03*mm2Tom2}" iyz="${2.8844444e+02*mm2Tom2}" izz="${4.4895027e+03*mm2Tom2}" />
         </inertial>
         <visual>
-          <origin xyz="0 0 0" rpy="-1.570796326795 1.570796326795 0"/>
+          <origin xyz="0 0 0" rpy="0 0 0"/>
           <geometry name="RElb_visual">
-            <mesh filename="package://bigman_urdf/meshes/collada/forearms/elbow.dae" scale="1.0 1.0 1.0" />
+            <mesh filename="package://bigman_urdf/meshes/Elbow.STL" scale="0.001 0.001 0.001" />
           </geometry>
         </visual>
         <collision>
-          <origin xyz="0 0 0" rpy="-1.570796326795 1.570796326795 0"/>
+          <origin xyz="0 0 0" rpy="0 0 0"/>
           <geometry name="RElb_collision">
-            <mesh filename="package://bigman_urdf/meshes/collada/simple/forearms/elbow.stl" scale="1.0 1.0 1.0" />
+            <mesh filename="package://bigman_urdf/meshes/simple/Elbow.STL" scale="0.001 0.001 0.001" />
           </geometry>
         </collision>
@@ -92,5 +93,5 @@
     <visual>
       <origin xyz="0 0 0" rpy="0 0 0"/>
-      <geometry name="RShp_visual">
+      <geometry name="LShp_visual">
         <mesh filename="package://bigman_urdf/meshes/ShoulderPitch.STL" scale="0.001 -0.001 0.001" />
       </geometry>
@@ -98,5 +99,5 @@
     <collision>
       <origin xyz="0 0 0" rpy="0 0 0"/>
-      <geometry name="RShp_collision">
+      <geometry name="LShp_collision">
         <mesh filename="package://bigman_urdf/meshes/simple/ShoulderPitch.STL" scale="0.001 -0.001 0.001" />
       </geometry>
@@ -111,5 +112,5 @@
     <visual>
       <origin xyz="0 0 0" rpy="0 0 0"/>
-      <geometry name="RShr_visual">
+      <geometry name="LShr_visual">
         <mesh filename="package://bigman_urdf/meshes/TopUpperArm.STL" scale="0.001 -0.001 0.001" />
       </geometry>
@@ -117,5 +118,5 @@
     <collision>
       <origin xyz="0 0 0" rpy="0 0 0"/>
-      <geometry name="RShr_collision">
+      <geometry name="LShr_collision">
         <mesh filename="package://bigman_urdf/meshes/simple/TopUpperArm.STL" scale="0.001 -0.001 0.001" />
       </geometry>
@@ -130,5 +131,5 @@
     <visual>
       <origin xyz="0 0 0" rpy="0 0 0"/>
-      <geometry name="RShy_visual">
+      <geometry name="LShy_visual">
         <mesh filename="package://bigman_urdf/meshes/BottomUpperArm.STL" scale="0.001 -0.001 0.001" />
       </geometry>
@@ -136,5 +137,5 @@
     <collision>
       <origin xyz="0 0 0" rpy="0 0 0"/>
-      <geometry name="RShy_collision">
+      <geometry name="LShy_collision">
         <mesh filename="package://bigman_urdf/meshes/simple/BottomUpperArm.STL" scale="0.001 -0.001 0.001" />
       </geometry>
@@ -143,18 +144,18 @@
     <link name ="LElb">
         <inertial>
-          <origin xyz="-6.5553403E-4 9.3464748E-4 -9.3101289E-4" rpy="0 0 0"/>
-          <mass value="0.63306933"/>
-          <inertia ixx="2.2599075E-4"  ixy="2.6376470E-7"  ixz="-9.8007285E-6" iyy="2.7781302E-4" iyz="2.0435288E-6" izz="2.1878992E-4" />
+          <origin xyz="${-5.5754915e+01*mmTom} ${7.5826040*mmTom} ${-4.3820396e+01*mmTom}" rpy="0 0 0"/>
+          <mass value="8.6765385e-01"/>
+          <inertia ixx="${4.0395238e+03*mm2Tom2}"  ixy="${-3.4973136e+02*mm2Tom2}"  ixz="${-6.8400465e+02*mm2Tom2}" iyy="${2.2460561e+03*mm2Tom2}" iyz="${-2.8844444e+02*mm2Tom2}" izz="${4.4895027e+03*mm2Tom2}" />
         </inertial>
         <visual>
-          <origin xyz="0 0 0" rpy="-1.570796326795 1.570796326795 0"/>
+          <origin xyz="0 0 0" rpy="0 0 0"/>
           <geometry name="LElb_visual">
-            <mesh filename="package://bigman_urdf/meshes/collada/forearms/elbow.dae" scale="1.0 1.0 1.0" />
+            <mesh filename="package://bigman_urdf/meshes/Elbow.STL" scale="0.001 -0.001 0.001" />
           </geometry>
         </visual>
         <collision>
-          <origin xyz="0 0 0" rpy="-1.570796326795 1.570796326795 0"/>
+          <origin xyz="0 0 0" rpy="0 0 0"/>
           <geometry name="LElb_collision">
-            <mesh filename="package://bigman_urdf/meshes/collada/simple/forearms/elbow.stl" scale="1.0 1.0 1.0" />
+            <mesh filename="package://bigman_urdf/meshes/simple/Elbow.STL" scale="0.001 -0.001 0.001" />
           </geometry>
         </collision>
@@ -191,5 +192,5 @@
     <origin xyz="0.036 0.0 -0.15" rpy="0 0 0" />
     <axis xyz="0 1 0" />
-    <limit velocity="4.0" effort="50" lower="-2.3562" upper="0.0" />
+    <limit velocity="6.283" effort="60" lower="-2.3562" upper="0.0" />
     <dynamics friction="0" damping="3.0"/>
   </joint>
@@ -224,5 +225,5 @@
     <origin xyz="0.036 0.0 -0.15" rpy="0 0 0" />
     <axis xyz="0 1 0" />
-    <limit velocity="4.0" effort="50" lower="-2.3562" upper="0.0" />
+    <limit velocity="6.283" effort="60" lower="-2.3562" upper="0.0" />
     <dynamics friction="0" damping="3.0"/>
   </joint>

File: bigman_urdf/urdf/parts/legs.urdf.xacro (robot description, xacro)
@@ -6,5 +6,4 @@
 <xacro:property name="PI" value="3.14159265359" />
 <xacro:property name="PI_2" value="1.57079632679" />
-<xacro:property name="SF" value="0.03937" /> <!-- Scale factor for meshes -->
 <!-- LINKS -->
 <!-- ********************RIGHT LEG******************** -->
@@ -132,5 +131,5 @@
     <visual>
       <origin xyz="0 0 0" rpy="0 0 0"/>
-      <geometry name="RHipMot_visual">
+      <geometry name="LHipMot_visual">
         <mesh filename="package://bigman_urdf/meshes/HipRoll.STL" scale="0.001 -0.001 0.001" />
       </geometry>
@@ -138,5 +137,5 @@
     <collision>
       <origin xyz="0 0 0" rpy="0 0 0"/>
-      <geometry name="RHipMot_collision">
+      <geometry name="LHipMot_collision">
         <mesh filename="package://bigman_urdf/meshes/simple/HipRoll.STL" scale="0.001 -0.001 0.001" />
       </geometry>
@@ -151,5 +150,5 @@
     <visual>
       <origin xyz="0 0 0" rpy="0 0 0"/>
-      <geometry name="RThighUpLeg_visual">
+      <geometry name="LThighUpLeg_visual">
         <mesh filename="package://bigman_urdf/meshes/HipYaw.STL" scale="0.001 -0.001 0.001" />
       </geometry>
@@ -157,5 +156,5 @@
     <collision>
       <origin xyz="0 0 0" rpy="0 0 0"/>
-      <geometry name="RThighUpLeg_collision">
+      <geometry name="LThighUpLeg_collision">
         <mesh filename="package://bigman_urdf/meshes/simple/HipYaw.STL" scale="0.001 -0.001 0.001" />
       </geometry>
@@ -170,5 +169,5 @@
     <visual>
       <origin xyz="0 0 0" rpy="0 0 0"/>
-      <geometry name="RThighLowLeg_visual">
+      <geometry name="LThighLowLeg_visual">
         <mesh filename="package://bigman_urdf/meshes/HipPitch.STL" scale="0.001 -0.001 0.001" />
       </geometry>
@@ -176,5 +175,5 @@
     <collision>
       <origin xyz="0 0 0" rpy="0 0 0"/>
-      <geometry name="RThighLowLeg_collision">
+      <geometry name="LThighLowLeg_collision">
         <mesh filename="package://bigman_urdf/meshes/simple/HipPitch.STL" scale="0.001 -0.001 0.001" />
       </geometry>
@@ -189,5 +188,5 @@
     <visual>
       <origin xyz="0 0 0" rpy="0 0 0"/>
-      <geometry name="RLowLeg_visual">
+      <geometry name="LLowLeg_visual">
         <mesh filename="package://bigman_urdf/meshes/KneePitch.STL" scale="0.001 0.001 0.001" />
       </geometry>
@@ -195,5 +194,5 @@
     <collision>
       <origin xyz="0 0 0" rpy="0 0 0"/>
-      <geometry name="RLowLeg_collision">
+      <geometry name="LLowLeg_collision">
         <mesh filename="package://bigman_urdf/meshes/simple/KneePitch.STL" scale="0.001 0.001 0.001" />
       </geometry>
@@ -208,5 +207,5 @@
     <visual>
       <origin xyz="0 0 0" rpy="0 0 0"/>
-      <geometry name="RFootmot_visual">
+      <geometry name="LFootmot_visual">
         <mesh filename="package://bigman_urdf/meshes/AnklePitch.STL" scale="0.001 -0.001 0.001" />
       </geometry>
@@ -214,5 +213,5 @@
     <collision>
       <origin xyz="0 0 0" rpy="0 0 0"/>
-      <geometry name="RFootmot_collision">
+      <geometry name="LFootmot_collision">
         <mesh filename="package://bigman_urdf/meshes/simple/AnklePitch.STL" scale="0.001 -0.001 0.001" />
       </geometry>

Commit message: Updated documentation. Added joint limits for elbow. Cleaned urdf of forearms

File: bigman_urdf/urdf/parts/arms.urdf.xacro (robot description, xacro)
@@ -192,5 +192,5 @@
     <origin xyz="0.036 0.0 -0.15" rpy="0 0 0" />
     <axis xyz="0 1 0" />
-    <limit velocity="6.283" effort="60" lower="-2.3562" upper="0.0" />
+    <limit velocity="6.283" effort="60" lower="-2.966" upper="0.523" />
     <dynamics friction="0" damping="3.0"/>
   </joint>
@@ -225,5 +225,5 @@
     <origin xyz="0.036 0.0 -0.15" rpy="0 0 0" />
     <axis xyz="0 1 0" />
-    <limit velocity="6.283" effort="60" lower="-2.3562" upper="0.0" />
+    <limit velocity="6.283" effort="60" lower="-2.966" upper="0.523" />
     <dynamics friction="0" damping="3.0"/>
   </joint>

File: bigman_urdf/urdf/parts/forearms.urdf.xacro (robot description, xacro)
@@ -3,10 +3,4 @@
 <xacro:property name="mmTom" value="0.001" />
 <xacro:property name="mm2Tom2" value="${0.001*0.001}" />
-<!-- distance from last motor to FT sensor
-		The value needs to be subtracted to the *FOrearmPlate joint z origin,
-		and in order to be compensated in the following joint and link,
-		it neeeds to be added in return to the following joint (*Wrj1) z origin
-		and to the z displacement of mass, visual and collision of *Forearm -->
-<xacro:property name="Wrj1_to_FT" value="0.0568" />
 <!-- ****************LINKS**************** -->
 <!-- ****************LEFT FOREARM**************** -->

Commit message: Added new torso. New reference frames for the shoulder. The axis of the ref frame are translated and rotated around Yaw, the joint roation axis is then roatated around x (this to simplify the implementation: the two rotations are then docupled) and to do not have to change anything from the previous version (inertia and visualization).

File: bigman_urdf/urdf/parts/arms.urdf.xacro (robot description, xacro)
@@ -166,5 +166,6 @@
     <parent link="DWYTorso"/>
     <child link="RShp"/>
-    <origin xyz="0.0 -0.2 0.0" rpy="0 0 0" />
+    <!--origin xyz="0.0 -0.2 0.0" rpy="0 0 0" /-->
+    <origin xyz="0.045646 -0.219164 0.001531" rpy="0 0 0.3491" />
     <axis xyz="0 ${cos_42} ${-sin_42}" />
     <limit velocity="6.283" effort="120" lower="-2.844" upper="2.844" />
@@ -199,6 +200,7 @@
     <parent link="DWYTorso"/>
     <child link="LShp"/>
-    <origin xyz="0.0 0.2 0.0" rpy="0 0 0" />
-    <axis xyz="0 ${cos_42} ${sin_42}" />
+    <!--origin xyz="0.0 0.2 0.0" rpy="0 0 0" /-->
+    <origin xyz="0.045646 0.219164 0.001531" rpy="0 0 -0.3491" />
+    <axis xyz="0.0 ${cos_42} ${sin_42}" />
     <limit velocity="6.283" effort="120" lower="-2.844" upper="2.844" />
     <dynamics friction="0" damping="3.0"/>

File: bigman_urdf/urdf/parts/torso.urdf.xacro (robot description, xacro)
@@ -81,5 +81,6 @@
       <origin xyz="0.0 0.0 0.0" rpy="0 0 0"/>
       <geometry name="DWYTorso_visual">
-        <mesh filename="package://bigman_urdf/meshes/Chest.STL" scale="0.001 0.001 0.001" />
+        <!--mesh filename="package://bigman_urdf/meshes/Chest.STL" scale="0.001 0.001 0.001" /-->
+        <mesh filename="package://bigman_urdf/meshes/NewChest.STL" scale="0.001 0.001 0.001" />
       </geometry>
     </visual>
@@ -87,5 +88,6 @@
       <origin xyz="0.0 0.0 0.0" rpy="0 0 0"/>
       <geometry name="DWYTorso_collision">
-        <mesh filename="package://bigman_urdf/meshes/simple/Chest.STL" scale="0.001 0.001 0.001" />
+        <!--mesh filename="package://bigman_urdf/meshes/simple/Chest.STL" scale="0.001 0.001 0.001" /-->
+        <mesh filename="package://bigman_urdf/meshes/simple/NewChest.STL" scale="0.001 0.001 0.001" />
       </geometry>
     </collision>
@@ -106,7 +108,6 @@
     <child link="DWL"/>
     <origin xyz="0.0715192 0 0.195982" rpy="0 0 0" />
-    <axis xyz="${cos_26} 0 ${sin_26}" />
+    <axis xyz="${cos_26} 0.0 ${sin_26}" />
     <limit velocity="6.283" effort="120" lower="-0.610" upper="0.610" />
-    <!-- dynamics friction="0" damping="0.3"/ -->
     <dynamics friction="0" damping="3.0"/>
 </joint>

Commit message: Added new joint limits to upper body

File: bigman_urdf/urdf/parts/arms.urdf.xacro (robot description, xacro)
@@ -6,4 +6,6 @@
 <xacro:property name="mmTom" value="0.001" />
 <xacro:property name="mm2Tom2" value="${0.001*0.001}" />
+<xacro:property name="toRad" value="${PI/180.0}" />
+<xacro:property name="safety" value="5.0" />
 <!-- LINKS -->
 <!-- RIGHT ARM -->
@@ -173,5 +175,5 @@
 </xacro:unless>
     <axis xyz="0 ${cos_42} ${-sin_42}" />
-    <limit velocity="6.283" effort="120" lower="-2.844" upper="2.844" />
+    <limit velocity="6.283" effort="120" lower="${(-163+safety)*toRad}" upper="${(161.0-safety)*toRad}" />
     <dynamics friction="0" damping="3.0"/>
 </joint>
@@ -181,5 +183,5 @@
     <origin xyz="0.0 -0.116568264 0.03364" rpy="0 0 0" />
     <axis xyz="1 0 0" />
-    <limit velocity="6.283" effort="120" lower="-3.699" upper="-0.052" />
+    <limit velocity="6.283" effort="120" lower="${(-221.0+safety)*toRad}" upper="${(-7.0-safety)*toRad}" />
     <dynamics friction="0" damping="3.0"/>
 </joint>
@@ -189,5 +191,5 @@
     <origin xyz="0.0 0.0 -0.222" rpy="0 0 0" />
     <axis xyz="0 0 1" />
-    <limit velocity="6.283" effort="120" lower="-2.844" upper="2.844" />
+    <limit velocity="6.283" effort="120" lower="${(-164+safety)*toRad}" upper="${(162.0-safety)*toRad}" />
     <dynamics friction="0" damping="3.0"/>
 </joint>
@@ -197,5 +199,5 @@
     <origin xyz="0.036 0.0 -0.15" rpy="0 0 0" />
     <axis xyz="0 1 0" />
-    <limit velocity="6.283" effort="60" lower="-2.966" upper="0.523" />
+    <limit velocity="6.283" effort="60" lower="${(-170.0+safety)*toRad}" upper="${(34.0-safety)*toRad}" />
     <dynamics friction="0" damping="3.0"/>
   </joint>
@@ -211,5 +213,5 @@
 </xacro:unless>
     <axis xyz="0.0 ${cos_42} ${sin_42}" />
-    <limit velocity="6.283" effort="120" lower="-2.844" upper="2.844" />
+    <limit velocity="6.283" effort="120" lower="${(-165.0+safety)*toRad}" upper="${(160.0-safety)*toRad}" />
     <dynamics friction="0" damping="3.0"/>
 </joint>
@@ -219,5 +221,5 @@
     <origin xyz="0.0 0.116568264 0.03364" rpy="0 0 0" />
     <axis xyz="1 0 0" />
-    <limit velocity="6.283" effort="120" lower="0.052" upper="3.699" />
+    <limit velocity="6.283" effort="120" lower="${(5.0+safety)*toRad}" upper="${(221.0-safety)*toRad}" />
     <dynamics friction="0" damping="3.0"/>
 </joint>
@@ -227,5 +229,5 @@
     <origin xyz="0.0 0.0 -0.222" rpy="0 0 0" />
     <axis xyz="0 0 1" />
-    <limit velocity="6.283" effort="120" lower="-2.844" upper="2.844" />
+    <limit velocity="6.283" effort="120" lower="${(-163.0+safety)*toRad}" upper="${(163.0-safety)*toRad}" />
     <dynamics friction="0" damping="3.0"/>
 </joint>
@@ -235,5 +237,5 @@
     <origin xyz="0.036 0.0 -0.15" rpy="0 0 0" />
     <axis xyz="0 1 0" />
-    <limit velocity="6.283" effort="60" lower="-2.966" upper="0.523" />
+    <limit velocity="6.283" effort="60" lower="${(-170.0+safety)*toRad}" upper="${(34.0-safety)*toRad}" />
     <dynamics friction="0" damping="3.0"/>
   </joint>

File: bigman_urdf/urdf/parts/torso.urdf.xacro (robot description, xacro)
@@ -8,4 +8,6 @@
 <xacro:property name="cos_26" value="0.89879991307" />
 <xacro:property name="sin_26" value="0.43835911792" />
+<xacro:property name="toRad" value="${PI/180.0}" />
+<xacro:property name="safety" value="5.0" />
 <!-- LINKS -->
 <!-- This links are defined in order to be compliant with http://www.ros.org/reps/rep-0120.html#coordinate-frames
@@ -91,5 +93,5 @@
     <origin xyz="0.0715192 0 0.195982" rpy="0 0 0" />
     <axis xyz="${cos_26} 0 ${sin_26}" />
-    <limit velocity="6.283" effort="120" lower="-0.610" upper="0.610" />
+    <limit velocity="6.283" effort="120" lower="${(-35.0+safety)*toRad}" upper="${(35.0-safety)*toRad}" />
     <dynamics friction="0" damping="3.0"/>
 </joint>
@@ -99,5 +101,5 @@
     <origin xyz="0 0 0" rpy="0 0 0" />
     <axis xyz="0 1 0" />
-    <limit velocity="6.283" effort="220" lower="-0.349" upper="1.396" />
+    <limit velocity="6.283" effort="220" lower="${(-20.0+safety)*toRad}" upper="${(80.0-safety)*toRad}" />
     <dynamics friction="0" damping="3.0"/>
   </joint>
@@ -107,5 +109,5 @@
     <origin xyz="0 0 0.22275" rpy="0 0 0" />
     <axis xyz="0 0 1" />
-    <limit velocity="6.283" effort="120" lower="-2.844" upper="2.844" />
+    <limit velocity="6.283" effort="120" lower="${(-120.0+safety)*toRad}" upper="${(120.0-safety)*toRad}" />
     <dynamics friction="0" damping="3.0"/>
   </joint>

Commit message: Removed safety magins. Joints limits for torso and arms (no forearms) are the same as robotMotorGui

File: bigman_urdf/urdf/parts/arms.urdf.xacro (robot description, xacro)
@@ -7,5 +7,5 @@
 <xacro:property name="mm2Tom2" value="${0.001*0.001}" />
 <xacro:property name="toRad" value="${PI/180.0}" />
-<xacro:property name="safety" value="5.0" />
+<xacro:property name="safety" value="0.0" />
 <!-- LINKS -->
 <!-- RIGHT ARM -->
@@ -175,5 +175,5 @@
 </xacro:unless>
     <axis xyz="0 ${cos_42} ${-sin_42}" />
-    <limit velocity="6.283" effort="120" lower="${(-163+safety)*toRad}" upper="${(161.0-safety)*toRad}" />
+    <limit velocity="6.283" effort="120" lower="${-163*toRad}" upper="${161.0*toRad}" />
     <dynamics friction="0" damping="3.0"/>
 </joint>
@@ -183,5 +183,5 @@
     <origin xyz="0.0 -0.116568264 0.03364" rpy="0 0 0" />
     <axis xyz="1 0 0" />
-    <limit velocity="6.283" effort="120" lower="${(-221.0+safety)*toRad}" upper="${(-7.0-safety)*toRad}" />
+    <limit velocity="6.283" effort="120" lower="${-221.0*toRad}" upper="${-7.0*toRad}" />
     <dynamics friction="0" damping="3.0"/>
 </joint>
@@ -191,5 +191,5 @@
     <origin xyz="0.0 0.0 -0.222" rpy="0 0 0" />
     <axis xyz="0 0 1" />
-    <limit velocity="6.283" effort="120" lower="${(-164+safety)*toRad}" upper="${(162.0-safety)*toRad}" />
+    <limit velocity="6.283" effort="120" lower="${-164*toRad}" upper="${162.0*toRad}" />
     <dynamics friction="0" damping="3.0"/>
 </joint>
@@ -199,5 +199,5 @@
     <origin xyz="0.036 0.0 -0.15" rpy="0 0 0" />
     <axis xyz="0 1 0" />
-    <limit velocity="6.283" effort="60" lower="${(-170.0+safety)*toRad}" upper="${(34.0-safety)*toRad}" />
+    <limit velocity="6.283" effort="60" lower="${-170.0*toRad}" upper="${34.0*toRad}" />
     <dynamics friction="0" damping="3.0"/>
   </joint>
@@ -213,5 +213,5 @@
 </xacro:unless>
     <axis xyz="0.0 ${cos_42} ${sin_42}" />
-    <limit velocity="6.283" effort="120" lower="${(-165.0+safety)*toRad}" upper="${(160.0-safety)*toRad}" />
+    <limit velocity="6.283" effort="120" lower="${-165.0*toRad}" upper="${160.0*toRad}" />
     <dynamics friction="0" damping="3.0"/>
 </joint>
@@ -221,5 +221,5 @@
     <origin xyz="0.0 0.116568264 0.03364" rpy="0 0 0" />
     <axis xyz="1 0 0" />
-    <limit velocity="6.283" effort="120" lower="${(5.0+safety)*toRad}" upper="${(221.0-safety)*toRad}" />
+    <limit velocity="6.283" effort="120" lower="${5.0*toRad}" upper="${221.0*toRad}" />
     <dynamics friction="0" damping="3.0"/>
 </joint>
@@ -229,5 +229,5 @@
     <origin xyz="0.0 0.0 -0.222" rpy="0 0 0" />
     <axis xyz="0 0 1" />
-    <limit velocity="6.283" effort="120" lower="${(-163.0+safety)*toRad}" upper="${(163.0-safety)*toRad}" />
+    <limit velocity="6.283" effort="120" lower="${-163.0*toRad}" upper="${163.0*toRad}" />
     <dynamics friction="0" damping="3.0"/>
 </joint>
@@ -237,5 +237,5 @@
     <origin xyz="0.036 0.0 -0.15" rpy="0 0 0" />
     <axis xyz="0 1 0" />
-    <limit velocity="6.283" effort="60" lower="${(-170.0+safety)*toRad}" upper="${(34.0-safety)*toRad}" />
+    <limit velocity="6.283" effort="60" lower="${-170.0*toRad}" upper="${34.0*toRad}" />
     <dynamics friction="0" damping="3.0"/>
   </joint>

File: bigman_urdf/urdf/parts/torso.urdf.xacro (robot description, xacro)
@@ -9,5 +9,4 @@
 <xacro:property name="sin_26" value="0.43835911792" />
 <xacro:property name="toRad" value="${PI/180.0}" />
-<xacro:property name="safety" value="5.0" />
 <!-- LINKS -->
 <!-- This links are defined in order to be compliant with http://www.ros.org/reps/rep-0120.html#coordinate-frames
@@ -93,5 +92,5 @@
     <origin xyz="0.0715192 0 0.195982" rpy="0 0 0" />
     <axis xyz="${cos_26} 0 ${sin_26}" />
-    <limit velocity="6.283" effort="120" lower="${(-35.0+safety)*toRad}" upper="${(35.0-safety)*toRad}" />
+    <limit velocity="6.283" effort="120" lower="${-35.0*toRad}" upper="${35.0*toRad}" />
     <dynamics friction="0" damping="3.0"/>
 </joint>
@@ -101,5 +100,5 @@
     <origin xyz="0 0 0" rpy="0 0 0" />
     <axis xyz="0 1 0" />
-    <limit velocity="6.283" effort="220" lower="${(-20.0+safety)*toRad}" upper="${(80.0-safety)*toRad}" />
+    <limit velocity="6.283" effort="220" lower="${-20.0*toRad}" upper="${80.0*toRad}" />
     <dynamics friction="0" damping="3.0"/>
   </joint>
@@ -109,5 +108,5 @@
     <origin xyz="0 0 0.22275" rpy="0 0 0" />
     <axis xyz="0 0 1" />
-    <limit velocity="6.283" effort="120" lower="${(-120.0+safety)*toRad}" upper="${(120.0-safety)*toRad}" />
+    <limit velocity="6.283" effort="120" lower="${-120.0*toRad}" upper="${120.0*toRad}" />
     <dynamics friction="0" damping="3.0"/>
   </joint>
