Commit message: Added NEW ELBOWS

File: bigman_urdf/urdf/parts/arms.urdf.xacro (robot description, xacro)
@@ -72,7 +72,7 @@
 <link name ="RElb">
         <inertial>
-          <origin xyz="${-5.5754915e+01*mmTom} ${-7.5826040*mmTom} ${-4.3820396e+01*mmTom}" rpy="0 0 0"/>
-          <mass value="8.6765385e-01"/>
-          <inertia ixx="${4.0395238e+03*mm2Tom2}"  ixy="${3.4973136e+02*mm2Tom2}"  ixz="${-6.8400465e+02*mm2Tom2}" iyy="${2.2460561e+03*mm2Tom2}" iyz="${2.8844444e+02*mm2Tom2}" izz="${4.4895027e+03*mm2Tom2}" />
+          <origin xyz="${-6.3655533e+01*mmTom} ${-4.4231462*mmTom} ${-1.3715758e+02*mmTom}" rpy="0 0 0"/>
+          <mass value="1.4874155"/>
+          <inertia ixx="${1.7815816e+04*mm2Tom2}"  ixy="${4.0170943e+02*mm2Tom2}"  ixz="${-2.4568192e+03*mm2Tom2}" iyy="${1.5706187e+04*mm2Tom2}" iyz="${8.9862025e+02*mm2Tom2}" izz="${6.2045522e+03*mm2Tom2}" />
         </inertial>
         <visual>
@@ -153,7 +153,7 @@
     <link name ="LElb">
         <inertial>
-          <origin xyz="${-5.5754915e+01*mmTom} ${7.5826040*mmTom} ${-4.3820396e+01*mmTom}" rpy="0 0 0"/>
-          <mass value="8.6765385e-01"/>
-          <inertia ixx="${4.0395238e+03*mm2Tom2}"  ixy="${-3.4973136e+02*mm2Tom2}"  ixz="${-6.8400465e+02*mm2Tom2}" iyy="${2.2460561e+03*mm2Tom2}" iyz="${-2.8844444e+02*mm2Tom2}" izz="${4.4895027e+03*mm2Tom2}" />
+          <origin xyz="${-6.3655533e+01*mmTom} ${4.4231462*mmTom} ${-1.3715758e+02*mmTom}" rpy="0 0 0"/>
+          <mass value="1.4874155"/>
+          <inertia ixx="${1.7815816e+04*mm2Tom2}"  ixy="${-4.0170943e+02*mm2Tom2}"  ixz="${-2.4568192e+03*mm2Tom2}" iyy="${1.5706187e+04*mm2Tom2}" iyz="${-8.9862025e+02*mm2Tom2}" izz="${6.2045522e+03*mm2Tom2}" />
         </inertial>
         <visual>

File: bigman_urdf/urdf/parts/forearms.urdf.xacro (robot description, xacro)
@@ -176,5 +176,5 @@
     <parent link="LElb"/>
     <child link="LForearm"/>
-    <origin xyz="-0.075 0.0 -0.1955" rpy="0 0 0"/>
+    <origin xyz="-0.075 0.0 -0.3745" rpy="0 0 0"/>
     <axis xyz="0 0 1" />
     <limit velocity="6.283" effort="60" lower="-2.529" upper="2.529" />
@@ -211,5 +211,5 @@
     <parent link="RElb"/>
     <child link="RForearm"/>
-    <origin xyz="-0.075 0.0 -0.1955" rpy="0 0 0"/>
+    <origin xyz="-0.075 0.0 -0.3745" rpy="0 0 0"/>
     <axis xyz="0 0 1" />
     <limit velocity="6.283" effort="60" lower="-2.529" upper="2.529" />

Commit message: Set back old forearms

File: bigman_urdf/urdf/parts/arms.urdf.xacro (robot description, xacro)
@@ -72,7 +72,7 @@
 <link name ="RElb">
         <inertial>
-          <origin xyz="${-6.3655533e+01*mmTom} ${-4.4231462*mmTom} ${-1.3715758e+02*mmTom}" rpy="0 0 0"/>
-          <mass value="1.4874155"/>
-          <inertia ixx="${1.7815816e+04*mm2Tom2}"  ixy="${4.0170943e+02*mm2Tom2}"  ixz="${-2.4568192e+03*mm2Tom2}" iyy="${1.5706187e+04*mm2Tom2}" iyz="${8.9862025e+02*mm2Tom2}" izz="${6.2045522e+03*mm2Tom2}" />
+          <origin xyz="${-5.5754915e+01*mmTom} ${-7.5826040*mmTom} ${-4.3820396e+01*mmTom}" rpy="0 0 0"/>
+          <mass value="8.6765385e-01"/>
+          <inertia ixx="${4.0395238e+03*mm2Tom2}"  ixy="${3.4973136e+02*mm2Tom2}"  ixz="${-6.8400465e+02*mm2Tom2}" iyy="${2.2460561e+03*mm2Tom2}" iyz="${2.8844444e+02*mm2Tom2}" izz="${4.4895027e+03*mm2Tom2}" />
         </inertial>
         <visual>
@@ -153,7 +153,7 @@
     <link name ="LElb">
         <inertial>
-          <origin xyz="${-6.3655533e+01*mmTom} ${4.4231462*mmTom} ${-1.3715758e+02*mmTom}" rpy="0 0 0"/>
-          <mass value="1.4874155"/>
-          <inertia ixx="${1.7815816e+04*mm2Tom2}"  ixy="${-4.0170943e+02*mm2Tom2}"  ixz="${-2.4568192e+03*mm2Tom2}" iyy="${1.5706187e+04*mm2Tom2}" iyz="${-8.9862025e+02*mm2Tom2}" izz="${6.2045522e+03*mm2Tom2}" />
+          <origin xyz="${-5.5754915e+01*mmTom} ${7.5826040*mmTom} ${-4.3820396e+01*mmTom}" rpy="0 0 0"/>
+          <mass value="8.6765385e-01"/>
+          <inertia ixx="${4.0395238e+03*mm2Tom2}"  ixy="${-3.4973136e+02*mm2Tom2}"  ixz="${-6.8400465e+02*mm2Tom2}" iyy="${2.2460561e+03*mm2Tom2}" iyz="${-2.8844444e+02*mm2Tom2}" izz="${4.4895027e+03*mm2Tom2}" />
         </inertial>
         <visual>
@@ -202,5 +202,5 @@
     <dynamics friction="0" damping="3.0"/>
 </joint>
-  <joint name="RElbj" type="revolute">
+   <joint name="RElbj" type="revolute">
     <parent link="RShy"/>
     <child link="RElb"/>

File: bigman_urdf/urdf/parts/forearms.urdf.xacro (robot description, xacro)
@@ -176,5 +176,5 @@
     <parent link="LElb"/>
     <child link="LForearm"/>
-    <origin xyz="-0.075 0.0 -0.3745" rpy="0 0 0"/>
+    <origin xyz="-0.075 0.0 -0.1955" rpy="0 0 0"/>
     <axis xyz="0 0 1" />
     <limit velocity="6.283" effort="60" lower="-2.529" upper="2.529" />
@@ -211,5 +211,5 @@
     <parent link="RElb"/>
     <child link="RForearm"/>
-    <origin xyz="-0.075 0.0 -0.3745" rpy="0 0 0"/>
+    <origin xyz="-0.075 0.0 -0.1955" rpy="0 0 0"/>
     <axis xyz="0 0 1" />
     <limit velocity="6.283" effort="60" lower="-2.529" upper="2.529" />

Commit message: Added new joint limits

File: bigman_urdf/urdf/parts/arms.urdf.xacro (robot description, xacro)
@@ -183,5 +183,6 @@
 </xacro:unless>
     <axis xyz="0 ${cos_42} ${-sin_42}" />
-    <limit velocity="6.283" effort="120" lower="${-163*toRad}" upper="${161.0*toRad}" />
+    <!--limit velocity="6.283" effort="120" lower="${-163*toRad}" upper="${161.0*toRad}" /-->
+    <limit velocity="6.283" effort="120" lower="${-57*toRad}" upper="${89.0*toRad}" />
     <dynamics friction="0" damping="3.0"/>
 </joint>
@@ -191,5 +192,6 @@
     <origin xyz="0.0 -0.116568264 0.03364" rpy="0 0 0" />
     <axis xyz="1 0 0" />
-    <limit velocity="6.283" effort="120" lower="${-221.0*toRad}" upper="${-7.0*toRad}" />
+    <!--limit velocity="6.283" effort="120" lower="${-221.0*toRad}" upper="${-7.0*toRad}" /-->
+    <limit velocity="6.283" effort="120" lower="${-170.0*toRad}" upper="${-7.0*toRad}" />
     <dynamics friction="0" damping="3.0"/>
 </joint>
@@ -221,5 +223,6 @@
 </xacro:unless>
     <axis xyz="0.0 ${cos_42} ${sin_42}" />
-    <limit velocity="6.283" effort="120" lower="${-165.0*toRad}" upper="${160.0*toRad}" />
+    <!--limit velocity="6.283" effort="120" lower="${-165.0*toRad}" upper="${160.0*toRad}" /-->
+    <limit velocity="6.283" effort="120" lower="${-57.0*toRad}" upper="${89.0*toRad}" />
     <dynamics friction="0" damping="3.0"/>
 </joint>
@@ -229,5 +232,6 @@
     <origin xyz="0.0 0.116568264 0.03364" rpy="0 0 0" />
     <axis xyz="1 0 0" />
-    <limit velocity="6.283" effort="120" lower="${5.0*toRad}" upper="${221.0*toRad}" />
+    <!--limit velocity="6.283" effort="120" lower="${5.0*toRad}" upper="${221.0*toRad}" /-->
+    <limit velocity="6.283" effort="120" lower="${5.0*toRad}" upper="${170.0*toRad}" />
     <dynamics friction="0" damping="3.0"/>
 </joint>

Commit message: arms, neck and torso joint limits updated.

File: bigman_urdf/urdf/parts/arms.urdf.xacro (robot description, xacro)
@@ -184,5 +184,5 @@
     <axis xyz="0 ${cos_42} ${-sin_42}" />
     <!--limit velocity="6.283" effort="120" lower="${-163*toRad}" upper="${161.0*toRad}" /-->
-    <limit velocity="6.283" effort="120" lower="${-57*toRad}" upper="${89.0*toRad}" />
+    <limit velocity="6.283" effort="120" lower="${-55*toRad}" upper="${85.0*toRad}" /> <!-- <limit velocity="6.283" effort="120" lower="${-57*toRad}" upper="${89.0*toRad}" /> -->
     <dynamics friction="0" damping="3.0"/>
 </joint>
@@ -193,5 +193,5 @@
     <axis xyz="1 0 0" />
     <!--limit velocity="6.283" effort="120" lower="${-221.0*toRad}" upper="${-7.0*toRad}" /-->
-    <limit velocity="6.283" effort="120" lower="${-170.0*toRad}" upper="${-7.0*toRad}" />
+    <limit velocity="6.283" effort="120" lower="${-120.0*toRad}" upper="${-7.0*toRad}" />
     <dynamics friction="0" damping="3.0"/>
 </joint>
@@ -224,5 +224,5 @@
     <axis xyz="0.0 ${cos_42} ${sin_42}" />
     <!--limit velocity="6.283" effort="120" lower="${-165.0*toRad}" upper="${160.0*toRad}" /-->
-    <limit velocity="6.283" effort="120" lower="${-57.0*toRad}" upper="${89.0*toRad}" />
+    <limit velocity="6.283" effort="120" lower="${-55.0*toRad}" upper="${85.0*toRad}" /><!-- <limit velocity="6.283" effort="120" lower="${-57*toRad}" upper="${89.0*toRad}" /> -->
     <dynamics friction="0" damping="3.0"/>
 </joint>
@@ -233,5 +233,5 @@
     <axis xyz="1 0 0" />
     <!--limit velocity="6.283" effort="120" lower="${5.0*toRad}" upper="${221.0*toRad}" /-->
-    <limit velocity="6.283" effort="120" lower="${5.0*toRad}" upper="${170.0*toRad}" />
+    <limit velocity="6.283" effort="120" lower="${5.0*toRad}" upper="${120.0*toRad}" />
     <dynamics friction="0" damping="3.0"/>
 </joint>

File: bigman_urdf/urdf/parts/neck.urdf.xacro (robot description, xacro)
@@ -55,6 +55,6 @@
     <origin xyz="0 0 0" rpy="0 0 0" />
     <axis xyz="0 0 1" />
-    <limit velocity="6.283" effort="120" lower="${(-175.0)*toRad}" upper="${(175.0)*toRad}" />
-    <!--limit velocity="6.283" effort="120" lower="${(-35.0)*toRad}" upper="${(35.0)*toRad}" /-->
+<!--     <limit velocity="6.283" effort="120" lower="${(-175.0)*toRad}" upper="${(175.0)*toRad}" /> -->
+    <limit velocity="6.283" effort="120" lower="${(-35.0)*toRad}" upper="${(35.0)*toRad}" />
     <dynamics friction="0" damping="3.0"/>
 </joint>
@@ -65,5 +65,5 @@
     <axis xyz="0 1 0" />
     <!--limit velocity="6.283" effort="120" lower="${(-30.0)*toRad}" upper="${(70.0)*toRad}" /-->
-    <limit velocity="6.283" effort="120" lower="${(-25.0)*toRad}" upper="${(60.0)*toRad}" />
+    <limit velocity="6.283" effort="120" lower="${(-15.0)*toRad}" upper="${(60.0)*toRad}" />
     <dynamics friction="0" damping="3.0"/>
 </joint>

File: bigman_urdf/urdf/parts/torso.urdf.xacro (robot description, xacro)
@@ -56,6 +56,6 @@
   <link name ="DWYTorso">
     <inertial>
-      <origin xyz="0.02049278 -0.00000767 -0.03249378" rpy="0 0 0"/>
-      <mass value="7.31313212"/>
+        <origin xyz="0.0 0.00 0.3" rpy="0 0 0"/>
+        <mass value="26"/>
       <inertia ixx="0.18629757"  ixy="0.00008160"  ixz="0.00030250" iyy="0.02013829" iyz="-0.00001790" izz="0.18850541" />
     </inertial>
@@ -155,5 +155,5 @@
     <origin xyz="0.1115 0 0.195982" rpy="0 0 0" />
     <axis xyz="${cos_26} 0 ${sin_26}" />
-    <limit velocity="6.283" effort="120" lower="${-35.0*toRad}" upper="${35.0*toRad}" />
+    <limit velocity="6.283" effort="120" lower="${-15.0*toRad}" upper="${15.0*toRad}" />
     <dynamics friction="0" damping="3.0"/>
 </joint>
@@ -163,5 +163,5 @@
     <origin xyz="0 0 0" rpy="0 0 0" />
     <axis xyz="0 1 0" />
-    <limit velocity="6.283" effort="220" lower="${-20.0*toRad}" upper="${80.0*toRad}" />
+    <limit velocity="6.283" effort="220" lower="${-10.0*toRad}" upper="${40.0*toRad}" />
     <dynamics friction="0" damping="3.0"/>
   </joint>
@@ -171,5 +171,5 @@
     <origin xyz="0 0 0.22275" rpy="0 0 0" />
     <axis xyz="0 0 1" />
-    <limit velocity="6.283" effort="120" lower="${-120.0*toRad}" upper="${120.0*toRad}" />
+    <limit velocity="6.283" effort="120" lower="${-100.0*toRad}" upper="${100.0*toRad}" />
     <dynamics friction="0" damping="3.0"/>
   </joint>

Commit message: Fixed torque limit on elbow

File: bigman_urdf/urdf/parts/arms.urdf.xacro (robot description, xacro)
@@ -217,5 +217,5 @@
     <origin xyz="0.036 0.0 -0.15" rpy="0 0 0" />
     <axis xyz="0 1 0" />
-    <limit velocity="6.283" effort="60" lower="${-170.0*toRad}" upper="${34.0*toRad}" />
+    <limit velocity="6.283" effort="120" lower="${-170.0*toRad}" upper="${34.0*toRad}" />
     <dynamics friction="0" damping="3.0"/>
   </joint>
@@ -265,5 +265,5 @@
     <origin xyz="0.036 0.0 -0.15" rpy="0 0 0" />
     <axis xyz="0 1 0" />
-    <limit velocity="6.283" effort="60" lower="${-170.0*toRad}" upper="${34.0*toRad}" />
+    <limit velocity="6.283" effort="120" lower="${-170.0*toRad}" upper="${34.0*toRad}" />
     <dynamics friction="0" damping="3.0"/>
   </joint>
