Commit message: Added inertia, CoM and Mass to left and right foot

File: bigman_urdf/urdf/parts/legs.urdf.xacro (robot description, xacro)
@@ -103,7 +103,7 @@
   <link name ="RFoot">
      <inertial>
-        <origin xyz="0.00969210464 -0.0090460227 -0.043062308" rpy="0 0 0"/>
-        <mass value="0.66646684"/>
-        <inertia ixx="0.0012944808"  ixy="-9.2387693E-5"  ixz="2.0080105E-4" iyy="0.0015851846" iyz="2.7599327E-4" izz="0.0013326766" />
+        <origin xyz="0.01282904 -0.00463694 -0.10109499" rpy="0 0 0"/>
+        <mass value="3.33109981"/>
+        <inertia ixx="0.01006627"  ixy="-0.00051955"  ixz="-0.00374069" iyy="0.02882577" iyz="0.00044505" izz="0.02819025" />
       </inertial>
     <visual>
@@ -218,7 +218,7 @@
   <link name ="LFoot">
       <inertial>
-        <origin xyz="0.0096921046 0.0090460227 -0.043062308" rpy="0 0 0"/>
-        <mass value="0.66646684"/>
-        <inertia ixx="0.0012944808"  ixy="9.2387693E-5"  ixz="2.0080105E-4" iyy="0.0015851846" iyz="-2.7599327E-4" izz="0.0013326766" />
+        <origin xyz="0.01282904 -0.00463694 -0.10109499" rpy="0 0 0"/>
+        <mass value="3.33109981"/>
+        <inertia ixx="0.01006627"  ixy="0.00051955"  ixz="-0.00374069" iyy="0.02882577" iyz="-0.00044505" izz="0.02819025" />
       </inertial>
       <visual>

Commit message: Added R/L HipYaw leg CoM, Inertia, Mass, visual and collision

File: bigman_urdf/urdf/parts/legs.urdf.xacro (robot description, xacro)
@@ -30,18 +30,18 @@
   <link name ="RThighUpLeg">
     <inertial>
-      <origin xyz="0.0012591632 -0.016896372 -0.058903336" rpy="0 0 0"/>
-      <mass value="1.0246101"/>
-      <inertia ixx="9.165719E-4"  ixy="-1.4449904E-6"  ixz="-1.6685011E-5" iyy="0.00104849584" iyz="2.5492874E-5" izz="6.8637197E-4" />
-    </inertial>
-    <visual>
-      <origin xyz="0.0 0.0726 -0.52" rpy="0 0 ${PI}"/>
+      <origin xyz="${-5.2929709*mmTom} ${-2.2561833e+01*mmTom} ${5.6701669*mmTom}" rpy="0 0 0"/>
+      <mass value="3.2402068"/>
+      <inertia ixx="${1.0102097e+04*mm2Tom2}"  ixy="${1.0858487e+02*mm2Tom2}"  ixz="${2.5291395e+02*mm2Tom2}" iyy="${6.7147000e+03*mm2Tom2}" iyz="${8.3447072e+01*mm2Tom2}" izz="${1.0485130e+04*mm2Tom2}" />
+    </inertial>
+    <visual>
+      <origin xyz="0 0 0" rpy="0 0 0"/>
       <geometry name="RThighUpLeg_visual">
-        <mesh filename="package://bigman_urdf/meshes/collada/asm0001_collada_19_prt.dae" scale="${SF} ${SF} ${SF}" />
-      </geometry>
-    </visual>
-    <collision>
-      <origin xyz="0.0 0.0726 -0.52" rpy="0 0 ${PI}"/>
+        <mesh filename="package://bigman_urdf/meshes/HipYaw.STL" scale="0.001 0.001 0.001" />
+      </geometry>
+    </visual>
+    <collision>
+      <origin xyz="0 0 0" rpy="0 0 0"/>
       <geometry name="RThighUpLeg_collision">
-        <mesh filename="package://bigman_urdf/meshes/collada/simple/simple_asm0001_collada_19_prt.stl" scale="${SF} ${SF} ${SF}" />
+        <mesh filename="package://bigman_urdf/meshes/simple/HipYaw.STL" scale="0.001 0.001 0.001" />
       </geometry>
     </collision>
@@ -145,18 +145,18 @@
   <link name ="LThighUpLeg">
     <inertial>
-      <origin xyz="0.0012591632 0.016896372 -0.058903336" rpy="0 0 0"/>
-      <mass value="1.0246101"/>
-      <inertia ixx="9.165719E-4"  ixy="1.4449904E-6"  ixz="-1.6685011E-5" iyy="0.00104849584" iyz="-2.5492874E-5" izz="6.8637197E-4" />
-    </inertial>
-    <visual>
-      <origin xyz="0.0 -0.0726 -0.52" rpy="0 0 ${PI}"/>
-      <geometry name="LThighUpLeg_visual">
-        <mesh filename="package://bigman_urdf/meshes/collada/asm0001_collada_05_prt.dae" scale="${SF} ${SF} ${SF}" />
-      </geometry>
-    </visual>
-    <collision>
-      <origin xyz="0.0 -0.0726 -0.52" rpy="0 0 ${PI}"/>
-      <geometry name="LThighUpLeg_collision">
-        <mesh filename="package://bigman_urdf/meshes/collada/simple/simple_asm0001_collada_05_prt.stl" scale="${SF} ${SF} ${SF}" />
+      <origin xyz="${-5.2929709*mmTom} ${2.2561833e+01*mmTom} ${5.6701669*mmTom}" rpy="0 0 0"/>
+      <mass value="3.2402068"/>
+      <inertia ixx="${1.0102097e+04*mm2Tom2}"  ixy="${-1.0858487e+02*mm2Tom2}"  ixz="${2.5291395e+02*mm2Tom2}" iyy="${6.7147000e+03*mm2Tom2}" iyz="${-8.3447072e+01*mm2Tom2}" izz="${1.0485130e+04*mm2Tom2}" />
+    </inertial>
+    <visual>
+      <origin xyz="0 0 0" rpy="0 0 0"/>
+      <geometry name="RThighUpLeg_visual">
+        <mesh filename="package://bigman_urdf/meshes/HipYaw.STL" scale="0.001 -0.001 0.001" />
+      </geometry>
+    </visual>
+    <collision>
+      <origin xyz="0 0 0" rpy="0 0 0"/>
+      <geometry name="RThighUpLeg_collision">
+        <mesh filename="package://bigman_urdf/meshes/simple/HipYaw.STL" scale="0.001 -0.001 0.001" />
       </geometry>
     </collision>
@@ -259,6 +259,6 @@
     <parent link="RThighUpLeg"/>
     <child link="RThighLowLeg"/>
-    <origin xyz="0.0 0.0 -0.1024" rpy="0 0 0" />
-    <axis xyz="0 0 1" />
+    <origin xyz="0.0 0.0 0.0" rpy="0 0 0" />
+    <axis xyz="0 1 0" />
     <limit velocity="4.0" effort="50" lower="-0.8727" upper="0.8727" />
     <dynamics friction="0" damping="3.0"/>
@@ -308,6 +308,6 @@
     <parent link="LThighUpLeg"/>
     <child link="LThighLowLeg"/>
-    <origin xyz="0.0 0.0 -0.1024" rpy="0 0 0" />
-    <axis xyz="0 0 1" />
+    <origin xyz="0.0 0.0 0.0" rpy="0 0 0" />
+    <axis xyz="0 1 0" />
     <limit velocity="4.0" effort="50" lower="-0.8727" upper="0.8727" />
     <dynamics friction="0" damping="3.0"/>

Commit message: Added L/R AnklePitch Visualization, Collision, CoM and Inertia

File: bigman_urdf/urdf/parts/legs.urdf.xacro (robot description, xacro)
@@ -87,18 +87,18 @@
   <link name ="RFootmot">
     <inertial>
-      <origin xyz="8.8067281E-4 -9.2224881E-4 2.3038476E-4" rpy="0 0 0"/>
-      <mass value="0.72992131"/>
-      <inertia ixx="3.2034425E-4"  ixy="7.6346303E-6"  ixz="2.5430158E-7" iyy="3.6584358E-4" iyz="-3.6889276E-6" izz="3.6065156E-4" />
-    </inertial>
-    <visual>
-      <origin xyz="0.0 0.0726 -0.0932" rpy="0 0 ${PI}"/>
+      <origin xyz="${-2.2024173e+01*mmTom} ${2.5677238*mmTom} ${9.4588455e-01*mmTom}" rpy="0 0 0"/>
+      <mass value="3.2844159"/>
+      <inertia ixx="${7.5550679e+03*mm2Tom2}"  ixy="${6.7488292e+02*mm2Tom2}"  ixz="${5.8332889e+01*mm2Tom2}" iyy="${1.1241163e+04*mm2Tom2}" iyz="${-1.4552081e+02*mm2Tom2}" izz="${1.3391865e+04*mm2Tom2}" />
+    </inertial>
+    <visual>
+      <origin xyz="0 0 0" rpy="0 0 0"/>
       <geometry name="RFootmot_visual">
-        <mesh filename="package://bigman_urdf/meshes/collada/asm0001_collada_16_prt.dae" scale="${SF} ${SF} ${SF}" />
-      </geometry>
-    </visual>
-    <collision>
-      <origin xyz="0.0 0.0726 -0.0932" rpy="0 0 ${PI}"/>
+        <mesh filename="package://bigman_urdf/meshes/AnklePitch.STL" scale="0.001 0.001 0.001" />
+      </geometry>
+    </visual>
+    <collision>
+      <origin xyz="0 0 0" rpy="0 0 0"/>
       <geometry name="RFootmot_collision">
-        <mesh filename="package://bigman_urdf/meshes/collada/simple/simple_asm0001_collada_16_prt.stl" scale="${SF} ${SF} ${SF}" />
+        <mesh filename="package://bigman_urdf/meshes/simple/AnklePitch.STL" scale="0.001 0.001 0.001" />
       </geometry>
     </collision>
@@ -202,18 +202,18 @@
   <link name ="LFootmot">
     <inertial>
-      <origin xyz="8.8067281E-4 9.2224881E-4 2.3038476E-4" rpy="0 0 0"/>
-      <mass value="0.72992131"/>
-      <inertia ixx="3.2034425E-4"  ixy="-7.6346303E-6"  ixz="2.5430158E-7" iyy="3.6584358E-4" iyz="3.6889276E-6" izz="3.6065156E-4" />
-    </inertial>
-    <visual>
-      <origin xyz="0.0 -0.0726 -0.0932" rpy="0 0 ${PI}"/>
-      <geometry name="LFootmot_visual">
-        <mesh filename="package://bigman_urdf/meshes/collada/asm0001_collada_02_prt.dae" scale="${SF} ${SF} ${SF}" />
-      </geometry>
-    </visual>
-    <collision>
-      <origin xyz="0.0 -0.0726 -0.0932" rpy="0 0 ${PI}"/>
-      <geometry name="LFootmot_collision">
-        <mesh filename="package://bigman_urdf/meshes/collada/simple/simple_asm0001_collada_02_prt.stl" scale="${SF} ${SF} ${SF}" />
+      <origin xyz="${-2.2024173e+01*mmTom} ${-2.5677238*mmTom} ${9.4588455e-01*mmTom}" rpy="0 0 0"/>
+      <mass value="3.2844159"/>
+      <inertia ixx="${7.5550679e+03*mm2Tom2}"  ixy="${-6.7488292e+02*mm2Tom2}"  ixz="${5.8332889e+01*mm2Tom2}" iyy="${1.1241163e+04*mm2Tom2}" iyz="${1.4552081e+02*mm2Tom2}" izz="${1.3391865e+04*mm2Tom2}" />
+    </inertial>
+    <visual>
+      <origin xyz="0 0 0" rpy="0 0 0"/>
+      <geometry name="RFootmot_visual">
+        <mesh filename="package://bigman_urdf/meshes/AnklePitch.STL" scale="0.001 -0.001 0.001" />
+      </geometry>
+    </visual>
+    <collision>
+      <origin xyz="0 0 0" rpy="0 0 0"/>
+      <geometry name="RFootmot_collision">
+        <mesh filename="package://bigman_urdf/meshes/simple/AnklePitch.STL" scale="0.001 -0.001 0.001" />
       </geometry>
     </collision>
@@ -284,5 +284,5 @@
       <child link="RFoot"/>
       <origin xyz="0.0 0.0 0.0" rpy="0 0 0" />
-      <axis xyz="0 1 0" />
+      <axis xyz="1 0 0" />
       <limit velocity="4.0" effort="50" lower="-1.2217" upper="1.2217" />
       <dynamics friction="0" damping="3.0"/>
@@ -333,5 +333,5 @@
     <child link="LFoot"/>
     <origin xyz="0.0 0.0 0.0" rpy="0 0 0" />
-    <axis xyz="0 1 0" />
+    <axis xyz="1 0 0" />
     <limit velocity="4.0" effort="50" lower="-1.2217" upper="1.2217" />
     <dynamics friction="0" damping="3.0"/>

Commit message: Added joint limits and torque limits. Added FAKE velocity limits!!!

File: bigman_urdf/urdf/parts/legs.urdf.xacro (robot description, xacro)
@@ -245,5 +245,5 @@
     <origin xyz="0.1059 -0.06 0.0" rpy="0 0 0" />
     <axis xyz="1 0 0" />
-    <limit velocity="4.0" effort="50" lower="-1.9199" upper="0.7854" />
+    <limit velocity="6.283" effort="220" lower="-0.87222" upper="0.697778" />
     <dynamics friction="0" damping="3.0"/>
   </joint>
@@ -253,5 +253,5 @@
     <origin xyz="-0.0889 -0.121032 -0.217872" rpy="0 0 0" />
     <axis xyz="0 0 1" />
-    <limit velocity="4.0" effort="50" lower="-1.0472" upper="0.4363" />
+    <limit velocity="6.283" effort="120" lower="-1.57" upper="0.872222" />
     <dynamics friction="0" damping="3.0"/>
   </joint>
@@ -261,5 +261,5 @@
     <origin xyz="0.0 0.0 0.0" rpy="0 0 0" />
     <axis xyz="0 1 0" />
-    <limit velocity="4.0" effort="50" lower="-0.8727" upper="0.8727" />
+    <limit velocity="6.283" effort="220" lower="-2.09333" upper="1.046667" />
     <dynamics friction="0" damping="3.0"/>
   </joint>
@@ -269,5 +269,5 @@
     <origin xyz="0.0 0.0 -0.356" rpy="0 0 0" />
     <axis xyz="0 1 0" />
-    <limit velocity="4.0" effort="50" lower="-0.1745" upper="1.9199" />
+    <limit velocity="6.283" effort="220" lower="0.0" upper="2.442222" />
     <dynamics friction="0" damping="3.0"/>
   </joint>
@@ -277,5 +277,5 @@
     <origin xyz="0.0 0.0 -0.4" rpy="0 0 0" />
     <axis xyz="0 1 0" />
-    <limit velocity="4.0" effort="50" lower="-0.6109" upper="0.6109" />
+    <limit velocity="6.283" effort="220" lower="-1.39556" upper="0.697778" />
     <dynamics friction="0" damping="3.0"/>
   </joint>
@@ -285,5 +285,5 @@
       <origin xyz="0.0 0.0 0.0" rpy="0 0 0" />
       <axis xyz="1 0 0" />
-      <limit velocity="4.0" effort="50" lower="-1.2217" upper="1.2217" />
+      <limit velocity="6.283" effort="120" lower="-0.785" upper="0.785" />
       <dynamics friction="0" damping="3.0"/>
     </joint>
@@ -294,5 +294,5 @@
     <origin xyz="0.1059 0.06 0.0" rpy="0 0 0" />
     <axis xyz="1 0 0" />
-    <limit velocity="4.0" effort="50" lower="-1.9199" upper="0.7854" />
+    <limit velocity="6.283" effort="220" lower="-0.697778" upper="0.87222" />
     <dynamics friction="0" damping="3.0"/>
   </joint>
@@ -302,5 +302,5 @@
     <origin xyz="-0.0889 0.121032 -0.217872" rpy="0 0 0" />
     <axis xyz="0 0 1" />
-    <limit velocity="4.0" effort="50" lower="-0.4363" upper="1.0472" />
+    <limit velocity="6.283" effort="120" lower="-0.872222" upper="1.57" />
     <dynamics friction="0" damping="3.0"/>
   </joint>
@@ -310,5 +310,5 @@
     <origin xyz="0.0 0.0 0.0" rpy="0 0 0" />
     <axis xyz="0 1 0" />
-    <limit velocity="4.0" effort="50" lower="-0.8727" upper="0.8727" />
+    <limit velocity="6.283" effort="220" lower="-2.09333" upper="1.046667" />
     <dynamics friction="0" damping="3.0"/>
   </joint>
@@ -318,5 +318,5 @@
     <origin xyz="0.0 0.0 -0.356" rpy="0 0 0" />
     <axis xyz="0 1 0" />
-    <limit velocity="4.0" effort="50" lower="-0.1745" upper="1.9199" />
+    <limit velocity="6.283" effort="220" lower="0.0" upper="2.442222" />
     <dynamics friction="0" damping="3.0"/>
   </joint>
@@ -326,5 +326,5 @@
     <origin xyz="0.0 0.0 -0.4" rpy="0 0 0" />
     <axis xyz="0 1 0" />
-    <limit velocity="4.0" effort="50" lower="-0.6109" upper="0.6109" />
+    <limit velocity="6.283" effort="220" lower="-1.39556" upper="0.697778" />
     <dynamics friction="0" damping="3.0"/>
   </joint>
@@ -334,5 +334,5 @@
     <origin xyz="0.0 0.0 0.0" rpy="0 0 0" />
     <axis xyz="1 0 0" />
-    <limit velocity="4.0" effort="50" lower="-1.2217" upper="1.2217" />
+    <limit velocity="6.283" effort="120" lower="-0.785" upper="0.785" />
     <dynamics friction="0" damping="3.0"/>
   </joint>

Commit message: Renamed legs joints according to the axis of rotation. Updated configuration files for the simulation

File: bigman_urdf/urdf/parts/legs.urdf.xacro (robot description, xacro)
@@ -240,5 +240,5 @@
 <!-- JOINTS -->
 <!-- ********************RIGHT LEG******************** -->
-  <joint name="RHipSag" type="revolute">
+  <joint name="RHipLat" type="revolute">
     <parent link="Waist"/>
     <child link="RHipMot"/>
@@ -248,5 +248,5 @@
     <dynamics friction="0" damping="3.0"/>
   </joint>
-  <joint name="RHipLat" type="revolute">
+  <joint name="RHipYaw" type="revolute">
     <parent link="RHipMot"/>
     <child link="RThighUpLeg"/>
@@ -256,5 +256,5 @@
     <dynamics friction="0" damping="3.0"/>
   </joint>
-  <joint name="RHipYaw" type="revolute">
+  <joint name="RHipSag" type="revolute">
     <parent link="RThighUpLeg"/>
     <child link="RThighLowLeg"/>
@@ -272,5 +272,5 @@
     <dynamics friction="0" damping="3.0"/>
   </joint>
-  <joint name="RAnkLat" type="revolute">
+  <joint name="RAnkSag" type="revolute">
     <parent link="RLowLeg"/>
     <child link="RFootmot"/>
@@ -280,5 +280,5 @@
     <dynamics friction="0" damping="3.0"/>
   </joint>
-    <joint name="RAnkSag" type="revolute">
+    <joint name="RAnkLat" type="revolute">
       <parent link="RFootmot"/>
       <child link="RFoot"/>
@@ -289,5 +289,5 @@
     </joint>
 <!-- ********************LEFT LEG******************** -->
-  <joint name="LHipSag" type="revolute">
+  <joint name="LHipLat" type="revolute">
     <parent link="Waist"/>
     <child link="LHipMot"/>
@@ -297,5 +297,5 @@
     <dynamics friction="0" damping="3.0"/>
   </joint>
-  <joint name="LHipLat" type="revolute">
+  <joint name="LHipYaw" type="revolute">
     <parent link="LHipMot"/>
     <child link="LThighUpLeg"/>
@@ -305,5 +305,5 @@
     <dynamics friction="0" damping="3.0"/>
   </joint>
-  <joint name="LHipYaw" type="revolute">
+  <joint name="LHipSag" type="revolute">
     <parent link="LThighUpLeg"/>
     <child link="LThighLowLeg"/>
@@ -321,5 +321,5 @@
     <dynamics friction="0" damping="3.0"/>
   </joint>
-  <joint name="LAnkLat" type="revolute">
+  <joint name="LAnkSag" type="revolute">
     <parent link="LLowLeg"/>
     <child link="LFootmot"/>
@@ -329,5 +329,5 @@
     <dynamics friction="0" damping="3.0"/>
   </joint>
-  <joint name="LAnkSag" type="revolute">
+  <joint name="LAnkLat" type="revolute">
     <parent link="LFootmot"/>
     <child link="LFoot"/>

Commit message: Added Part for weigths in only_legs model

File: bigman_urdf/urdf/parts/legs.urdf.xacro (robot description, xacro)
@@ -7,4 +7,25 @@
 <xacro:property name="PI_2" value="1.57079632679" />
 <!-- LINKS -->
+<xacro:if value="${BIGMAN_ONLY_LEGS}">
+<link name ="PelvisWeightBench">
+    <inertial>
+      <origin xyz="0.0 0.0 ${1.8846109e+02*mmTom}" rpy="0 0 0"/>
+      <mass value="5.5278386"/>
+      <inertia ixx="${1.5195067e+05*mm2Tom2}"  ixy="0.0"  ixz="${-2.4191890e-01*mm2Tom2}" iyy="${1.5213465e+05*mm2Tom2}" iyz="0.0" izz="${5.1389419e+03*mm2Tom2}" />
+    </inertial>
+    <visual>
+      <origin xyz="0 0 0" rpy="0 0 0"/>
+      <geometry name="PelvisWeightBench_visual">
+        <mesh filename="package://bigman_urdf/meshes/PelvisWeightBench.STL" scale="0.001 0.001 0.001" />
+      </geometry>
+    </visual>
+    <collision>
+      <origin xyz="0 0 0" rpy="0 0 0"/>
+      <geometry name="PelvisWeightBench_collision">
+        <mesh filename="package://bigman_urdf/meshes/simple/PelvisWeightBench.STL" scale="0.001 0.001 0.001" />
+      </geometry>
+    </collision>
+</link>
+</xacro:if>
 <!-- ********************RIGHT LEG******************** -->
 <link name ="RHipMot">
@@ -248,4 +269,11 @@
    </link>
 <!-- JOINTS -->
+<xacro:if value="${BIGMAN_ONLY_LEGS}">
+       <joint name="PelvisWeightBench_joint" type="fixed">
+           <parent link="Waist"/>
+           <child link="PelvisWeightBench"/>
+           <origin xyz="-0.035 0 0.075" rpy="0 0 ${PI_2}" />
+       </joint>
+</xacro:if>
 <!-- ********************RIGHT LEG******************** -->
   <joint name="RHipLat" type="revolute">

Commit message: Added new knee pitch stl with calf

File: bigman_urdf/urdf/parts/legs.urdf.xacro (robot description, xacro)
@@ -95,5 +95,5 @@
       <origin xyz="0 0 0" rpy="0 0 0"/>
       <geometry name="RLowLeg_visual">
-        <mesh filename="package://bigman_urdf/meshes/KneePitch.STL" scale="0.001 0.001 0.001" />
+        <mesh filename="package://bigman_urdf/meshes/KneePitchCalf.STL" scale="0.001 0.001 0.001" />
       </geometry>
     </visual>
@@ -101,5 +101,5 @@
       <origin xyz="0 0 0" rpy="0 0 0"/>
       <geometry name="RLowLeg_collision">
-        <mesh filename="package://bigman_urdf/meshes/simple/KneePitch.STL" scale="0.001 0.001 0.001" />
+        <mesh filename="package://bigman_urdf/meshes/simple/KneePitchCalf.STL" scale="0.001 0.001 0.001" />
       </geometry>
     </collision>
@@ -214,5 +214,5 @@
       <origin xyz="0 0 0" rpy="0 0 0"/>
       <geometry name="LLowLeg_visual">
-        <mesh filename="package://bigman_urdf/meshes/KneePitch.STL" scale="0.001 0.001 0.001" />
+        <mesh filename="package://bigman_urdf/meshes/KneePitchCalf.STL" scale="0.001 0.001 0.001" />
       </geometry>
     </visual>
@@ -220,5 +220,5 @@
       <origin xyz="0 0 0" rpy="0 0 0"/>
       <geometry name="LLowLeg_collision">
-        <mesh filename="package://bigman_urdf/meshes/simple/KneePitch.STL" scale="0.001 0.001 0.001" />
+        <mesh filename="package://bigman_urdf/meshes/simple/KneePitchCalf.STL" scale="0.001 0.001 0.001" />
       </geometry>
     </collision>

Commit message: Fixed bug in left leg

File: bigman_urdf/urdf/parts/legs.urdf.xacro (robot description, xacro)
@@ -202,5 +202,5 @@
       <origin xyz="0 0 0" rpy="0 0 0"/>
       <geometry name="LLowLeg_visual">
-        <mesh filename="package://bigman_urdf/meshes/KneePitchCalf.STL" scale="0.001 0.001 0.001" />
+        <mesh filename="package://bigman_urdf/meshes/KneePitchCalf.STL" scale="0.001 -0.001 0.001" />
       </geometry>
       <material name="dark_grey"/>
@@ -209,5 +209,5 @@
       <origin xyz="0 0 0" rpy="0 0 0"/>
       <geometry name="LLowLeg_collision">
-        <mesh filename="package://bigman_urdf/meshes/simple/KneePitchCalf.STL" scale="0.001 0.001 0.001" />
+        <mesh filename="package://bigman_urdf/meshes/simple/KneePitchCalf.STL" scale="0.001 -0.001 0.001" />
       </geometry>
     </collision>
