Commit message: - updated the leg joints torque limits to the latest specs (from Francesca)

File: bigman_urdf/urdf/parts/legs.urdf.xacro (robot description, xacro)
@@ -306,5 +306,5 @@
     <origin xyz="0.1059 -0.06 0.0" rpy="0 0 0" />
     <axis xyz="1 0 0" />
-    <limit velocity="6.283" effort="220" lower="-0.87222" upper="0.697778" />
+    <limit velocity="6.283" effort="400" lower="-0.87222" upper="0.697778" />
     <dynamics friction="0" damping="3.0"/>
   </joint>
@@ -314,5 +314,5 @@
     <origin xyz="-0.0889 -0.121032 -0.217872" rpy="0 0 0" />
     <axis xyz="0 0 1" />
-    <limit velocity="6.283" effort="120" lower="-1.57" upper="0.872222" />
+    <limit velocity="6.283" effort="140" lower="-1.57" upper="0.872222" />
     <dynamics friction="0" damping="3.0"/>
   </joint>
@@ -322,5 +322,5 @@
     <origin xyz="0.0 0.0 0.0" rpy="0 0 0" />
     <axis xyz="0 1 0" />
-    <limit velocity="6.283" effort="220" lower="-2.09333" upper="1.046667" />
+    <limit velocity="6.283" effort="400" lower="-2.09333" upper="1.046667" />
     <dynamics friction="0" damping="3.0"/>
   </joint>
@@ -330,5 +330,5 @@
     <origin xyz="0.0 0.0 -0.356" rpy="0 0 0" />
     <axis xyz="0 1 0" />
-    <limit velocity="6.283" effort="220" lower="0.0" upper="2.442222" />
+    <limit velocity="6.283" effort="400" lower="0.0" upper="2.442222" />
     <dynamics friction="0" damping="3.0"/>
   </joint>
@@ -338,5 +338,5 @@
     <origin xyz="0.0 0.0 -0.4" rpy="0 0 0" />
     <axis xyz="0 1 0" />
-    <limit velocity="6.283" effort="220" lower="-1.39556" upper="0.697778" />
+    <limit velocity="6.283" effort="330" lower="-1.39556" upper="0.697778" />
     <dynamics friction="0" damping="3.0"/>
   </joint>
@@ -346,5 +346,5 @@
       <origin xyz="0.0 0.0 0.0" rpy="0 0 0" />
       <axis xyz="1 0 0" />
-      <limit velocity="6.283" effort="120" lower="-0.785" upper="0.785" />
+      <limit velocity="6.283" effort="210" lower="-0.785" upper="0.785" />
       <dynamics friction="0" damping="3.0"/>
     </joint>
@@ -355,5 +355,5 @@
     <origin xyz="0.1059 0.06 0.0" rpy="0 0 0" />
     <axis xyz="1 0 0" />
-    <limit velocity="6.283" effort="220" lower="-0.697778" upper="0.87222" />
+    <limit velocity="6.283" effort="400" lower="-0.697778" upper="0.87222" />
     <dynamics friction="0" damping="3.0"/>
   </joint>
@@ -363,5 +363,5 @@
     <origin xyz="-0.0889 0.121032 -0.217872" rpy="0 0 0" />
     <axis xyz="0 0 1" />
-    <limit velocity="6.283" effort="120" lower="-0.872222" upper="1.57" />
+    <limit velocity="6.283" effort="140" lower="-0.872222" upper="1.57" />
     <dynamics friction="0" damping="3.0"/>
   </joint>
@@ -371,5 +371,5 @@
     <origin xyz="0.0 0.0 0.0" rpy="0 0 0" />
     <axis xyz="0 1 0" />
-    <limit velocity="6.283" effort="220" lower="-2.09333" upper="1.046667" />
+    <limit velocity="6.283" effort="400" lower="-2.09333" upper="1.046667" />
     <dynamics friction="0" damping="3.0"/>
   </joint>
@@ -379,5 +379,5 @@
     <origin xyz="0.0 0.0 -0.356" rpy="0 0 0" />
     <axis xyz="0 1 0" />
-    <limit velocity="6.283" effort="220" lower="0.0" upper="2.442222" />
+    <limit velocity="6.283" effort="400" lower="0.0" upper="2.442222" />
     <dynamics friction="0" damping="3.0"/>
   </joint>
@@ -387,5 +387,5 @@
     <origin xyz="0.0 0.0 -0.4" rpy="0 0 0" />
     <axis xyz="0 1 0" />
-    <limit velocity="6.283" effort="220" lower="-1.39556" upper="0.697778" />
+    <limit velocity="6.283" effort="330" lower="-1.39556" upper="0.697778" />
     <dynamics friction="0" damping="3.0"/>
   </joint>
@@ -395,5 +395,5 @@
     <origin xyz="0.0 0.0 0.0" rpy="0 0 0" />
     <axis xyz="1 0 0" />
-    <limit velocity="6.283" effort="120" lower="-0.785" upper="0.785" />
+    <limit velocity="6.283" effort="210" lower="-0.785" upper="0.785" />
     <dynamics friction="0" damping="3.0"/>
   </joint>

Commit message: Fixed wrong inertia for the LFoot

File: bigman_urdf/urdf/parts/legs.urdf.xacro (robot description, xacro)
@@ -258,5 +258,5 @@
           <origin xyz="-0.00653584 0.00479384 -0.10180375" rpy="0 0 0"/>
           <mass value="3.42638110"/>
-          <inertia ixx="0.01032886"  ixy="-0.00016407"  ixz="-0.00201294" iyy="0.02854025" iyz="0.00046315" izz="0.02799499" />
+          <inertia ixx="0.01032886"  ixy="0.00016407"  ixz="-0.00201294" iyy="0.02854025" iyz="-0.00046315" izz="0.02799499" />
         </xacro:if>
         <xacro:unless value="${BIGMAN_NEW_FEET}">
