Commit message: Moved soft hand.

File: bigman_urdf/urdf/parts/soft_hand.urdf.xacro (robot description, xacro)
@@ -45,10 +45,10 @@
         <parent link="RWrMot3"/>
         <child link="RSoftHand"/>
-        <origin xyz="0 0 -0.07" rpy="0 0 0"/>
+        <origin xyz="0 0 -0.11" rpy="0 0 0"/>
   </joint>
   <joint name="l_handj" type="fixed">
         <parent link="LWrMot3"/>
         <child link="LSoftHand"/>
-        <origin xyz="0 0 -0.07" rpy="0 0 0"/>
+        <origin xyz="0 0 -0.11" rpy="0 0 0"/>
   </joint>
 </xacro:if>

Commit message: Added reference frames

File: bigman_urdf/urdf/parts/soft_hand.urdf.xacro (robot description, xacro)
@@ -59,5 +59,5 @@
         <parent link="RSoftHand"/>
         <child link="r_palm"/>
-        <origin xyz="0 0.05 0.0" rpy="0 0 0"/>
+        <origin xyz="0 ${2.0696923e+01*mmTom+5.0*mmTom} 0.0" rpy="0 0 0"/>
   </joint>
   <joint name="l_handj" type="fixed">
@@ -74,5 +74,5 @@
         <parent link="LSoftHand"/>
         <child link="l_palm"/>
-        <origin xyz="0 -0.05 0.0" rpy="0 0 0"/>
+        <origin xyz="0 ${-2.0696923e+01*mmTom-5.0*mmTom} 0.0" rpy="0 0 0"/>
   </joint>
 </xacro:if>

Commit message: Added inertia, CoM and Mass

File: bigman_urdf/urdf/parts/soft_hand.urdf.xacro (robot description, xacro)
@@ -2,4 +2,8 @@
 <robot xmlns:xacro="http://ros.org/wiki/xacro" name="SoftHand">
 <xacro:if value="${BIGMAN_FIXED_HANDS}">
+<xacro:property name="a" value="0.08" />
+<xacro:property name="b" value="0.08" />
+<xacro:property name="c" value="0.1" />
+<!-- For the hand we use the inertia of a parallelepiped -->
 <!-- LINKS -->
 <link name="RSoftHand"/>
@@ -7,7 +11,7 @@
 <link name="RSoftHandLink">
     <inertial>
-      <origin xyz="0 0 0" rpy="0 0 0"/>
-      <mass value="0.3"/>
-      <inertia ixx="0.001"  ixy="0"  ixz="0" iyy="0.001" iyz="0" izz="0.001" />
+      <origin xyz="${1.1908576e+01*mmTom} ${2.1833446*mmTom} ${-1.5361558e+02*mmTom}" rpy="0 0 0"/>
+      <mass value="5.0e-01"/>
+      <inertia ixx="${5.0e-01*(a*a+c*c)/12.0}"  ixy="0"  ixz="0" iyy="${5.0e-01*(b*b+c*c)/12.0}" iyz="0" izz="${5.0e-01*(a*a+b*b)/12.0}" />
     </inertial>
     <visual>
@@ -28,7 +32,7 @@
   <link name="LSoftHandLink">
     <inertial>
-      <origin xyz="0 0 0" rpy="0 0 0"/>
-      <mass value="0.3"/>
-      <inertia ixx="0.001"  ixy="0"  ixz="0" iyy="0.001" iyz="0" izz="0.001" />
+      <origin xyz="${1.1908576e+01*mmTom} ${-2.1833446*mmTom} ${-1.5361558e+02*mmTom}" rpy="0 0 0"/>
+      <mass value="5.0e-01"/>
+      <inertia ixx="${5.0e-01*(a*a+c*c)/12.0}"  ixy="0"  ixz="0" iyy="${5.0e-01*(b*b+c*c)/12.0}" iyz="0" izz="${5.0e-01*(a*a+b*b)/12.0}" />
     </inertial>
     <visual>
@@ -82,7 +86,7 @@
   <link name="RSoftHand">
     <inertial>
-      <origin xyz="0 0 0" rpy="0 0 0"/>
-      <mass value="0.3"/>
-      <inertia ixx="0.001"  ixy="0"  ixz="0" iyy="0.001" iyz="0" izz="0.001" />
+      <origin xyz="${1.1908576e+01*mmTom} ${2.1833446*mmTom} ${-1.5361558e+02*mmTom}" rpy="0 0 0"/>
+      <mass value="5.0e-01"/>
+      <inertia ixx="${5.0e-01*(a*a+c*c)/12.0}"  ixy="0"  ixz="0" iyy="${5.0e-01*(b*b+c*c)/12.0}" iyz="0" izz="${5.0e-01*(a*a+b*b)/12.0}" />
     </inertial>
     <visual>
@@ -104,7 +108,7 @@
   <link name="LSoftHand">
     <inertial>
-      <origin xyz="0 0 0" rpy="0 0 0"/>
-      <mass value="0.3"/>
-      <inertia ixx="0.001"  ixy="0"  ixz="0" iyy="0.001" iyz="0" izz="0.001" />
+      <origin xyz="${1.1908576e+01*mmTom} ${-2.1833446*mmTom} ${-1.5361558e+02*mmTom}" rpy="0 0 0"/>
+      <mass value="5.0e-01"/>
+      <inertia ixx="${5.0e-01*(a*a+c*c)/12.0}"  ixy="0"  ixz="0" iyy="${5.0e-01*(b*b+c*c)/12.0}" iyz="0" izz="${5.0e-01*(a*a+b*b)/12.0}" />
     </inertial>
     <visual>

Commit message: Reverted left_hand joint sign, increased P gain for both hands

File: bigman_urdf/urdf/parts/soft_hand.urdf.xacro (robot description, xacro)
@@ -141,6 +141,6 @@
         <child link="LSoftHand"/>
         <origin xyz="0 0 -0.04" rpy="0 0 0"/>
-        <axis xyz="1 0 0" />
-        <limit velocity="4.0" effort="5" lower="-1.57075" upper="0.0" />
+        <axis xyz="-1 0 0" />
+        <limit velocity="4.0" effort="5" lower="0" upper="1.57075.0" />
         <dynamics friction="0" damping="3.0"/>
 </joint>

Commit message: Fixed typo from previous commit which prevented model from compiling

File: bigman_urdf/urdf/parts/soft_hand.urdf.xacro (robot description, xacro)
@@ -142,5 +142,5 @@
         <origin xyz="0 0 -0.04" rpy="0 0 0"/>
         <axis xyz="-1 0 0" />
-        <limit velocity="4.0" effort="5" lower="0" upper="1.57075.0" />
+        <limit velocity="4.0" effort="5" lower="0" upper="1.57075" />
         <dynamics friction="0" damping="3.0"/>
 </joint>

Commit message: First attemp at a proper joint limit for the hands

File: bigman_urdf/urdf/parts/soft_hand.urdf.xacro (robot description, xacro)
@@ -134,5 +134,5 @@
         <origin xyz="0 0 -0.04" rpy="0 0 0"/>
         <axis xyz="1 0 0" />
-        <limit velocity="4.0" effort="5" lower="0.0" upper="1.57075" />
+        <limit velocity="4.0" effort="5" lower="0.0" upper="5.0" />
         <dynamics friction="0" damping="3.0"/>
 </joint>
@@ -142,5 +142,5 @@
         <origin xyz="0 0 -0.04" rpy="0 0 0"/>
         <axis xyz="-1 0 0" />
-        <limit velocity="4.0" effort="5" lower="0" upper="1.57075" />
+        <limit velocity="4.0" effort="5" lower="0" upper="5.0" />
         <dynamics friction="0" damping="3.0"/>
 </joint>

Commit message: Added new hands visualization and collision

File: bigman_urdf/urdf/parts/soft_hand.urdf.xacro (robot description, xacro)
@@ -8,5 +8,4 @@
 <!-- LINKS -->
 <link name="RSoftHand"/>
-<link name="r_palm"/>
 <link name="RSoftHandLink">
     <inertial>
@@ -20,5 +19,5 @@
         <mesh filename="package://bigman_urdf/meshes/SoftHandOpen.STL" scale="0.001 0.001 0.001" />
       </geometry>
-      <material name="black"/>
+      <material name="grey"/>
    </visual>
    <collision>
@@ -30,5 +29,4 @@
   </link>
   <link name="LSoftHand"/>
-  <link name="l_palm"/>
   <link name="LSoftHandLink">
     <inertial>
@@ -42,5 +40,5 @@
         <mesh filename="package://bigman_urdf/meshes/SoftHandOpen.STL" scale="0.001 -0.001 0.001" />
       </geometry>
-      <material name="black"/>
+      <material name="grey"/>
    </visual>
    <collision>
@@ -62,9 +60,4 @@
         <origin xyz="${1.1908576e+01*mmTom} ${2.1833446*mmTom} ${-1.5361558e+02*mmTom}" rpy="0 0 0"/>
   </joint>
-  <joint name="r_handj3" type="fixed">
-        <parent link="RSoftHand"/>
-        <child link="r_palm"/>
-        <origin xyz="0 ${2.0696923e+01*mmTom+5.0*mmTom} 0.0" rpy="0 0 0"/>
-  </joint>
   <joint name="l_handj" type="fixed">
         <parent link="LWrMot3"/>
@@ -76,9 +69,4 @@
         <child link="LSoftHand"/>
         <origin xyz="${1.1908576e+01*mmTom} ${-2.1833446*mmTom} ${-1.5361558e+02*mmTom}" rpy="0 0 0"/>
-  </joint>
-  <joint name="l_handj3" type="fixed">
-        <parent link="LSoftHand"/>
-        <child link="l_palm"/>
-        <origin xyz="0 ${-2.0696923e+01*mmTom-5.0*mmTom} 0.0" rpy="0 0 0"/>
   </joint>
 </xacro:if>

Commit message: Added new reference frames for control

File: bigman_urdf/urdf/parts/soft_hand.urdf.xacro (robot description, xacro)
@@ -11,5 +11,5 @@
     <inertial>
       <origin xyz="${1.1908576e+01*mmTom} ${2.1833446*mmTom} ${-1.5361558e+02*mmTom}" rpy="0 0 0"/>
-      <mass value="5.0e-01"/>
+      <mass value="1.2"/>
       <inertia ixx="${5.0e-01*(a*a+c*c)/12.0}"  ixy="0"  ixz="0" iyy="${5.0e-01*(b*b+c*c)/12.0}" iyz="0" izz="${5.0e-01*(a*a+b*b)/12.0}" />
     </inertial>
@@ -32,5 +32,5 @@
     <inertial>
       <origin xyz="${1.1908576e+01*mmTom} ${-2.1833446*mmTom} ${-1.5361558e+02*mmTom}" rpy="0 0 0"/>
-      <mass value="5.0e-01"/>
+      <mass value="1.2"/>
       <inertia ixx="${5.0e-01*(a*a+c*c)/12.0}"  ixy="0"  ixz="0" iyy="${5.0e-01*(b*b+c*c)/12.0}" iyz="0" izz="${5.0e-01*(a*a+b*b)/12.0}" />
     </inertial>
@@ -58,5 +58,5 @@
         <parent link="RSoftHandLink"/>
         <child link="RSoftHand"/>
-        <origin xyz="${1.1908576e+01*mmTom} ${2.1833446*mmTom} ${-1.5361558e+02*mmTom}" rpy="0 0 0"/>
+        <origin xyz="0 0.0305 -0.21" rpy="0 0 0"/>
   </joint>
   <joint name="l_handj" type="fixed">
@@ -68,5 +68,5 @@
         <parent link="LSoftHandLink"/>
         <child link="LSoftHand"/>
-        <origin xyz="${1.1908576e+01*mmTom} ${-2.1833446*mmTom} ${-1.5361558e+02*mmTom}" rpy="0 0 0"/>
+        <origin xyz="0 -0.0305 -0.21" rpy="0 0 0"/>
   </joint>
 </xacro:if>
@@ -77,5 +77,5 @@
     <inertial>
       <origin xyz="${1.1908576e+01*mmTom} ${2.1833446*mmTom} ${-1.5361558e+02*mmTom}" rpy="0 0 0"/>
-      <mass value="5.0e-01"/>
+      <mass value="1.2"/>
       <inertia ixx="${5.0e-01*(a*a+c*c)/12.0}"  ixy="0"  ixz="0" iyy="${5.0e-01*(b*b+c*c)/12.0}" iyz="0" izz="${5.0e-01*(a*a+b*b)/12.0}" />
     </inertial>
@@ -99,5 +99,5 @@
     <inertial>
       <origin xyz="${1.1908576e+01*mmTom} ${-2.1833446*mmTom} ${-1.5361558e+02*mmTom}" rpy="0 0 0"/>
-      <mass value="5.0e-01"/>
+      <mass value="1.2"/>
       <inertia ixx="${5.0e-01*(a*a+c*c)/12.0}"  ixy="0"  ixz="0" iyy="${5.0e-01*(b*b+c*c)/12.0}" iyz="0" izz="${5.0e-01*(a*a+b*b)/12.0}" />
     </inertial>

Commit message: Added real mass but approximated com and inertia for the hands

File: bigman_urdf/urdf/parts/soft_hand.urdf.xacro (robot description, xacro)
@@ -2,7 +2,7 @@
 <robot xmlns:xacro="http://ros.org/wiki/xacro" name="SoftHand">
 <xacro:if value="${BIGMAN_FIXED_HANDS}">
-<xacro:property name="a" value="0.08" />
-<xacro:property name="b" value="0.08" />
-<xacro:property name="c" value="0.1" />
+<xacro:property name="a" value="0.1" />
+<xacro:property name="b" value="0.06" />
+<xacro:property name="c" value="0.14" />
 <!-- For the hand we use the inertia of a parallelepiped -->
 <!-- LINKS -->
@@ -10,7 +10,7 @@
 <link name="RSoftHandLink">
     <inertial>
-      <origin xyz="${1.1908576e+01*mmTom} ${2.1833446*mmTom} ${-1.5361558e+02*mmTom}" rpy="0 0 0"/>
+      <origin xyz="0 0 -0.17" rpy="0 0 0"/>
       <mass value="1.2"/>
-      <inertia ixx="${5.0e-01*(a*a+c*c)/12.0}"  ixy="0"  ixz="0" iyy="${5.0e-01*(b*b+c*c)/12.0}" iyz="0" izz="${5.0e-01*(a*a+b*b)/12.0}" />
+      <inertia ixx="${1.2*(b*b+c*c)/12.0}"  ixy="0"  ixz="0" iyy="${1.2*(a*a+c*c)/12.0}" iyz="0" izz="${1.2*(a*a+b*b)/12.0}" />
     </inertial>
     <visual>
@@ -31,7 +31,7 @@
   <link name="LSoftHandLink">
     <inertial>
-      <origin xyz="${1.1908576e+01*mmTom} ${-2.1833446*mmTom} ${-1.5361558e+02*mmTom}" rpy="0 0 0"/>
+      <origin xyz="0 0 -0.17" rpy="0 0 0"/>
       <mass value="1.2"/>
-      <inertia ixx="${5.0e-01*(a*a+c*c)/12.0}"  ixy="0"  ixz="0" iyy="${5.0e-01*(b*b+c*c)/12.0}" iyz="0" izz="${5.0e-01*(a*a+b*b)/12.0}" />
+      <inertia ixx="${1.2*(b*b+c*c)/12.0}"  ixy="0"  ixz="0" iyy="${1.2*(a*a+c*c)/12.0}" iyz="0" izz="${1.2*(a*a+b*b)/12.0}" />
     </inertial>
     <visual>
@@ -76,7 +76,7 @@
   <link name="RSoftHand">
     <inertial>
-      <origin xyz="${1.1908576e+01*mmTom} ${2.1833446*mmTom} ${-1.5361558e+02*mmTom}" rpy="0 0 0"/>
+      <origin xyz="0 0 -0.17" rpy="0 0 0"/>
       <mass value="1.2"/>
-      <inertia ixx="${5.0e-01*(a*a+c*c)/12.0}"  ixy="0"  ixz="0" iyy="${5.0e-01*(b*b+c*c)/12.0}" iyz="0" izz="${5.0e-01*(a*a+b*b)/12.0}" />
+      <inertia ixx="${1.2*(b*b+c*c)/12.0}"  ixy="0"  ixz="0" iyy="${1.2*(a*a+c*c)/12.0}" iyz="0" izz="${1.2*(a*a+b*b)/12.0}" />
     </inertial>
     <visual>
@@ -98,7 +98,7 @@
   <link name="LSoftHand">
     <inertial>
-      <origin xyz="${1.1908576e+01*mmTom} ${-2.1833446*mmTom} ${-1.5361558e+02*mmTom}" rpy="0 0 0"/>
+      <origin xyz="0 0 -0.17" rpy="0 0 0"/>
       <mass value="1.2"/>
-      <inertia ixx="${5.0e-01*(a*a+c*c)/12.0}"  ixy="0"  ixz="0" iyy="${5.0e-01*(b*b+c*c)/12.0}" iyz="0" izz="${5.0e-01*(a*a+b*b)/12.0}" />
+      <inertia ixx="${1.2*(b*b+c*c)/12.0}"  ixy="0"  ixz="0" iyy="${1.2*(a*a+c*c)/12.0}" iyz="0" izz="${1.2*(a*a+b*b)/12.0}" />
     </inertial>
     <visual>

Commit message: added hands useful links

File: bigman_urdf/urdf/parts/soft_hand.urdf.xacro (robot description, xacro)
@@ -28,4 +28,8 @@
    </collision>
   </link>
+<link name="r_hand_upper_right_link"/>
+<link name="r_hand_lower_right_link"/>
+<link name="r_hand_upper_left_link"/>
+<link name="r_hand_lower_left_link"/>
   <link name="LSoftHand"/>
   <link name="LSoftHandLink">
@@ -49,4 +53,8 @@
    </collision>
   </link>
+<link name="l_hand_upper_right_link"/>
+<link name="l_hand_lower_right_link"/>
+<link name="l_hand_upper_left_link"/>
+<link name="l_hand_lower_left_link"/>
 <!-- JOINTS -->
   <joint name="r_handj" type="fixed">
@@ -60,4 +68,24 @@
         <origin xyz="0 0.0305 -0.21" rpy="0 0 0"/>
   </joint>
+  <joint name="r_handj3" type="fixed">
+        <parent link="RSoftHand"/>
+        <child link="r_hand_upper_right_link"/>
+        <origin xyz="0.05 0.0 0.0" rpy="0 0 0"/>
+  </joint>
+  <joint name="r_handj4" type="fixed">
+        <parent link="RSoftHand"/>
+        <child link="r_hand_lower_right_link"/>
+        <origin xyz="-0.05 0.0 0.0" rpy="0 0 0"/>
+  </joint>
+  <joint name="r_handj5" type="fixed">
+        <parent link="RSoftHand"/>
+        <child link="r_hand_upper_left_link"/>
+        <origin xyz="0.05 0.0 0.1" rpy="0 0 0"/>
+  </joint>
+  <joint name="r_handj6" type="fixed">
+        <parent link="RSoftHand"/>
+        <child link="r_hand_lower_left_link"/>
+        <origin xyz="-0.05 0.0 0.1" rpy="0 0 0"/>
+  </joint>
   <joint name="l_handj" type="fixed">
         <parent link="LWrMot3"/>
@@ -69,4 +97,24 @@
         <child link="LSoftHand"/>
         <origin xyz="0 -0.0305 -0.21" rpy="0 0 0"/>
+  </joint>
+  <joint name="l_handj3" type="fixed">
+        <parent link="LSoftHand"/>
+        <child link="l_hand_upper_right_link"/>
+        <origin xyz="0.05 0.0 0.0" rpy="0 0 0"/>
+  </joint>
+  <joint name="l_handj4" type="fixed">
+        <parent link="LSoftHand"/>
+        <child link="l_hand_lower_right_link"/>
+        <origin xyz="-0.05 0.0 0.0" rpy="0 0 0"/>
+  </joint>
+  <joint name="l_handj5" type="fixed">
+        <parent link="LSoftHand"/>
+        <child link="l_hand_upper_left_link"/>
+        <origin xyz="0.05 0.0 0.1" rpy="0 0 0"/>
+  </joint>
+  <joint name="l_handj6" type="fixed">
+        <parent link="LSoftHand"/>
+        <child link="l_hand_lower_left_link"/>
+        <origin xyz="-0.05 0.0 0.1" rpy="0 0 0"/>
   </joint>
 </xacro:if>

Commit message: Added new TCP_L and TCP_R frames to be compiant with ARMARX code

File: bigman_urdf/urdf/parts/soft_hand.urdf.xacro (robot description, xacro)
@@ -2,4 +2,6 @@
 <robot xmlns:xacro="http://ros.org/wiki/xacro" name="SoftHand">
 <xacro:if value="${BIGMAN_FIXED_HANDS}">
+<xacro:property name="PI" value="3.14159265359" />
+<xacro:property name="PI_2" value="1.57079632679" />
 <xacro:property name="a" value="0.1" />
 <xacro:property name="b" value="0.06" />
@@ -8,4 +10,5 @@
 <!-- LINKS -->
 <link name="RSoftHand"/>
+<link name="TCP_R"/>
 <link name="RSoftHandLink">
     <inertial>
@@ -33,4 +36,5 @@
 <link name="r_hand_lower_left_link"/>
   <link name="LSoftHand"/>
+  <link name="TCP_L"/>
   <link name="LSoftHandLink">
     <inertial>
@@ -117,4 +121,14 @@
         <child link="l_hand_lower_left_link"/>
         <origin xyz="-0.05 0.0 0.1" rpy="0 0 0"/>
+  </joint>
+  <joint name="TCP_Ljoint" type="fixed">
+        <parent link="LSoftHand"/>
+        <child link="TCP_L"/>
+        <origin xyz="0.0 0.0 0.0" rpy="${PI_2} ${PI} 0"/>
+  </joint>
+  <joint name="TCP_Rjoint" type="fixed">
+        <parent link="RSoftHand"/>
+        <child link="TCP_R"/>
+        <origin xyz="0.0 0.0 0.0" rpy="-${PI_2} 0 0"/>
   </joint>
 </xacro:if>

Commit message: Updated hands and doc

File: bigman_urdf/urdf/parts/soft_hand.urdf.xacro (robot description, xacro)
@@ -7,9 +7,12 @@
 <xacro:property name="b" value="0.06" />
 <xacro:property name="c" value="0.14" />
+<xacro:property name="mmTom" value="0.001" />
+<xacro:property name="mm2Tom2" value="${0.001*0.001}" />
+<xacro:property name="tonsToKg" value="1000.0" />
 <!-- For the hand we use the inertia of a parallelepiped -->
 <!-- LINKS -->
 <link name="RSoftHand"/>
 <link name="TCP_R"/>
-<link name="RSoftHandLink">
+<!--link name="RSoftHandLink">
     <inertial>
       <origin xyz="0 0 -0.17" rpy="0 0 0"/>
@@ -30,5 +33,25 @@
       </geometry>
    </collision>
-  </link>
+</link-->
+<link name="RSoftHandLink">
+    <inertial>
+      <origin xyz="${2.0955992*mmTom} ${4.3009755*mmTom} ${-6.0792229e+01*mmTom}" rpy="0 0 0"/>
+      <mass value="1.4"/>
+      <inertia ixx="${4.6340021e+03*mm2Tom2}"  ixy="${-5.6301252e+01*mm2Tom2}"  ixz="${2.1001241e+02*mm2Tom2}" iyy="${5.2222303e+03*mm2Tom2}" iyz="${2.0916976e+02*mm2Tom2}" izz="${1.3961628e+03*mm2Tom2}" />
+    </inertial>
+    <visual>
+      <origin xyz="0.0 0.0 0.0" rpy="0.0 0.0 0.0"/>
+      <geometry name="RSoftHandLink_visual">
+        <mesh filename="package://bigman_urdf/meshes/SoftHandOpen2.STL" scale="0.001 0.001 0.001" />
+      </geometry>
+      <material name="grey"/>
+   </visual>
+   <collision>
+      <origin xyz="0.0 0.0 0.0" rpy="0.0 0.0 0.0"/>
+      <geometry name="RSoftHandLink_collision">
+        <mesh filename="package://bigman_urdf/meshes/simple/SoftHandOpen2.STL" scale="0.001 0.001 0.001" />
+      </geometry>
+   </collision>
+</link>
 <link name="r_hand_upper_right_link"/>
 <link name="r_hand_lower_right_link"/>
@@ -37,5 +60,5 @@
   <link name="LSoftHand"/>
   <link name="TCP_L"/>
-  <link name="LSoftHandLink">
+  <!--link name="LSoftHandLink">
     <inertial>
       <origin xyz="0 0 -0.17" rpy="0 0 0"/>
@@ -56,5 +79,25 @@
       </geometry>
    </collision>
-  </link>
+  </link-->
+<link name="LSoftHandLink">
+    <inertial>
+      <origin xyz="${2.0955992*mmTom} ${-4.3009755*mmTom} ${-6.0792229e+01*mmTom}" rpy="0 0 0"/>
+      <mass value="1.4"/>
+      <inertia ixx="${4.6340021e+03*mm2Tom2}"  ixy="${5.6301252e+01*mm2Tom2}"  ixz="${2.1001241e+02*mm2Tom2}" iyy="${5.2222303e+03*mm2Tom2}" iyz="${-2.0916976e+02*mm2Tom2}" izz="${1.3961628e+03*mm2Tom2}" />
+    </inertial>
+    <visual>
+      <origin xyz="0.0 0.0 0.0" rpy="0.0 0.0 0.0"/>
+      <geometry name="LSoftHandLink_visual">
+        <mesh filename="package://bigman_urdf/meshes/SoftHandOpen2.STL" scale="0.001 -0.001 0.001" />
+      </geometry>
+      <material name="grey"/>
+   </visual>
+   <collision>
+      <origin xyz="0.0 0.0 0.0" rpy="0.0 0.0 0.0"/>
+      <geometry name="LSoftHandLink_collision">
+        <mesh filename="package://bigman_urdf/meshes/simple/SoftHandOpen2.STL" scale="0.001 -0.001 0.001" />
+      </geometry>
+   </collision>
+</link>
 <link name="l_hand_upper_right_link"/>
 <link name="l_hand_lower_right_link"/>
@@ -62,8 +105,13 @@
 <link name="l_hand_lower_left_link"/>
 <!-- JOINTS -->
+  <!--joint name="r_handj" type="fixed">
+        <parent link="RWrMot3"/>
+        <child link="RSoftHandLink"/>
+        <origin xyz="0 0 0" rpy="0 0 0"/>
+  </joint-->
   <joint name="r_handj" type="fixed">
         <parent link="RWrMot3"/>
         <child link="RSoftHandLink"/>
-        <origin xyz="0 0 0" rpy="0 0 0"/>
+        <origin xyz="0 0 ${-69.5*mmTom}" rpy="0 0 0"/>
   </joint>
   <joint name="r_handj2" type="fixed">
@@ -92,8 +140,13 @@
         <origin xyz="-0.05 0.0 0.1" rpy="0 0 0"/>
   </joint>
+  <!--joint name="l_handj" type="fixed">
+        <parent link="LWrMot3"/>
+        <child link="LSoftHandLink"/>
+        <origin xyz="0 0 0" rpy="0 0 0"/>
+  </joint-->
   <joint name="l_handj" type="fixed">
         <parent link="LWrMot3"/>
         <child link="LSoftHandLink"/>
-        <origin xyz="0 0 0" rpy="0 0 0"/>
+        <origin xyz="0 0 ${-69.5*mmTom}" rpy="0 0 0"/>
   </joint>
   <joint name="l_handj2" type="fixed">
@@ -139,6 +192,6 @@
     <inertial>
       <origin xyz="0 0 -0.17" rpy="0 0 0"/>
-      <mass value="1.2"/>
-      <inertia ixx="${1.2*(b*b+c*c)/12.0}"  ixy="0"  ixz="0" iyy="${1.2*(a*a+c*c)/12.0}" iyz="0" izz="${1.2*(a*a+b*b)/12.0}" />
+      <mass value="1.4"/>
+      <inertia ixx="${1.4*(b*b+c*c)/12.0}"  ixy="0"  ixz="0" iyy="${1.4*(a*a+c*c)/12.0}" iyz="0" izz="${1.4*(a*a+b*b)/12.0}" />
     </inertial>
     <visual>
@@ -161,6 +214,6 @@
     <inertial>
       <origin xyz="0 0 -0.17" rpy="0 0 0"/>
-      <mass value="1.2"/>
-      <inertia ixx="${1.2*(b*b+c*c)/12.0}"  ixy="0"  ixz="0" iyy="${1.2*(a*a+c*c)/12.0}" iyz="0" izz="${1.2*(a*a+b*b)/12.0}" />
+      <mass value="1.4"/>
+      <inertia ixx="${1.4*(b*b+c*c)/12.0}"  ixy="0"  ixz="0" iyy="${1.4*(a*a+c*c)/12.0}" iyz="0" izz="${1.4*(a*a+b*b)/12.0}" />
     </inertial>
     <visual>

Commit message: Added new frames for ctrl. Removed extra frames for the hands

File: bigman_urdf/urdf/parts/soft_hand.urdf.xacro (robot description, xacro)
@@ -54,8 +54,10 @@
    </collision>
 </link>
+<!--
 <link name="r_hand_upper_right_link"/>
 <link name="r_hand_lower_right_link"/>
 <link name="r_hand_upper_left_link"/>
 <link name="r_hand_lower_left_link"/>
+-->
   <link name="LSoftHand"/>
   <link name="TCP_L"/>
@@ -100,8 +102,10 @@
    </collision>
 </link>
+<!--
 <link name="l_hand_upper_right_link"/>
 <link name="l_hand_lower_right_link"/>
 <link name="l_hand_upper_left_link"/>
 <link name="l_hand_lower_left_link"/>
+-->
 <!-- JOINTS -->
   <!--joint name="r_handj" type="fixed">
@@ -115,9 +119,15 @@
         <origin xyz="0 0 ${-69.5*mmTom}" rpy="0 0 0"/>
   </joint>
+  <!--joint name="r_handj2" type="fixed">
+        <parent link="RSoftHandLink"/>
+        <child link="RSoftHand"/>
+        <origin xyz="0 0.0305 -0.21" rpy="0 0 0"/>
+  </joint-->
   <joint name="r_handj2" type="fixed">
         <parent link="RSoftHandLink"/>
         <child link="RSoftHand"/>
-        <origin xyz="0 0.0305 -0.21" rpy="0 0 0"/>
-  </joint>
+        <origin xyz="${16.*mmTom}0 0.0 ${-125.5*mmTom}" rpy="0 0 0"/>
+  </joint>
+<!--
   <joint name="r_handj3" type="fixed">
         <parent link="RSoftHand"/>
@@ -140,4 +150,5 @@
         <origin xyz="-0.05 0.0 0.1" rpy="0 0 0"/>
   </joint>
+-->
   <!--joint name="l_handj" type="fixed">
         <parent link="LWrMot3"/>
@@ -150,9 +161,15 @@
         <origin xyz="0 0 ${-69.5*mmTom}" rpy="0 0 0"/>
   </joint>
+  <!--joint name="l_handj2" type="fixed">
+        <parent link="LSoftHandLink"/>
+        <child link="LSoftHand"/>
+        <origin xyz="0 -0.0305 -0.21" rpy="0 0 0"/>
+  </joint-->
   <joint name="l_handj2" type="fixed">
         <parent link="LSoftHandLink"/>
         <child link="LSoftHand"/>
-        <origin xyz="0 -0.0305 -0.21" rpy="0 0 0"/>
-  </joint>
+        <origin xyz="${16.*mmTom}0 0.0 ${-125.5*mmTom}" rpy="0 0 0"/>
+  </joint>
+<!--
   <joint name="l_handj3" type="fixed">
         <parent link="LSoftHand"/>
@@ -175,4 +192,5 @@
         <origin xyz="-0.05 0.0 0.1" rpy="0 0 0"/>
   </joint>
+-->
   <joint name="TCP_Ljoint" type="fixed">
         <parent link="LSoftHand"/>
