Commit message: Corrected control frame and documentation

File: bigman_urdf/urdf/parts/soft_hand.urdf.xacro (robot description, xacro)
@@ -127,5 +127,5 @@
         <parent link="RSoftHandLink"/>
         <child link="RSoftHand"/>
-        <origin xyz="${16.*mmTom}0 0.0 ${-125.5*mmTom}" rpy="0 0 0"/>
+        <origin xyz="${16.*mmTom} ${33.1261*mmTom} ${-125.5*mmTom}" rpy="0 0 0"/>
   </joint>
 <!--
@@ -169,5 +169,5 @@
         <parent link="LSoftHandLink"/>
         <child link="LSoftHand"/>
-        <origin xyz="${16.*mmTom}0 0.0 ${-125.5*mmTom}" rpy="0 0 0"/>
+        <origin xyz="${16.*mmTom} ${-33.1261*mmTom} ${-125.5*mmTom}" rpy="0 0 0"/>
   </joint>
 <!--
