Commit message: Added simplified contact model

File: bigman_urdf/urdf/gazebo/bigman.gazebo.xacro (robot description, xacro)
@@ -5,18 +5,18 @@
      <kp>1000000.0</kp>
      <kd>100.0</kd>
-     <mu1>1.5</mu1>
-     <mu2>1.5</mu2>
+     <mu1>1.0</mu1>
+     <mu2>0.9</mu2>
      <fdir1>1 0 0</fdir1>
      <maxVel>1.0</maxVel>
-     <minDepth>0.00</minDepth>
+     <minDepth>0.003</minDepth>
    </gazebo>
    <gazebo reference="RFoot">
      <kp>1000000.0</kp>
      <kd>100.0</kd>
-     <mu1>1.5</mu1>
-     <mu2>1.5</mu2>
+     <mu1>1.0</mu1>
+     <mu2>0.9</mu2>
      <fdir1>1 0 0</fdir1>
      <maxVel>1.0</maxVel>
-     <minDepth>0.00</minDepth>
+     <minDepth>0.003</minDepth>
    </gazebo>
 <!-- contact model for hand surface -->

File: bigman_urdf/urdf/gazebo/force_torque.gazebo.xacro (robot description, xacro)
@@ -27,9 +27,11 @@
 	<gazebo reference="LAnkSag">
 		<sensor type="force_torque" name="left_leg">
-    	<!--<sensor type="force_torque" name="LAnkSag_FT">-->
 			<always_on>true</always_on>
 			<visualize>true</visualize>
 			<update_rate>1000</update_rate>
 			<pose>0.005 0 -0.107 0 0 0</pose>
+                     <force_torque>
+                            <frame>sensor</frame>
+                     </force_torque>
 			<plugin name="LAnkSag_FT_plugin" filename="libgazebo_yarp_forcetorque.so">
 				<yarpConfigurationFile>model://bigman_urdf/conf/bigman/bigman_gazebo_left_leg_ft.ini</yarpConfigurationFile>
@@ -39,9 +41,11 @@
 	<gazebo reference="RAnkSag">
 		<sensor type="force_torque" name="right_leg">
-			<!--<sensor type="force_torque" name="RAnkSag_FT">-->
 			<always_on>true</always_on>
 			<visualize>true</visualize>
 			<update_rate>1000</update_rate>
 			<pose>0.005 0 -0.107 0 0 0</pose>
+                     <force_torque>
+                            <frame>sensor</frame>
+                     </force_torque>
 			<plugin name="RAnkSag_FT_plugin" filename="libgazebo_yarp_forcetorque.so">
 				<yarpConfigurationFile>model://bigman_urdf/conf/bigman/bigman_gazebo_right_leg_ft.ini</yarpConfigurationFile>

File: bigman_urdf/urdf/parts/legs.urdf.xacro (robot description, xacro)
@@ -116,8 +116,12 @@
     </visual>
     <collision>
-      <origin xyz="0 0 0" rpy="0 0 0"/>
+      <!--<origin xyz="0 0 0" rpy="0 0 0"/>
       <geometry name="RFoot_collision">
         <mesh filename="package://bigman_urdf/meshes/simple/Foot.STL" scale="0.001 -0.001 0.001"/>
-      </geometry>
+      </geometry>-->
+     <origin xyz="0.047 -0.01 -0.1359" rpy="0 0 0"/>
+     <geometry>
+       <box size="0.306 0.16 0.015" />
+     </geometry>
     </collision>
   </link>
@@ -231,8 +235,14 @@
     </visual>
     <collision>
+      <!--
       <origin xyz="0 0 0" rpy="0 0 0"/>
       <geometry name="LFoot_collision">
         <mesh filename="package://bigman_urdf/meshes/simple/Foot.STL" scale="0.001 0.001 0.001"/>
       </geometry>
+      -->
+     <origin xyz="0.047 0.01 -0.1359" rpy="0 0 0"/>
+     <geometry>
+       <box size="0.306 0.16 0.015" />
+     </geometry>
     </collision>
    </link>
