Commit message: Updated colors

File: bigman_urdf/urdf/gazebo/bigman_materials.gazebo.xacro (robot description, xacro)
@@ -1,5 +1,5 @@
 <?xml version="1.0"?>
 <robot xmlns:xacro="http://ros.org/wiki/xacro">
-<gazebo reference="Waist">
+<gazebo reference="base_link">
   <material>Gazebo/Grey</material>
 </gazebo>
@@ -109,3 +109,9 @@
   <material>Gazebo/Black</material>
 </gazebo>
+<gazebo reference="NeckYaw">
+  <material>Gazebo/Grey</material>
+</gazebo>
+<gazebo reference="NeckPitch">
+  <material>Gazebo/Grey</material>
+</gazebo>
 </robot>
