Commit message: hands joint are now represented by red cubes which rotates in the fixed version of walkman robot

File: bigman_urdf/urdf/gazebo/yarp_control.gazebo.xacro (robot description, xacro)
@@ -47,5 +47,5 @@
     </plugin>
 	<!-- HANDS -->
-	<xacro:unless value="${BIGMAN_FIXED_HANDS}">
+    <xacro:unless value="${BIGMAN_FIXED_HANDS}">    </xacro:unless>
 		<plugin name="bigman_yarp_gazebo_plugin_left_hand" filename="libgazebo_yarp_controlboard.so">
 			<yarpConfigurationFile>model://bigman_urdf/conf/bigman/bigman_gazebo_left_hand.ini</yarpConfigurationFile>
@@ -56,5 +56,4 @@
 			<initialConfiguration>0.0</initialConfiguration>
 		</plugin>
-	</xacro:unless>
 </xacro:if>
 <xacro:if value="${BIGMAN_LEGS}">
@@ -82,5 +81,5 @@
 </xacro:if>
 <!-- Plugin to apply external wrenches to the robot & show the CoM in simulation-->
-<!-- plugin name="bigman_yarp_gazebo_plugin_external_wrench" filename="libgazebo_yarp_externalwrench.so"/ -->
+<plugin name="bigman_yarp_gazebo_plugin_external_wrench" filename="libgazebo_yarp_externalwrench.so"/>
 <plugin name="bigman_add_objects" filename="libgazebo_yarp_objects.so"/>
 <plugin name="bigman_show_model_com" filename="libgazebo_yarp_showmodelcom.so"/>

File: bigman_urdf/urdf/parts/soft_hand.urdf.xacro (robot description, xacro)
@@ -9,4 +9,20 @@
 <link name="RSoftHand"/>
 <link name="r_palm"/>
+<link name="R_visual_cube">
+    <inertial>
+        <origin xyz="0 0 0" rpy="0 0 0"/>
+        <mass value="1.0e-5"/>
+        <inertia ixx="0"  ixy="0"  ixz="0" iyy="0" iyz="0" izz="0" />
+    </inertial>
+    <visual>
+        <origin xyz="0 0 0" rpy="0 0 0" />
+        <geometry>
+            <box size="0.08 0.08 0.08" />
+        </geometry>
+    </visual>
+</link>
+<gazebo reference="R_visual_cube">
+    <material>Gazebo/RedBright</material>
+</gazebo>
 <link name="RSoftHandLink">
     <inertial>
@@ -31,4 +47,20 @@
   <link name="LSoftHand"/>
   <link name="l_palm"/>
+  <link name="L_visual_cube">
+      <inertial>
+          <origin xyz="0 0 0" rpy="0 0 0"/>
+          <mass value="1.0e-5"/>
+          <inertia ixx="0"  ixy="0"  ixz="0" iyy="0" iyz="0" izz="0" />
+      </inertial>
+      <visual>
+          <origin xyz="0 0 0" rpy="0 0 0" />
+          <geometry>
+              <box size="0.08 0.08 0.08" />
+          </geometry>
+      </visual>
+  </link>
+  <gazebo reference="L_visual_cube">
+      <material>Gazebo/RedBright</material>
+  </gazebo>
   <link name="LSoftHandLink">
     <inertial>
@@ -52,5 +84,13 @@
   </link>
 <!-- JOINTS -->
-  <joint name="r_handj" type="fixed">
+  <joint name="r_handj" type="revolute">
+      <parent link="RWrMot3"/>
+      <child link="R_visual_cube"/>
+      <origin xyz="0 0 -0.04" rpy="0 0 0"/>
+      <axis xyz="1 0 0" />
+      <limit velocity="4.0" effort="5" lower="0.0" upper="1.7" />
+      <dynamics friction="0" damping="3.0"/>
+  </joint>
+  <joint name="r_handj1" type="fixed">
         <parent link="RWrMot3"/>
         <child link="RSoftHandLink"/>
@@ -67,5 +107,13 @@
         <origin xyz="0 ${2.0696923e+01*mmTom+5.0*mmTom} 0.0" rpy="0 0 0"/>
   </joint>
-  <joint name="l_handj" type="fixed">
+  <joint name="l_handj" type="revolute">
+      <parent link="LWrMot3"/>
+      <child link="L_visual_cube"/>
+      <origin xyz="0 0 -0.04" rpy="0 0 0"/>
+      <axis xyz="-1 0 0" />
+      <limit velocity="4.0" effort="5" lower="0" upper="1.7" />
+      <dynamics friction="0" damping="3.0"/>
+  </joint>
+  <joint name="l_handj1" type="fixed">
         <parent link="LWrMot3"/>
         <child link="LSoftHandLink"/>
