Commit message: added new imu

File: bigman_urdf/urdf/gazebo/microstrain_3dmgx2_imu.gazebo.xacro (robot description, xacro)
@@ -36,3 +36,33 @@
         </sensor>
        </gazebo>
+       <gazebo reference="imu_link2">
+        <sensor name="imu_sensor2" type="imu">
+         <always_on>1</always_on>
+         <update_rate>1000</update_rate>
+         <visualize>true</visualize>
+         <topic>__default_topic__</topic>
+	 <imu>
+          <!--
+          <noise>
+           <type>gaussian</type>
+            <rate>
+             <mean>0.0</mean>
+             <stddev>2e-4</stddev>
+             <bias_mean>0.0000075</bias_mean>
+             <bias_stddev>0.0000008</bias_stddev>
+            </rate>
+            <accel>
+             <mean>0.0</mean>
+             <stddev>1.7e-2</stddev>
+             <bias_mean>0.1</bias_mean>
+             <bias_stddev>0.001</bias_stddev>
+            </accel>
+          </noise>
+          -->
+         </imu>
+         <plugin name="bigman_yarp_gazebo_plugin_IMU2" filename="libgazebo_yarp_imu.so">
+           <yarpConfigurationFile>model://bigman_urdf/conf/bigman/bigman_gazebo_inertial2.ini</yarpConfigurationFile>
+         </plugin>
+        </sensor>
+       </gazebo>
 </robot>

File: bigman_urdf/urdf/sensors/imu.urdf.xacro (robot description, xacro)
@@ -3,4 +3,17 @@
 <xacro:property name="PI" value="3.14159265359" />
 <link name="imu_link">
+    <inertial>
+      <mass value="0.01"/>
+      <origin xyz="0 0 0"/>
+      <inertia ixx="1.0E-6" ixy="0" ixz="0" iyy="1.0E-6" iyz="0" izz="1.0E-6"/>
+    </inertial>
+    <visual>
+      <origin rpy="0 0 0" xyz="0 0 0"/>
+      <geometry>
+        <box size="0.01 0.01 0.01"/>
+      </geometry>
+    </visual>
+  </link>
+<link name="imu_link2">
     <inertial>
       <mass value="0.01"/>
@@ -20,3 +33,8 @@
     <origin xyz="-0.072 -0.0068 0.044" rpy="0 0 0"/>
 </joint>
+<joint name="imu_joint2" type="fixed">
+    <parent link="imu_link"/>
+    <child link="imu_link2"/>
+    <origin xyz="0 0 0.01" rpy="0 0 0"/>
+</joint>
 </robot>
