Commit message: Added an upper_body model for simulation

File: bigman_urdf/urdf/config/bigman_only_upper_body_gazebo.urdf.xacro (robot description, xacro)
@@ -1,5 +1,5 @@
 <?xml version="1.0"?>
 <robot xmlns:xacro="http://ros.org/wiki/xacro" name="BIGMAN">
-<xacro:property name="model_name" value="IIT Bigman Upper Body Ctrl" />
+<xacro:property name="model_name" value="IIT Bigman Upper Body" />
 <xacro:property name="model_version" value="0.1" />
 <!--
@@ -45,5 +45,5 @@
 ####################################################
 -->
-<xacro:property name="BIGMAN_FIXED_HANDS" value="true" />
+<xacro:property name="BIGMAN_FIXED_HANDS" value="false" />
 <!--
 ####################################################
@@ -57,4 +57,4 @@
 ####################################################
 -->
-<xacro:property name="BIGMAN_FIXED_MULTISENSE" value="true" />
+<xacro:property name="BIGMAN_FIXED_MULTISENSE" value="false" />
 </robot>
