Commit message: Added multisense in bigman real

File: bigman_urdf/urdf/config/bigman_real.urdf.xacro (robot description, xacro)
@@ -76,5 +76,5 @@
 ####################################################
 -->
-<xacro:property name="BIGMAN_FIXED_MULTISENSE" value="true" />
+<xacro:property name="BIGMAN_FIXED_MULTISENSE" value="false" />
 <!--
 ####################################################
@@ -90,5 +90,5 @@
 ####################################################
 -->
-<xacro:property name="BIGMAN_HEAD" value="false" />
+<xacro:property name="BIGMAN_HEAD" value="true" />
 <!--
 ####################################################
@@ -100,5 +100,5 @@
 ####################################################
 -->
-<xacro:property name="BIGMAN_ADD_PROTECTIONS" value="true" />
+<xacro:property name="BIGMAN_ADD_PROTECTIONS" value="false" />
 <!--
 ####################################################

File: bigman_urdf/urdf/sensors/multisense_sl.urdf.xacro (robot description, xacro)
@@ -128,4 +128,10 @@
       </geometry>
     </visual>
+    <collision>
+      <origin rpy="0 0 0" xyz="0 0 0"/>
+      <geometry>
+        <box size="0.01 0.01 0.01"/>
+      </geometry>
+    </collision>
   </link>
   <joint name="head_imu_joint" type="fixed">
