Commit message: Changed configs

File: bigman_urdf/urdf/config/bigman_gazebo.urdf.xacro (robot description, xacro)
@@ -64,5 +64,5 @@
 ####################################################
 -->
-<xacro:property name="BIGMAN_FIXED_HANDS" value="false" />
+<xacro:property name="BIGMAN_FIXED_HANDS" value="true" />
 <!--
 ####################################################

File: bigman_urdf/urdf/config/bigman_real.urdf.xacro (robot description, xacro)
@@ -90,5 +90,5 @@
 ####################################################
 -->
-<xacro:property name="BIGMAN_HEAD" value="true" />
+<xacro:property name="BIGMAN_HEAD" value="false" />
 <!--
 ####################################################
@@ -100,5 +100,5 @@
 ####################################################
 -->
-<xacro:property name="BIGMAN_ADD_PROTECTIONS" value="false" />
+<xacro:property name="BIGMAN_ADD_PROTECTIONS" value="true" />
 <!--
 ####################################################
@@ -154,4 +154,4 @@
 ####################################################
 -->
-<xacro:property name="BIGMAN_MAGNETIC_ATTACH_ROS" value="true" />
+<xacro:property name="BIGMAN_MAGNETIC_ATTACH_ROS" value="false" />
 </robot>
