Commit message: changed orientation of IMU link

File: bigman_urdf/urdf/sensors/imu.urdf.xacro (robot description, xacro)
@@ -18,5 +18,5 @@
     <parent link="Waist"/>
     <child link="imu_link"/>
-    <origin xyz="-0.072 -0.0068 0.044" rpy="0 ${PI} 0"/>
+    <origin xyz="-0.072 -0.0068 0.044" rpy="0 0 0"/>
 </joint>
 </robot>

Commit message: Updated imu pose in urdf

File: bigman_urdf/urdf/sensors/imu.urdf.xacro (robot description, xacro)
@@ -18,5 +18,5 @@
     <parent link="Waist"/>
     <child link="imu_link"/>
-    <origin xyz="-0.072 -0.0068 0.044" rpy="0 0 0"/>
+    <origin xyz="0.07199 -0.06098 -0.045" rpy="0 0 0"/>
 </joint>
 </robot>

Commit message: Moved pose IMUs.

File: bigman_urdf/urdf/sensors/imu.urdf.xacro (robot description, xacro)
@@ -31,10 +31,10 @@
     <parent link="Waist"/>
     <child link="imu_link"/>
-    <origin xyz="-0.072 -0.0068 0.044" rpy="0 0 0"/>
+    <origin xyz="0.0535 0.0 0.0601" rpy="0 0 0"/>
 </joint>
 <joint name="imu_joint2" type="fixed">
-    <parent link="imu_link"/>
+    <parent link="Waist"/>
     <child link="imu_link2"/>
-    <origin xyz="0 0 0.01" rpy="0 0 0"/>
+    <origin xyz="0.0135 0.0 0.0601" rpy="0 0 0"/>
 </joint>
 </robot>
