Commit message: Deleted and added files

File: bigman_srdf/srdf/bigman.srdf.xacro (robot description, xacro)
@@ -11,5 +11,5 @@
     <!--CHAINS: When a chain is specified, all the links along the chain (including endpoints) are included in the group. Additionally, all the joints that are parents to included links are also included. This means that joints along the chain and the parent joint of the base link are included in the group-->
     <!--SUBGROUPS: Groups can also be formed by referencing to already defined group names-->
-<xacro:if value="${GAZEBO_bigman_USES_7DOF_FOREARMS_DRC_14}">
+<xacro:if value="${GAZEBO_BIGMAN_USES_7DOF_FOREARMS_DRC_14}">
     <group name="left_arm">
         <joint name="LShSag" />
@@ -31,5 +31,5 @@
     </group>
 </xacro:if>
-<xacro:unless value="${GAZEBO_bigman_USES_7DOF_FOREARMS_DRC_14}">
+<xacro:unless value="${GAZEBO_BIGMAN_USES_7DOF_FOREARMS_DRC_14}">
     <group name="left_arm">
         <joint name="LShSag" />

File: bigman_urdf/urdf/bigman_config.urdf.xacro (robot description, xacro)
@@ -1,4 +1,4 @@
 <?xml version="1.0"?>
-<robot xmlns:xacro="http://ros.org/wiki/xacro" name="bigman">
+<robot xmlns:xacro="http://ros.org/wiki/xacro" name="BIGMAN">
 <xacro:property name="model_name" value="IIT Bigman w/ Softhand" />
 <xacro:property name="model_version" value="0.1" />

File: bigman_urdf/urdf/config/bigman.urdf.xacro (robot description, xacro)
@@ -1,5 +1,5 @@
 <?xml version="1.0"?>
 <robot xmlns:xacro="http://ros.org/wiki/xacro" name="BIGMAN">
-<xacro:property name="model_name" value="IIT Coman w/ Softhand" />
+<xacro:property name="model_name" value="IIT Bigman w/ Softhand" />
 <xacro:property name="model_version" value="0.1" />
 <!--

File: bigman_urdf/urdf/config/bigman_hands.urdf.xacro (robot description, xacro)
@@ -1,5 +1,5 @@
 <?xml version="1.0"?>
 <robot xmlns:xacro="http://ros.org/wiki/xacro" name="BIGMAN">
-<xacro:property name="model_name" value="IIT Coman" />
+<xacro:property name="model_name" value="IIT Bigman" />
 <xacro:property name="model_version" value="1.0" />
 <!--

File: bigman_urdf/urdf/config/bigman_no_forearms.urdf.xacro (robot description, xacro)
@@ -1,5 +1,5 @@
 <?xml version="1.0"?>
 <robot xmlns:xacro="http://ros.org/wiki/xacro" name="BIGMAN">
-<xacro:property name="model_name" value="IIT Coman 2013" />
+<xacro:property name="model_name" value="IIT Bigman 2013" />
 <xacro:property name="model_version" value="1.0" />
 <!--

Commit message: Deleted useless variable in srdf.xacro

File: bigman_srdf/srdf/bigman.srdf.xacro (robot description, xacro)
@@ -11,5 +11,4 @@
     <!--CHAINS: When a chain is specified, all the links along the chain (including endpoints) are included in the group. Additionally, all the joints that are parents to included links are also included. This means that joints along the chain and the parent joint of the base link are included in the group-->
     <!--SUBGROUPS: Groups can also be formed by referencing to already defined group names-->
-<xacro:if value="${GAZEBO_BIGMAN_USES_7DOF_FOREARMS_DRC_14}">
     <group name="left_arm">
         <joint name="LShSag" />
@@ -30,19 +29,4 @@
         <joint name="RWrj2" />
     </group>
-</xacro:if>
-<xacro:unless value="${GAZEBO_BIGMAN_USES_7DOF_FOREARMS_DRC_14}">
-    <group name="left_arm">
-        <joint name="LShSag" />
-        <joint name="LShLat" />
-        <joint name="LShYaw" />
-        <joint name="LElbj" />
-    </group>
-    <group name="right_arm">
-        <joint name="RShSag" />
-        <joint name="RShLat" />
-        <joint name="RShYaw" />
-        <joint name="RElbj" />
-    </group>
-</xacro:unless>
     <group name="left_leg">
         <joint name="LHipSag" />

Commit message: Updated to new version of srdf

File: bigman_srdf/srdf/bigman.srdf.xacro (robot description, xacro)
@@ -11,42 +11,32 @@
     <!--CHAINS: When a chain is specified, all the links along the chain (including endpoints) are included in the group. Additionally, all the joints that are parents to included links are also included. This means that joints along the chain and the parent joint of the base link are included in the group-->
     <!--SUBGROUPS: Groups can also be formed by referencing to already defined group names-->
+    <group name="base">
+        <link name="Waist"/>
+    </group>
+    <group name="sensors">
+        <joint name="l_ankle_joint"/>
+        <joint name="r_ankle_joint"/>
+    </group>
     <group name="left_arm">
-        <joint name="LShSag" />
-        <joint name="LShLat" />
-        <joint name="LShYaw" />
-        <joint name="LElbj" />
-        <joint name="LForearmPlate" />
-        <joint name="LWrj1" />
-        <joint name="LWrj2" />
+        <chain base_link="DWYTorso" tip_link="l_wrist"/>
     </group>
     <group name="right_arm">
-        <joint name="RShSag" />
-        <joint name="RShLat" />
-        <joint name="RShYaw" />
-        <joint name="RElbj" />
-        <joint name="RForearmPlate" />
-        <joint name="RWrj1" />
-        <joint name="RWrj2" />
+        <chain base_link="DWYTorso" tip_link="r_wrist"/>
     </group>
     <group name="left_leg">
-        <joint name="LHipSag" />
-        <joint name="LHipLat" />
-        <joint name="LHipYaw" />
-        <joint name="LKneeSag" />
-        <joint name="LAnkLat" />
-        <joint name="LAnkSag" />
+        <chain base_link="Waist" tip_link="l_sole"/>
     </group>
     <group name="right_leg">
-        <joint name="RHipSag" />
-        <joint name="RHipLat" />
-        <joint name="RHipYaw" />
-        <joint name="RKneeSag" />
-        <joint name="RAnkLat" />
-        <joint name="RAnkSag" />
+        <chain base_link="Waist" tip_link="r_sole"/>
     </group>
     <group name="torso">
-        <joint name="WaistLat" />
-        <joint name="WaistSag" />
-        <joint name="WaistYaw" />
+        <chain base_link="Waist" tip_link="DWYTorso"/>
+    </group>
+    <group name="chains"> <!--THIS HAS TO BE THE LAST GROUP IN THE FILE -->
+        <group name="left_arm"/>
+        <group name="right_arm"/>
+        <group name="left_leg"/>
+        <group name="right_leg"/>
+        <group name="torso"/>
     </group>
 </robot>

Commit message: Tuned (by trial and error) position PIDs for legs (in simulation). Changed sensors name in urdf. Added possibility to have bigman fixed in simulation.

File: bigman_srdf/srdf/bigman.srdf.xacro (robot description, xacro)
@@ -15,6 +15,6 @@
     </group>
     <group name="sensors">
-        <joint name="l_ankle_joint"/>
-        <joint name="r_ankle_joint"/>
+        <joint name="l_leg_ft_joint"/>
+        <joint name="r_leg_ft_joint"/>
     </group>
     <group name="left_arm">

File: bigman_urdf/urdf/bigman_robot.urdf.xacro (robot description, xacro)
@@ -6,4 +6,14 @@
   This file groups files to use BIGMAN in GAZEBO
   -->
+  <!-- Uncomment this to have the robot rigidly connected to the world -->
+<!--
+  <link name="world"/>
+   <joint name="fixed" type="fixed">
+    <parent link="world"/>
+    <child link="base_link"/>
+  </joint>
+  <origin xyz="0.0 0.0 1.5" rpy="0 0 0" /> -->
+  <origin xyz="0.0 0.0 1.12" rpy="0 0 0" />
+  <!-- ROBOT -->
   <xacro:include filename="$(find bigman_urdf)/urdf/bigman.urdf.xacro" />
   <xacro:include filename="$(find bigman_urdf)/urdf/gazebo/microstrain_3dmgx2_imu.gazebo.xacro" />
@@ -12,4 +22,3 @@
 <!-- YARP PLUGINS for GAZEBO SIMULATION -->
   <xacro:include filename="$(find bigman_urdf)/urdf/gazebo/yarp_control.gazebo.xacro" />
-  <origin xyz="0.0 0.0 1.12" rpy="0 0 0" />
 </robot>

Commit message: Deleted group sensor, added group force_torque_sensors

File: bigman_srdf/srdf/bigman.srdf.xacro (robot description, xacro)
@@ -14,7 +14,7 @@
         <link name="Waist"/>
     </group>
-    <group name="sensors">
-        <joint name="l_leg_ft_joint"/>
-        <joint name="r_leg_ft_joint"/>
+    <group name="force_torque_sensors">
+            <joint name="l_leg_ft_joint"/>
+            <joint name="r_leg_ft_joint"/>
     </group>
     <group name="left_arm">

Commit message: Added proper position and frames for ft sensors in arm.

File: bigman_srdf/srdf/bigman.srdf.xacro (robot description, xacro)
@@ -17,4 +17,6 @@
             <joint name="l_leg_ft_joint"/>
             <joint name="r_leg_ft_joint"/>
+            <joint name="l_arm_ft_joint"/>
+            <joint name="r_arm_ft_joint"/>
     </group>
     <group name="left_arm">

File: bigman_urdf/urdf/bigman.urdf.xacro (robot description, xacro)
@@ -35,4 +35,16 @@
     <origin xyz="0.005 0 -0.107" rpy="0 0 0" />
 </joint>
+<link name="l_arm_ft"/>
+<link name="r_arm_ft"/>
+<joint name="l_arm_ft_joint" type="fixed">
+    <parent link="LWrMot3"/>
+    <child link="l_arm_ft"/>
+    <origin xyz="0 0 -0.0565" rpy="0 0 0" />
+</joint>
+<joint name="r_arm_ft_joint" type="fixed">
+    <parent link="RWrMot3"/>
+    <child link="r_arm_ft"/>
+    <origin xyz="0 0 -0.0565" rpy="0 0 0" />
+</joint>
 <!-- ************ FOREARMS ************ -->
 <!-- This links are defined in order to be compliant with http://www.ros.org/reps/rep-0120.html#coordinate-frames

File: bigman_urdf/urdf/gazebo/force_torque.gazebo.xacro (robot description, xacro)
@@ -1,5 +1,5 @@
 <?xml version="1.0"?>
-<robot xmlns:xacro="http://ros.org/wiki/xacro">
-	<gazebo reference="RForearmPlate">
+<robot xmlns:xacro="http:/ros.org/wiki/xacro">
+	<gazebo reference="RWrj2">
 		<sensor type="force_torque" name="right_arm">
 			<!--<sensor type="force_torque" name="LAnkSag_FT">-->
@@ -7,4 +7,5 @@
 			<visualize>true</visualize>
 			<update_rate>1000</update_rate>
+                     <pose>0 0 -0.0565 0 0 0</pose>
 			<plugin name="RForearmPlate_FT_plugin" filename="libgazebo_yarp_forcetorque.so">
 				<yarpConfigurationFile>model://bigman_urdf/conf/bigman/bigman_gazebo_right_arm_ft.ini</yarpConfigurationFile>
@@ -12,5 +13,5 @@
 		</sensor>
 	</gazebo>
-	<gazebo reference="LForearmPlate">
+	<gazebo reference="LWrj2">
 		<sensor type="force_torque" name="left_arm">
 			<!--<sensor type="force_torque" name="LAnkSag_FT">-->
@@ -18,4 +19,5 @@
 			<visualize>true</visualize>
 			<update_rate>1000</update_rate>
+                     <pose>0 0 -0.0565 0 0 0</pose>
 			<plugin name="LForearmPlate_FT_plugin" filename="libgazebo_yarp_forcetorque.so">
 				<yarpConfigurationFile>model://bigman_urdf/conf/bigman/bigman_gazebo_left_arm_ft.ini</yarpConfigurationFile>
