Commit message: Added model of bigman only legs

File: bigman_srdf/srdf/bigman.srdf.xacro (robot description, xacro)
@@ -17,7 +17,10 @@
             <joint name="l_leg_ft_joint"/>
             <joint name="r_leg_ft_joint"/>
-            <joint name="l_arm_ft_joint"/>
-            <joint name="r_arm_ft_joint"/>
+            <xacro:unless value="${BIGMAN_ONLY_LEGS}">
+              <joint name="l_arm_ft_joint"/>
+              <joint name="r_arm_ft_joint"/>
+            </xacro:unless>
     </group>
+ <xacro:unless value="${BIGMAN_ONLY_LEGS}">
     <group name="left_arm">
         <chain base_link="DWYTorso" tip_link="l_wrist"/>
@@ -26,4 +29,5 @@
         <chain base_link="DWYTorso" tip_link="r_wrist"/>
     </group>
+</xacro:unless>
     <group name="left_leg">
         <chain base_link="Waist" tip_link="l_sole"/>
@@ -32,13 +36,19 @@
         <chain base_link="Waist" tip_link="r_sole"/>
     </group>
+ <xacro:unless value="${BIGMAN_ONLY_LEGS}">
     <group name="torso">
         <chain base_link="Waist" tip_link="DWYTorso"/>
     </group>
+</xacro:unless>
     <group name="chains"> <!--THIS HAS TO BE THE LAST GROUP IN THE FILE -->
+<xacro:unless value="${BIGMAN_ONLY_LEGS}">
         <group name="left_arm"/>
         <group name="right_arm"/>
+</xacro:unless>
         <group name="left_leg"/>
         <group name="right_leg"/>
+<xacro:unless value="${BIGMAN_ONLY_LEGS}">
         <group name="torso"/>
+</xacro:unless>
     </group>
 </robot>

File: bigman_urdf/urdf/bigman.urdf.xacro (robot description, xacro)
@@ -10,4 +10,5 @@
 <!-- ************ MODEL CONFIGURATION ************ -->
 <xacro:include filename="$(find bigman_urdf)/urdf/bigman_config.urdf.xacro" />
+<xacro:unless value="${BIGMAN_ONLY_LEGS}">
 <!-- Head -->
 <!-- This links are defined in order to be compliant with http://www.ros.org/reps/rep-0120.html#coordinate-frames
@@ -20,4 +21,5 @@
 	<origin xyz="0 0 0.1" rpy="0 0 0" />
 </joint>
+</xacro:unless>
 <!-- ************ BIGMAN BASE ************** -->
 <xacro:include filename="$(find bigman_urdf)/urdf/bigman_base.urdf.xacro"/>
@@ -35,4 +37,5 @@
     <origin xyz="0.005 0 -0.107" rpy="0 0 0"/>
 </joint>
+<xacro:unless value="${BIGMAN_ONLY_LEGS}">
 <link name="l_arm_ft"/>
 <link name="r_arm_ft"/>
@@ -58,6 +61,4 @@
 <!-- Reference frames in hands -->
 <xacro:include filename="$(find bigman_urdf)/urdf/parts/hand_reference_frame.urdf.xacro" />
-<!-- IMU -->
-<xacro:include filename="$(find bigman_urdf)/urdf/sensors/imu.urdf.xacro"/>
 <!-- multisense_sl_v4 with fixed joints (NOT FOR SIMULATION) -->
 <xacro:include filename="$(find bigman_urdf)/urdf/sensors/multisense_sl.urdf.xacro"/>
@@ -67,3 +68,6 @@
     <origin xyz="0.05 0 0.05" rpy="0 0 0" />
 </joint>
+</xacro:unless>
+<!-- IMU -->
+<xacro:include filename="$(find bigman_urdf)/urdf/sensors/imu.urdf.xacro"/>
 </robot>

File: bigman_urdf/urdf/bigman_base.urdf.xacro (robot description, xacro)
@@ -8,7 +8,36 @@
   Velocity and effort limits are fake!
 -->
-<!-- ********************TORSO******************** -->
-<!-- first real link of the robot, inertial reference frame -->
-<xacro:include filename="$(find bigman_urdf)/urdf/parts/torso.urdf.xacro" />
+<!--
+The coordinate frame called base_link is rigidly attached to the robot root body. It is recommended to choose the robot waist as its root body. The base_link can be attached to the root in any arbitrary position or orientation; for every hardware platform there will be a different place on the base that provides an obvious point of reference. Note that REP 103 [1] specifies a preferred orientation for frames. -->
+<link name="base_link"/>
+<link name="Waist">
+    <inertial>
+      <origin xyz="${-3.2862932e+01*mmTom} ${-5.0930727e-01*mmTom} ${-1.2899617*mmTom}" rpy="0.0 0.0 0.0"/>
+      <mass value="6.4080904"/>
+      <inertia ixx="${3.8826078e+04*mm2Tom2}"  ixy="${2.9047605e+02*mm2Tom2}"  ixz="${6.8975598e+02*mm2Tom2}" iyy="${2.5050374e+04*mm2Tom2}" iyz="${-1.3370623e+01*mm2Tom2}" izz="${4.8055286e+04*mm2Tom2}" />
+    </inertial>
+    <visual>
+      <origin xyz="0 0 0" rpy="0 0 0"/>
+      <geometry name="Waist_visual">
+        <mesh filename="package://bigman_urdf/meshes/Waist.STL" scale="0.001 0.001 0.001"/>
+      </geometry>
+    </visual>
+    <collision>
+      <origin xyz="0 0 0" rpy="0 0 0"/>
+      <geometry name="Waist_collision">
+        <mesh filename="package://bigman_urdf/meshes/simple/Waist.STL" scale="0.001 0.001 0.001"/>
+      </geometry>
+    </collision>
+</link>
+<joint name="base_joint" type="fixed">
+    <parent link="base_link"/>
+    <child link="Waist"/>
+    <origin xyz="0 0 0" rpy="0 0 0" />
+</joint>
+<xacro:unless value="${BIGMAN_ONLY_LEGS}">
+       <!-- ********************TORSO******************** -->
+       <!-- first real link of the robot, inertial reference frame -->
+       <xacro:include filename="$(find bigman_urdf)/urdf/parts/torso.urdf.xacro" />
+</xacro:unless>
 <!-- ********************LEGS******************** -->
 <!-- This links are defined in order to be compliant with http://www.ros.org/reps/rep-0120.html#coordinate-frames
@@ -56,5 +85,7 @@
 <!-- Reference frames in feet -->
 <xacro:include filename="$(find bigman_urdf)/urdf/parts/foot_reference_frame.urdf.xacro" />
-<!-- ********************ARMS******************** -->
-<xacro:include filename="$(find bigman_urdf)/urdf/parts/arms.urdf.xacro" />
+<xacro:unless value="${BIGMAN_ONLY_LEGS}">
+       <!-- ********************ARMS******************** -->
+       <xacro:include filename="$(find bigman_urdf)/urdf/parts/arms.urdf.xacro" />
+</xacro:unless>
 </robot>

File: bigman_urdf/urdf/bigman_config.urdf.xacro (robot description, xacro)
@@ -3,4 +3,17 @@
 <xacro:property name="model_name" value="IIT Bigman Ctrl" />
 <xacro:property name="model_version" value="0.1" />
+<!--
+####################################################
+##
+##  BIGMAN_ONLY_LEGS
+##  if "true" only the kinematic chains of the legs
+##  will be used to generate the model, the flags
+##  regarding the upper body will not be taken in
+##  consideration.
+##
+##
+####################################################
+-->
+<xacro:property name="BIGMAN_ONLY_LEGS" value="false" />
 <!--
 ####################################################

File: bigman_urdf/urdf/bigman_robot.urdf.xacro (robot description, xacro)
@@ -17,5 +17,7 @@
   <!-- ROBOT -->
   <xacro:include filename="$(find bigman_urdf)/urdf/bigman.urdf.xacro" />
-  <xacro:include filename="$(find bigman_urdf)/urdf/gazebo/microstrain_3dmgx2_imu.gazebo.xacro" />
+  <xacro:unless value="${BIGMAN_ONLY_LEGS}">
+       <xacro:include filename="$(find bigman_urdf)/urdf/gazebo/microstrain_3dmgx2_imu.gazebo.xacro" />
+  </xacro:unless>
   <xacro:include filename="$(find bigman_urdf)/urdf/gazebo/force_torque.gazebo.xacro" />
   <xacro:include filename="$(find bigman_urdf)/urdf/gazebo/bigman.gazebo.xacro" />

File: bigman_urdf/urdf/config/bigman_gazebo.urdf.xacro (robot description, xacro)
@@ -3,4 +3,17 @@
 <xacro:property name="model_name" value="IIT Bigman" />
 <xacro:property name="model_version" value="0.1" />
+<!--
+####################################################
+##
+##  BIGMAN_ONLY_LEGS
+##  if "true" only the kinematic chains of the legs
+##  will be used to generate the model, the flags
+##  regarding the upper body will not be taken in
+##  consideration.
+##
+##
+####################################################
+-->
+<xacro:property name="BIGMAN_ONLY_LEGS" value="false" />
 <!--
 ####################################################

File: bigman_urdf/urdf/gazebo/bigman.gazebo.xacro (robot description, xacro)
@@ -47,4 +47,5 @@
 </xacro:if>
 -->
+<xacro:unless value="${BIGMAN_ONLY_LEGS}">
 <!-- Other parameters... -->
    <gazebo reference="WaistSag">
@@ -60,53 +61,5 @@
     <provideFeedback>true</provideFeedback>
    </gazebo>
-   <gazebo reference="RHipSag">
-    <implicitSpringDamper>1</implicitSpringDamper>
-    <provideFeedback>true</provideFeedback>
-   </gazebo>
-   <gazebo reference="RHipLat">
-    <implicitSpringDamper>1</implicitSpringDamper>
-    <provideFeedback>true</provideFeedback>
-   </gazebo>
-   <gazebo reference="RHipYaw">
-    <implicitSpringDamper>1</implicitSpringDamper>
-    <provideFeedback>true</provideFeedback>
-   </gazebo>
-   <gazebo reference="RKneeSag">
-    <implicitSpringDamper>1</implicitSpringDamper>
-    <provideFeedback>true</provideFeedback>
-   </gazebo>
-   <gazebo reference="RAnkLat">
-    <implicitSpringDamper>1</implicitSpringDamper>
-    <provideFeedback>true</provideFeedback>
-   </gazebo>
-   <gazebo reference="RAnkSag">
-    <implicitSpringDamper>1</implicitSpringDamper>
-    <provideFeedback>true</provideFeedback>
-  </gazebo>
-   <gazebo reference="LHipSag">
-    <implicitSpringDamper>1</implicitSpringDamper>
-    <provideFeedback>true</provideFeedback>
-   </gazebo>
-   <gazebo reference="LHipLat">
-    <implicitSpringDamper>1</implicitSpringDamper>
-    <provideFeedback>true</provideFeedback>
-   </gazebo>
-   <gazebo reference="LHipYaw">
-    <implicitSpringDamper>1</implicitSpringDamper>
-    <provideFeedback>true</provideFeedback>
-   </gazebo>
-   <gazebo reference="LKneeSag">
-    <implicitSpringDamper>1</implicitSpringDamper>
-    <provideFeedback>true</provideFeedback>
-   </gazebo>
-   <gazebo reference="LAnkLat">
-    <implicitSpringDamper>1</implicitSpringDamper>
-    <provideFeedback>true</provideFeedback>
-   </gazebo>
-   <gazebo reference="LAnkSag">
-    <implicitSpringDamper>1</implicitSpringDamper>
-    <provideFeedback>true</provideFeedback>
-   </gazebo>
-   <gazebo reference="RShSag">
+<gazebo reference="RShSag">
     <implicitSpringDamper>1</implicitSpringDamper>
     <provideFeedback>true</provideFeedback>
@@ -176,3 +129,52 @@
       </gazebo>
     </xacro:unless>
+</xacro:unless>
+   <gazebo reference="RHipSag">
+    <implicitSpringDamper>1</implicitSpringDamper>
+    <provideFeedback>true</provideFeedback>
+   </gazebo>
+   <gazebo reference="RHipLat">
+    <implicitSpringDamper>1</implicitSpringDamper>
+    <provideFeedback>true</provideFeedback>
+   </gazebo>
+   <gazebo reference="RHipYaw">
+    <implicitSpringDamper>1</implicitSpringDamper>
+    <provideFeedback>true</provideFeedback>
+   </gazebo>
+   <gazebo reference="RKneeSag">
+    <implicitSpringDamper>1</implicitSpringDamper>
+    <provideFeedback>true</provideFeedback>
+   </gazebo>
+   <gazebo reference="RAnkLat">
+    <implicitSpringDamper>1</implicitSpringDamper>
+    <provideFeedback>true</provideFeedback>
+   </gazebo>
+   <gazebo reference="RAnkSag">
+    <implicitSpringDamper>1</implicitSpringDamper>
+    <provideFeedback>true</provideFeedback>
+  </gazebo>
+   <gazebo reference="LHipSag">
+    <implicitSpringDamper>1</implicitSpringDamper>
+    <provideFeedback>true</provideFeedback>
+   </gazebo>
+   <gazebo reference="LHipLat">
+    <implicitSpringDamper>1</implicitSpringDamper>
+    <provideFeedback>true</provideFeedback>
+   </gazebo>
+   <gazebo reference="LHipYaw">
+    <implicitSpringDamper>1</implicitSpringDamper>
+    <provideFeedback>true</provideFeedback>
+   </gazebo>
+   <gazebo reference="LKneeSag">
+    <implicitSpringDamper>1</implicitSpringDamper>
+    <provideFeedback>true</provideFeedback>
+   </gazebo>
+   <gazebo reference="LAnkLat">
+    <implicitSpringDamper>1</implicitSpringDamper>
+    <provideFeedback>true</provideFeedback>
+   </gazebo>
+   <gazebo reference="LAnkSag">
+    <implicitSpringDamper>1</implicitSpringDamper>
+    <provideFeedback>true</provideFeedback>
+   </gazebo>
 </robot>

File: bigman_urdf/urdf/gazebo/force_torque.gazebo.xacro (robot description, xacro)
@@ -7,4 +7,5 @@
 -->
 <robot xmlns:xacro="http:/ros.org/wiki/xacro">
+<xacro:unless value="${BIGMAN_ONLY_LEGS}">
 	<gazebo reference="RWrj2">
 		<sensor type="force_torque" name="right_arm">
@@ -37,4 +38,5 @@
 		</sensor>
 	</gazebo>
+</xacro:unless>
 	<gazebo reference="LAnkLat">
 		<sensor type="force_torque" name="left_leg">

File: bigman_urdf/urdf/gazebo/yarp_control.gazebo.xacro (robot description, xacro)
@@ -2,4 +2,5 @@
 <robot xmlns:xacro="http://ros.org/wiki/xacro">
 <gazebo>
+<xacro:unless value="${BIGMAN_ONLY_LEGS}">
 <!-- TORSO -->
 <plugin name="bigman_yarp_gazebo_plugin_torso" filename="libgazebo_yarp_controlboard.so">
@@ -12,25 +13,4 @@
 <plugin name="bigman_yarp_gazebo_plugin_torso_torque" filename="libgazebo_yarp_jointsensors.so">
     <yarpConfigurationFile>model://bigman_urdf/conf/bigman/bigman_gazebo_torso_torque.ini</yarpConfigurationFile>
-</plugin>
-<!-- LEGS -->
-<plugin name="bigman_yarp_gazebo_plugin_left_leg" filename="libgazebo_yarp_controlboard.so">
-	<yarpConfigurationFile>model://bigman_urdf/conf/bigman/bigman_gazebo_left_leg.ini</yarpConfigurationFile>
-        <initialConfiguration>0.0 0.0 0.0 0.0 0.0 0.0</initialConfiguration>
-</plugin>
-<plugin name="bigman_yarp_gazebo_plugin_left_leg_speed" filename="libgazebo_yarp_jointsensors.so">
-	<yarpConfigurationFile>model://bigman_urdf/conf/bigman/bigman_gazebo_left_leg_speed.ini</yarpConfigurationFile>
-</plugin>
-<plugin name="bigman_yarp_gazebo_plugin_left_leg_torque" filename="libgazebo_yarp_jointsensors.so">
-    <yarpConfigurationFile>model://bigman_urdf/conf/bigman/bigman_gazebo_left_leg_torque.ini</yarpConfigurationFile>
-</plugin>
-<plugin name="bigman_yarp_gazebo_plugin_right_leg" filename="libgazebo_yarp_controlboard.so">
-	<yarpConfigurationFile>model://bigman_urdf/conf/bigman/bigman_gazebo_right_leg.ini</yarpConfigurationFile>
-        <initialConfiguration>0.0 0.0 0.0 0.0 0.0 0.0</initialConfiguration>
-</plugin>
-<plugin name="bigman_yarp_gazebo_plugin_right_leg_speed" filename="libgazebo_yarp_jointsensors.so">
-    <yarpConfigurationFile>model://bigman_urdf/conf/bigman/bigman_gazebo_right_leg_speed.ini</yarpConfigurationFile>
-</plugin>
-<plugin name="bigman_yarp_gazebo_plugin_right_leg_torque" filename="libgazebo_yarp_jointsensors.so">
-    <yarpConfigurationFile>model://bigman_urdf/conf/bigman/bigman_gazebo_right_leg_torque.ini</yarpConfigurationFile>
 </plugin>
 <!-- ARMS -->
@@ -66,4 +46,26 @@
 		</plugin>
 	</xacro:unless>
+</xacro:unless>
+<!-- LEGS -->
+<plugin name="bigman_yarp_gazebo_plugin_left_leg" filename="libgazebo_yarp_controlboard.so">
+	<yarpConfigurationFile>model://bigman_urdf/conf/bigman/bigman_gazebo_left_leg.ini</yarpConfigurationFile>
+        <initialConfiguration>0.0 0.0 0.0 0.0 0.0 0.0</initialConfiguration>
+</plugin>
+<plugin name="bigman_yarp_gazebo_plugin_left_leg_speed" filename="libgazebo_yarp_jointsensors.so">
+	<yarpConfigurationFile>model://bigman_urdf/conf/bigman/bigman_gazebo_left_leg_speed.ini</yarpConfigurationFile>
+</plugin>
+<plugin name="bigman_yarp_gazebo_plugin_left_leg_torque" filename="libgazebo_yarp_jointsensors.so">
+    <yarpConfigurationFile>model://bigman_urdf/conf/bigman/bigman_gazebo_left_leg_torque.ini</yarpConfigurationFile>
+</plugin>
+<plugin name="bigman_yarp_gazebo_plugin_right_leg" filename="libgazebo_yarp_controlboard.so">
+	<yarpConfigurationFile>model://bigman_urdf/conf/bigman/bigman_gazebo_right_leg.ini</yarpConfigurationFile>
+        <initialConfiguration>0.0 0.0 0.0 0.0 0.0 0.0</initialConfiguration>
+</plugin>
+<plugin name="bigman_yarp_gazebo_plugin_right_leg_speed" filename="libgazebo_yarp_jointsensors.so">
+    <yarpConfigurationFile>model://bigman_urdf/conf/bigman/bigman_gazebo_right_leg_speed.ini</yarpConfigurationFile>
+</plugin>
+<plugin name="bigman_yarp_gazebo_plugin_right_leg_torque" filename="libgazebo_yarp_jointsensors.so">
+    <yarpConfigurationFile>model://bigman_urdf/conf/bigman/bigman_gazebo_right_leg_torque.ini</yarpConfigurationFile>
+</plugin>
 <!-- Plugin to apply external wrenches to the robot -->
 <plugin name="bigman_yarp_gazebo_plugin_external_wrench" filename="libgazebo_yarp_externalwrench.so"/>

File: bigman_urdf/urdf/parts/torso.urdf.xacro (robot description, xacro)
@@ -10,28 +10,7 @@
 <!-- LINKS -->
 <!-- This links are defined in order to be compliant with http://www.ros.org/reps/rep-0120.html#coordinate-frames
-and to define the end effectors of the robot
-The coordinate frame called base_link is rigidly attached to the robot root body. It is recommended to choose the robot waist as its root body. The base_link can be attached to the root in any arbitrary position or orientation; for every hardware platform there will be a different place on the base that provides an obvious point of reference. Note that REP 103 [1] specifies a preferred orientation for frames. -->
-<link name="base_link"/>
+and to define the end effectors of the robot-->
 <!-- The coordinate frame called torso is attached to the lowest body of the model which is a parent of l_gripper, r_gripper and gaze. -->
  <link name="torso"/>
-<link name="Waist">
-    <inertial>
-      <origin xyz="${-3.2862932e+01*mmTom} ${-5.0930727e-01*mmTom} ${-1.2899617*mmTom}" rpy="0.0 0.0 0.0"/>
-      <mass value="6.4080904"/>
-      <inertia ixx="${3.8826078e+04*mm2Tom2}"  ixy="${2.9047605e+02*mm2Tom2}"  ixz="${6.8975598e+02*mm2Tom2}" iyy="${2.5050374e+04*mm2Tom2}" iyz="${-1.3370623e+01*mm2Tom2}" izz="${4.8055286e+04*mm2Tom2}" />
-    </inertial>
-    <visual>
-      <origin xyz="0 0 0" rpy="0 0 0"/>
-      <geometry name="Waist_visual">
-        <mesh filename="package://bigman_urdf/meshes/Waist.STL" scale="0.001 0.001 0.001"/>
-      </geometry>
-    </visual>
-    <collision>
-      <origin xyz="0 0 0" rpy="0 0 0"/>
-      <geometry name="Waist_collision">
-        <mesh filename="package://bigman_urdf/meshes/simple/Waist.STL" scale="0.001 0.001 0.001"/>
-      </geometry>
-    </collision>
-</link>
   <link name ="DWL">
     <inertial>
@@ -82,4 +61,5 @@
       <geometry name="DWYTorso_visual">
         <mesh filename="package://bigman_urdf/meshes/Chest.STL" scale="0.001 0.001 0.001" />
+        <!--mesh filename="package://bigman_urdf/meshes/NewChest.STL" scale="0.001 0.001 0.001" /-->
       </geometry>
     </visual>
@@ -88,13 +68,9 @@
       <geometry name="DWYTorso_collision">
         <mesh filename="package://bigman_urdf/meshes/simple/Chest.STL" scale="0.001 0.001 0.001" />
+        <!--mesh filename="package://bigman_urdf/meshes/simple/NewChest.STL" scale="0.001 0.001 0.001" /-->
       </geometry>
     </collision>
   </link>
 <!-- JOINTS -->
-<joint name="base_joint" type="fixed">
-    <parent link="base_link"/>
-    <child link="Waist"/>
-    <origin xyz="0 0 0" rpy="0 0 0" />
-</joint>
 <joint name="torso_joint" type="fixed">
     <parent link="DWYTorso"/>

Commit message: Updated srdf.xacro and urdf.xacro. Need to be tested.

File: bigman_srdf/srdf/bigman.srdf.xacro (robot description, xacro)
@@ -15,12 +15,14 @@
     </group>
     <group name="force_torque_sensors">
-            <joint name="l_leg_ft_joint"/>
-            <joint name="r_leg_ft_joint"/>
-            <xacro:unless value="${BIGMAN_ONLY_LEGS}">
-              <joint name="l_arm_ft_joint"/>
-              <joint name="r_arm_ft_joint"/>
-            </xacro:unless>
+            <xacro:if value="${BIGMAN_LEGS}">
+		    <joint name="l_leg_ft_joint"/>
+		    <joint name="r_leg_ft_joint"/>
+	    </xacro:if>
+            <xacro:if value="${BIGMAN_UPPER_BODY}">
+		      <joint name="l_arm_ft_joint"/>
+		      <joint name="r_arm_ft_joint"/>
+            </xacro:if>
     </group>
- <xacro:unless value="${BIGMAN_ONLY_LEGS}">
+ <xacro:if value="${BIGMAN_UPPER_BODY}">
     <group name="left_arm">
         <chain base_link="DWYTorso" tip_link="l_wrist"/>
@@ -29,5 +31,6 @@
         <chain base_link="DWYTorso" tip_link="r_wrist"/>
     </group>
-</xacro:unless>
+</xacro:if>
+<xacro:if value="${BIGMAN_LEGS}">
     <group name="left_leg">
         <chain base_link="Waist" tip_link="l_sole"/>
@@ -36,19 +39,22 @@
         <chain base_link="Waist" tip_link="r_sole"/>
     </group>
- <xacro:unless value="${BIGMAN_ONLY_LEGS}">
+</xacro:if>
+ <xacro:if value="${BIGMAN_UPPER_BODY}">>
     <group name="torso">
         <chain base_link="Waist" tip_link="DWYTorso"/>
     </group>
-</xacro:unless>
+</xacro:if>
     <group name="chains"> <!--THIS HAS TO BE THE LAST GROUP IN THE FILE -->
-<xacro:unless value="${BIGMAN_ONLY_LEGS}">
+<xacro:if value="${BIGMAN_UPPER_BODY}">
         <group name="left_arm"/>
         <group name="right_arm"/>
-</xacro:unless>
+</xacro:if>
+<xacro:if value="${BIGMAN_LEGS}">
         <group name="left_leg"/>
         <group name="right_leg"/>
-<xacro:unless value="${BIGMAN_ONLY_LEGS}">
+</xacro:if>
+<xacro:if value="${BIGMAN_UPPER_BODY}">
         <group name="torso"/>
-</xacro:unless>
+</xacro:if>
     </group>
 </robot>

File: bigman_urdf/urdf/bigman.urdf.xacro (robot description, xacro)
@@ -70,5 +70,7 @@
 	</joint>
 </xacro:if>
-<!-- IMU -->
-<xacro:include filename="$(find bigman_urdf)/urdf/sensors/imu.urdf.xacro"/>
+<xacro:if value="${BIGMAN_LEGS}">
+	<!-- IMU -->
+	<xacro:include filename="$(find bigman_urdf)/urdf/sensors/imu.urdf.xacro"/>
+</xacro:if>
 </robot>

File: bigman_urdf/urdf/bigman_robot.urdf.xacro (robot description, xacro)
@@ -14,8 +14,20 @@
   </joint>
   <origin xyz="0.0 0.0 1.5" rpy="0 0 0" /> -->
-  <origin xyz="0.0 0.0 1.12" rpy="0 0 0" />
   <!-- ROBOT -->
   <xacro:include filename="$(find bigman_urdf)/urdf/bigman.urdf.xacro" />
+<xacro:if value="${BIGMAN_UPPER_BODY}">
+       <xacro:unless value="${BIGMAN_LEGS}">
+		  <link name="world"/>
+		   <joint name="fixed" type="fixed">
+		    <parent link="world"/>
+		    <child link="base_link"/>
+		  </joint>
+		  <origin xyz="0.0 0.0 1.5" rpy="0 0 0" />
+	</xacro:unless>
+</xacro:if>
+<xacro:if value="${BIGMAN_LEGS}">
+  <origin xyz="0.0 0.0 1.12" rpy="0 0 0" />
   <xacro:include filename="$(find bigman_urdf)/urdf/gazebo/microstrain_3dmgx2_imu.gazebo.xacro" />
+</xacro:if>
   <xacro:include filename="$(find bigman_urdf)/urdf/gazebo/force_torque.gazebo.xacro" />
   <xacro:include filename="$(find bigman_urdf)/urdf/gazebo/bigman.gazebo.xacro" />

Commit message: Added imu_sensors group

File: bigman_srdf/srdf/bigman.srdf.xacro (robot description, xacro)
@@ -21,4 +21,7 @@
               <joint name="r_arm_ft_joint"/>
             </xacro:unless>
+    </group>
+    <group name="imu_sensors">
+            <link name="imu_link"/>
     </group>
  <xacro:unless value="${BIGMAN_ONLY_LEGS}">
