Commit message: Updated head. Added new meshes for head. Added neck group in srdf

File: bigman_srdf/srdf/bigman.srdf.xacro (robot description, xacro)
@@ -44,4 +44,7 @@
         <chain base_link="Waist" tip_link="DWYTorso"/>
     </group>
+    <group name="head">
+        <chain base_link="NeckYaw" tip_link="NeckPitch"/>
+    </group>
 </xacro:if>
     <group name="chains"> <!--THIS HAS TO BE THE LAST GROUP IN THE FILE -->
@@ -56,4 +59,5 @@
 <xacro:if value="${BIGMAN_UPPER_BODY}">
         <group name="torso"/>
+        <group name="head"/>
 </xacro:if>
     </group>

File: bigman_urdf/urdf/sensors/multisense_sl.urdf.xacro (robot description, xacro)
@@ -12,7 +12,7 @@
     </inertial>
     <visual>
-            <origin xyz="-0.0446 0 0.0880" rpy="0 0 1.570795" />
+            <origin xyz="0 0 0" rpy="0 0 0" />
             <geometry>
-                <mesh filename="package://bigman_urdf/meshes/multisense.STL"/>
+                <mesh filename="package://bigman_urdf/meshes/Head.STL" scale="0.001 0.001 0.001"/>
             </geometry>
             <material name="">
@@ -21,13 +21,7 @@
         </visual>
   <collision>
-    <origin xyz="-0.0503 0 -0.00195" rpy="0 0 0" />
+    <origin xyz="0 0 0" rpy="0 0 0" />
     <geometry>
-      <box size="0.1311 0.12 0.0591"/>
-    </geometry>
-  </collision>
-  <collision>
-    <origin xyz="-0.093 0 0.0868" rpy="0 0 0" />
-    <geometry>
-      <box size="0.0468 0.12 0.1184"/>
+      <mesh filename="package://bigman_urdf/meshes/simple/Head.STL" scale="0.001 0.001 0.001"/>
     </geometry>
   </collision>

Commit message: Added imu group in srdf

File: bigman_srdf/srdf/bigman.srdf.xacro (robot description, xacro)
@@ -33,4 +33,7 @@
 </xacro:if>
 <xacro:if value="${BIGMAN_LEGS}">
+    <group name="imu_sensors">
+            <link name="imu_link"/>
+    </group>
     <group name="left_leg">
         <chain base_link="Waist" tip_link="l_sole"/>

Commit message: Added second imu in srdf

File: bigman_srdf/srdf/bigman.srdf.xacro (robot description, xacro)
@@ -35,4 +35,5 @@
     <group name="imu_sensors">
             <link name="imu_link"/>
+            <link name="imu_link2"/>
     </group>
     <group name="left_leg">

Commit message: Changed head link to original NeckPitch

File: bigman_srdf/srdf/bigman.srdf.xacro (robot description, xacro)
@@ -49,5 +49,5 @@
     </group>
     <group name="head">
-        <chain base_link="DWYTorso" tip_link="head"/>
+        <chain base_link="DWYTorso" tip_link="NeckPitch"/>
     </group>
 </xacro:if>

File: bigman_urdf/urdf/bigman.urdf.xacro (robot description, xacro)
@@ -57,5 +57,5 @@
        <xacro:if value="${BIGMAN_HEAD}">
                 <joint name="neck_joint" type="fixed">
-                     <parent link="head"/>
+                     <parent link="NeckPitch"/>
                      <child link="${multisense_namespace}head_multisense"/>
                      <origin xyz="0.08765 0 0.06475" rpy="0 0 0" />

File: bigman_urdf/urdf/parts/neck.urdf.xacro (robot description, xacro)
@@ -29,5 +29,5 @@
     </collision>
   </link>
-  <link name ="head">
+  <link name ="NeckPitch">
     <inertial>
       <origin xyz="${-1.020e+02*mmTom} 0.0 ${2.6575000e+02*mmTom}" rpy="0 0 0"/>
@@ -61,5 +61,5 @@
 <joint name="NeckPitchj" type="revolute">
     <parent link="NeckYaw"/>
-    <child link="head"/>
+    <child link="NeckPitch"/>
     <origin xyz="0 0 0.1155" rpy="0 0 0" />
     <axis xyz="0 1 0" />
